File: PCBs/Eyebrow_warning_indicators/Left/EWI_Left.sch (KiCad schematic (older format))
At the start: 43 parts, among them J2 Conn_01x06_Male, J3 Conn_01x08_Male, SW1 IN SWTCH, SW2 OUT SWTCH

Commit message: footprint
Parts:
- D31, D32: renamed from D?; footprint (none) -> Diode_THT:D_A-405_P7.62mm_Horizontal
- J1, J4, J5: renamed from J?; footprint (none) -> Connector_PinHeader_2.54mm:PinHeader_1x02_P2.54mm_Vertical
- J2: symbol Connector:Conn_01x06_Male -> Connector:Conn_01x06_Female
- J3: symbol Connector:Conn_01x08_Male -> Connector:Conn_01x08_Female
- R1: renamed from R?; footprint (none) -> Resistor_THT:R_Axial_DIN0207_L6.3mm_D2.5mm_P7.62mm_Horizontal
Connections:
- wire segments 148 -> 155
Other:
- note removed: "1) INSTALL 120 OHM RESISTOR ACROSS A AND B OF MAX487 ONLY \nFOR BUS TERMINATION.\n\n2) INSTALL JUMPER BETWEEN PIN 1 AND 2 OF PGM SEL FOR RS487 BUS \nENABLE. REMOVE JUMPER FOR PROGRAMMING ARDUINO NANO."
- note removed: "NOTES: (UNLESS OTHERWISE SPECIFIED)"
- moved on the sheet: D31, D32, J1, J4, J5, R1, SW1, SW2

Commit message: PCB
Parts:
- D31, D32: footprint Diode_THT:D_A-405_P7.62mm_Horizontal -> PT_Library_v001:D_Signal_P7.62mm_Horizontal
- J1: value Conn_01x02_Female -> Backlight; footprint Connector_PinHeader_2.54mm:PinHeader_1x02_P2.54mm_Vertical -> PT_Library_v001:Molex_1x02_P2.54mm_Vertical
- J2: value Conn_01x06_Male -> Led Cathode; footprint Connector_PinHeader_2.54mm:PinHeader_1x06_P2.54mm_Vertical -> PT_Library_v001:Molex_1x06_P2.54mm_Vertical
- J3: value Conn_01x08_Male -> Led Annode; footprint Connector_PinHeader_2.54mm:PinHeader_1x08_P2.54mm_Vertical -> PT_Library_v001:Molex_1x08_P2.54mm_Vertical
- J4: value Conn_01x02_Female -> SwitchCol; footprint Connector_PinHeader_2.54mm:PinHeader_1x02_P2.54mm_Vertical -> PT_Library_v001:Molex_1x02_P2.54mm_Vertical
- J5: value Conn_01x02_Female -> SwitchRow; footprint Connector_PinHeader_2.54mm:PinHeader_1x02_P2.54mm_Vertical -> PT_Library_v001:Molex_1x02_P2.54mm_Vertical
- R1: value R -> 330
Connections:
- net labels removed: 7
- wire segments 155 -> 148
Other:
- moved on the sheet: D31, SW1, SW2
Changed lines of the file:
@@
 L PT_Symbol_Library_v001:PT_Tactile_Switch_Led SW1
 U 1 1 5A4585C5
-P 2300 2350
-F 0 "SW1" H 2300 2475 50  0000 C CNN
-F 1 "IN SWTCH" H 2600 2500 50  0000 C CNN
-F 2 "PT_Library_v001:PT_Small_Tactile_Switch_With_LED" H 2300 2350 50  0001 C CNN
-F 3 "" H 2300 2350 50  0001 C CNN
-F 4 "GX06400" H 2300 2350 60  0001 C CNN "PN"
-	1    2300 2350
+P 2250 2200
+F 0 "SW1" H 2250 2325 50  0000 C CNN
+F 1 "IN SWTCH" H 2200 2100 50  0000 C CNN
+F 2 "PT_Library_v001:PT_Small_Tactile_Switch_With_LED" H 2250 2200 50  0001 C CNN
+F 3 "" H 2250 2200 50  0001 C CNN
+F 4 "GX06400" H 2250 2200 60  0001 C CNN "PN"
+	1    2250 2200
 	1    0    0    -1
 $EndComp
@@
 L PT_Symbol_Library_v001:PT_Tactile_Switch_Led SW2
 U 1 1 5A4586CB
-P 3750 2000
-F 0 "SW2" H 3750 2125 50  0000 C CNN
-F 1 "OUT SWTCH" H 4100 2000 50  0000 C CNN
-F 2 "PT_Library_v001:PT_Small_Tactile_Switch_With_LED" H 3750 2000 50  0001 C CNN
-F 3 "" H 3750 2000 50  0001 C CNN
-F 4 "GX06400" H 3750 2000 60  0001 C CNN "PN"
-	1    3750 2000
+P 3500 2200
+F 0 "SW2" H 3500 2325 50  0000 C CNN
+F 1 "OUT SWTCH" H 3400 2100 50  0000 C CNN
+F 2 "PT_Library_v001:PT_Small_Tactile_Switch_With_LED" H 3500 2200 50  0001 C CNN
+F 3 "" H 3500 2200 50  0001 C CNN
+F 4 "GX06400" H 3500 2200 60  0001 C CNN "PN"
+	1    3500 2200
 	1    0    0    -1
 $EndComp
@@
 Wire Notes Line
 	7700 5700 7700 2950
-Text Label 2000 2350 0    60   ~ 0
-7
 Wire Notes Line
 	5800 3750 5800 4650
@@
 P 2800 4450
 F 0 "J2" H 2908 4831 50  0000 C CNN
-F 1 "Conn_01x06_Male" H 2908 4740 50  0000 C CNN
-F 2 "Connector_PinHeader_2.54mm:PinHeader_1x06_P2.54mm_Vertical" H 2800 4450 50  0001 C CNN
+F 1 "Led Cathode" H 2908 4740 50  0000 C CNN
+F 2 "PT_Library_v001:Molex_1x06_P2.54mm_Vertical" H 2800 4450 50  0001 C CNN
 F 3 "~" H 2800 4450 50  0001 C CNN
 	1    2800 4450
@@
 P 6350 1900
 F 0 "J3" V 6185 1828 50  0000 C CNN
-F 1 "Conn_01x08_Male" V 6276 1828 50  0000 C CNN
-F 2 "Connector_PinHeader_2.54mm:PinHeader_1x08_P2.54mm_Vertical" H 6350 1900 50  0001 C CNN
+F 1 "Led Annode" V 6450 1850 50  0000 C CNN
+F 2 "PT_Library_v001:Molex_1x08_P2.54mm_Vertical" H 6350 1900 50  0001 C CNN
 F 3 "~" H 6350 1900 50  0001 C CNN
 	1    6350 1900
@@
 Wire Wire Line
 	3500 5650 4200 5650
-$Comp
-L Device:D D31
-U 1 1 5EE6136F
-P 1500 2150
-F 0 "D31" H 1500 2366 50  0000 C CNN
-F 1 "D" H 1500 2275 50  0000 C CNN
-F 2 "Diode_THT:D_A-405_P7.62mm_Horizontal" H 1500 2150 50  0001 C CNN
-F 3 "~" H 1500 2150 50  0001 C CNN
-	1    1500 2150
-	-1   0    0    -1
-$EndComp
-Wire Wire Line
-	1650 2350 2100 2350
-$Comp
-L Device:D D32
-U 1 1 5EE66971
-P 2950 2000
-F 0 "D32" H 2950 2216 50  0000 C CNN
-F 1 "D" H 2950 2125 50  0000 C CNN
-F 2 "Diode_THT:D_A-405_P7.62mm_Horizontal" H 2950 2000 50  0001 C CNN
-F 3 "~" H 2950 2000 50  0001 C CNN
-	1    2950 2000
-	-1   0    0    -1
-$EndComp
-Wire Wire Line
-	3100 2000 3250 2000
-Wire Wire Line
-	2100 2350 2100 2250
-Wire Wire Line
-	2100 2250 2000 2250
-Wire Wire Line
-	2400 2250 2400 2350
-Wire Wire Line
-	2400 2350 2100 2350
-Connection ~ 2100 2350
-Wire Wire Line
-	2000 1800 2000 1850
-Wire Wire Line
-	2400 1800 2400 1850
-Wire Wire Line
-	2000 1800 2200 1800
-Wire Wire Line
-	3450 1400 3850 1400
-Wire Wire Line
-	3850 1400 3850 1500
-Wire Wire Line
-	3450 1900 3250 1900
-Wire Wire Line
-	3250 1900 3250 2000
-Wire Wire Line
-	3450 1900 3850 1900
 $Comp
 L Connector:Conn_01x02_Female J5
@@
 P 1800 850
 F 0 "J5" H 1692 1035 50  0000 C CNN
-F 1 "Conn_01x02_Female" H 1692 944 50  0000 C CNN
-F 2 "Connector_PinHeader_2.54mm:PinHeader_1x02_P2.54mm_Vertical" H 1800 850 50  0001 C CNN
+F 1 "SwitchRow" H 1692 944 50  0000 C CNN
+F 2 "PT_Library_v001:Molex_1x02_P2.54mm_Vertical" H 1800 850 50  0001 C CNN
 F 3 "~" H 1800 850 50  0001 C CNN
 	1    1800 850
@@
 P 1600 1600
 F 0 "J4" H 1492 1785 50  0000 C CNN
-F 1 "Conn_01x02_Female" H 1492 1694 50  0000 C CNN
-F 2 "Connector_PinHeader_2.54mm:PinHeader_1x02_P2.54mm_Vertical" H 1600 1600 50  0001 C CNN
+F 1 "SwitchCol" H 1492 1694 50  0000 C CNN
+F 2 "PT_Library_v001:Molex_1x02_P2.54mm_Vertical" H 1600 1600 50  0001 C CNN
 F 3 "~" H 1600 1600 50  0001 C CNN
 	1    1600 1600
@@
 P 1100 2500
 F 0 "J1" H 992 2685 50  0000 C CNN
-F 1 "Conn_01x02_Female" H 992 2594 50  0000 C CNN
-F 2 "Connector_PinHeader_2.54mm:PinHeader_1x02_P2.54mm_Vertical" H 1100 2500 50  0001 C CNN
+F 1 "Backlight" H 992 2594 50  0000 C CNN
+F 2 "PT_Library_v001:Molex_1x02_P2.54mm_Vertical" H 1100 2500 50  0001 C CNN
 F 3 "~" H 1100 2500 50  0001 C CNN
 	1    1100 2500
@@
 P 1700 2500
 F 0 "R1" V 1907 2500 50  0000 C CNN
-F 1 "R" V 1816 2500 50  0000 C CNN
+F 1 "330" V 1816 2500 50  0000 C CNN
 F 2 "Resistor_THT:R_Axial_DIN0207_L6.3mm_D2.5mm_P7.62mm_Horizontal" V 1630 2500 50  0001 C CNN
 F 3 "~" H 1700 2500 50  0001 C CNN
@@
 $EndComp
 Wire Wire Line
-	1850 2500 2050 2500
-Wire Wire Line
-	2450 2500 2950 2500
-Wire Wire Line
-	2950 2500 2950 2150
-Wire Wire Line
-	2950 2150 3500 2150
+	1850 2500 1900 2500
 Wire Wire Line
 	1300 2500 1550 2500
 Wire Wire Line
-	2200 1800 2200 1450
-Wire Wire Line
-	2200 1450 2350 1450
-Connection ~ 2200 1800
-Wire Wire Line
-	2200 1800 2400 1800
-Wire Wire Line
 	6050 2800 4500 2800
 Wire Wire Line
-	3900 2150 3900 2400
-Wire Wire Line
-	3900 2400 3250 2400
-Wire Wire Line
-	3250 2400 3250 2750
-Wire Wire Line
-	3250 2750 1300 2750
-Wire Wire Line
 	1300 2750 1300 2600
 Wire Wire Line
-	3450 1400 3450 1450
-Connection ~ 3450 1450
-Wire Wire Line
-	3450 1450 3450 1500
-Connection ~ 3450 1900
-Wire Wire Line
-	1650 2350 1650 2150
-Wire Wire Line
-	1800 1700 1800 1950
-Wire Wire Line
-	1800 1950 1350 1950
-Wire Wire Line
-	1350 1950 1350 2150
+	1800 1700 1800 1800
+Wire Wire Line
+	1800 1800 1350 1800
+Wire Wire Line
+	1350 1800 1350 2000
 Wire Wire Line
 	1800 1600 2800 1600
@@
 Wire Wire Line
 	2350 850  2350 1450
-Connection ~ 2350 1450
-Wire Wire Line
-	2350 1450 3450 1450
+Wire Wire Line
+	2350 1450 2500 1450
 Wire Wire Line
 	6650 2100 6650 2300
 Wire Wire Line
 	3150 3650 4200 3650
+$Comp
+L Device:D D31
+U 1 1 5EE6136F
+P 1500 2000
+F 0 "D31" H 1500 2216 50  0000 C CNN
+F 1 "D" H 1500 2125 50  0000 C CNN
+F 2 "PT_Library_v001:D_Signal_P7.62mm_Horizontal" H 1500 2000 50  0001 C CNN
+F 3 "~" H 1500 2000 50  0001 C CNN
+	1    1500 2000
+	-1   0    0    -1
+$EndComp
+Wire Wire Line
+	1900 1900 1900 2000
+Wire Wire Line
+	1650 2000 1900 2000
+Connection ~ 1900 2000
+Wire Wire Line
+	1900 2000 1900 2100
+Wire Wire Line
+	2450 1900 2450 2000
+Wire Wire Line
+	2500 1450 2500 1500
+Wire Wire Line
+	2500 2000 2450 2000
+Connection ~ 2450 2000
+Wire Wire Line
+	2450 2000 2450 2100
+Wire Wire Line
+	1900 2200 1900 2500
+$Comp
+L Device:D D32
+U 1 1 5EF80AE6
+P 2950 2000
+F 0 "D32" H 2950 2216 50  0000 C CNN
+F 1 "D" H 2950 2125 50  0000 C CNN
+F 2 "PT_Library_v001:D_Signal_P7.62mm_Horizontal" H 2950 2000 50  0001 C CNN
+F 3 "~" H 2950 2000 50  0001 C CNN
+	1    2950 2000
+	-1   0    0    -1
+$EndComp
+Wire Wire Line
+	3150 1900 3150 2000
+Wire Wire Line
+	3100 2000 3150 2000
+Connection ~ 3150 2000
+Wire Wire Line
+	3150 2000 3150 2100
+Wire Wire Line
+	3700 1900 3700 2000
+Wire Wire Line
+	2500 1500 3800 1500
+Wire Wire Line
+	3800 1500 3800 2000
+Wire Wire Line
+	3800 2000 3700 2000
+Connection ~ 2500 1500
+Wire Wire Line
+	2500 1500 2500 2000
+Connection ~ 3700 2000
+Wire Wire Line
+	3700 2000 3700 2100
+Wire Wire Line
+	3150 2200 2450 2200
+Wire Wire Line
+	3700 2200 3700 2750
+Wire Wire Line
+	1300 2750 3700 2750
 $EndSCHEMATC
