File: PCBs/Eyebrow_warning_indicators/Left/EWI_Left.kicad_pcb (KiCad board)
At the start: 2 copper layers, 96.1 x 78.8 mm, 38 parts, among them J1 PWR, J2 Conn_01x06_Male, J3 Conn_01x08_Male, SW1 IN SWTCH, SW2 OUT SWTCH

Commit message: footprint
Parts:
- added D31: D, Diode_THT:D_A-405_P7.62mm_Horizontal, F.Cu at (54.4, 63.1)
- added D32: D, Diode_THT:D_A-405_P7.62mm_Horizontal, F.Cu at (88.4, 63.2)
- added J4: Conn_01x02_Female, Connector_PinHeader_2.54mm:PinHeader_1x02_P2.54mm_Vertical, F.Cu at (69.9, 66.9)
- added J5: Conn_01x02_Female, Connector_PinHeader_2.54mm:PinHeader_1x02_P2.54mm_Vertical, F.Cu at (94.7, 67.6)
- added R1: R, Resistor_THT:R_Axial_DIN0207_L6.3mm_D2.5mm_P7.62mm_Horizontal, F.Cu at (65.2, 62.8)
- J1: value PWR -> Conn_01x02_Female; footprint Connectors_Molex:Molex_KK-6410-04_04x2.54mm_Straight -> Connector_PinHeader_2.54mm:PinHeader_1x02_P2.54mm_Vertical; moved to F.Cu
- SW1, SW2: footprint KiCAD Libraries:SWITCH_SNAP_DOME_6.3mm_DIA_SINGLE_SIDE_PCB -> PT_Library_v001:PT_Small_Tactile_Switch_With_LED
- moved J1 23.0 mm to (77.0, 48.8), turned to 0 degrees
Connections:
- J1 pad 1: GND -> Net-(J1-Pad1)
- J1 pad 2: +3V3 -> Net-(J1-Pad2)
- J2 pad 1: Net-(J2-Pad1) -> /Dig0
- J2 pad 2: Net-(J2-Pad2) -> /Dig1
- J2 pad 3: Net-(J2-Pad3) -> /Dig2
- J2 pad 4: Net-(J2-Pad4) -> /Dig3
- J2 pad 5: Net-(J2-Pad5) -> /Dig4
- J2 pad 6: Net-(J2-Pad6) -> /Dig5
- J3 pad 1: /SegG -> /SegDP
- J3 pad 2: /SegF -> /SegA
- J3 pad 3: /SegE -> /SegB
- J3 pad 4: /SegD -> /SegC
- J3 pad 5: /SegC -> /SegD
- J3 pad 6: /SegB -> /SegE
- J3 pad 7: /SegA -> /SegF
- J3 pad 8: /SegDP -> /SegG
- SW1 pad 1: /7 -> Net-(J5-Pad1)
- SW1 pad 2: Net-(SW1-Pad2) -> Net-(J5-Pad1)
- SW2 pad 1: /8 -> Net-(J5-Pad1)
- SW2 pad 2: Net-(SW1-Pad2) -> Net-(J5-Pad1)
Routing:
- net Net-(J5-Pad1): track 0.00 -> 90.1 mm, vias 0 -> 2
- net Net-(D32-Pad1): track 0.00 -> 80.7 mm, vias 0 -> 1
- net Net-(SW1-Pad2): track 55.1 -> 0.00 mm
- net /SegDP: track 104.0 -> 158.8 mm
- net /SegA: track 96.9 -> 142.3 mm
- net Net-(SW1-Pad6): track 0.00 -> 43.2 mm, vias 0 -> 1
- net /Dig5: track 9.35 -> 46.5 mm
- net Net-(D32-Pad2): track 0.00 -> 28.8 mm
- net /SegG: track 23.5 -> 49.1 mm, vias 0 -> 2
- net /7: track 1.25 -> 24.1 mm
- net /Dig0: track 26.5 -> 49.4 mm
- net Net-(J1-Pad1): track 0.00 -> 22.4 mm
- net /Dig4: track 26.5 -> 44.4 mm, vias 0 -> 1
- net Net-(J1-Pad2): track 0.00 -> 14.7 mm
- net Net-(D31-Pad2): track 0.00 -> 12.5 mm
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Other:
- board text removed: "+12V"
- board text removed: "+3.3V"
- board text removed: "+5V"
- board text removed: "GND"
- board text removed: "REMOVE JUMPER FROM J4 TO ENABLE NANO PROGRAMMING"

Commit message: PCB
Parts:
- moved J1 5.29 mm to (77.6, 54.0)
- moved D25 2.22 mm to (86.0, 49.0)
- moved D23 2.20 mm to (97.8, 49.1)
- moved D26 2.19 mm to (85.9, 60.4)
- moved D24 2.15 mm to (97.7, 60.4)
- moved D27 2.10 mm to (73.7, 49.2)
- moved D28 2.02 mm to (73.7, 60.2)
- moved D30 1.98 mm to (62.0, 60.1)
- moved D29 1.91 mm to (62.1, 49.4)
- moved J2 1.36 mm to (102.9, 51.0)
Changed lines of the file:
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@@
     )
     (fp_line (start -4.318 -3.81) (end -3.048 -3.81) (layer F.SilkS) (width 0.12))
-    (fp_line (start -4.318 4.318) (end -4.318 -3.81) (layer F.SilkS) (width 0.12))
-    (fp_line (start 4.064 4.318) (end -4.318 4.318) (layer F.SilkS) (width 0.12))
-    (fp_line (start 4.064 -3.81) (end 4.064 4.318) (layer F.SilkS) (width 0.12))
+    (fp_line (start -4.32 3.81) (end -4.318 -3.81) (layer F.SilkS) (width 0.12))
+    (fp_line (start 4.07 3.81) (end -4.312 3.81) (layer F.SilkS) (width 0.12))
+    (fp_line (start 4.064 -3.81) (end 4.05 3.81) (layer F.SilkS) (width 0.12))
     (fp_line (start -4.064 -3.81) (end 4.064 -3.81) (layer F.SilkS) (width 0.12))
     (fp_text user - (at -1.524 3.302 90) (layer F.SilkS)
@@
       (effects (font (size 1 1) (thickness 0.15)))
     )
-    (pad 6 thru_hole circle (at 0 3.429 270) (size 1.524 1.524) (drill 0.762) (layers *.Cu *.Mask)
+    (pad 6 thru_hole circle (at 0.04 2.87 270) (size 1.524 1.524) (drill 0.762) (layers *.Cu *.Mask)
       (net 19 "Net-(J1-Pad2)"))
     (pad 5 thru_hole circle (at 0 -2.921 270) (size 1.524 1.524) (drill 0.762) (layers *.Cu *.Mask)
@@
     )
     (fp_line (start -4.318 -3.81) (end -3.048 -3.81) (layer F.SilkS) (width 0.12))
-    (fp_line (start -4.318 4.318) (end -4.318 -3.81) (layer F.SilkS) (width 0.12))
-    (fp_line (start 4.064 4.318) (end -4.318 4.318) (layer F.SilkS) (width 0.12))
-    (fp_line (start 4.064 -3.81) (end 4.064 4.318) (layer F.SilkS) (width 0.12))
+    (fp_line (start -4.32 3.81) (end -4.318 -3.81) (layer F.SilkS) (width 0.12))
+    (fp_line (start 4.07 3.81) (end -4.312 3.81) (layer F.SilkS) (width 0.12))
+    (fp_line (start 4.064 -3.81) (end 4.05 3.81) (layer F.SilkS) (width 0.12))
     (fp_line (start -4.064 -3.81) (end 4.064 -3.81) (layer F.SilkS) (width 0.12))
     (fp_text user - (at -1.524 3.302 90) (layer F.SilkS)
@@
       (effects (font (size 1 1) (thickness 0.15)))
     )
-    (pad 6 thru_hole circle (at 0 3.429 270) (size 1.524 1.524) (drill 0.762) (layers *.Cu *.Mask)
+    (pad 6 thru_hole circle (at 0.04 2.87 270) (size 1.524 1.524) (drill 0.762) (layers *.Cu *.Mask)
       (net 24 "Net-(SW1-Pad6)"))
     (pad 5 thru_hole circle (at 0 -2.921 270) (size 1.524 1.524) (drill 0.762) (layers *.Cu *.Mask)
@@
   )
   (module Connector_PinHeader_2.54mm:PinHeader_1x02_P2.54mm_Vertical (layer F.Cu)
-    (at 77 48.76)
+    (at 77.59 54.02)
     (descr "Through hole straight pin header, 1x02, 2.54mm pitch, single row")
     (tags "Through hole pin header THT 1x02 2.54mm single row")
@@
       (effects (font (size 1 1) (thickness 0.15)))
     )
-    (fp_text user K (at 0 -1.9) (layer F.SilkS)
+    (fp_text user K (at 0 -1.9) (layer F.Fab)
       (effects (font (size 1 1) (thickness 0.15)))
     )
@@
       (effects (font (size 1 1) (thickness 0.15)))
     )
-    (fp_text user K (at 0 -1.9) (layer F.SilkS)
+    (fp_text user K (at 0 -1.9) (layer F.Fab)
       (effects (font (size 1 1) (thickness 0.15)))
     )
@@
   )
   (module Connector_PinHeader_2.54mm:PinHeader_1x06_P2.54mm_Vertical (layer F.Cu)
-    (at 102.17 52.18)
+    (at 102.92 51.05)
     (descr "Through hole straight pin header, 1x06, 2.54mm pitch, single row")
     (tags "Through hole pin header THT 1x06 2.54mm single row")
@@
   )
   (module LED_THT:LED_D3.0mm_FlatTop (layer F.Cu)
-    (at 63.8268 59.2589 90)
+    (at 62.02 60.07 90)
     (descr "LED, Round, FlatTop, diameter 3.0mm, 2 pins, http://www.kingbright.com/attachments/file/psearch/000/00/00/L-47XEC(Ver.9A).pdf")
     (tags "LED Round FlatTop diameter 3.0mm 2 pins")
@@
   )
   (module LED_THT:LED_D3.0mm_FlatTop (layer F.Cu)
-    (at 63.8268 50.2689 270)
+    (at 62.13 49.39 270)
     (descr "LED, Round, FlatTop, diameter 3.0mm, 2 pins, http://www.kingbright.com/attachments/file/psearch/000/00/00/L-47XEC(Ver.9A).pdf")
     (tags "LED Round FlatTop diameter 3.0mm 2 pins")
@@
   )
   (module LED_THT:LED_D3.0mm_FlatTop (layer F.Cu)
-    (at 71.8969 59.2589 90)
+    (at 73.66 60.25 90)
     (descr "LED, Round, FlatTop, diameter 3.0mm, 2 pins, http://www.kingbright.com/attachments/file/psearch/000/00/00/L-47XEC(Ver.9A).pdf")
     (tags "LED Round FlatTop diameter 3.0mm 2 pins")
@@
   )
   (module LED_THT:LED_D3.0mm_FlatTop (layer F.Cu)
-    (at 71.8969 50.2689 270)
+    (at 73.69 49.18 270)
     (descr "LED, Round, FlatTop, diameter 3.0mm, 2 pins, http://www.kingbright.com/attachments/file/psearch/000/00/00/L-47XEC(Ver.9A).pdf")
     (tags "LED Round FlatTop diameter 3.0mm 2 pins")
@@
   )
   (module LED_THT:LED_D3.0mm_FlatTop (layer F.Cu)
-    (at 87.7969 59.2589 90)
+    (at 85.94 60.42 90)
     (descr "LED, Round, FlatTop, diameter 3.0mm, 2 pins, http://www.kingbright.com/attachments/file/psearch/000/00/00/L-47XEC(Ver.9A).pdf")
     (tags "LED Round FlatTop diameter 3.0mm 2 pins")
@@
   )
   (module LED_THT:LED_D3.0mm_FlatTop (layer F.Cu)
-    (at 87.7969 50.2689 270)
+    (at 85.97 49 270)
     (descr "LED, Round, FlatTop, diameter 3.0mm, 2 pins, http://www.kingbright.com/attachments/file/psearch/000/00/00/L-47XEC(Ver.9A).pdf")
     (tags "LED Round FlatTop diameter 3.0mm 2 pins")
@@
   )
   (module LED_THT:LED_D3.0mm_FlatTop (layer F.Cu)
-    (at 95.8669 59.2589 90)
+    (at 97.72 60.35 90)
     (descr "LED, Round, FlatTop, diameter 3.0mm, 2 pins, http://www.kingbright.com/attachments/file/psearch/000/00/00/L-47XEC(Ver.9A).pdf")
     (tags "LED Round FlatTop diameter 3.0mm 2 pins")
@@
   )
   (module LED_THT:LED_D3.0mm_FlatTop (layer F.Cu)
-    (at 95.8669 50.2689 270)
-    (descr "LED, Round, FlatTop, diameter 3.0mm, 2 pins, http://www.kingbright.com/attachments/file/psearch/000/00/00/L-47XEC(Ver.9A).pdf")
-    (tags "LED Round FlatTop diameter 3.0mm 2 pins")
+    (at 97.75 49.14 270)
+    (descr "LED, Round, FlatTop, diameter 3.0mm, 2 pins, http://www.kingbright.com/attachments/file/psearch/000/00/00/L-47XEC(Ver.9A).pdf")
+    (tags "LED Round FlatTop diameter 3.0mm 2 pins")

Commit message: PCB
Parts:
- D31, D32: footprint Diode_THT:D_A-405_P7.62mm_Horizontal -> PT_Library_v001:D_Signal_P7.62mm_Horizontal
- J1: value Conn_01x02_Female -> Backlight; footprint Connector_PinHeader_2.54mm:PinHeader_1x02_P2.54mm_Vertical -> PT_Library_v001:Molex_1x02_P2.54mm_Vertical; moved to B.Cu
- J2: value Conn_01x06_Male -> Led Cathode; footprint Connector_PinHeader_2.54mm:PinHeader_1x06_P2.54mm_Vertical -> PT_Library_v001:Molex_1x06_P2.54mm_Vertical; moved to B.Cu
- J3: value Conn_01x08_Male -> Led Annode; footprint Connector_PinHeader_2.54mm:PinHeader_1x08_P2.54mm_Vertical -> PT_Library_v001:Molex_1x08_P2.54mm_Vertical; moved to B.Cu
- J4: value Conn_01x02_Female -> SwitchCol; footprint Connector_PinHeader_2.54mm:PinHeader_1x02_P2.54mm_Vertical -> PT_Library_v001:Molex_1x02_P2.54mm_Vertical; moved to B.Cu
- J5: value Conn_01x02_Female -> SwitchRow; footprint Connector_PinHeader_2.54mm:PinHeader_1x02_P2.54mm_Vertical -> PT_Library_v001:Molex_1x02_P2.54mm_Vertical; moved to B.Cu
- R1: value R -> 330
- moved J3 41.2 mm to (121.6, 39.3), turned to 270 degrees
- moved J4 38.8 mm to (103.8, 48.0), turned to 270 degrees
- moved J1 27.0 mm to (103.5, 61.4), turned to 270 degrees
- moved J2 22.6 mm to (121.3, 64.2), turned to 270 degrees
- moved J5 16.3 mm to (103.8, 54.0), turned to 270 degrees
- moved D32 12.1 mm to (76.9, 66.7)
- moved R1 3.66 mm to (65.4, 66.5)
- moved D31 3.43 mm to (54.5, 66.5)
- moved D25 2.69 mm to (86.0, 51.7), turned to 90 degrees
- moved D23 2.55 mm to (97.8, 51.7), turned to 90 degrees
- moved D27 2.55 mm to (73.7, 51.7), turned to 90 degrees
- moved D29 2.34 mm to (62.1, 51.7), turned to 90 degrees
- moved D1 0.75 mm to (134.3, 41.3)
- moved D2 0.75 mm to (134.3, 50.3)
- moved D3 0.75 mm to (134.3, 59.3)
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Connections:
- D31 pad 1: /7 -> Net-(D31-Pad1)
- SW1 pad 1: Net-(J5-Pad1) -> Net-(D31-Pad1)
- SW1 pad 2: Net-(J5-Pad1) -> Net-(D31-Pad1)
- SW1 pad 3: /7 -> Net-(J5-Pad1)
- SW1 pad 4: /7 -> Net-(J5-Pad1)
- SW2 pad 1: Net-(J5-Pad1) -> Net-(D32-Pad1)
- SW2 pad 2: Net-(J5-Pad1) -> Net-(D32-Pad1)
- SW2 pad 3: Net-(D32-Pad1) -> Net-(J5-Pad1)
- SW2 pad 4: Net-(D32-Pad1) -> Net-(J5-Pad1)
Routing:
- net /SegDP: track 158.8 -> 0.00 mm
- net /SegA: track 142.3 -> 0.00 mm
- net /SegB: track 93.7 -> 0.00 mm
- net Net-(J5-Pad1): track 90.1 -> 0.00 mm, vias 2 -> 0
- net Net-(D32-Pad1): track 80.7 -> 0.00 mm, vias 1 -> 0
- net /Dig1: track 78.2 -> 0.00 mm
- net /Dig2: track 73.1 -> 0.00 mm
- net /SegC: track 70.5 -> 0.00 mm, vias 1 -> 0
- net /Dig0: track 49.4 -> 0.00 mm
- net /SegG: track 49.1 -> 0.00 mm, vias 2 -> 0
- net /Dig5: track 46.5 -> 0.00 mm
- net /Dig4: track 44.4 -> 0.00 mm, vias 1 -> 0
- net Net-(SW1-Pad6): track 43.2 -> 0.00 mm, vias 1 -> 0
- net /Dig3: track 38.4 -> 0.00 mm, vias 1 -> 0
- net Net-(D32-Pad2): track 28.8 -> 0.00 mm
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Other:
- board text added: "+"
- board text added: "330"
- board text added: "ASPJ ON"
- board text added: "Amber"
- board text added: "Backlight"
- board text added: "Fire"
- board text added: "GO"
- board text added: "Green"
- board text added: "L BAR"
- board text added: "L BLEED"
- board text added: "LED Annode"
- board text added: "LED Cathode"
- board text added: "Master Caution"
- board text added: "NO GO"
- board text added: "Orange"
- board text added: "R BLEED"
- board text added: "REC"
- board text added: "Red"
- board text added: "SD BRK"
- board text added: "STBY"
- board text added: "Switch Col"
- board text added: "Switch Row"
- board text added: "XMT"

Commit message: PCB
Routing:
- net /Dig1: track 0.00 -> 93.8 mm
- net /Dig2: track 0.00 -> 83.7 mm
- net /SegG: track 0.00 -> 71.3 mm
- net /SegDP: track 0.00 -> 63.3 mm
- net /SegF: track 0.00 -> 58.7 mm
- net Net-(J5-Pad1): track 0.00 -> 56.5 mm
- net Net-(D31-Pad2): track 0.00 -> 55.8 mm
- net /SegA: track 0.00 -> 53.3 mm
- net /SegC: track 0.00 -> 52.3 mm
- net /Dig0: track 0.00 -> 50.6 mm
- net /SegB: track 0.00 -> 48.0 mm
- net /SegE: track 0.00 -> 46.1 mm, vias 0 -> 1
- net Net-(J1-Pad1): track 0.00 -> 40.2 mm
- net Net-(D32-Pad2): track 0.00 -> 38.6 mm
- net Net-(J1-Pad2): track 0.00 -> 35.5 mm
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
Commit message: PCB prior to Gerber
Other:
- board text added: "Left Eyebrow v001"
Changed lines of the file:
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@@
   (general
     (thickness 1.2)
-    (drawings 93)
+    (drawings 94)
     (tracks 267)
     (zones 0)
@@
     (pad 1 np_thru_hole circle (at 0 0) (size 2.7 2.7) (drill 2.7) (layers *.Cu *.Mask))
   )
+  (gr_text "Left Eyebrow\nv001\n" (at 128.17 91.386) (layer F.SilkS)
+    (effects (font (size 1.5 1.5) (thickness 0.3)))
+  )
   (gr_text Backlight (at 101.754 66.748) (layer B.SilkS)

Commit message: eyebrow
Other:
- board text added: "Left Eyebrow v002"
- board text removed: "Left Eyebrow v001"
Changed lines of the file:
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@@
     (pad 1 np_thru_hole circle (at 0 0) (size 2.7 2.7) (drill 2.7) (layers *.Cu *.Mask))
   )
-  (gr_text "Left Eyebrow\nv001\n" (at 128.17 91.386) (layer F.SilkS)
+  (gr_text "Left Eyebrow\nv002\n" (at 128.17 91.386) (layer F.SilkS)
     (effects (font (size 1.5 1.5) (thickness 0.3)))
   )
@@
     (effects (font (size 1 1) (thickness 0.15)))
   )
-  (gr_text Green (at 126.9 63.7) (layer F.SilkS)
+  (gr_text Orange (at 126.9 63.7) (layer F.SilkS)
     (effects (font (size 1 1) (thickness 0.15)))
   )
-  (gr_text Green (at 134.266 63.7) (layer F.SilkS)
+  (gr_text Orange (at 134.266 63.7) (layer F.SilkS)
     (effects (font (size 1 1) (thickness 0.15)))
   )
@@
     (effects (font (size 1 1) (thickness 0.15)))
   )
-  (gr_text Red (at 127.916 36.522) (layer F.SilkS)
+  (gr_text Orange (at 127.916 36.522) (layer F.SilkS)
     (effects (font (size 1 1) (thickness 0.15)))
   )
@@
     (effects (font (size 1 1) (thickness 0.15)))
   )
-  (gr_text Red (at 133.758 36.522) (layer F.SilkS)
+  (gr_text Orange (at 133.758 36.522) (layer F.SilkS)
     (effects (font (size 1 1) (thickness 0.15)))
   )
