File: PCBs/55_SQ_Indicator/sq_indicator.sch (KiCad schematic (older format))
At the start: 9 parts, among them J1 Conn_01x02_Female, J2 Conn_01x02_Female, J3 Conn_01x02_Female, J4 Conn_01x02_Female, SW1 push

Commit message: PCB
Parts:
- added D5: 1N4148, Diode_THT:D_DO-35_SOD27_P7.62mm_Horizontal, symbol Diode:1N4148
- J1: value Conn_01x02_Female -> LedAnode
- J2: value Conn_01x02_Female -> LedCathode
- J3: value Conn_01x02_Female -> SwitchCol
- J4: value Conn_01x02_Female -> SwitchRow
Connections:
- net at SW1.1, SW1.2: now also D5.1 (K); no longer J3.1 (Pin_1)
- new net: D5.2 (A), J3.1 (Pin_1)
Changed lines of the file:
@@
 P 5050 1300
 F 0 "J3" H 4942 1485 50  0000 C CNN
-F 1 "Conn_01x02_Female" H 4942 1394 50  0000 C CNN
+F 1 "SwitchCol" H 4942 1394 50  0000 C CNN
 F 2 "Connector_PinHeader_2.54mm:PinHeader_1x02_P2.54mm_Vertical" H 5050 1300 50  0001 C CNN
 F 3 "~" H 5050 1300 50  0001 C CNN
@@
 P 5050 1750
 F 0 "J4" H 4942 1935 50  0000 C CNN
-F 1 "Conn_01x02_Female" H 4942 1844 50  0000 C CNN
+F 1 "SwitchRow" H 4942 1844 50  0000 C CNN
 F 2 "Connector_PinHeader_2.54mm:PinHeader_1x02_P2.54mm_Vertical" H 5050 1750 50  0001 C CNN
 F 3 "~" H 5050 1750 50  0001 C CNN
@@
 P 2850 3450
 F 0 "J2" H 2742 3635 50  0000 C CNN
-F 1 "Conn_01x02_Female" H 2742 3544 50  0000 C CNN
+F 1 "LedCathode" H 2742 3544 50  0000 C CNN
 F 2 "Connector_PinHeader_2.54mm:PinHeader_1x02_P2.54mm_Vertical" H 2850 3450 50  0001 C CNN
 F 3 "~" H 2850 3450 50  0001 C CNN
@@
 P 2850 2600
 F 0 "J1" H 2742 2785 50  0000 C CNN
-F 1 "Conn_01x02_Female" H 2742 2694 50  0000 C CNN
+F 1 "LedAnode" H 2742 2694 50  0000 C CNN
 F 2 "Connector_PinHeader_2.54mm:PinHeader_1x02_P2.54mm_Vertical" H 2850 2600 50  0001 C CNN
 F 3 "~" H 2850 2600 50  0001 C CNN
@@
 $EndComp
 Wire Wire Line
-	5250 1300 5850 1300
-Wire Wire Line
-	5850 1300 5850 1350
-Wire Wire Line
-	5850 1350 5850 1550
-Connection ~ 5850 1350
+	5850 1350 5850 1450
 Wire Wire Line
 	6400 1550 6400 1400
@@
 Wire Wire Line
 	3550 2700 3050 2700
+$Comp
+L Diode:1N4148 D5
+U 1 1 5EEF607D
+P 5400 1300
+F 0 "D5" H 5400 1084 50  0000 C CNN
+F 1 "1N4148" H 5400 1175 50  0000 C CNN
+F 2 "Diode_THT:D_DO-35_SOD27_P7.62mm_Horizontal" H 5400 1125 50  0001 C CNN
+F 3 "https://assets.nexperia.com/documents/data-sheet/1N4148_1N4448.pdf" H 5400 1300 50  0001 C CNN
+	1    5400 1300
+	-1   0    0    1
+$EndComp
+Wire Wire Line
+	5550 1300 5550 1450
+Wire Wire Line
+	5550 1450 5850 1450
+Connection ~ 5850 1450
+Wire Wire Line
+	5850 1450 5850 1550
 $EndSCHEMATC

Commit message: PCB prior to Gerber
Parts:
- added H1, H2: MountingHole, MountingHole:MountingHole_2.2mm_M2, symbol Mechanical:MountingHole
- added H3, H4: MountingHole, MountingHole:MountingHole_3.2mm_M3, symbol Mechanical:MountingHole
Changed lines of the file:
@@
 Wire Wire Line
 	5850 1450 5850 1550
+$Comp
+L Mechanical:MountingHole H1
+U 1 1 5EEECC41
+P 8050 3550
+F 0 "H1" H 8150 3596 50  0000 L CNN
+F 1 "MountingHole" H 8150 3505 50  0000 L CNN
+F 2 "MountingHole:MountingHole_2.2mm_M2" H 8050 3550 50  0001 C CNN
+F 3 "~" H 8050 3550 50  0001 C CNN
+	1    8050 3550
+	1    0    0    -1
+$EndComp
+$Comp
+L Mechanical:MountingHole H2
+U 1 1 5EEED081
+P 8050 3800
+F 0 "H2" H 8150 3846 50  0000 L CNN
+F 1 "MountingHole" H 8150 3755 50  0000 L CNN
+F 2 "MountingHole:MountingHole_2.2mm_M2" H 8050 3800 50  0001 C CNN
+F 3 "~" H 8050 3800 50  0001 C CNN
+	1    8050 3800
+	1    0    0    -1
+$EndComp
+$Comp
+L Mechanical:MountingHole H3
+U 1 1 5EEED377
+P 8050 4050
+F 0 "H3" H 8150 4096 50  0000 L CNN
+F 1 "MountingHole" H 8150 4005 50  0000 L CNN
+F 2 "MountingHole:MountingHole_3.2mm_M3" H 8050 4050 50  0001 C CNN
+F 3 "~" H 8050 4050 50  0001 C CNN
+	1    8050 4050
+	1    0    0    -1
+$EndComp
+$Comp
+L Mechanical:MountingHole H4
+U 1 1 5EEED746
+P 8050 4350
+F 0 "H4" H 8150 4396 50  0000 L CNN
+F 1 "MountingHole" H 8150 4305 50  0000 L CNN
+F 2 "MountingHole:MountingHole_3.2mm_M3" H 8050 4350 50  0001 C CNN
+F 3 "~" H 8050 4350 50  0001 C CNN
+	1    8050 4350
+	1    0    0    -1
+$EndComp
 $EndSCHEMATC
