File: PCBs/IFEI/IFEI.kicad_pcb (KiCad board)
At the start: 2 copper layers, 24.3 x 104.3 mm, 13 parts, among them J1 Conn_02x04_Male, SW1 mode, SW2 qty, SW3 up, SW4 down, SW5 zone, SW6 ET

Commit message: PCB prior to Gerber
Parts:
- removed G***: LOGO, KiCAD Libraries:CC-BY-NC-SA-Small
- removed G***: LOGO, KiCAD Libraries:OH_LOGO_37.7mm_5.9mm
- added D1: 1N4148, Diode_THT:D_DO-35_SOD27_P7.62mm_Horizontal, F.Cu at (133.0, 65.0)
- added D2: 1N4148, Diode_THT:D_DO-35_SOD27_P7.62mm_Horizontal, F.Cu at (133.0, 68.8)
- added D3: 1N4148, Diode_THT:D_DO-35_SOD27_P7.62mm_Horizontal, F.Cu at (133.2, 83.6)
- added D4: 1N4148, Diode_THT:D_DO-35_SOD27_P7.62mm_Horizontal, F.Cu at (133.2, 110.5)
- added D5: 1N4148, Diode_THT:D_DO-35_SOD27_P7.62mm_Horizontal, F.Cu at (133.2, 126.0)
- added D6: 1N4148, Diode_THT:D_DO-35_SOD27_P7.62mm_Horizontal, F.Cu at (133.2, 129.8)
- added J2: SwitchRow, PT_Library_v001:Molex_1x03_P2.54mm_Vertical, F.Cu at (129.4, 99.6)
- added J3: BackLight, PT_Library_v001:Molex_1x02_P2.54mm_Vertical, F.Cu at (144.4, 98.5)
- added R1: 150, PT_Library_v001:R_Axial_DIN0207_L6.3mm_D2.5mm_P7.62mm_Horizontal, F.Cu at (140.8, 80.3)
- added R2: 150, PT_Library_v001:R_Axial_DIN0207_L6.3mm_D2.5mm_P7.62mm_Horizontal, F.Cu at (133.2, 114.3)
- J1: value Conn_02x04_Male -> SwithCol; footprint Connector_PinHeader_2.54mm:PinHeader_2x04_P2.54mm_Horizontal -> PT_Library_v001:Molex_1x02_P2.54mm_Vertical; moved to F.Cu
- MK1, MK2, MK3, MK4: footprint KiCAD Libraries:Mouting_Hole_1.85mm -> MountingHole:MountingHole_2.2mm_M2
- SW1, SW2, SW3, SW4, SW5, SW6: footprint KiCAD Libraries:SWITCH_SNAP_DOME_6.3mm_DIA_SINGLE_SIDE_PCB -> PT_Library_v001:PT_Small_Tactile_Switch_With_LED
- moved J1 4.06 mm to (136.8, 98.5)
Connections:
- J1 pad 1: GND -> /Col1
- J1 pad 2: GND -> /Col2
- SW1 pad 1: /A -> Net-(D1-Pad1)
- SW1 pad 2: GND -> Net-(D1-Pad1)
- SW2 pad 1: /B -> Net-(D2-Pad1)
- SW2 pad 2: GND -> Net-(D2-Pad1)
- SW3 pad 1: /C -> Net-(D3-Pad1)
- SW3 pad 2: GND -> Net-(D3-Pad1)
- SW4 pad 1: /D -> Net-(D4-Pad1)
- SW4 pad 2: GND -> Net-(D4-Pad1)
- SW5 pad 1: /E -> Net-(D5-Pad1)
- SW5 pad 2: GND -> Net-(D5-Pad1)
- SW6 pad 1: /F -> Net-(D6-Pad1)
- SW6 pad 2: GND -> Net-(D6-Pad1)
Routing:
- net GND: track 174.0 -> 0.00 mm
- net /Row3: track 0.00 -> 65.1 mm
- net /Row1: track 0.00 -> 64.3 mm
- net /Row2: track 0.00 -> 63.4 mm
- net /A: track 53.2 -> 0.00 mm, vias 2 -> 0
- net /-BckLght: track 0.00 -> 52.5 mm
- net /F: track 44.5 -> 0.00 mm, vias 1 -> 0
- net /+BckLght: track 0.00 -> 42.0 mm
- net /Col2: track 0.00 -> 37.3 mm
- net /Col1: track 0.00 -> 36.2 mm
- net /B: track 31.2 -> 0.00 mm, vias 2 -> 0
- net /E: track 25.1 -> 0.00 mm, vias 1 -> 0
- net Net-(SW2-Pad6): track 0.00 -> 22.0 mm
- net Net-(SW5-Pad6): track 0.00 -> 22.0 mm
- net Net-(SW1-Pad6): track 0.00 -> 22.0 mm
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Other:
- board text added: "150"
- board text added: "Backlight"
- board text added: "Switch Row"
