File: PCBs/Arduino_NW_I2C/Arduino_NW_I2C.kicad_pcb (KiCad board)
At the start: 2 copper layers, 68.6 x 53.3 mm, 12 parts, among them J4 PT_Conn_01x06, J5 PT_Conn_01x06, J6 Conn_01x08_Female, J7 Conn_01x08_Female, J8 Conn_01x08_Female, U1 PT_Ethernet_Shield

Commit message: MUX PCB
Parts:
- added J1: PT_Conn_01x06, PT_Library_v001:PT_PinHeader_1x06_P2.54mm_Vertical, F.Cu at (150.2, 79.7)
- added J10: PT_Conn_01x06, PT_Library_v001:PT_PinHeader_1x06_P2.54mm_Vertical, F.Cu at (150.5, 106.7)
- added J11: PT_Conn_01x06, PT_Library_v001:PT_PinHeader_1x06_P2.54mm_Vertical, F.Cu at (160.4, 72.2)
- added J12: PT_Conn_01x06, PT_Library_v001:PT_PinHeader_1x06_P2.54mm_Vertical, F.Cu at (160.4, 64.8)
- added J13: PT_Conn_01x06, PT_Library_v001:PT_PinHeader_1x06_P2.54mm_Vertical, F.Cu at (160.4, 57.3)
- added J2: PT_Conn_01x06, PT_Library_v001:PT_PinHeader_1x06_P2.54mm_Vertical, F.Cu at (150.2, 86.3)
- added J3: PT_Conn_01x06, PT_Library_v001:PT_PinHeader_1x06_P2.54mm_Vertical, F.Cu at (150.5, 93.1)
- added J9: PT_Conn_01x06, PT_Library_v001:PT_PinHeader_1x06_P2.54mm_Vertical, F.Cu at (150.4, 99.7)
- added U2: MUX, PT_Library_v001:Adafruit_TCA9548A, F.Cu at (126.8, 95.7)
- moved J4 5.77 mm to (150.4, 72.8)
Other:
- board text added: "FIX ADDRESS PIN ISSUE!!!!!"

Commit message: OLED PCB
Parts:
- added J14: Conn_01x02_Female, Connector_PinHeader_2.54mm:PinHeader_1x02_P2.54mm_Vertical, F.Cu at (146.2, 65.8)
Connections:
- net Net-(J13-Pad3) renamed /SC6
- net Net-(J13-Pad4) renamed /SD6
- J1 pad 1: Net-(J1-Pad1) -> +5V
- J1 pad 2: Net-(J1-Pad2) -> GND
- J1 pad 3: Net-(J1-Pad3) -> /SC7
- J1 pad 4: Net-(J1-Pad4) -> /SD7
- J13 pad 1: Net-(J13-Pad1) -> +5V
- J13 pad 2: Net-(J13-Pad2) -> GND
- U2 pad SC7: Net-(U2-PadSC7) -> /SC7
- U2 pad SD7: Net-(U2-PadSD7) -> /SD7

Commit message: I2C PCB
Parts:
- J1, J10, J11, J12, J13, J9: value PT_Conn_01x06 -> PT_Conn_01x04; footprint PT_Library_v001:PT_PinHeader_1x06_P2.54mm_Vertical -> PT_Library_v001:PT_PinHeader_1x04_P2.54mm_Vertical
- moved J13 46.5 mm to (145.1, 101.2), turned to 0 degrees
- moved J12 34.4 mm to (145.3, 95.6)
- moved J11 20.1 mm to (142.8, 81.9), turned to 0 degrees
- moved J3 15.9 mm to (156.4, 78.3), turned to 0 degrees
- moved J2 15.2 mm to (163.0, 78.2), turned to 0 degrees
- moved J9 9.24 mm to (159.6, 101.0), turned to 0 degrees
- moved J10 5.99 mm to (152.4, 101.0), turned to 0 degrees
- moved U2 5.86 mm to (126.1, 101.5)
- moved J5 1.40 mm to (120.1, 84.4)
- moved J1 0.87 mm to (149.6, 80.3), turned to 0 degrees

Commit message: I2C
Connections:
- J10 pad 1: Net-(J10-Pad1) -> +5V
- J10 pad 2: Net-(J10-Pad2) -> GND
- J10 pad 3: Net-(J10-Pad3) -> /SC3
- J10 pad 4: Net-(J10-Pad4) -> /SD3
- J11 pad 1: Net-(J11-Pad1) -> +5V
- J11 pad 2: Net-(J11-Pad2) -> GND
- J11 pad 3: Net-(J11-Pad3) -> /SC4
- J11 pad 4: Net-(J11-Pad4) -> /SD4
- J12 pad 1: Net-(J12-Pad1) -> +5V
- J12 pad 2: Net-(J12-Pad2) -> GND
- J12 pad 3: Net-(J12-Pad3) -> /SC5
- J12 pad 4: Net-(J12-Pad4) -> /SD5
- J2 pad 1: Net-(J2-Pad1) -> +5V
- J2 pad 2: Net-(J2-Pad2) -> GND
- J2 pad 3: Net-(J2-Pad3) -> /SC0
- J2 pad 4: Net-(J2-Pad4) -> /SD0
- J2 pad 5: Net-(J2-Pad5) -> /RST
- J3 pad 1: Net-(J3-Pad1) -> +5V
- J3 pad 2: Net-(J3-Pad2) -> GND
- J3 pad 3: Net-(J3-Pad3) -> /SC1
- J3 pad 4: Net-(J3-Pad4) -> /SD1
- J3 pad 5: Net-(J3-Pad5) -> /RST
- J9 pad 1: Net-(J9-Pad1) -> +5V
- J9 pad 2: Net-(J9-Pad2) -> GND
- J9 pad 3: Net-(J9-Pad3) -> /SC2
- J9 pad 4: Net-(J9-Pad4) -> /SD2
- R3 pad 2: Net-(R3-Pad2) -> /RST
- U1 pad 1: Net-(R3-Pad2) -> /RST
- U2 pad RST: Net-(R3-Pad2) -> /RST
- U2 pad SC0: Net-(U2-PadSC0) -> /SC0
- U2 pad SC1: Net-(U2-PadSC1) -> /SC1
- U2 pad SC2: Net-(U2-PadSC2) -> /SC2
- U2 pad SC3: Net-(U2-PadSC3) -> /SC3
- U2 pad SC4: Net-(U2-PadSC4) -> /SC4
- U2 pad SC5: Net-(U2-PadSC5) -> /SC5
- U2 pad SC6: Net-(U2-PadSC6) -> /SC6
- U2 pad SD0: Net-(U2-PadSD0) -> /SD0
- U2 pad SD1: Net-(U2-PadSD1) -> /SD1
- U2 pad SD2: Net-(U2-PadSD2) -> /SD2
- U2 pad SD3: Net-(U2-PadSD3) -> /SD3
- U2 pad SD4: Net-(U2-PadSD4) -> /SD4
- U2 pad SD5: Net-(U2-PadSD5) -> /SD5
- U2 pad SD6: Net-(U2-PadSD6) -> /SD6
Routing:
- net GND: track 0.00 -> 170.0 mm
- net +5V: track 0.00 -> 125.6 mm
- net /RST: track 0.00 -> 70.7 mm
- net Net-(J14-Pad1): track 0.00 -> 59.9 mm
- net Net-(J14-Pad2): track 0.00 -> 56.5 mm
- net /SC0: track 0.00 -> 54.8 mm
- net /SD0: track 0.00 -> 45.7 mm
- net Net-(J4-Pad5): track 0.00 -> 45.0 mm
- net /SC1: track 0.00 -> 43.5 mm
- net Net-(J5-Pad5): track 0.00 -> 42.5 mm
- net /SD7: track 0.00 -> 42.4 mm
- net Net-(J4-Pad3): track 0.00 -> 41.2 mm
- net Net-(J5-Pad6): track 0.00 -> 40.5 mm
- net /SC7: track 0.00 -> 39.2 mm
- net Net-(J4-Pad4): track 0.00 -> 37.4 mm
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
Commit message: PCB WORK
Parts:
- removed the J10 at (152.4, 101.0)
- added J1: A0, Connector_PinHeader_2.54mm:PinHeader_1x02_P2.54mm_Vertical, F.Cu at (139.8, 83.3)
- added J14: PT_Conn_01x04, PT_Library_v001:Molex_1x04_P2.54mm_Vertical, F.Cu at (146.2, 98.6)
- added J2: A1, Connector_PinHeader_2.54mm:PinHeader_1x02_P2.54mm_Vertical, F.Cu at (135.7, 83.3)
- added J3: A2, Connector_PinHeader_2.54mm:PinHeader_1x02_P2.54mm_Vertical, F.Cu at (131.4, 83.3)
- J10: renamed from J1; footprint PT_Library_v001:PT_PinHeader_1x04_P2.54mm_Vertical -> PT_Library_v001:Molex_1x04_P2.54mm_Vertical
- J11: renamed from J2; footprint PT_Library_v001:PT_PinHeader_1x06_P2.54mm_Vertical -> PT_Library_v001:Molex_1x06_P2.54mm_Vertical
- J12: renamed from J3; footprint PT_Library_v001:PT_PinHeader_1x06_P2.54mm_Vertical -> PT_Library_v001:Molex_1x06_P2.54mm_Vertical
- J13: renamed from J9; footprint PT_Library_v001:PT_PinHeader_1x04_P2.54mm_Vertical -> PT_Library_v001:Molex_1x04_P2.54mm_Vertical
- J15: renamed from J11; footprint PT_Library_v001:PT_PinHeader_1x04_P2.54mm_Vertical -> PT_Library_v001:Molex_1x04_P2.54mm_Vertical
- J16: renamed from J12; footprint PT_Library_v001:PT_PinHeader_1x04_P2.54mm_Vertical -> PT_Library_v001:Molex_1x04_P2.54mm_Vertical
- J17: renamed from J13; footprint PT_Library_v001:PT_PinHeader_1x04_P2.54mm_Vertical -> PT_Library_v001:Molex_1x04_P2.54mm_Vertical
- J4: footprint PT_Library_v001:PT_PinHeader_1x06_P2.54mm_Vertical -> PT_Library_v001:Molex_1x06_P2.54mm_Vertical
- J5: footprint PT_Library_v001:PT_PinHeader_1x06_P2.54mm_Vertical -> PT_Library_v001:Molex_1x04_P2.54mm_Vertical
- R1, R2, R3: footprint PT_Library_v001:PT_R_Axial_DIN0204_L3.6mm_D1.6mm_P2.54mm_Vertical -> PT_Library_v001:R_Axial_DIN0207_L6.3mm_D2.5mm_P7.62mm_Horizontal
- moved J15 30.3 mm to (154.9, 109.7), turned to 90 degrees
- moved J10 23.0 mm to (163.7, 98.6), turned to 90 degrees
- moved J17 20.4 mm to (163.7, 109.7), turned to 90 degrees
- moved J11 19.0 mm to (146.2, 86.9), turned to 90 degrees
- moved J13 16.0 mm to (146.2, 109.7), turned to 90 degrees
- moved J4 15.0 mm to (161.4, 83.1)
- moved J16 10.1 mm to (154.9, 98.6)
- moved J12 8.89 mm to (154.0, 86.9), turned to 90 degrees
- moved J5 6.61 mm to (124.1, 89.7)
- moved R2 5.08 mm to (128.9, 70.9)
- moved R3 2.97 mm to (100.7, 111.8)
- moved J9 0.90 mm to (146.9, 66.3)
- renumbered J14 to J9
Connections:
- R3 pad 2: /RST -> +5V
- U1 pad 1: /RST -> Net-(C1-Pad1)
- U1 pad 24: Net-(J5-Pad4) -> Net-(J5-Pad3)
- U1 pad 25: Net-(J5-Pad5) -> Net-(J5-Pad4)
- U1 pad 26: Net-(J5-Pad6) -> Net-(J3-Pad1)
- U2 pad +5V: Net-(U2-Pad+5V) -> +5V
- U2 pad GND: Net-(U2-PadGND) -> GND
- U2 pad RST: /RST -> Net-(C1-Pad1)
Routing:
- net /RST: track 70.7 -> 7.87 mm
- net Net-(J5-Pad5): track 42.5 -> 0.00 mm
- net Net-(J5-Pad6): track 40.5 -> 0.00 mm
- net Net-(J3-Pad1): track 0.00 -> 36.4 mm
- net Net-(J2-Pad1): track 0.00 -> 31.2 mm
- net /SD6: track 34.9 -> 61.5 mm
- net Net-(J1-Pad1): track 0.00 -> 26.0 mm
- net Net-(J5-Pad3): track 0.00 -> 25.0 mm
- net Net-(C1-Pad1): track 8.89 -> 32.8 mm
- net /SC0: track 54.8 -> 33.4 mm
- net /SC6: track 31.3 -> 50.8 mm
- net /SC4: track 16.5 -> 34.4 mm
- net /SC7: track 39.2 -> 54.1 mm
- net /SD7: track 42.4 -> 56.0 mm
- net /SD2: track 29.3 -> 16.1 mm, vias 0 -> 1
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Other:
- net class POWER added: clearance 0.2, trace_width 0.5, via_dia 0.8, via_drill 0.4
- board text added: "+"
- board text added: "-"
- board text added: "330"
- board text added: "47UF"
- board text added: "500"
- board text added: "D11"
- board text added: "D12"
- board text added: "I2C 0"
- board text added: "I2C 1"
- board text added: "I2C 2"
- board text added: "I2C 3"
- board text added: "I2C 4"
- board text added: "I2C 5"
- board text added: "I2C 6"
- board text added: "I2C 7"
- board text added: "I2C in"
- board text added: "SCL"
- board text added: "SDA"
- board text removed: "D10 - D13"
- board text removed: "FIX ADDRESS PIN ISSUE!!!!!"
- board text removed: "To Max7219"
- board text removed: "To Panel A0-A7"

Commit message: PCB prior to Gerber
Connections:
- R3 pad 2: +5V -> Net-(R3-Pad2)
- U1 pad 1: Net-(C1-Pad1) -> Net-(R3-Pad2)
- U2 pad RST: Net-(C1-Pad1) -> Net-(R3-Pad2)
Routing:
- net Net-(C1-Pad1): track 32.8 -> 9.03 mm
- net /SC7: track 54.1 -> 72.7 mm
- net Net-(R3-Pad2): track 0.00 -> 18.5 mm
- net /SD6: track 61.5 -> 56.4 mm
- net +5V: track 136.1 -> 131.5 mm
- net /SD2: track 16.1 -> 13.5 mm
- net Net-(J9-Pad2): track 52.0 -> 53.3 mm
- net /SD5: track 36.3 -> 35.2 mm
- net GND: track 173.6 -> 173.0 mm

Commit message: PCB
Parts:
- removed J5: PT_Conn_01x06, PT_Library_v001:Molex_1x04_P2.54mm_Vertical
- J13: footprint PT_Library_v001:Molex_1x04_P2.54mm_Vertical -> PT_Library_v001:Molex_1x06_P2.54mm_Vertical
- moved J13 29.9 mm to (164.2, 85.9), turned to 180 degrees
- moved J11 23.4 mm to (164.2, 71.9), turned to 180 degrees
- moved J15 19.0 mm to (163.9, 93.0), turned to 180 degrees
- moved J4 17.0 mm to (144.4, 83.8), turned to 180 degrees
- moved J12 12.9 mm to (164.2, 79.0), turned to 180 degrees
- moved J1 12.2 mm to (127.6, 82.3)
- moved J3 12.2 mm to (119.2, 82.3)
- moved J2 12.2 mm to (123.6, 82.3)
- moved J17 9.40 mm to (163.9, 100.3), turned to 180 degrees
- moved J10 9.23 mm to (165.0, 107.7), turned to 180 degrees
- moved J14 8.46 mm to (152.5, 93.0), turned to 180 degrees
- moved J16 3.00 mm to (152.5, 100.3), turned to 180 degrees
Connections:
- J11 pad 5: /RST -> /RST_1
- J12 pad 5: /RST -> /RST_2
- U1 pad 15: Net-(U1-Pad15) -> /RST_1
- U1 pad 24: Net-(J5-Pad3) -> /RST_2
- U1 pad 25: Net-(J5-Pad4) -> /RST_3
Routing:
- net /RST_3: track 0.00 -> 68.2 mm
- net /RST_2: track 0.00 -> 49.2 mm
- net /SC0: track 33.4 -> 62.2 mm
- net Net-(J5-Pad4): track 28.3 -> 0.00 mm
- net Net-(J5-Pad3): track 25.3 -> 0.00 mm
- net /SC7: track 72.7 -> 52.0 mm
- net /RST_1: track 0.00 -> 20.4 mm
- net Net-(J9-Pad2): track 53.3 -> 73.3 mm
- net /SD0: track 37.1 -> 55.6 mm
- net Net-(J3-Pad1): track 36.7 -> 22.2 mm
- net /SD6: track 56.4 -> 42.5 mm
- net GND: track 173.0 -> 161.7 mm
- net Net-(J1-Pad1): track 26.1 -> 36.3 mm
- net /SD2: track 13.5 -> 23.5 mm, vias 1 -> 0
- net /SC2: track 13.9 -> 23.5 mm
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Other:
- board text added: "Ethernet Shield I2C V002"
- board text removed: "D11"
- board text removed: "D12"
- board text removed: "Ethernet Shield I2C V001"
