File: PCBs/OH - Left Console - 14 - Auxiliary Power Unit Panel/OH - Left Console - 14 - Auxiliary Power Unit Panel.sch (KiCad schematic (older format))
At the start: 10 parts, among them J1 Input Columns, J2 Input Rows, SW1 EXT_PWR_SW

Commit message: Panels
Parts:
- removed J1: Input Columns, PT_Library_v001:Molex_1x06_P2.54mm_Vertical, symbol Connector:Conn_01x06_Female
- removed RV?: R_POT_US, PT_Library_v001:Molex_1x03_P2.54mm_Vertical, symbol Device:R_POT_US
- removed SW?: SW_Push, PT_Library_v001:Molex_1x02_P2.54mm_Vertical, symbol Switch:SW_Push
- removed SW?: Rotary_Encoder_Switch, PT_Library_v001:Molex_1x03_P2.54mm_Vertical, symbol Device:Rotary_Encoder_Switch
- removed SW?: SW_Rotary6, symbol OpenHornet2:SW_Rotary6
- removed SW?: SW_Rotary3x4, symbol Switch:SW_Rotary3x4
- added D1, D5: D, Diode_THT:D_DO-41_SOD81_P10.16mm_Horizontal, symbol Diode:1N4001
- added D3: D, PT_Library_v001:D_Signal_P7.62mm_Horizontal, symbol Device:D
- added D4: LED, symbol Device:LED
- added J1: Coil 1, PT_Library_v001:Molex_1x02_P2.54mm_Vertical, symbol Connector:Conn_01x02_Female
- added J2: Ready LED, PT_Library_v001:Molex_1x02_P2.54mm_Vertical, symbol Connector:Conn_01x02_Female
- added J3: Input Columns, PT_Library_v001:Molex_1x02_P2.54mm_Vertical, symbol Connector:Conn_01x02_Female
- added J4: Optional Coil, PT_Library_v001:Molex_1x02_P2.54mm_Vertical, symbol Connector:Conn_01x02_Female
- added L1, L2: L, symbol Device:L
- gave numbers to parts that had none: 1
- renumbered D1 to D2, J2 to J5
Connections:
- net at SW1.1: now also J5.1 (Pin_1), SW2.2 (B)
- net at SW1.2: now also D2.1 (K)
- net at SW1.3: now also J5.2 (Pin_2)
- net at D2.2 (A): now also J3.1 (Pin_1)
- net at SW2.1 (A): now also D3.1 (K)
- new net: D3.2 (A), J3.2 (Pin_2)
- new net: D4.1 (K), J2.2 (Pin_2)
- new net: D4.2 (A), J2.1 (Pin_1)
- new net: D5.1 (K), J4.1 (Pin_1), L2.1
- new net: D5.2 (A), J4.2 (Pin_2), L2.2
- new net: D1.1 (K), J1.1 (Pin_1), L1.1
- new net: D1.2 (A), J1.2 (Pin_2), L1.2
Other:
- note added: "Coil for Magentic Switch"
- note added: "Second Coil for Magentic Switch optional - not needed for a real Honeywell Switch"
- note removed: "1: Copy section from Inputs-Outputs-from-DCS-BIOS in Templates directory to top of Input-Output-from DCS-BIOS, and panel into top left hand corner\n\n2: Grab section of image from NeoEngress_FA-18C_Full_Layout_-_4220x5200 and paste \n\n3: Don’t forget outputs such as gauges, lights and Mag Switches\n\n4: After editing diagram reset numbering during Net generation\n"
- note removed: "Instructions"
- moved on the sheet: D2, J5, SW1, SW2

Commit message: pcbs
Parts:
- removed J1: Coil 1, PT_Library_v001:Molex_1x02_P2.54mm_Vertical, symbol Connector:Conn_01x02_Female
- removed J4: Optional Coil, PT_Library_v001:Molex_1x02_P2.54mm_Vertical, symbol Connector:Conn_01x02_Female
- removed J5: Input Rows, PT_Library_v001:Molex_1x02_P2.54mm_Vertical, symbol Connector:Conn_01x02_Female
- added H1, H2, H3: MountingHole, MountingHole:MountingHole_4.3mm_M4, symbol Mechanical:MountingHole
- added J1: Coil Inputs, PT_Library_v001:Molex_1x04_P2.54mm_Vertical, symbol Connector:Conn_01x04_Female
- D4: value LED -> Ready LED Out; footprint (none) -> PT_Library_v001:Molex_1x02_P2.54mm_Vertical
- J2: value Ready LED -> Ready LED In
- J3: footprint PT_Library_v001:Molex_1x02_P2.54mm_Vertical -> PT_Library_v001:Molex_1x04_P2.54mm_Vertical; symbol Connector:Conn_01x02_Female -> Connector:Conn_01x04_Female
- L1: value L -> Crank Coil; footprint (none) -> PT_Library_v001:Molex_1x02_P2.54mm_Vertical
- L2: value L -> APU Coil; footprint (none) -> PT_Library_v001:Molex_1x02_P2.54mm_Vertical
- SW1: value EXT_PWR_SW -> ENG CRANK
- SW2: value SW_SPST -> APU
Connections:
- net Row1: now reaches SW1.1, SW2.2 (B)
- net Row1: now also J3.3 (Pin_3)
- net Row2: now reaches SW1.3
- net Row2: now also J3.4 (Pin_4)
- net Col1: now reaches D2.2 (A), J3.1 (Pin_1)
- net Col2: now reaches D3.2 (A), J3.2 (Pin_2)
- net at D5.1 (K), L2.1: now also J1.3 (Pin_3)
- net at D5.2 (A), L2.2: now also J1.4 (Pin_4)
- net at D1.1 (K), L1.1: now also J1.1 (Pin_1)
- net at D1.2 (A), L1.2: now also J1.2 (Pin_2)
Other:
- note added: "Coil for APU\nMagentic Switch"
- note added: "Coil for Engine Crank\nMagentic Switch"
- note removed: "Coil for Magentic Switch"
- note removed: "Second Coil for Magentic Switch optional - not needed for a real Honeywell Switch"
- moved on the sheet: D1, L1
Changed lines of the file:
@@
 P 5000 3450
 F 0 "SW1" H 5000 3735 50  0000 C CNN
-F 1 "EXT_PWR_SW" H 5000 3644 50  0000 C CNN
+F 1 "ENG CRANK" H 5000 3644 50  0000 C CNN
 F 2 "PT_Library_v001:Molex_1x03_P2.54mm_Vertical" H 5000 3450 50  0001 C CNN
 F 3 "~" H 5000 3450 50  0001 C CNN
@@
 $EndComp
 $Comp
-L Connector:Conn_01x02_Female J5
-U 1 1 5FC37DA5
-P 6250 3700
-F 0 "J5" H 6278 3676 50  0000 L CNN
-F 1 "Input Rows" H 6278 3585 50  0000 L CNN
-F 2 "PT_Library_v001:Molex_1x02_P2.54mm_Vertical" H 6250 3700 50  0001 C CNN
-F 3 "~" H 6250 3700 50  0001 C CNN
-	1    6250 3700
-	1    0    0    -1
-$EndComp
-$Comp
 L Switch:SW_SPST SW2
 U 1 1 5FC61E34
 P 5000 4200
 F 0 "SW2" H 5000 4435 50  0000 C CNN
-F 1 "SW_SPST" H 5000 4344 50  0000 C CNN
+F 1 "APU" H 5000 4344 50  0000 C CNN
 F 2 "PT_Library_v001:Molex_1x02_P2.54mm_Vertical" H 5000 4200 50  0001 C CNN
 F 3 "~" H 5000 4200 50  0001 C CNN
@@
 $EndComp
 $Comp
-L Connector:Conn_01x02_Female J3
+L Connector:Conn_01x04_Female J3
 U 1 1 5FC98150
-P 3500 3750
-F 0 "J3" H 3528 3726 50  0000 L CNN
-F 1 "Input Columns" H 3528 3635 50  0000 L CNN
-F 2 "PT_Library_v001:Molex_1x02_P2.54mm_Vertical" H 3500 3750 50  0001 C CNN
-F 3 "~" H 3500 3750 50  0001 C CNN
-	1    3500 3750
+P 3500 3850
+F 0 "J3" H 3528 3826 50  0000 L CNN
+F 1 "Input Columns" H 3528 3735 50  0000 L CNN
+F 2 "PT_Library_v001:Molex_1x04_P2.54mm_Vertical" H 3500 3850 50  0001 C CNN
+F 3 "~" H 3500 3850 50  0001 C CNN
+	1    3500 3850
 	-1   0    0    -1
 $EndComp
@@
 P 4650 4950
 F 0 "D4" V 4689 5028 50  0000 L CNN
-F 1 "LED" V 4598 5028 50  0000 L CNN
-F 2 "" H 4650 4950 50  0001 C CNN
+F 1 "Ready LED Out" V 4598 5028 50  0000 L CNN
+F 2 "PT_Library_v001:Molex_1x02_P2.54mm_Vertical" H 4650 4950 50  0001 C CNN
 F 3 "~" H 4650 4950 50  0001 C CNN
 	1    4650 4950
@@
 P 3450 4900
 F 0 "J2" H 3478 4876 50  0000 L CNN
-F 1 "Ready LED" H 3478 4785 50  0000 L CNN
+F 1 "Ready LED In" H 3478 4785 50  0000 L CNN
 F 2 "PT_Library_v001:Molex_1x02_P2.54mm_Vertical" H 3450 4900 50  0001 C CNN
 F 3 "~" H 3450 4900 50  0001 C CNN
@@
 	5200 3350 5800 3350
 Wire Wire Line
-	5800 3350 5800 3700
-Wire Wire Line
-	5800 3700 6050 3700
-Wire Wire Line
-	5200 3550 5500 3550
-Wire Wire Line
-	5500 3550 5500 3800
-Wire Wire Line
-	5500 3800 6050 3800
-Wire Wire Line
 	5200 4200 5800 4200
 Wire Wire Line
-	5800 4200 5800 3700
-Connection ~ 5800 3700
-Wire Wire Line
 	3650 4900 3950 4900
 Wire Wire Line
@@
 Wire Wire Line
 	3950 5000 3650 5000
-$Comp
-L Connector:Conn_01x02_Female J4
-U 1 1 5FC9D626
-P 5650 2650
-F 0 "J4" H 5678 2626 50  0000 L CNN
-F 1 "Optional Coil" H 5678 2535 50  0000 L CNN
-F 2 "PT_Library_v001:Molex_1x02_P2.54mm_Vertical" H 5650 2650 50  0001 C CNN
-F 3 "~" H 5650 2650 50  0001 C CNN
-	1    5650 2650
-	-1   0    0    -1
-$EndComp
 $Comp
 L Device:L L2
@@
 P 6850 2700
 F 0 "L2" H 6903 2746 50  0000 L CNN
-F 1 "L" H 6903 2655 50  0000 L CNN
-F 2 "" H 6850 2700 50  0001 C CNN
+F 1 "APU Coil" H 6903 2655 50  0000 L CNN
+F 2 "PT_Library_v001:Molex_1x02_P2.54mm_Vertical" H 6850 2700 50  0001 C CNN
 F 3 "~" H 6850 2700 50  0001 C CNN
 	1    6850 2700
@@
 Wire Wire Line
 	6850 2550 6500 2550
-Wire Wire Line
-	6500 2550 5850 2550
-Wire Wire Line
-	5850 2550 5850 2650
 Connection ~ 6500 2550
-Wire Wire Line
-	5850 2750 5900 2750
 Wire Wire Line
 	5900 2750 5900 2850
@@
 Connection ~ 6500 2850
 Text Notes 7000 2700 0    50   ~ 0
-Coil for Magentic Switch
-$Comp
-L Connector:Conn_01x02_Female J1
-U 1 1 5FCAC0EF
-P 2600 2700
-F 0 "J1" H 2628 2676 50  0000 L CNN
-F 1 "Coil 1" H 2628 2585 50  0000 L CNN
-F 2 "PT_Library_v001:Molex_1x02_P2.54mm_Vertical" H 2600 2700 50  0001 C CNN
-F 3 "~" H 2600 2700 50  0001 C CNN
-	1    2600 2700
-	-1   0    0    -1
-$EndComp
+Coil for APU\nMagentic Switch
 $Comp
 L Device:L L1
 U 1 1 5FCAC0F9
-P 3800 2750
-F 0 "L1" H 3853 2796 50  0000 L CNN
-F 1 "L" H 3853 2705 50  0000 L CNN
-F 2 "" H 3800 2750 50  0001 C CNN
-F 3 "~" H 3800 2750 50  0001 C CNN
-	1    3800 2750
+P 6850 2150
+F 0 "L1" H 6903 2196 50  0000 L CNN
+F 1 "Crank Coil" H 6903 2105 50  0000 L CNN
+F 2 "PT_Library_v001:Molex_1x02_P2.54mm_Vertical" H 6850 2150 50  0001 C CNN
+F 3 "~" H 6850 2150 50  0001 C CNN
+	1    6850 2150
 	1    0    0    -1
 $EndComp
@@
 L Diode:1N4001 D1
 U 1 1 5FCAC103
-P 3450 2750
-F 0 "D1" V 3404 2671 50  0000 R CNN
-F 1 "D" V 3495 2671 50  0000 R CNN
-F 2 "Diode_THT:D_DO-41_SOD81_P10.16mm_Horizontal" H 3450 2750 50  0001 C CNN
-F 3 "http://www.vishay.com/docs/88503/1n4001.pdf" H 3450 2750 50  0001 C CNN
-	1    3450 2750
+P 6500 2150
+F 0 "D1" V 6454 2071 50  0000 R CNN
+F 1 "D" V 6545 2071 50  0000 R CNN
+F 2 "Diode_THT:D_DO-41_SOD81_P10.16mm_Horizontal" H 6500 2150 50  0001 C CNN
+F 3 "http://www.vishay.com/docs/88503/1n4001.pdf" H 6500 2150 50  0001 C CNN
+	1    6500 2150
 	0    -1   1    0
 $EndComp
 Wire Wire Line
-	3800 2600 3450 2600
-Wire Wire Line
-	3450 2600 2800 2600
-Wire Wire Line
-	2800 2600 2800 2700
-Connection ~ 3450 2600
-Wire Wire Line
-	2800 2800 2850 2800
-Wire Wire Line
-	2850 2800 2850 2900
-Wire Wire Line
-	2850 2900 3450 2900
-Wire Wire Line
-	3800 2900 3450 2900
-Connection ~ 3450 2900
-Text Notes 3950 2750 0    50   ~ 0
-Coil for Magentic Switch
-Text Notes 5350 3000 0    50   ~ 0
-Second Coil for Magentic Switch optional - not needed for a real Honeywell Switch
+	6850 2000 6500 2000
+Wire Wire Line
+	6500 2000 5850 2000
+Wire Wire Line
+	5850 2000 5850 2100
+Connection ~ 6500 2000
+Wire Wire Line
+	5900 2200 5900 2300
+Wire Wire Line
+	5900 2300 6500 2300
+Wire Wire Line
+	6850 2300 6500 2300
+Connection ~ 6500 2300
+Text Notes 7000 2150 0    50   ~ 0
+Coil for Engine Crank\nMagentic Switch
+Text Label 5800 3400 0    50   ~ 0
+Row1
+Text Label 5200 3550 0    50   ~ 0
+Row2
+Text Label 4050 3450 0    50   ~ 0
+Col1
+Text Label 4150 4200 0    50   ~ 0
+Col2
+Text Label 3700 3950 0    50   ~ 0
+Row1
+Text Label 3700 4050 0    50   ~ 0
+Row2
+Wire Wire Line
+	5800 3350 5800 4200
+$Comp
+L Connector:Conn_01x04_Female J1
+U 1 1 6049B816
+P 4900 2200
+F 0 "J1" H 4928 2176 50  0000 L CNN
+F 1 "Coil Inputs" H 4928 2085 50  0000 L CNN
+F 2 "PT_Library_v001:Molex_1x04_P2.54mm_Vertical" H 4900 2200 50  0001 C CNN
+F 3 "~" H 4900 2200 50  0001 C CNN
+	1    4900 2200
+	-1   0    0    -1
+$EndComp
+Wire Wire Line
+	5850 2100 5100 2100
+Wire Wire Line
+	5100 2200 5900 2200
+Wire Wire Line
+	5650 2550 5650 2300
+Wire Wire Line
+	5650 2300 5100 2300
+Wire Wire Line
+	5100 2400 5600 2400
+Wire Wire Line
+	5600 2400 5600 2750
+Wire Wire Line
+	5600 2750 5900 2750
+Wire Wire Line
+	5650 2550 6500 2550
+$Comp
+L Mechanical:MountingHole H1
+U 1 1 604A2B2F
+P 7700 4000
+F 0 "H1" H 7800 4046 50  0000 L CNN
+F 1 "MountingHole" H 7800 3955 50  0000 L CNN
+F 2 "MountingHole:MountingHole_4.3mm_M4" H 7700 4000 50  0001 C CNN
+F 3 "~" H 7700 4000 50  0001 C CNN
+	1    7700 4000
+	1    0    0    -1
+$EndComp
+$Comp
+L Mechanical:MountingHole H2
+U 1 1 604A2ED8
+P 7700 4350
+F 0 "H2" H 7800 4396 50  0000 L CNN
+F 1 "MountingHole" H 7800 4305 50  0000 L CNN
+F 2 "MountingHole:MountingHole_4.3mm_M4" H 7700 4350 50  0001 C CNN
+F 3 "~" H 7700 4350 50  0001 C CNN
+	1    7700 4350
+	1    0    0    -1
+$EndComp
+$Comp
+L Mechanical:MountingHole H3
+U 1 1 604A317B
+P 7700 4700
+F 0 "H3" H 7800 4746 50  0000 L CNN
+F 1 "MountingHole" H 7800 4655 50  0000 L CNN
+F 2 "MountingHole:MountingHole_4.3mm_M4" H 7700 4700 50  0001 C CNN
+F 3 "~" H 7700 4700 50  0001 C CNN
+	1    7700 4700
+	1    0    0    -1
+$EndComp
 $EndSCHEMATC

Commit message: PCB
Parts:
- J3: value Input Columns -> Switch Inputs
Connections:
- net at D5.1 (K), L2.1: now also J1.1 (Pin_1); no longer J1.3 (Pin_3)
- net at D5.2 (A), L2.2: now also J1.2 (Pin_2); no longer J1.4 (Pin_4)
- net at D1.1 (K), L1.1: now also J1.3 (Pin_3); no longer J1.1 (Pin_1)
- net at D1.2 (A), L1.2: now also J1.4 (Pin_4); no longer J1.2 (Pin_2)
Other:
- moved on the sheet: D1, D5, L1, L2
Changed lines of the file:
@@
 P 3500 3850
 F 0 "J3" H 3528 3826 50  0000 L CNN
-F 1 "Input Columns" H 3528 3735 50  0000 L CNN
+F 1 "Switch Inputs" H 3528 3735 50  0000 L CNN
 F 2 "PT_Library_v001:Molex_1x04_P2.54mm_Vertical" H 3500 3850 50  0001 C CNN
 F 3 "~" H 3500 3850 50  0001 C CNN
@@
 L Device:L L2
 U 1 1 5FCA743C
-P 6850 2700
-F 0 "L2" H 6903 2746 50  0000 L CNN
-F 1 "APU Coil" H 6903 2655 50  0000 L CNN
-F 2 "PT_Library_v001:Molex_1x02_P2.54mm_Vertical" H 6850 2700 50  0001 C CNN
-F 3 "~" H 6850 2700 50  0001 C CNN
-	1    6850 2700
+P 7050 2150
+F 0 "L2" H 7103 2196 50  0000 L CNN
+F 1 "APU Coil" H 7103 2105 50  0000 L CNN
+F 2 "PT_Library_v001:Molex_1x02_P2.54mm_Vertical" H 7050 2150 50  0001 C CNN
+F 3 "~" H 7050 2150 50  0001 C CNN
+	1    7050 2150
 	1    0    0    -1
 $EndComp
@@
 L Diode:1N4001 D5
 U 1 1 5FCA8CD7
-P 6500 2700
-F 0 "D5" V 6454 2621 50  0000 R CNN
-F 1 "D" V 6545 2621 50  0000 R CNN
-F 2 "Diode_THT:D_DO-41_SOD81_P10.16mm_Horizontal" H 6500 2700 50  0001 C CNN
-F 3 "http://www.vishay.com/docs/88503/1n4001.pdf" H 6500 2700 50  0001 C CNN
-	1    6500 2700
+P 6700 2150
+F 0 "D5" V 6654 2071 50  0000 R CNN
+F 1 "D" V 6745 2071 50  0000 R CNN
+F 2 "Diode_THT:D_DO-41_SOD81_P10.16mm_Horizontal" H 6700 2150 50  0001 C CNN
+F 3 "http://www.vishay.com/docs/88503/1n4001.pdf" H 6700 2150 50  0001 C CNN
+	1    6700 2150
 	0    -1   1    0
 $EndComp
 Wire Wire Line
-	6850 2550 6500 2550
-Connection ~ 6500 2550
-Wire Wire Line
-	5900 2750 5900 2850
-Wire Wire Line
-	5900 2850 6500 2850
-Wire Wire Line
-	6850 2850 6500 2850
-Connection ~ 6500 2850
-Text Notes 7000 2700 0    50   ~ 0
+	7050 2000 6700 2000
+Connection ~ 6700 2000
+Wire Wire Line
+	7050 2300 6700 2300
+Connection ~ 6700 2300
+Text Notes 7200 2150 0    50   ~ 0
 Coil for APU\nMagentic Switch
 $Comp
 L Device:L L1
 U 1 1 5FCAC0F9
-P 6850 2150
-F 0 "L1" H 6903 2196 50  0000 L CNN
-F 1 "Crank Coil" H 6903 2105 50  0000 L CNN
-F 2 "PT_Library_v001:Molex_1x02_P2.54mm_Vertical" H 6850 2150 50  0001 C CNN
-F 3 "~" H 6850 2150 50  0001 C CNN
-	1    6850 2150
+P 7050 2750
+F 0 "L1" H 7103 2796 50  0000 L CNN
+F 1 "Crank Coil" H 7103 2705 50  0000 L CNN
+F 2 "PT_Library_v001:Molex_1x02_P2.54mm_Vertical" H 7050 2750 50  0001 C CNN
+F 3 "~" H 7050 2750 50  0001 C CNN
+	1    7050 2750
 	1    0    0    -1
 $EndComp
@@
 L Diode:1N4001 D1
 U 1 1 5FCAC103
-P 6500 2150
-F 0 "D1" V 6454 2071 50  0000 R CNN
-F 1 "D" V 6545 2071 50  0000 R CNN
-F 2 "Diode_THT:D_DO-41_SOD81_P10.16mm_Horizontal" H 6500 2150 50  0001 C CNN
-F 3 "http://www.vishay.com/docs/88503/1n4001.pdf" H 6500 2150 50  0001 C CNN
-	1    6500 2150
+P 6700 2750
+F 0 "D1" V 6654 2671 50  0000 R CNN
+F 1 "D" V 6745 2671 50  0000 R CNN
+F 2 "Diode_THT:D_DO-41_SOD81_P10.16mm_Horizontal" H 6700 2750 50  0001 C CNN
+F 3 "http://www.vishay.com/docs/88503/1n4001.pdf" H 6700 2750 50  0001 C CNN
+	1    6700 2750
 	0    -1   1    0
 $EndComp
 Wire Wire Line
-	6850 2000 6500 2000
-Wire Wire Line
-	6500 2000 5850 2000
+	7050 2600 6700 2600
 Wire Wire Line
 	5850 2000 5850 2100
-Connection ~ 6500 2000
+Connection ~ 6700 2600
 Wire Wire Line
 	5900 2200 5900 2300
 Wire Wire Line
-	5900 2300 6500 2300
-Wire Wire Line
-	6850 2300 6500 2300
-Connection ~ 6500 2300
-Text Notes 7000 2150 0    50   ~ 0
+	7050 2900 6700 2900
+Connection ~ 6700 2900
+Text Notes 7200 2750 0    50   ~ 0
 Coil for Engine Crank\nMagentic Switch
 Text Label 5800 3400 0    50   ~ 0
@@
 	5100 2200 5900 2200
 Wire Wire Line
-	5650 2550 5650 2300
-Wire Wire Line
 	5650 2300 5100 2300
 Wire Wire Line
@@
 	5600 2750 5900 2750
 Wire Wire Line
-	5650 2550 6500 2550
+	5850 2000 6700 2000
 $Comp
 L Mechanical:MountingHole H1
@@
 	1    0    0    -1
 $EndComp
+Wire Wire Line
+	5900 2300 6700 2300
+Wire Wire Line
+	5650 2600 6700 2600
+Wire Wire Line
+	5650 2300 5650 2600
+Wire Wire Line
+	5900 2750 5900 2900
+Wire Wire Line
+	5900 2900 6700 2900
 $EndSCHEMATC
