File: PCBs/OH - Left Console - 18 - Left Essential Circuit Breakers/OH - Left Console - 18 - Left Essential Circuit Breakers.sch (KiCad schematic (older format))
At the start: 12 parts, among them J1 Input Columns, J2 Input Rows, SW1 SW_Push, SW2 SW_Push, SW3 SW_Push, SW4 SW_Push, SW5 SW_Push

Commit message: PCBs
Parts:
- removed J2: Input Rows, PT_Library_v001:Molex_1x02_P2.54mm_Vertical, symbol Connector:Conn_01x02_Female
- added H1, H2, H3, H4: MountingHole, MountingHole:MountingHole_3.2mm_M3, symbol Mechanical:MountingHole
- J1: value Input Columns -> Switch Inputs; footprint (none) -> PT_Library_v001:Molex_1x06_P2.54mm_Vertical; symbol Connector:Conn_01x03_Female -> Connector:Conn_01x06_Female
- SW1: value SW_Push -> CMSD_DISPENSE_BTN
- SW2: value SW_Push -> CB_FCS_CHAN1
- SW3: value SW_Push -> CB_FCS_CHAN2
- SW4: value SW_Push -> CB_SPD_BRK
- SW5: value SW_Push -> CB_LAUNCH_BAR
Connections:
- net labels added: Col1, Col2, Col3, Row1, Row2
- wire segments 30 -> 26
Changed lines of the file:
@@
-$EndComp
-$Comp
-L Connector:Conn_01x02_Female J2
-U 1 1 5FC37DA5
-P 4850 3550
-F 0 "J2" H 4878 3526 50  0000 L CNN
-F 1 "Input Rows" H 4878 3435 50  0000 L CNN
-F 2 "PT_Library_v001:Molex_1x02_P2.54mm_Vertical" H 4850 3550 50  0001 C CNN
-F 3 "~" H 4850 3550 50  0001 C CNN
-	1    4850 3550
-	1    0    0    -1
 $EndComp
 $Comp
@@
 P 3250 2600
 F 0 "SW1" H 3250 2885 50  0000 C CNN
-F 1 "SW_Push" H 3250 2794 50  0000 C CNN
+F 1 "CMSD_DISPENSE_BTN" H 3250 2794 50  0000 C CNN
 F 2 "PT_Library_v001:Molex_1x02_P2.54mm_Vertical" H 3250 2800 50  0001 C CNN
 F 3 "~" H 3250 2800 50  0001 C CNN
@@
 P 3250 3300
 F 0 "SW2" H 3250 3585 50  0000 C CNN
-F 1 "SW_Push" H 3250 3494 50  0000 C CNN
+F 1 "CB_FCS_CHAN1" H 3250 3494 50  0000 C CNN
 F 2 "PT_Library_v001:Molex_1x02_P2.54mm_Vertical" H 3250 3500 50  0001 C CNN
 F 3 "~" H 3250 3500 50  0001 C CNN
@@
 P 3250 3950
 F 0 "SW3" H 3250 4235 50  0000 C CNN
-F 1 "SW_Push" H 3250 4144 50  0000 C CNN
+F 1 "CB_FCS_CHAN2" H 3250 4144 50  0000 C CNN
 F 2 "PT_Library_v001:Molex_1x02_P2.54mm_Vertical" H 3250 4150 50  0001 C CNN
 F 3 "~" H 3250 4150 50  0001 C CNN
@@
 P 3250 4550
 F 0 "SW4" H 3250 4835 50  0000 C CNN
-F 1 "SW_Push" H 3250 4744 50  0000 C CNN
+F 1 "CB_SPD_BRK" H 3250 4744 50  0000 C CNN
 F 2 "PT_Library_v001:Molex_1x02_P2.54mm_Vertical" H 3250 4750 50  0001 C CNN
 F 3 "~" H 3250 4750 50  0001 C CNN
@@
 P 3250 5100
 F 0 "SW5" H 3250 5385 50  0000 C CNN
-F 1 "SW_Push" H 3250 5294 50  0000 C CNN
+F 1 "CB_LAUNCH_BAR" H 3250 5294 50  0000 C CNN
 F 2 "PT_Library_v001:Molex_1x02_P2.54mm_Vertical" H 3250 5300 50  0001 C CNN
 F 3 "~" H 3250 5300 50  0001 C CNN
@@
 	3050 5100 2600 5100
 $Comp
-L Connector:Conn_01x03_Female J1
+L Connector:Conn_01x06_Female J1
 U 1 1 5FCC4B59
-P 1250 3450
-F 0 "J1" H 1142 3735 50  0000 C CNN
-F 1 "Input Columns" H 1142 3644 50  0000 C CNN
-F 2 "" H 1250 3450 50  0001 C CNN
-F 3 "~" H 1250 3450 50  0001 C CNN
-	1    1250 3450
+P 1250 3550
+F 0 "J1" H 1142 3835 50  0000 C CNN
+F 1 "Switch Inputs" H 1600 3500 50  0000 C CNN
+F 2 "PT_Library_v001:Molex_1x06_P2.54mm_Vertical" H 1250 3550 50  0001 C CNN
+F 3 "~" H 1250 3550 50  0001 C CNN
+	1    1250 3550
 	-1   0    0    -1
 $EndComp
@@
 	3450 3950 4000 3950
 Wire Wire Line
-	4000 3950 4000 3550
-Wire Wire Line
-	4000 3550 4650 3550
-Wire Wire Line
 	3500 2600 4000 2600
-Wire Wire Line
-	4000 2600 4000 3550
-Connection ~ 4000 3550
 Wire Wire Line
 	3450 5100 4000 5100
@@
 Wire Wire Line
 	3700 4550 3450 4550
-Wire Wire Line
-	3700 3300 3700 3650
-Wire Wire Line
-	4650 3650 3700 3650
-Connection ~ 3700 3650
-Wire Wire Line
-	3700 3650 3700 4550
+Text Label 2050 2600 0    50   ~ 0
+Col1
+Text Label 2200 3950 0    50   ~ 0
+Col2
+Text Label 2150 5100 0    50   ~ 0
+Col3
+Text Label 4000 3050 0    50   ~ 0
+Row1
+Text Label 3700 3800 0    50   ~ 0
+Row2
+Wire Wire Line
+	4000 2600 4000 3950
+Wire Wire Line
+	3700 3300 3700 4550
+Text Label 1450 3650 0    50   ~ 0
+Row1
+Text Label 1450 3750 0    50   ~ 0
+Row2
+$Comp
+L Mechanical:MountingHole H1
+U 1 1 604CC05E
+P 4900 3900
+F 0 "H1" H 5000 3946 50  0000 L CNN
+F 1 "MountingHole" H 5000 3855 50  0000 L CNN
+F 2 "MountingHole:MountingHole_3.2mm_M3" H 4900 3900 50  0001 C CNN
+F 3 "~" H 4900 3900 50  0001 C CNN
+	1    4900 3900
+	1    0    0    -1
+$EndComp
+$Comp
+L Mechanical:MountingHole H2
+U 1 1 604CC22A
+P 4900 4150
+F 0 "H2" H 5000 4196 50  0000 L CNN
+F 1 "MountingHole" H 5000 4105 50  0000 L CNN
+F 2 "MountingHole:MountingHole_3.2mm_M3" H 4900 4150 50  0001 C CNN
+F 3 "~" H 4900 4150 50  0001 C CNN
+	1    4900 4150
+	1    0    0    -1
+$EndComp
+$Comp
+L Mechanical:MountingHole H3
+U 1 1 604CC547
+P 4900 4450
+F 0 "H3" H 5000 4496 50  0000 L CNN
+F 1 "MountingHole" H 5000 4405 50  0000 L CNN
+F 2 "MountingHole:MountingHole_3.2mm_M3" H 4900 4450 50  0001 C CNN
+F 3 "~" H 4900 4450 50  0001 C CNN
+	1    4900 4450
+	1    0    0    -1
+$EndComp
+$Comp
+L Mechanical:MountingHole H4
+U 1 1 604CC8A4
+P 4900 4750
+F 0 "H4" H 5000 4796 50  0000 L CNN
+F 1 "MountingHole" H 5000 4705 50  0000 L CNN
+F 2 "MountingHole:MountingHole_3.2mm_M3" H 4900 4750 50  0001 C CNN
+F 3 "~" H 4900 4750 50  0001 C CNN
+	1    4900 4750
+	1    0    0    -1
+$EndComp
 $EndSCHEMATC

Commit message: pcbs
Connections:
- no-connect marks 0 -> 1
Changed lines of the file:
@@
 	3450 3950 4000 3950
-Wire Wire Line
-	3500 2600 4000 2600
 Wire Wire Line
 	3450 5100 4000 5100
@@
 	1    0    0    -1
 $EndComp
+NoConn ~ 1450 3850
+Wire Wire Line
+	3450 2600 4000 2600
 $EndSCHEMATC
