File: PCBs/OH - Left Console - 6 - Flight Control Systems Panel /OH - Left Console - 6 - Flight Control Systems Panel .kicad_pcb (KiCad board)
At the start: 2 copper layers, 44.5 x 44.7 mm, 15 parts, among them J1 Switch Inputs, J2 FCS_Analog, J3 Backlighting In, J4 Backlighting Out, SW1 FCS_RESET_BTN, SW2 TO_TRIM_BTN, SW3 GAIN_SWITCH

Commit message: FCS PCB
Parts:
- moved J1 4.70 mm to (79.5, 116.3)
- moved SW2 4.46 mm to (83.3, 126.4)
- moved SW1 2.07 mm to (94.1, 126.4)
- moved SW3 0.63 mm to (73.3, 126.4)
Routing:
- net Net-(D2-Pad1): track 13.7 -> 20.7 mm
- net /Row2: track 23.7 -> 19.6 mm
- net /Col1: track 30.1 -> 31.2 mm
- net /Row1: track 24.4 -> 23.8 mm
Other:
- board text added: "+"
- board text added: "-"
- board text added: "Col 1"
- board text added: "Col 2"
- board text added: "Row 1"
- board text added: "Row 2"

Commit message: pcbs
Parts:
- moved D1 0.76 mm to (92.5, 110.4)
- moved D2 0.76 mm to (92.5, 113.7)
- moved D3 0.76 mm to (92.5, 116.8)
Routing:
- net Net-(D2-Pad1): track 20.7 -> 16.6 mm
- net /Row2: track 19.6 -> 16.1 mm
- net Net-(D3-Pad1): track 23.9 -> 26.0 mm
- net /Col2: track 20.3 -> 19.5 mm
- net /Col1: track 31.2 -> 30.5 mm
- net /Row1: track 23.8 -> 23.2 mm
Changed lines of the file:
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@@
     (thickness 1.6)
     (drawings 18)
-    (tracks 68)
+    (tracks 63)
     (zones 0)
     (modules 15)
@@
   )
   (module Diode_THT:D_DO-35_SOD27_P7.62mm_Horizontal (layer F.Cu)
-    (at 93.218 116.84)
+    (at 92.456 116.84)
     (descr "Diode, DO-35_SOD27 series, Axial, Horizontal, pin pitch=7.62mm, , length*diameter=4*2mm^2, , http://www.diodes.com/_files/packages/DO-35.pdf")
     (tags "Diode DO-35_SOD27 series Axial Horizontal pin pitch 7.62mm  length 4mm diameter 2mm")
@@
   )
   (module Diode_THT:D_DO-35_SOD27_P7.62mm_Horizontal (layer F.Cu)
-    (at 93.218 113.665)
+    (at 92.456 113.665)
     (descr "Diode, DO-35_SOD27 series, Axial, Horizontal, pin pitch=7.62mm, , length*diameter=4*2mm^2, , http://www.diodes.com/_files/packages/DO-35.pdf")
     (tags "Diode DO-35_SOD27 series Axial Horizontal pin pitch 7.62mm  length 4mm diameter 2mm")
@@
   )
   (module Diode_THT:D_DO-35_SOD27_P7.62mm_Horizontal (layer F.Cu)
-    (at 93.218 110.363)
+    (at 92.456 110.363)
     (descr "Diode, DO-35_SOD27 series, Axial, Horizontal, pin pitch=7.62mm, , length*diameter=4*2mm^2, , http://www.diodes.com/_files/packages/DO-35.pdf")
     (tags "Diode DO-35_SOD27 series Axial Horizontal pin pitch 7.62mm  length 4mm diameter 2mm")
@@
   (gr_line (start 68.58 152.146) (end 78.994 152.146) (layer Edge.Cuts) (width 0.12))
   (gr_line (start 68.58 107.442) (end 68.58 152.146) (layer Edge.Cuts) (width 0.12))
-  (segment (start 100.838 116.84) (end 100.838 115.7147) (width 0.25) (layer F.Cu) (net 1))
-  (segment (start 100.838 110.363) (end 100.838 111.4883) (width 0.25) (layer F.Cu) (net 1))
-  (segment (start 100.838 111.4883) (end 101.9633 112.6136) (width 0.25) (layer F.Cu) (net 1))
-  (segment (start 101.9633 112.6136) (end 101.9633 114.5894) (width 0.25) (layer F.Cu) (net 1))
-  (segment (start 101.9633 114.5894) (end 100.838 115.7147) (width 0.25) (layer F.Cu) (net 1))
-  (segment (start 100.838 110.363) (end 99.7127 110.363) (width 0.25) (layer B.Cu) (net 1))
-  (segment (start 99.7127 110.363) (end 98.5874 111.4883) (width 0.25) (layer B.Cu) (net 1))
-  (segment (start 98.5874 111.4883) (end 84.3457 111.4883) (width 0.25) (layer B.Cu) (net 1))
+  (segment (start 100.076 116.84) (end 100.076 115.7147) (width 0.25) (layer F.Cu) (net 1))
+  (segment (start 100.076 110.363) (end 100.076 111.4883) (width 0.25) (layer F.Cu) (net 1))
+  (segment (start 100.076 111.4883) (end 101.2013 112.6136) (width 0.25) (layer F.Cu) (net 1))
+  (segment (start 101.2013 112.6136) (end 101.2013 114.5894) (width 0.25) (layer F.Cu) (net 1))
+  (segment (start 101.2013 114.5894) (end 100.076 115.7147) (width 0.25) (layer F.Cu) (net 1))
+  (segment (start 100.076 110.363) (end 98.9507 110.363) (width 0.25) (layer B.Cu) (net 1))
+  (segment (start 98.9507 110.363) (end 97.8254 111.4883) (width 0.25) (layer B.Cu) (net 1))
+  (segment (start 97.8254 111.4883) (end 84.3457 111.4883) (width 0.25) (layer B.Cu) (net 1))
   (segment (start 84.3457 111.4883) (end 79.502 116.332) (width 0.25) (layer B.Cu) (net 1))
-  (segment (start 93.218 110.363) (end 93.218 111.4883) (width 0.25) (layer F.Cu) (net 2))
-  (segment (start 93.218 111.4883) (end 94.3434 112.6137) (width 0.25) (layer F.Cu) (net 2))
-  (segment (start 94.3434 112.6137) (end 94.3434 126.1286) (width 0.25) (layer F.Cu) (net 2))
-  (segment (start 94.3434 126.1286) (end 94.107 126.365) (width 0.25) (layer F.Cu) (net 2))
+  (segment (start 92.456 110.363) (end 92.456 111.4883) (width 0.25) (layer F.Cu) (net 2))
+  (segment (start 92.456 111.4883) (end 94.107 113.1393) (width 0.25) (layer F.Cu) (net 2))
+  (segment (start 94.107 113.1393) (end 94.107 126.365) (width 0.25) (layer F.Cu) (net 2))
   (segment (start 82.042 116.332) (end 83.2373 116.332) (width 0.25) (layer B.Cu) (net 3))
-  (segment (start 100.838 113.665) (end 99.7127 113.665) (width 0.25) (layer B.Cu) (net 3))
-  (segment (start 99.7127 113.665) (end 98.5874 114.7903) (width 0.25) (layer B.Cu) (net 3))
-  (segment (start 98.5874 114.7903) (end 84.1813 114.7903) (width 0.25) (layer B.Cu) (net 3))
+  (segment (start 100.076 113.665) (end 98.9507 113.665) (width 0.25) (layer B.Cu) (net 3))
+  (segment (start 98.9507 113.665) (end 97.8254 114.7903) (width 0.25) (layer B.Cu) (net 3))
+  (segment (start 97.8254 114.7903) (end 84.1813 114.7903) (width 0.25) (layer B.Cu) (net 3))
   (segment (start 84.1813 114.7903) (end 83.2373 115.7343) (width 0.25) (layer B.Cu) (net 3))
   (segment (start 83.2373 115.7343) (end 83.2373 116.332) (width 0.25) (layer B.Cu) (net 3))
-  (segment (start 93.218 113.665) (end 93.218 114.7903) (width 0.25) (layer F.Cu) (net 4))
-  (segment (start 93.218 114.7903) (end 93.0772 114.7903) (width 0.25) (layer F.Cu) (net 4))
-  (segment (start 93.0772 114.7903) (end 92.0927 115.7748) (width 0.25) (layer F.Cu) (net 4))
-  (segment (start 92.0927 115.7748) (end 92.0927 122.0614) (width 0.25) (layer F.Cu) (net 4))
-  (segment (start 92.0927 122.0614) (end 86.3387 127.8154) (width 0.25) (layer F.Cu) (net 4))
-  (segment (start 86.3387 127.8154) (end 84.7624 127.8154) (width 0.25) (layer F.Cu) (net 4))
-  (segment (start 84.7624 127.8154) (end 83.312 126.365) (width 0.25) (layer F.Cu) (net 4))
-  (segment (start 93.218 116.84) (end 92.0927 116.84) (width 0.25) (layer B.Cu) (net 5))
-  (segment (start 92.0927 116.84) (end 90.9674 117.9653) (width 0.25) (layer B.Cu) (net 5))
-  (segment (start 90.9674 117.9653) (end 81.6787 117.9653) (width 0.25) (layer B.Cu) (net 5))
-  (segment (start 81.6787 117.9653) (end 73.279 126.365) (width 0.25) (layer B.Cu) (net 5))
+  (segment (start 92.456 113.665) (end 92.456 114.7903) (width 0.25) (layer F.Cu) (net 4))
+  (segment (start 92.456 114.7903) (end 92.3153 114.7903) (width 0.25) (layer F.Cu) (net 4))
+  (segment (start 92.3153 114.7903) (end 83.312 123.7936) (width 0.25) (layer F.Cu) (net 4))
+  (segment (start 83.312 123.7936) (end 83.312 126.365) (width 0.25) (layer F.Cu) (net 4))
+  (segment (start 92.456 116.84) (end 92.456 117.9653) (width 0.25) (layer F.Cu) (net 5))
+  (segment (start 92.456 117.9653) (end 92.3153 117.9653) (width 0.25) (layer F.Cu) (net 5))
+  (segment (start 92.3153 117.9653) (end 84.64 125.6406) (width 0.25) (layer F.Cu) (net 5))
+  (segment (start 84.64 125.6406) (end 84.64 127.3601) (width 0.25) (layer F.Cu) (net 5))
+  (segment (start 84.64 127.3601) (end 84.1878 127.8123) (width 0.25) (layer F.Cu) (net 5))
+  (segment (start 84.1878 127.8123) (end 74.7263 127.8123) (width 0.25) (layer F.Cu) (net 5))
+  (segment (start 74.7263 127.8123) (end 73.279 126.365) (width 0.25) (layer F.Cu) (net 5))
   (segment (start 75.819 126.365) (end 77.0143 126.365) (width 0.25) (layer F.Cu) (net 6))
   (segment (start 87.122 116.332) (end 85.9267 116.332) (width 0.25) (layer F.Cu) (net 6))
-  (segment (start 85.9267 116.332) (end 85.9267 115.7344) (width 0.25) (layer F.Cu) (net 6))
-  (segment (start 85.9267 115.7344) (end 85.0873 114.895) (width 0.25) (layer F.Cu) (net 6))
-  (segment (start 85.0873 114.895) (end 84.0701 114.895) (width 0.25) (layer F.Cu) (net 6))
-  (segment (start 84.0701 114.895) (end 83.3111 115.654) (width 0.25) (layer F.Cu) (net 6))
-  (segment (start 83.3111 115.654) (end 83.3111 120.0682) (width 0.25) (layer F.Cu) (net 6))
-  (segment (start 83.3111 120.0682) (end 77.0143 126.365) (width 0.25) (layer F.Cu) (net 6))
-  (segment (start 85.852 126.365) (end 84.6567 126.365) (width 0.25) (layer F.Cu) (net 7))
-  (segment (start 84.582 116.332) (end 84.582 126.2903) (width 0.25) (layer F.Cu) (net 7))
-  (segment (start 84.582 126.2903) (end 84.6567 126.365) (width 0.25) (layer F.Cu) (net 7))
+  (segment (start 85.9267 116.332) (end 85.9267 117.4526) (width 0.25) (layer F.Cu) (net 6))
+  (segment (start 85.9267 117.4526) (end 77.0143 126.365) (width 0.25) (layer F.Cu) (net 6))
+  (segment (start 85.852 124.8829) (end 85.852 124.9397) (width 0.25) (layer B.Cu) (net 7))
+  (segment (start 85.7773 116.332) (end 85.7773 124.8082) (width 0.25) (layer B.Cu) (net 7))
+  (segment (start 85.7773 124.8082) (end 85.852 124.8829) (width 0.25) (layer B.Cu) (net 7))
+  (segment (start 85.852 124.8829) (end 94.9408 124.8829) (width 0.25) (layer B.Cu) (net 7))
+  (segment (start 94.9408 124.8829) (end 95.4517 125.3938) (width 0.25) (layer B.Cu) (net 7))
+  (segment (start 95.4517 125.3938) (end 95.4517 126.365) (width 0.25) (layer B.Cu) (net 7))
   (segment (start 96.647 126.365) (end 95.4517 126.365) (width 0.25) (layer B.Cu) (net 7))
-  (segment (start 85.852 126.365) (end 87.0473 126.365) (width 0.25) (layer B.Cu) (net 7))
-  (segment (start 87.0473 126.365) (end 88.5068 124.9055) (width 0.25) (layer B.Cu) (net 7))
-  (segment (start 88.5068 124.9055) (end 94.9634 124.9055) (width 0.25) (layer B.Cu) (net 7))
-  (segment (start 94.9634 124.9055) (end 95.4517 125.3938) (width 0.25) (layer B.Cu) (net 7))
-  (segment (start 95.4517 125.3938) (end 95.4517 126.365) (width 0.25) (layer B.Cu) (net 7))
+  (segment (start 85.852 126.365) (end 85.852 124.9397) (width 0.25) (layer B.Cu) (net 7))
+  (segment (start 84.582 116.332) (end 85.7773 116.332) (width 0.25) (layer B.Cu) (net 7))
   (segment (start 89.154 136.398) (end 87.9587 136.398) (width 0.25) (layer B.Cu) (net 8))
   (segment (start 76.835 136.017) (end 78.0303 136.017) (width 0.25) (layer B.Cu) (net 8))
