File: PCBs/OH - Left Console - 4 - Exterior Lights Panel/OH - Left Console - 4 - Exterior Lights Panel.kicad_pcb (KiCad board)
At the start: 2 copper layers, 51 x 51 mm, 17 parts, among them J1 Columns In, J2 Backlight In, J3 Backlight Out, J4 Rows In, J5 Analog In, SW1 INT_WNG_TANK_SW, SW2 STROBE_SW, SW3 GEN_TIE_SW

Commit message: ext lights
Parts:
- removed H4: MountingHole, MountingHole:MountingHole_3.2mm_M3
Other:
- outline, holes or cut-outs redrawn
Changed lines of the file:
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@@
   (general
     (thickness 1.6)
-    (drawings 18)
+    (drawings 20)
     (tracks 83)
     (zones 0)
-    (modules 17)
+    (modules 16)
     (nets 14)
   )
@@
   )
   (module MountingHole:MountingHole_3.2mm_M3 locked (layer F.Cu)
-    (at 145 100)
-    (descr "Mounting Hole 3.2mm, no annular, M3")
-    (tags "mounting hole 3.2mm no annular m3")
-    (attr virtual)
-    (fp_text reference H4 (at 0 -4.2) (layer F.SilkS) hide
-      (effects (font (size 1 1) (thickness 0.15)))
-    )
-    (fp_text value MountingHole (at 0 4.2) (layer F.Fab) hide
-      (effects (font (size 1 1) (thickness 0.15)))
-    )
-    (fp_circle (center 0 0) (end 3.45 0) (layer F.CrtYd) (width 0.05))
-    (fp_circle (center 0 0) (end 3.2 0) (layer Cmts.User) (width 0.15))
-    (fp_text user %R (at 0.3 0) (layer F.Fab)
-      (effects (font (size 1 1) (thickness 0.15)))
-    )
-    (pad 1 np_thru_hole circle (at 0 0) (size 3.2 3.2) (drill 3.2) (layers *.Cu *.Mask))
-  )
-  (module MountingHole:MountingHole_3.2mm_M3 locked (layer F.Cu)
     (at 145 145)
     (descr "Mounting Hole 3.2mm, no annular, M3")
@@
     )
   )
+  (gr_line (start 143.002 129) (end 148 129) (layer Edge.Cuts) (width 0.05))
+  (gr_line (start 143 97) (end 143.002 129) (layer Edge.Cuts) (width 0.05))
   (gr_text - (at 141.859 130.937) (layer F.SilkS)
     (effects (font (size 1 1) (thickness 0.15)))
   )
   (gr_line (start 97 148) (end 97 97) (layer Edge.Cuts) (width 0.05))
-  (gr_line (start 148 97) (end 148 148) (layer Edge.Cuts) (width 0.05))
+  (gr_line (start 148 129) (end 148 148) (layer Edge.Cuts) (width 0.05))
   (gr_line (start 97 148) (end 148 148) (layer Edge.Cuts) (width 0.12))
-  (gr_line (start 97 97) (end 148 97) (layer Edge.Cuts) (width 0.12))
+  (gr_line (start 97 97) (end 143 97) (layer Edge.Cuts) (width 0.12))
   (gr_text "Pos\n" (at 108.712 129.286 90) (layer F.SilkS)
     (effects (font (size 1 1) (thickness 0.15)))

Commit message: pcb
Parts:
- removed the J4 at (113.5, 107.6)
- J1: value Columns In -> Switch_Inputs; footprint PT_Library_v001:Molex_1x02_P2.54mm_Vertical -> PT_Library_v001:Molex_1x04_P2.54mm_Vertical
- moved J1 6.02 mm to (108.6, 105.7)
- renumbered J5 to J4
Connections:
- net Net-(D1-Pad2) renamed /Col2
- net Net-(D2-Pad2) renamed /Col1
- SW1 pad 2: Net-(J4-Pad1) (its old number) -> /Row1
- SW2 pad 1: Net-(J4-Pad1) (its old number) -> /Row1
- SW2 pad 3: Net-(J4-Pad2) (its old number) -> /Row2
- SW3 pad 2: Net-(J4-Pad2) (its old number) -> /Row2
Routing:
- net /Row2: track 0.00 -> 40.0 mm
- net Net-(J4-Pad2) (its old number): track 38.8 -> 0.00 mm
- net /Row1: track 0.00 -> 38.7 mm
- net Net-(J4-Pad1) (its old number): track 36.2 -> 0.00 mm
- net /Col2: track 37.7 -> 33.1 mm
- net Net-(D2-Pad1): track 23.4 -> 22.2 mm
- net /Col1: track 12.3 -> 11.1 mm
Other:
- board text added: "Col1"
- board text added: "Col2"
- board text added: "Row1"
- board text added: "Row2"

Commit message: PCBs
Parts:
- moved SW1 6.22 mm to (128.7, 122.2)
- moved SW2 5.71 mm to (114.8, 122.2)
- moved D1 4.42 mm to (127.1, 114.3)
- moved D2 4.42 mm to (100.1, 114.0)
- moved D3 4.42 mm to (114.0, 114.2)
- moved RV1 2.84 mm to (136.3, 137.8)
- moved RV2 2.84 mm to (120.9, 137.8)
- moved J4 2.84 mm to (103.0, 137.4)
- moved SW3 2.54 mm to (102.5, 122.2)
Routing:
- net /Row2: track 40.0 -> 34.0 mm
- net /Col2: track 33.1 -> 28.4 mm
- net /Row1: track 38.7 -> 36.1 mm
- net /Col1: track 11.1 -> 8.75 mm
- net Net-(D3-Pad1): track 15.9 -> 14.9 mm
- net Net-(D2-Pad1): track 22.2 -> 21.2 mm
- net Net-(D1-Pad1): track 7.95 -> 8.51 mm
Other:
- outline, holes or cut-outs redrawn
