File: PCBs/OH - Left Console - 8 - LOX Indicator/OH - Left Console - 8 - LOX Indicator.kicad_pcb (KiCad board)
At the start: 2 copper layers, 47 x 46.2 mm, 11 parts, among them J1 Switch_Inputs, J2 LOX Analog, SW1 OBOGS_SW, SW2 OBOGS_FLOW

Commit message: PCBs
Other:
- board text added: "Row 1"
- board text removed: "Col 2"
Changed lines of the file:
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@@
     (effects (font (size 2 2) (thickness 0.15)))
   )
-  (gr_text "Row 2" (at 153.416 79.248 90) (layer F.SilkS)
+  (gr_text "Row 2" (at 153.416 79.509905 90) (layer F.SilkS)
     (effects (font (size 1 1) (thickness 0.15)))
   )
-  (gr_text "Col 2" (at 150.876 79.509905 90) (layer F.SilkS)
+  (gr_text "Row 1" (at 150.876 79.509905 90) (layer F.SilkS)
     (effects (font (size 1 1) (thickness 0.15)))
   )
-  (gr_text "Col 1" (at 148.336 79.509905 90) (layer F.SilkS)
+  (gr_text "Col 1" (at 148.336 79.77181 90) (layer F.SilkS)
     (effects (font (size 1 1) (thickness 0.15)))
   )
