File: PCBs/Eyebrow_warning_indicators/Right/EWI_Right.kicad_pcb (KiCad board)
At the start: 2 copper layers, 96.1 x 78.8 mm, 37 parts, among them J2 Conn_01x06_Male, J3 Conn_01x08_Male, SW1 IN SWTCH, SW2 OUT SWTCH

Commit message: footprint
Parts:
- added D31: D, Diode_THT:D_A-405_P7.62mm_Horizontal, F.Cu at (196.3, 75.6)
- added D32: D, Diode_THT:D_A-405_P7.62mm_Horizontal, F.Cu at (196.3, 79.8)
- added J1: Conn_01x02_Female, Connector_PinHeader_2.54mm:PinHeader_1x02_P2.54mm_Vertical, F.Cu at (208.0, 79.8)
- added J4: Conn_01x02_Female, Connector_PinHeader_2.54mm:PinHeader_1x02_P2.54mm_Vertical, F.Cu at (218.7, 75.8)
- added J5: Conn_01x02_Female, Connector_PinHeader_2.54mm:PinHeader_1x02_P2.54mm_Vertical, F.Cu at (212.6, 79.8)
- added R1: R, Resistor_THT:R_Axial_DIN0207_L6.3mm_D2.5mm_P7.62mm_Horizontal, F.Cu at (207.2, 75.5)
Connections:
- J3 pad 1: /SegG -> /SegDP
- J3 pad 2: /SegF -> /SegA
- J3 pad 3: /SegE -> /SegB
- J3 pad 4: /SegD -> /SegC
- J3 pad 5: /SegC -> /SegD
- J3 pad 6: /SegB -> /SegE
- J3 pad 7: /SegA -> /SegF
- J3 pad 8: /SegDP -> /SegG
- SW1 pad 1: /7 -> Net-(J5-Pad1)
- SW1 pad 2: Net-(SW1-Pad2) -> Net-(J5-Pad1)
- SW1 pad 3: (no net) -> /7
- SW1 pad 4: (no net) -> /7
- SW1 pad 5: (no net) -> Net-(R1-Pad2)
- SW1 pad 6: (no net) -> Net-(SW1-Pad6)
- SW2 pad 1: /8 -> Net-(J5-Pad1)
- SW2 pad 2: Net-(SW1-Pad2) -> Net-(J5-Pad1)
- SW2 pad 3: (no net) -> Net-(D32-Pad1)
- SW2 pad 4: (no net) -> Net-(D32-Pad1)
- SW2 pad 5: (no net) -> Net-(SW1-Pad6)
- SW2 pad 6: (no net) -> Net-(J1-Pad2)
Routing:
- net Net-(SW1-Pad2): track 24.9 -> 0.00 mm
- net Net-(J5-Pad1): track 0.00 -> 24.9 mm
Other:
- board text added: "Check all diodes in same direction add labels for connectors move leds around switches"
- board text removed: "+12V"
- board text removed: "+3.3V"
- board text removed: "+5V"
- board text removed: "REMOVE JUMPER FROM J4 TO ENABLE NANO PROGRAMMING"

Commit message: pcb
Parts:
- D32: footprint Diode_THT:D_A-405_P7.62mm_Horizontal -> Diode_THT:D_DO-35_SOD27_P7.62mm_Horizontal
Changed lines of the file:
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@@
     (uvia_drill 0.1)
+  )
+  (module Diode_THT:D_DO-35_SOD27_P7.62mm_Horizontal (layer F.Cu)
+    (at 196.34 79.83)
+    (descr "Diode, DO-35_SOD27 series, Axial, Horizontal, pin pitch=7.62mm, , length*diameter=4*2mm^2, , http://www.diodes.com/_files/packages/DO-35.pdf")
+    (tags "Diode DO-35_SOD27 series Axial Horizontal pin pitch 7.62mm  length 4mm diameter 2mm")
+    (fp_text reference D32 (at 3.81 -2.12) (layer F.SilkS)
+      (effects (font (size 1 1) (thickness 0.15)))
+    )
+    (fp_text value D (at 3.81 2.12) (layer F.Fab)
+      (effects (font (size 1 1) (thickness 0.15)))
+    )
+    (fp_text user K (at 0 -1.8) (layer F.Fab)
+      (effects (font (size 1 1) (thickness 0.15)))
+    )
+    (fp_text user K (at 0 -1.8) (layer F.Fab)
+      (effects (font (size 1 1) (thickness 0.15)))
+    )
+    (fp_text user %R (at 4.11 0) (layer F.Fab)
+      (effects (font (size 0.8 0.8) (thickness 0.12)))
+    )
+    (fp_line (start 8.67 -1.25) (end -1.05 -1.25) (layer F.CrtYd) (width 0.05))
+    (fp_line (start 8.67 1.25) (end 8.67 -1.25) (layer F.CrtYd) (width 0.05))
+    (fp_line (start -1.05 1.25) (end 8.67 1.25) (layer F.CrtYd) (width 0.05))
+    (fp_line (start -1.05 -1.25) (end -1.05 1.25) (layer F.CrtYd) (width 0.05))
+    (fp_line (start 2.29 -1.12) (end 2.29 1.12) (layer F.SilkS) (width 0.12))
+    (fp_line (start 2.53 -1.12) (end 2.53 1.12) (layer F.SilkS) (width 0.12))
+    (fp_line (start 2.41 -1.12) (end 2.41 1.12) (layer F.SilkS) (width 0.12))
+    (fp_line (start 6.58 0) (end 5.93 0) (layer F.SilkS) (width 0.12))
+    (fp_line (start 1.04 0) (end 1.69 0) (layer F.SilkS) (width 0.12))
+    (fp_line (start 5.93 -1.12) (end 1.69 -1.12) (layer F.SilkS) (width 0.12))
+    (fp_line (start 5.93 1.12) (end 5.93 -1.12) (layer F.SilkS) (width 0.12))
+    (fp_line (start 1.69 1.12) (end 5.93 1.12) (layer F.SilkS) (width 0.12))
+    (fp_line (start 1.69 -1.12) (end 1.69 1.12) (layer F.SilkS) (width 0.12))
+    (fp_line (start 2.31 -1) (end 2.31 1) (layer F.Fab) (width 0.1))
+    (fp_line (start 2.51 -1) (end 2.51 1) (layer F.Fab) (width 0.1))
+    (fp_line (start 2.41 -1) (end 2.41 1) (layer F.Fab) (width 0.1))
+    (fp_line (start 7.62 0) (end 5.81 0) (layer F.Fab) (width 0.1))
+    (fp_line (start 0 0) (end 1.81 0) (layer F.Fab) (width 0.1))
+    (fp_line (start 5.81 -1) (end 1.81 -1) (layer F.Fab) (width 0.1))
+    (fp_line (start 5.81 1) (end 5.81 -1) (layer F.Fab) (width 0.1))
+    (fp_line (start 1.81 1) (end 5.81 1) (layer F.Fab) (width 0.1))
+    (fp_line (start 1.81 -1) (end 1.81 1) (layer F.Fab) (width 0.1))
+    (pad 2 thru_hole oval (at 7.62 0) (size 1.6 1.6) (drill 0.8) (layers *.Cu *.Mask)
+      (net 17 "Net-(D32-Pad2)"))
+    (pad 1 thru_hole rect (at 0 0) (size 1.6 1.6) (drill 0.8) (layers *.Cu *.Mask)
+      (net 18 "Net-(D32-Pad1)"))
+    (model ${KISYS3DMOD}/Diode_THT.3dshapes/D_DO-35_SOD27_P7.62mm_Horizontal.wrl
+      (at (xyz 0 0 0))
+      (scale (xyz 1 1 1))
+      (rotate (xyz 0 0 0))
+    )
   )
   (module Resistor_THT:R_Axial_DIN0207_L6.3mm_D2.5mm_P7.62mm_Horizontal (layer F.Cu)
@@
   )
   (module Diode_THT:D_A-405_P7.62mm_Horizontal (layer F.Cu)
-    (at 196.34 79.83)
-    (descr "Diode, A-405 series, Axial, Horizontal, pin pitch=7.62mm, , length*diameter=5.2*2.7mm^2, , http://www.diodes.com/_files/packages/A-405.pdf")
-    (tags "Diode A-405 series Axial Horizontal pin pitch 7.62mm  length 5.2mm diameter 2.7mm")
-    (fp_text reference D32 (at 3.81 -2.47) (layer F.SilkS)
-      (effects (font (size 1 1) (thickness 0.15)))
-    )
-    (fp_text value D (at 3.81 2.47) (layer F.Fab)
-      (effects (font (size 1 1) (thickness 0.15)))
-    )
-    (fp_text user K (at 0 -1.9) (layer F.SilkS)
-      (effects (font (size 1 1) (thickness 0.15)))
-    )
-    (fp_text user K (at 0 -1.9) (layer F.Fab)
-      (effects (font (size 1 1) (thickness 0.15)))
-    )
-    (fp_text user %R (at 4.2 0) (layer F.Fab)
-      (effects (font (size 1 1) (thickness 0.15)))
-    )
-    (fp_line (start 8.77 -1.6) (end -1.15 -1.6) (layer F.CrtYd) (width 0.05))
-    (fp_line (start 8.77 1.6) (end 8.77 -1.6) (layer F.CrtYd) (width 0.05))
-    (fp_line (start -1.15 1.6) (end 8.77 1.6) (layer F.CrtYd) (width 0.05))
-    (fp_line (start -1.15 -1.6) (end -1.15 1.6) (layer F.CrtYd) (width 0.05))
-    (fp_line (start 1.87 -1.47) (end 1.87 1.47) (layer F.SilkS) (width 0.12))
-    (fp_line (start 2.11 -1.47) (end 2.11 1.47) (layer F.SilkS) (width 0.12))
-    (fp_line (start 1.99 -1.47) (end 1.99 1.47) (layer F.SilkS) (width 0.12))
-    (fp_line (start 6.53 1.47) (end 6.53 1.14) (layer F.SilkS) (width 0.12))
-    (fp_line (start 1.09 1.47) (end 6.53 1.47) (layer F.SilkS) (width 0.12))
-    (fp_line (start 1.09 1.14) (end 1.09 1.47) (layer F.SilkS) (width 0.12))
-    (fp_line (start 6.53 -1.47) (end 6.53 -1.14) (layer F.SilkS) (width 0.12))
-    (fp_line (start 1.09 -1.47) (end 6.53 -1.47) (layer F.SilkS) (width 0.12))
-    (fp_line (start 1.09 -1.14) (end 1.09 -1.47) (layer F.SilkS) (width 0.12))
-    (fp_line (start 1.89 -1.35) (end 1.89 1.35) (layer F.Fab) (width 0.1))
-    (fp_line (start 2.09 -1.35) (end 2.09 1.35) (layer F.Fab) (width 0.1))
-    (fp_line (start 1.99 -1.35) (end 1.99 1.35) (layer F.Fab) (width 0.1))
-    (fp_line (start 7.62 0) (end 6.41 0) (layer F.Fab) (width 0.1))
-    (fp_line (start 0 0) (end 1.21 0) (layer F.Fab) (width 0.1))
-    (fp_line (start 6.41 -1.35) (end 1.21 -1.35) (layer F.Fab) (width 0.1))
-    (fp_line (start 6.41 1.35) (end 6.41 -1.35) (layer F.Fab) (width 0.1))
-    (fp_line (start 1.21 1.35) (end 6.41 1.35) (layer F.Fab) (width 0.1))
-    (fp_line (start 1.21 -1.35) (end 1.21 1.35) (layer F.Fab) (width 0.1))
-    (pad 2 thru_hole oval (at 7.62 0) (size 1.8 1.8) (drill 0.9) (layers *.Cu *.Mask)
-      (net 17 "Net-(D32-Pad2)"))
-    (pad 1 thru_hole rect (at 0 0) (size 1.8 1.8) (drill 0.9) (layers *.Cu *.Mask)
-      (net 18 "Net-(D32-Pad1)"))
-    (model ${KISYS3DMOD}/Diode_THT.3dshapes/D_A-405_P7.62mm_Horizontal.wrl
-      (at (xyz 0 0 0))
-      (scale (xyz 1 1 1))
-      (rotate (xyz 0 0 0))
-    )
-  )
-  (module Diode_THT:D_A-405_P7.62mm_Horizontal (layer F.Cu)
     (at 196.34 75.58)
     (descr "Diode, A-405 series, Axial, Horizontal, pin pitch=7.62mm, , length*diameter=5.2*2.7mm^2, , http://www.diodes.com/_files/packages/A-405.pdf")
@@
       (effects (font (size 1 1) (thickness 0.15)))
     )
-    (fp_text user K (at 0 -1.9) (layer F.SilkS)
+    (fp_text user K (at 0 -1.9) (layer F.Fab)
       (effects (font (size 1 1) (thickness 0.15)))
     )
@@
     )
     (fp_line (start -4.318 -3.81) (end -3.048 -3.81) (layer F.SilkS) (width 0.12))
-    (fp_line (start -4.318 4.318) (end -4.318 -3.81) (layer F.SilkS) (width 0.12))
-    (fp_line (start 4.064 4.318) (end -4.318 4.318) (layer F.SilkS) (width 0.12))
-    (fp_line (start 4.064 -3.81) (end 4.064 4.318) (layer F.SilkS) (width 0.12))
+    (fp_line (start -4.32 3.81) (end -4.318 -3.81) (layer F.SilkS) (width 0.12))
+    (fp_line (start 4.07 3.81) (end -4.312 3.81) (layer F.SilkS) (width 0.12))
+    (fp_line (start 4.064 -3.81) (end 4.05 3.81) (layer F.SilkS) (width 0.12))
     (fp_line (start -4.064 -3.81) (end 4.064 -3.81) (layer F.SilkS) (width 0.12))
     (fp_text user - (at -1.524 3.302 90) (layer F.SilkS)
@@
       (effects (font (size 1 1) (thickness 0.15)))
     )
-    (pad 6 thru_hole circle (at 0 3.429 270) (size 1.524 1.524) (drill 0.762) (layers *.Cu *.Mask)
+    (pad 6 thru_hole circle (at 0.04 2.87 270) (size 1.524 1.524) (drill 0.762) (layers *.Cu *.Mask)
       (net 19 "Net-(J1-Pad2)"))
     (pad 5 thru_hole circle (at 0 -2.921 270) (size 1.524 1.524) (drill 0.762) (layers *.Cu *.Mask)
@@
     )
     (fp_line (start -4.318 -3.81) (end -3.048 -3.81) (layer F.SilkS) (width 0.12))
-    (fp_line (start -4.318 4.318) (end -4.318 -3.81) (layer F.SilkS) (width 0.12))
-    (fp_line (start 4.064 4.318) (end -4.318 4.318) (layer F.SilkS) (width 0.12))
-    (fp_line (start 4.064 -3.81) (end 4.064 4.318) (layer F.SilkS) (width 0.12))
+    (fp_line (start -4.32 3.81) (end -4.318 -3.81) (layer F.SilkS) (width 0.12))
+    (fp_line (start 4.07 3.81) (end -4.312 3.81) (layer F.SilkS) (width 0.12))
+    (fp_line (start 4.064 -3.81) (end 4.05 3.81) (layer F.SilkS) (width 0.12))
     (fp_line (start -4.064 -3.81) (end 4.064 -3.81) (layer F.SilkS) (width 0.12))
     (fp_text user - (at -1.524 3.302 90) (layer F.SilkS)
@@
       (effects (font (size 1 1) (thickness 0.15)))
     )
-    (pad 6 thru_hole circle (at 0 3.429 270) (size 1.524 1.524) (drill 0.762) (layers *.Cu *.Mask)
+    (pad 6 thru_hole circle (at 0.04 2.87 270) (size 1.524 1.524) (drill 0.762) (layers *.Cu *.Mask)
       (net 24 "Net-(SW1-Pad6)"))
     (pad 5 thru_hole circle (at 0 -2.921 270) (size 1.524 1.524) (drill 0.762) (layers *.Cu *.Mask)

Commit message: PCB
Parts:
- D31: footprint Diode_THT:D_A-405_P7.62mm_Horizontal -> PT_Library_v001:D_Signal_P7.62mm_Horizontal
- D32: footprint Diode_THT:D_DO-35_SOD27_P7.62mm_Horizontal -> PT_Library_v001:D_Signal_P7.62mm_Horizontal
- J1: value Conn_01x02_Female -> Backlight; footprint Connector_PinHeader_2.54mm:PinHeader_1x02_P2.54mm_Vertical -> PT_Library_v001:Molex_1x02_P2.54mm_Vertical; moved to B.Cu
- J2: value Conn_01x06_Male -> Led Cathode; footprint Connector_PinHeader_2.54mm:PinHeader_1x06_P2.54mm_Vertical -> PT_Library_v001:Molex_1x06_P2.54mm_Vertical; moved to B.Cu
- J3: value Conn_01x08_Male -> Led Annode; footprint Connector_PinHeader_2.54mm:PinHeader_1x08_P2.54mm_Vertical -> PT_Library_v001:Molex_1x08_P2.54mm_Vertical; moved to B.Cu
- J4: value Conn_01x02_Female -> SwitchCol; footprint Connector_PinHeader_2.54mm:PinHeader_1x02_P2.54mm_Vertical -> PT_Library_v001:Molex_1x02_P2.54mm_Vertical; moved to B.Cu
- J5: value Conn_01x02_Female -> SwitchRow; footprint Connector_PinHeader_2.54mm:PinHeader_1x02_P2.54mm_Vertical -> PT_Library_v001:Molex_1x02_P2.54mm_Vertical; moved to B.Cu
- R1: value R -> 330
- moved J4 55.1 mm to (170.9, 48.3), turned to 270 degrees
- moved J5 48.7 mm to (170.9, 54.6), turned to 270 degrees
- moved J2 48.5 mm to (152.7, 64.0), turned to 270 degrees
- moved J1 41.3 mm to (170.7, 62.0), turned to 270 degrees
- moved J3 32.7 mm to (152.7, 39.4), turned to 270 degrees
- moved R1 16.3 mm to (193.5, 66.5)
- moved D31 16.0 mm to (183.1, 66.5)
- moved D32 15.3 mm to (204.0, 66.5)
- moved D27 2.64 mm to (200.4, 52.8), turned to 90 degrees
- moved D23 2.55 mm to (176.4, 52.4), turned to 90 degrees
- moved D25 2.55 mm to (188.0, 52.4), turned to 90 degrees
- moved D29 2.55 mm to (212.1, 52.8), turned to 90 degrees
- moved D1 0.84 mm to (140.0, 41.3)
- moved D2 0.84 mm to (140.0, 50.3)
- moved D3 0.84 mm to (140.0, 59.3)
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Connections:
- D31 pad 1: /7 -> Net-(D31-Pad1)
- SW1 pad 1: Net-(J5-Pad1) -> Net-(D31-Pad1)
- SW1 pad 2: Net-(J5-Pad1) -> Net-(D31-Pad1)
- SW1 pad 3: /7 -> Net-(J5-Pad1)
- SW1 pad 4: /7 -> Net-(J5-Pad1)
- SW2 pad 1: Net-(J5-Pad1) -> Net-(D32-Pad1)
- SW2 pad 2: Net-(J5-Pad1) -> Net-(D32-Pad1)
- SW2 pad 3: Net-(D32-Pad1) -> Net-(J5-Pad1)
- SW2 pad 4: Net-(D32-Pad1) -> Net-(J5-Pad1)
Routing:
- net /Dig5: track 83.4 -> 19.6 mm
- net Net-(D32-Pad2): track 0.00 -> 52.5 mm
- net /Dig4: track 77.2 -> 27.9 mm
- net /Dig3: track 70.9 -> 29.3 mm
- net /SegDP: track 102.4 -> 63.4 mm
- net /SegA: track 90.8 -> 53.2 mm
- net Net-(D31-Pad1): track 0.00 -> 35.7 mm
- net Net-(D31-Pad2): track 0.00 -> 32.8 mm
- net Net-(D32-Pad1): track 0.00 -> 29.7 mm
- net /Dig0: track 77.6 -> 51.9 mm
- net Net-(J1-Pad1): track 0.00 -> 25.7 mm
- net /SegE: track 20.8 -> 45.3 mm
- net /SegB: track 69.4 -> 44.8 mm
- net Net-(J5-Pad1): track 24.9 -> 49.0 mm
- net /SegF: track 34.6 -> 58.3 mm
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Other:
- board text added: "+"
- board text added: "330"
- board text added: "AAA"
- board text added: "AI"
- board text added: "APU FIRE"
- board text added: "Backlight"
- board text added: "CW"
- board text added: "DISP"
- board text added: "FIRE"
- board text added: "Green"
- board text added: "LED Annode"
- board text added: "LED Cathode"
- board text added: "RCDR ON"
- board text added: "Red"
- board text added: "SAM"
- board text added: "Switch Col"
- board text added: "Switch Row"
- board text removed: "Check all diodes in same direction add labels for connectors move leds around switches"

Commit message: PCB prior to Gerber
Other:
- board text added: "Right Eyebrow v001"
Changed lines of the file:
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@@
   (general
     (thickness 1.2)
-    (drawings 95)
+    (drawings 96)
     (tracks 274)
     (zones 0)
@@
     (pad 1 np_thru_hole circle (at 0 0 180) (size 2.7 2.7) (drill 2.7) (layers *.Cu *.Mask))
   )
+  (gr_text "Right Eyebrow\nv001" (at 144.272 92.964) (layer F.SilkS)
+    (effects (font (size 1 1) (thickness 0.15)))
+  )
   (gr_text Green (at 165.1 36.83) (layer F.SilkS)

Commit message: update
Other:
- board text added: "Right Eyebrow v002"
- board text removed: "Right Eyebrow v001"
Changed lines of the file:
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@@
     (pad 1 np_thru_hole circle (at 0 0 180) (size 2.7 2.7) (drill 2.7) (layers *.Cu *.Mask))
   )
-  (gr_text "Right Eyebrow\nv001" (at 144.272 92.964) (layer F.SilkS)
+  (gr_text "Right Eyebrow\nv002" (at 144.272 92.964) (layer F.SilkS)
     (effects (font (size 1 1) (thickness 0.15)))
   )
@@
     (effects (font (size 1 1) (thickness 0.15)))
   )
-  (gr_text Red (at 165.1 63.754) (layer F.SilkS)
+  (gr_text Green (at 165.1 63.754) (layer F.SilkS)
     (effects (font (size 1 1) (thickness 0.15)))
   )
-  (gr_text Red (at 157.48 63.754) (layer F.SilkS)
+  (gr_text Green (at 157.48 63.754) (layer F.SilkS)
     (effects (font (size 1 1) (thickness 0.15)))
   )
-  (gr_text Red (at 165.1 72.644) (layer F.SilkS)
+  (gr_text Green (at 165.1 72.644) (layer F.SilkS)
     (effects (font (size 1 1) (thickness 0.15)))
   )
-  (gr_text Red (at 157.48 72.644) (layer F.SilkS)
+  (gr_text Green (at 157.48 72.644) (layer F.SilkS)
     (effects (font (size 1 1) (thickness 0.15)))
   )
-  (gr_text Red (at 147.828 72.898) (layer F.SilkS)
+  (gr_text Green (at 147.828 72.898) (layer F.SilkS)
     (effects (font (size 1 1) (thickness 0.15)))
   )
-  (gr_text Red (at 140.208 72.644) (layer F.SilkS)
+  (gr_text Green (at 140.208 72.644) (layer F.SilkS)
     (effects (font (size 1 1) (thickness 0.15)))
   )
-  (gr_text Red (at 147.828 81.534) (layer F.SilkS)
+  (gr_text Green (at 147.828 81.534) (layer F.SilkS)
     (effects (font (size 1 1) (thickness 0.15)))
   )
-  (gr_text Red (at 140.208 81.534) (layer F.SilkS)
+  (gr_text Green (at 140.208 81.534) (layer F.SilkS)
     (effects (font (size 1 1) (thickness 0.15)))
   )
