File: PCBs/OH - Upper Mixed Small PCBs/COPY OF PEDEAL OUTsch.sch (KiCad schematic (older format))
At the start: 5 parts, among them J26 PEDAL POWER IN, J27 To Motor, J28 Rear Limit Switch, J29 Directional Move Switch, J30 Forward Limit Switch

Commit message: PCBS
Parts:
- added H1, H11, H12, H14, H15, H16, H17, H18, H19, H20, H21, H22, H23, H24, H25, H26, H27, H28, H29, H30, H31, H32, H5, H8: MountingHole, MountingHole:MountingHole_4.3mm_M4, symbol Mechanical:MountingHole
- J26: footprint PT_Library_v001:Molex_1x02_P2.54mm_Vertical -> Connector_BarrelJack:BarrelJack_Horizontal
- J28: value Rear Limit Switch -> Rear Limit
- J30: value Forward Limit Switch -> Forward Limit
