File: PCBs/OH - Vid Record and IFEI/Vid Record and IFEI.kicad_pcb (KiCad board)
At the start: 2 copper layers, 22 parts, among them J1 IFEI NEXTRON, J10 BKLGHT, J2 IFEI BRIGHTNESS, J3 IFEI Buttons, J4 SWITCH INPUTS, J5 BKLGHT, J6 BKLGHT, J7 BKLGHT, J8 BKLGHT, J9 BKLGHT, SW1 IFEI Off, SW2 L DDI / HUD, SW3 MAN OFF AUTO

Commit message: PCBs
Other:
- board text added: "5V IN GND"
Changed lines of the file:
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@@
   (general
     (thickness 1.6)
-    (drawings 6)
+    (drawings 10)
     (tracks 148)
     (zones 0)
@@
     )
   )
+  (gr_text "5V IN GND" (at 159.5755 101.5365) (layer F.SilkS)
+    (effects (font (size 1 1) (thickness 0.15)))
+  )
+  (gr_text "5V IN GND" (at 145.8595 101.854) (layer F.SilkS)
+    (effects (font (size 1 1) (thickness 0.15)))
+  )
+  (gr_text "5V IN GND" (at 185.547 101.473) (layer F.SilkS)
+    (effects (font (size 1 1) (thickness 0.15)))
+  )
+  (gr_text "5V IN GND" (at 173.609 101.473) (layer F.SilkS)
+    (effects (font (size 1 1) (thickness 0.15)))
+  )
   (gr_text V001 (at 143.637 117.7925) (layer F.SilkS)

Commit message: IFEI COMBINED INPUT ORDERED
Parts:
- J1: value IFEI NEXTRON -> IFEI NEXTION
Changed lines of the file:
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@@
       (outputformat 1)
       (mirror false)
-      (drillshape 1)
+      (drillshape 0)
       (scaleselection 1)
-      (outputdirectory ""))
+      (outputdirectory "MANUFACTURING"))
   )
   (net 0 "")
@@
     (tags "mounting hole 4.3mm no annular m4")
     (attr virtual)
-    (fp_text reference H4 (at 0 -5.3) (layer F.SilkS)
+    (fp_text reference H4 (at 0 -5.3) (layer F.Fab)
       (effects (font (size 1 1) (thickness 0.15)))
     )
@@
     (tags "mounting hole 4.3mm no annular m4")
     (attr virtual)
-    (fp_text reference H3 (at 0 -5.3) (layer F.SilkS)
+    (fp_text reference H3 (at 0.049 -3.2765) (layer F.Fab)
       (effects (font (size 1 1) (thickness 0.15)))
     )
@@
     (tags "mounting hole 4.3mm no annular m4")
     (attr virtual)
-    (fp_text reference H1 (at 0 -5.3) (layer F.SilkS)
+    (fp_text reference H1 (at 0 -5.3) (layer F.Fab)
       (effects (font (size 1 1) (thickness 0.15)))
     )
@@
       (effects (font (size 1 1) (thickness 0.15)) (justify mirror))
     )
-    (fp_text value "IFEI NEXTRON" (at 2.54 4.08) (layer F.SilkS)
+    (fp_text value "IFEI NEXTION" (at 2.54 4.08) (layer F.SilkS)
       (effects (font (size 1 1) (thickness 0.15)))
     )
@@
     (descr "Diode, DO-35_SOD27 series, Axial, Horizontal, pin pitch=7.62mm, , length*diameter=4*2mm^2, , http://www.diodes.com/_files/packages/DO-35.pdf")
     (tags "Diode DO-35_SOD27 series Axial Horizontal pin pitch 7.62mm  length 4mm diameter 2mm")
-    (fp_text reference D3 (at 3.81 -2.12) (layer F.SilkS)
-      (effects (font (size 1 1) (thickness 0.15)))
+    (fp_text reference D3 (at 4.0635 0.0635) (layer B.SilkS)
+      (effects (font (size 1 1) (thickness 0.15)) (justify mirror))
     )
     (fp_text value D (at 3.81 2.12) (layer F.Fab)
@@
     (descr "Diode, DO-35_SOD27 series, Axial, Horizontal, pin pitch=7.62mm, , length*diameter=4*2mm^2, , http://www.diodes.com/_files/packages/DO-35.pdf")
     (tags "Diode DO-35_SOD27 series Axial Horizontal pin pitch 7.62mm  length 4mm diameter 2mm")
-    (fp_text reference D2 (at 3.81 -2.12) (layer F.SilkS)
-      (effects (font (size 1 1) (thickness 0.15)))
+    (fp_text reference D2 (at 4.0635 0.127) (layer B.SilkS)
+      (effects (font (size 1 1) (thickness 0.15)) (justify mirror))
     )
     (fp_text value D (at 3.81 2.12) (layer F.Fab)
@@
     (descr "Diode, DO-35_SOD27 series, Axial, Horizontal, pin pitch=7.62mm, , length*diameter=4*2mm^2, , http://www.diodes.com/_files/packages/DO-35.pdf")
     (tags "Diode DO-35_SOD27 series Axial Horizontal pin pitch 7.62mm  length 4mm diameter 2mm")
-    (fp_text reference D1 (at 3.81 -2.12) (layer F.SilkS)
-      (effects (font (size 1 1) (thickness 0.15)))
+    (fp_text reference D1 (at 3.8735 0) (layer B.SilkS)
+      (effects (font (size 1 1) (thickness 0.15)) (justify mirror))
     )
     (fp_text value D (at 3.81 2.12) (layer F.Fab)
