File: PCBs/OH - Hornet Forward Output Shield/Hornet Forward Output Shield.sch (KiCad schematic (older format))
At the start: 21 parts, among them J1 MATRIX INPUT, J10 DIGITAL B, J11 DIGITAL C, J2 5V to Max7219, J3 7219 OUT, J4 ANALOG B, J6 ANALOG A, J7 Address Select 0, J8 Address Select 1, J9 DIGITAL A, P1 Power, P2 Analog, P3 Analog, P4 Digital, P5 PWM, P6 PWM, P7 Communication

Commit message: PCBS
Parts:
- added J12: LEFT SERVO, PT_Library_v001:Molex_1x03_P2.54mm_Vertical, symbol Connector:Conn_01x03_Female
- added J13: RIGHT OUTPUT DIST, PT_Library_v001:Molex_1x06_P2.54mm_Vertical, symbol Connector:Conn_01x06_Female
- added J14: LEFT STEPPER, PT_Library_v001:Molex_1x04_P2.54mm_Vertical, symbol Connector:Conn_01x04_Female
- added J5: LEFT OUTPUT DIST, PT_Library_v001:Molex_1x10_P2.54mm_Vertical, symbol Connector:Conn_01x08_Female
- J1: value MATRIX INPUT -> OUTPUT

Commit message: PCBS
Parts:
- removed J10: DIGITAL B, PT_Library_v001:Molex_1x06_P2.54mm_Vertical, symbol Connector:Conn_01x06_Female
- removed J11: DIGITAL C, PT_Library_v001:Molex_1x06_P2.54mm_Vertical, symbol Connector:Conn_01x06_Female
- removed J4: ANALOG B, PT_Library_v001:Molex_1x10_P2.54mm_Vertical, symbol Connector:Conn_01x10_Female
- removed J6: ANALOG A, PT_Library_v001:Molex_1x10_P2.54mm_Vertical, symbol Connector:Conn_01x08_Female
- removed J9: DIGITAL A, PT_Library_v001:Molex_1x06_P2.54mm_Vertical, symbol Connector:Conn_01x06_Female
- added J4: RIGHT SERVO, PT_Library_v001:Molex_1x06_P2.54mm_Vertical, symbol Connector:Conn_01x06_Female
- added J6: RIGHT STEPPER, PT_Library_v001:Molex_1x04_P2.54mm_Vertical, symbol Connector:Conn_01x04_Female
- J5: footprint PT_Library_v001:Molex_1x10_P2.54mm_Vertical -> PT_Library_v001:Molex_1x08_P2.54mm_Vertical
Connections:
- net labels added: APU_MAG, BLEED_AIR_SOL, BP_STEP_COIL_A, BP_STEP_COIL_B, BP_STEP_COIL_C, BP_STEP_COIL_D, CANOPY_MAG, D14, D15, D16, D17, D18, ENGINE_CRANK_MAG, FUEL_DUMP_MAG, HOOK_BYPASS_MAG, LANDING_GEAR_SOL, LASER_ARM_MAG, LAUNCH_BAR_MAG, PITOT_HEAT_MAG, R_ALT_STEP_COIL_A, R_ALT_STEP_COIL_B, R_ALT_STEP_COIL_C, R_ALT_STEP_COIL_D, SERVO_5V, SERVO_ALT_FLAG, SERVO_BATT_E, SERVO_BATT_U, SERVO_GND, SERVO_HYD_PRS_1, SERVO_HYD_PRS_2, SERVO_TRIM
- net labels removed: 0(Rx0), 1(Tx0), 11(**), 12(**), 13(**), 2(**), 3(**), 5(**), 6(**), 7(**), 8(**), 9(**), ENC-1-A, ENC-1-B, ENC-2-A, ENC-2-B, ENC-3-A, ENC-3-B, ENC-4-A, ENC-4-B
- wire segments 98 -> 95
- no-connect marks 22 -> 24
Other:
- note added: "CORRECT SERVO POWER"
- moved on the sheet: J12, P4

Commit message: PCBS
Parts:
- removed J1: OUTPUT, Connector_IDC:IDC-Header_2x17_P2.54mm_Vertical, symbol Connector:Conn_01x34_Female
- added J1: CABIN ALT, PT_Library_v001:Molex_1x04_P2.54mm_Vertical, symbol Connector:Conn_01x04_Female
- added J10: I2C, PT_Library_v001:Molex_1x04_P2.54mm_Vertical, symbol Connector:Conn_01x04_Female
- added J11: NEXTION, PT_Library_v001:Molex_1x04_P2.54mm_Vertical, symbol Connector:Conn_01x04_Female
- added J9: PIXEL LEDS, PT_Library_v001:Molex_1x08_P2.54mm_Vertical, symbol Connector:Conn_01x08_Female
- J14: value LEFT STEPPER -> BRAKE PRESSURE
- J6: value RIGHT STEPPER -> RADAR ALT
- J7, J8: footprint PT_Library_v001:Molex_1x02_P2.54mm_Vertical -> Connector_PinHeader_2.54mm:PinHeader_1x02_P2.54mm_Vertical
Connections:
- net labels added: ADDRESS_SELECT_0, ADDRESS_SELECT_1, CA_STEP_COIL_A, CA_STEP_COIL_B, CA_STEP_COIL_C, CA_STEP_COIL_D, GREEN_LED, LED_CHAIN_1, LED_CHAIN_2, LED_CHAIN_3, LED_CHAIN_4, LED_CHAIN_5, LED_CHAIN_6, NEXTION_RX, NEXTION_TX, RED_LED, SCL, SDA
- net labels removed: COL0, COL1, COL10, COL2, COL3, COL4, COL5, COL6, COL7, COL8, COL9, D18, ROW0, ROW1, ROW10, ROW11, ROW12, ROW13, ROW14, ROW15, ROW2, ROW3, ROW4, ROW5, ROW6, ROW7, ROW8, ROW9
- wire segments 95 -> 102
- no-connect marks 24 -> 16
Other:
- note removed: "Output block which can be removed"
- note removed: "To dos\nOutput Channels for Lukes LEDs (Max 6 Channels)\nIdeally catch I2C bus\nSPI Bus\nServos - how many needed\ndirect outputs for Mag switches etc"
- moved on the sheet: J12, J13, J14, J4, J5, J6, J7, J8

Commit message: PCBS
Parts:
- removed J4: RIGHT SERVO, PT_Library_v001:Molex_1x06_P2.54mm_Vertical, symbol Connector:Conn_01x06_Female
- added J15: 5V IN, Connector_BarrelJack:BarrelJack_Horizontal, symbol Connector:Conn_01x02_Female
- added J16: UPPER 5V OUT, PT_Library_v001:Molex_1x02_P2.54mm_Vertical, symbol Connector:Conn_01x02_Female
- added J4: RIGHT_SERVO, PT_Library_v001:Molex_1x08_P2.54mm_Vertical, symbol Connector:Conn_01x08_Female
- J2: value 5V to Max7219 -> LOWER 5V IN
Connections:
- net +5V: no longer J10.1 (Pin_1), J11.1 (Pin_1), J2.1 (Pin_1)
- net +5VL: no longer J12.2 (Pin_2)
- net D11: now also J4.3 (Pin_3)
- net D6: now also J4.7 (Pin_7)
- net D7: now also J4.6 (Pin_6)
- net D8: now also J4.5 (Pin_5)
- net D9: now also J4.4 (Pin_4)
- net GND: now also J2.2 (Pin_2)
- net GNDD: now also J15.2 (Pin_2), J16.2 (Pin_2), J4.2 (Pin_2)
- net LOWER_OUTPUT_5V: now reaches J3.1 (Pin_1)
- net LOWER_OUTPUT_5V: now also J10.1 (Pin_1), J11.1 (Pin_1), J2.1 (Pin_1); no longer J2.2 (Pin_2)
- new net UPPER_OUTPUT_5V: J12.2 (Pin_2), J15.1 (Pin_1), J16.1 (Pin_1), J4.1 (Pin_1)
- no-connect marks 16 -> 17
Other:
- note added: "Powering the Servos and LEDs and Nextron is done through a barrel connect to the upper board and then carried across to \nthe lower board through stand headers. As boards are split, separate 5V buses are used in this diagram."
- note removed: "CORRECT SERVO POWER"
- moved on the sheet: J2, J3, J5
Changed lines of the file:
@@
 Red LED - solid\non until a packet\nis succesfully \nsent to controller
 Wire Wire Line
-	2850 4500 2850 4800
-Wire Wire Line
-	2850 4800 3200 4800
-Wire Wire Line
-	3200 4900 2850 4900
-NoConn ~ 3200 5300
-Text Notes 3450 5000 0    50   ~ 0
+	3400 4850 3050 4850
+NoConn ~ 3400 5250
+Text Notes 3650 4950 0    50   ~ 0
 DATA IN - ORANGE
-Text Notes 3450 5100 0    50   ~ 0
+Text Notes 3650 5050 0    50   ~ 0
 LOAD/CS - YELLOW
-Text Notes 3450 5200 0    50   ~ 0
+Text Notes 3650 5150 0    50   ~ 0
 CLOCK - GREEN
 Text Notes 2800 5800 0    50   ~ 0
@@
 L Connector:Conn_01x06_Female J3
 U 1 1 61726457
-P 3400 5000
-F 0 "J3" H 3050 5300 50  0000 L CNN
-F 1 "7219 OUT" H 3200 5300 50  0000 L CNN
-F 2 "PT_Library_v001:Molex_1x06_P2.54mm_Vertical" H 3400 5000 50  0001 C CNN
-F 3 "~" H 3400 5000 50  0001 C CNN
-	1    3400 5000
+P 3600 4950
+F 0 "J3" H 3250 5250 50  0000 L CNN
+F 1 "7219 OUT" H 3400 5250 50  0000 L CNN
+F 2 "PT_Library_v001:Molex_1x06_P2.54mm_Vertical" H 3600 4950 50  0001 C CNN
+F 3 "~" H 3600 4950 50  0001 C CNN
+	1    3600 4950
 	1    0    0    -1
 $EndComp
@@
 L Connector:Conn_01x02_Female J2
 U 1 1 61728B28
-P 3050 4400
-F 0 "J2" H 3078 4376 50  0000 L CNN
-F 1 "5V to Max7219" H 3078 4285 50  0000 L CNN
-F 2 "PT_Library_v001:Molex_1x02_P2.54mm_Vertical" H 3050 4400 50  0001 C CNN
-F 3 "~" H 3050 4400 50  0001 C CNN
-	1    3050 4400
+P 2900 950
+F 0 "J2" H 2928 926 50  0000 L CNN
+F 1 "LOWER 5V IN" H 2928 835 50  0000 L CNN
+F 2 "PT_Library_v001:Molex_1x02_P2.54mm_Vertical" H 2900 950 50  0001 C CNN
+F 3 "~" H 2900 950 50  0001 C CNN
+	1    2900 950
 	1    0    0    -1
 $EndComp
@@
 L Connector:Conn_01x08_Female J5
 U 1 1 6171CCFC
-P 1700 3150
-F 0 "J5" H 1728 3126 50  0000 L CNN
-F 1 "LEFT OUTPUT DIST" H 1728 3035 50  0000 L CNN
-F 2 "PT_Library_v001:Molex_1x08_P2.54mm_Vertical" H 1700 3150 50  0001 C CNN
-F 3 "~" H 1700 3150 50  0001 C CNN
-	1    1700 3150
+P 1600 3050
+F 0 "J5" H 1628 3026 50  0000 L CNN
+F 1 "LEFT OUTPUT DIST" H 1628 2935 50  0000 L CNN
+F 2 "PT_Library_v001:Molex_1x08_P2.54mm_Vertical" H 1600 3050 50  0001 C CNN
+F 3 "~" H 1600 3050 50  0001 C CNN
+	1    1600 3050
 	1    0    0    -1
 $EndComp
@@
 L power:GND #PWR0101
 U 1 1 617259A2
-P 1500 3550
-F 0 "#PWR0101" H 1500 3300 50  0001 C CNN
-F 1 "GND" H 1505 3377 50  0000 C CNN
-F 2 "" H 1500 3550 50  0001 C CNN
-F 3 "" H 1500 3550 50  0001 C CNN
-	1    1500 3550
+P 1400 3450
+F 0 "#PWR0101" H 1400 3200 50  0001 C CNN
+F 1 "GND" H 1405 3277 50  0000 C CNN
+F 2 "" H 1400 3450 50  0001 C CNN
+F 3 "" H 1400 3450 50  0001 C CNN
+	1    1400 3450
 	1    0    0    -1
 $EndComp
@@
 Text Notes 9150 5000 2    50   ~ 0
 USED BY\nETHERNET\nSHIELD
-Text Label 1500 2850 2    50   ~ 0
+Text Label 1400 2750 2    50   ~ 0
 LANDING_GEAR_SOL
-Text Label 1500 2950 2    50   ~ 0
+Text Label 1400 2850 2    50   ~ 0
 LAUNCH_BAR_MAG
-Text Label 1500 3050 2    50   ~ 0
+Text Label 1400 2950 2    50   ~ 0
 HOOK_BYPASS_MAG
-Text Label 1500 3150 2    50   ~ 0
+Text Label 1400 3050 2    50   ~ 0
 FUEL_DUMP_MAG
-Text Label 1500 3250 2    50   ~ 0
+Text Label 1400 3150 2    50   ~ 0
 APU_MAG
-Text Label 1500 3350 2    50   ~ 0
+Text Label 1400 3250 2    50   ~ 0
 ENGINE_CRANK_MAG
-NoConn ~ 1500 3450
+NoConn ~ 1400 3350
 Text Label 10350 4850 1    50   ~ 0
 LANDING_GEAR_SOL
@@
 Text Label 1450 1500 2    50   ~ 0
 SERVO_TRIM
-Text Label 1450 1600 2    50   ~ 0
-SERVO_5V
 Text Label 1450 1700 2    50   ~ 0
 SERVO_GND
-Wire Wire Line
-	4200 900  4450 900
 Text Label 4200 900  2    50   ~ 0
-SERVO_5V
+UPPER_OUTPUT_5V
 Text Label 4200 1050 2    50   ~ 0
 SERVO_GND
 Wire Wire Line
-	4200 1050 4450 1050
-Text Notes 5750 1500 2    118  Italic 24
-CORRECT SERVO POWER
+	4200 1050 4350 1050
 Text Label 6150 2750 2    50   ~ 0
 BP_STEP_COIL_A
@@
 Wire Wire Line
 	10600 1650 10150 1650
-$Comp
-L Connector:Conn_01x06_Female J4
-U 1 1 617A8F9A
-P 1650 2250
-F 0 "J4" H 1678 2226 50  0000 L CNN
-F 1 "RIGHT SERVO" H 1678 2135 50  0000 L CNN
-F 2 "PT_Library_v001:Molex_1x06_P2.54mm_Vertical" H 1650 2250 50  0001 C CNN
-F 3 "~" H 1650 2250 50  0001 C CNN
-	1    1650 2250
-	1    0    0    -1
-$EndComp
 Text Label 1450 2050 2    50   ~ 0
 SERVO_ALT_FLAG
@@
 Text Label 10600 3600 0    50   ~ 0
 D16
-Text Label 3200 5200 2    50   ~ 0
+Text Label 3400 5150 2    50   ~ 0
 D14
-Text Label 3200 5100 2    50   ~ 0
+Text Label 3400 5050 2    50   ~ 0
 D15
-Text Label 3200 5000 2    50   ~ 0
+Text Label 3400 4950 2    50   ~ 0
 D16
 Text Label 10400 2450 0    50   ~ 0
@@
 Text Label 10400 2550 0    50   ~ 0
 SERVO_HYD_PRS_2
-Text Label 1450 2550 2    50   ~ 0
+Text Label 1450 1950 2    50   ~ 0
 SERVO_GND
 $Comp
@@
 $EndComp
 $Comp
-L power:+5VL #PWR0104
-U 1 1 617CDED4
-P 4450 900
-F 0 "#PWR0104" H 4450 750 50  0001 C CNN
-F 1 "+5VL" H 4465 1073 50  0000 C CNN
-F 2 "" H 4450 900 50  0001 C CNN
-F 3 "" H 4450 900 50  0001 C CNN
-	1    4450 900
-	1    0    0    -1
-$EndComp
-$Comp
 L power:GND #PWR0105
 U 1 1 617D4C60
-P 2850 4900
-F 0 "#PWR0105" H 2850 4650 50  0001 C CNN
-F 1 "GND" H 2855 4727 50  0000 C CNN
-F 2 "" H 2850 4900 50  0001 C CNN
-F 3 "" H 2850 4900 50  0001 C CNN
-	1    2850 4900
-	1    0    0    -1
-$EndComp
-$Comp
-L power:+5V #PWR0106
-U 1 1 617D5A76
-P 2850 4400
-F 0 "#PWR0106" H 2850 4250 50  0001 C CNN
-F 1 "+5V" H 2850 4540 50  0000 C CNN
-F 2 "" H 2850 4400 50  0000 C CNN
-F 3 "" H 2850 4400 50  0000 C CNN
-	1    2850 4400
+P 3050 4850
+F 0 "#PWR0105" H 3050 4600 50  0001 C CNN
+F 1 "GND" H 3055 4677 50  0000 C CNN
+F 2 "" H 3050 4850 50  0001 C CNN
+F 3 "" H 3050 4850 50  0001 C CNN
+	1    3050 4850
 	1    0    0    -1
 $EndComp
@@
 	1    0    0    -1
 $EndComp
-$Comp
-L power:+5V #PWR0107
-U 1 1 617A5FA6
-P 2950 3350
-F 0 "#PWR0107" H 2950 3200 50  0001 C CNN
-F 1 "+5V" H 2950 3490 50  0000 C CNN
-F 2 "" H 2950 3350 50  0000 C CNN
-F 3 "" H 2950 3350 50  0000 C CNN
-	1    2950 3350
-	1    0    0    -1
-$EndComp
-$Comp
-L power:+5V #PWR0108
-U 1 1 617A6CD5
-P 4000 3350
-F 0 "#PWR0108" H 4000 3200 50  0001 C CNN
-F 1 "+5V" H 4000 3490 50  0000 C CNN
-F 2 "" H 4000 3350 50  0000 C CNN
-F 3 "" H 4000 3350 50  0000 C CNN
-	1    4000 3350
-	1    0    0    -1
-$EndComp
 Wire Wire Line
-	2300 3450 2950 3450
+	2400 3450 2950 3450
 Wire Wire Line
 	4000 3450 3650 3450
@@
 L power:GND #PWR0110
 U 1 1 617AE279
-P 2300 3450
-F 0 "#PWR0110" H 2300 3200 50  0001 C CNN
-F 1 "GND" H 2305 3277 50  0000 C CNN
-F 2 "" H 2300 3450 50  0001 C CNN
-F 3 "" H 2300 3450 50  0001 C CNN
-	1    2300 3450
+P 2400 3450
+F 0 "#PWR0110" H 2400 3200 50  0001 C CNN
+F 1 "GND" H 2405 3277 50  0000 C CNN
+F 2 "" H 2400 3450 50  0001 C CNN
+F 3 "" H 2400 3450 50  0001 C CNN
+	1    2400 3450
 	1    0    0    -1
 $EndComp
@@
 Text Label 10600 3900 0    50   ~ 0
 NEXTION_RX
+$Comp
+L Connector:Conn_01x02_Female J15
+U 1 1 6173779C
+P 4900 900
+F 0 "J15" H 4928 876 50  0000 L CNN
+F 1 "5V IN" H 4928 785 50  0000 L CNN
+F 2 "Connector_BarrelJack:BarrelJack_Horizontal" H 4900 900 50  0001 C CNN
+F 3 "~" H 4900 900 50  0001 C CNN
+	1    4900 900
+	1    0    0    -1
+$EndComp
+Wire Wire Line
+	4200 900  4700 900
+Wire Wire Line
+	4700 1000 4350 1000
+Wire Wire Line
+	4350 1000 4350 1050
+Connection ~ 4350 1050
+Wire Wire Line
+	4350 1050 4450 1050
+Text Notes 3200 6500 0    50   ~ 0
+Powering the Servos and LEDs and Nextron is done through a barrel connect to the upper board and then carried across to \nthe lower board through stand headers.  As boards are split, separate 5V buses are used in this diagram.
+$Comp
+L Connector:Conn_01x08_Female J4
+U 1 1 61749FE1
+P 1650 2150
+F 0 "J4" H 1678 2126 50  0000 L CNN
+F 1 "RIGHT_SERVO" H 1678 2035 50  0000 L CNN
+F 2 "PT_Library_v001:Molex_1x08_P2.54mm_Vertical" H 1650 2150 50  0001 C CNN
+F 3 "~" H 1650 2150 50  0001 C CNN
+	1    1650 2150
+	1    0    0    -1
+$EndComp
+NoConn ~ 1450 2550
+Text Label 1450 1600 2    50   ~ 0
+UPPER_OUTPUT_5V
+Text Label 1450 1850 2    50   ~ 0
+UPPER_OUTPUT_5V
+Text Label 2950 3350 2    50   ~ 0
+LOWER_OUTPUT_5V
+Text Label 4000 3350 2    50   ~ 0
+LOWER_OUTPUT_5V
+Text Label 3400 4750 2    50   ~ 0
+LOWER_OUTPUT_5V
+$Comp
+L power:GND #PWR01
+U 1 1 61778DBA
+P 2700 1050
+F 0 "#PWR01" H 2700 800 50  0001 C CNN
+F 1 "GND" H 2705 877 50  0000 C CNN
+F 2 "" H 2700 1050 50  0001 C CNN
+F 3 "" H 2700 1050 50  0001 C CNN
+	1    2700 1050
+	1    0    0    -1
+$EndComp
+Text Label 2700 950  2    50   ~ 0
+LOWER_OUTPUT_5V
+$Comp
+L Connector:Conn_01x02_Female J16
+U 1 1 6177A219
+P 2950 1400
+F 0 "J16" H 2978 1376 50  0000 L CNN
+F 1 "UPPER 5V OUT" H 2978 1285 50  0000 L CNN
+F 2 "PT_Library_v001:Molex_1x02_P2.54mm_Vertical" H 2950 1400 50  0001 C CNN
+F 3 "~" H 2950 1400 50  0001 C CNN
+	1    2950 1400
+	1    0    0    -1
+$EndComp
+Text Label 2750 1400 2    50   ~ 0
+UPPER_OUTPUT_5V
+$Comp
+L power:GNDD #PWR02
+U 1 1 61782A2B
+P 2750 1500
+F 0 "#PWR02" H 2750 1250 50  0001 C CNN
+F 1 "GNDD" H 2754 1345 50  0000 C CNN
+F 2 "" H 2750 1500 50  0001 C CNN
+F 3 "" H 2750 1500 50  0001 C CNN
+	1    2750 1500
+	1    0    0    -1
+$EndComp
 $EndSCHEMATC

Commit message: PCBS
Parts:
- added J15: ANALOG, PT_Library_v001:Molex_1x06_P2.54mm_Vertical, symbol Connector:Conn_01x06_Female
- R1: renamed from R12; value R -> 330
- R2: renamed from R13; value R -> 330
- renumbered J5 to J1, J15 to J11, J1 to J12, J14 to J13, J6 to J14, J7 to J16, J8 to J17, J13 to J2, J12 to J3, J2 to J5, J16 to J6, J11 to J7, J3 to J8
Connections:
- net +5VL: now also J15.1 (Pin_1)
- net A0: now also J15.3 (Pin_3)
- net A1: now also J15.4 (Pin_4)
- net A2: now also J15.5 (Pin_5)
- net A3: now also J15.6 (Pin_6)
- net GNDD: now also J15.2 (Pin_2)
- no-connect marks 17 -> 29

Commit message: ALL PCBS ORDERED
Parts:
- added J18: NEXTION ANA, PT_Library_v001:Molex_1x03_P2.54mm_Vertical, symbol Connector:Conn_01x03_Female
Connections:
- net +5VL: now also J18.1 (Pin_1)
- net A4: now also J18.2 (Pin_2)
- net GND: no longer J9.7 (Pin_7)
- net GNDD: now also J18.3 (Pin_3)
Changed lines of the file:
@@
 1
 $Comp
-L power:+3V3 #PWR018
+L power:+3V3 #PWR020
 U 1 1 56D71AA9
 P 9100 1200
-F 0 "#PWR018" H 9100 1050 50  0001 C CNN
+F 0 "#PWR020" H 9100 1050 50  0001 C CNN
 F 1 "+3.3V" V 9100 1450 50  0000 C CNN
 F 2 "" H 9100 1200 50  0000 C CNN
@@
 	8950 5050 8700 5050
 $Comp
-L power:GND #PWR016
+L power:GND #PWR018
 U 1 1 56D758F6
 P 8700 5950
-F 0 "#PWR016" H 8700 5700 50  0001 C CNN
+F 0 "#PWR018" H 8700 5700 50  0001 C CNN
 F 1 "GND" H 8700 5800 50  0000 C CNN
 F 2 "" H 8700 5950 50  0000 C CNN
@@
 	10800 5050 10650 5050
 $Comp
-L power:+5V #PWR021
+L power:+5V #PWR023
 U 1 1 56D75AB8
 P 10800 4750
-F 0 "#PWR021" H 10800 4600 50  0001 C CNN
+F 0 "#PWR023" H 10800 4600 50  0001 C CNN
 F 1 "+5V" H 10800 4890 50  0000 C CNN
 F 2 "" H 10800 4750 50  0000 C CNN
@@
 Vin
 $Comp
-L power:+5VL #PWR017
+L power:+5VL #PWR019
 U 1 1 616FD070
 P 9000 1050
-F 0 "#PWR017" H 9000 900 50  0001 C CNN
+F 0 "#PWR019" H 9000 900 50  0001 C CNN
 F 1 "+5VL" H 9015 1223 50  0000 C CNN
 F 2 "" H 9000 1050 50  0001 C CNN
@@
 $EndComp
 $Comp
-L power:GNDD #PWR019
+L power:GNDD #PWR021
 U 1 1 616FDC1F
 P 9250 2150
-F 0 "#PWR019" H 9250 1900 50  0001 C CNN
+F 0 "#PWR021" H 9250 1900 50  0001 C CNN
 F 1 "GNDD" H 9254 1995 50  0000 C CNN
 F 2 "" H 9250 2150 50  0001 C CNN
@@
 $EndComp
 $Comp
-L power:GNDD #PWR020
+L power:GNDD #PWR022
 U 1 1 616FEA6D
 P 10250 2150
-F 0 "#PWR020" H 10250 1900 50  0001 C CNN
+F 0 "#PWR022" H 10250 1900 50  0001 C CNN
 F 1 "GNDD" H 10254 1995 50  0000 C CNN
 F 2 "" H 10250 2150 50  0001 C CNN
@@
 L power:GND #PWR07
 U 1 1 6178A8D7
-P 3300 2600
-F 0 "#PWR07" H 3300 2350 50  0001 C CNN
-F 1 "GND" H 3305 2427 50  0000 C CNN
-F 2 "" H 3300 2600 50  0001 C CNN
-F 3 "" H 3300 2600 50  0001 C CNN
-	1    3300 2600
-	1    0    0    -1
-$EndComp
-Wire Wire Line
-	3500 2500 3400 2500
-Wire Wire Line
-	3300 2500 3300 2600
+P 3400 2600
+F 0 "#PWR07" H 3400 2350 50  0001 C CNN
+F 1 "GND" H 3405 2427 50  0000 C CNN
+F 2 "" H 3400 2600 50  0001 C CNN
+F 3 "" H 3400 2600 50  0001 C CNN
+	1    3400 2600
+	1    0    0    -1
+$EndComp
 Wire Wire Line
 	3500 2600 3400 2600
-Wire Wire Line
-	3400 2600 3400 2500
-Connection ~ 3400 2500
-Wire Wire Line
-	3400 2500 3300 2500
 Text Label 9650 4850 1    50   ~ 0
 LED_CHAIN_1
@@
 	1    0    0    -1
 $EndComp
-NoConn ~ 8900 2850
 NoConn ~ 8900 2950
 NoConn ~ 10400 3150
@@
 Wire Wire Line
 	6700 1100 6400 1100
+$Comp
+L Connector:Conn_01x03_Female J18
+U 1 1 61766056
+P 7750 1250
+F 0 "J18" H 7778 1276 50  0000 L CNN
+F 1 "NEXTION ANA" H 7778 1185 50  0000 L CNN
+F 2 "PT_Library_v001:Molex_1x03_P2.54mm_Vertical" H 7750 1250 50  0001 C CNN
+F 3 "~" H 7750 1250 50  0001 C CNN
+	1    7750 1250
+	1    0    0    -1
+$EndComp
+$Comp
+L power:+5VL #PWR016
+U 1 1 617677BF
+P 7550 1150
+F 0 "#PWR016" H 7550 1000 50  0001 C CNN
+F 1 "+5VL" H 7565 1323 50  0000 C CNN
+F 2 "" H 7550 1150 50  0001 C CNN
+F 3 "" H 7550 1150 50  0001 C CNN
+	1    7550 1150
+	1    0    0    -1
+$EndComp
+Text Label 7550 1250 2    50   ~ 0
+A4
+$Comp
+L power:GNDD #PWR017
+U 1 1 6176CA45
+P 7550 1350
+F 0 "#PWR017" H 7550 1100 50  0001 C CNN
+F 1 "GNDD" H 7554 1195 50  0000 C CNN
+F 2 "" H 7550 1350 50  0001 C CNN
+F 3 "" H 7550 1350 50  0001 C CNN
+	1    7550 1350
+	1    0    0    -1
+$EndComp
+NoConn ~ 3500 2500
 $EndSCHEMATC

Commit message: pcbs
Other:
- note added: "LedControl lc=LedControl(16,14,15,2);\n16 - DATA IN\n14 - CLK\n15 - LOAD/CS"
- note removed: "LEDCONTROL Ic_2=LEDCONTROL(9,8,7,1);\n9 - DATA IN\n8 - CLK\n7 - LOAD/CS"
Changed lines of the file:
@@
 CLOCK - GREEN
 Text Notes 2800 5800 0    50   ~ 0
-LEDCONTROL Ic_2=LEDCONTROL(9,8,7,1);\n9 - DATA IN\n8 - CLK\n7 - LOAD/CS
+LedControl lc=LedControl(16,14,15,2);\n16 - DATA IN\n14 - CLK\n15 - LOAD/CS
 $Comp
 L Connector_Generic:Conn_01x08 P1
