File: PCBs/OH - LEFT CONSOLE - OUTPUT DISTRIBUTION/OH - LEFT CONSOLE - OUTPUT DISTRIBUTION.kicad_pcb (KiCad board)
At the start: 2 copper layers, 85.5 x 49.8 mm, 20 parts, among them J1 Central Output, J10 APU, J11 Trim Servo Out, J12 Trim Servo Out, J2 Power In, J3 Brake Pressure In, J4 APU LED, J5 Landing Gear Sol, J6 Landing Gear Handle, J7 Select Jet, J8 Fuel Dump, J9 Brake Pressure Out, U1 ULN2003A, U2 ULN2003A

Commit message: PCBs
Parts:
- J11: value Trim Servo Out -> Trim Servo In
Connections:
- U1 pad 10: (no net) -> Net-(U1-Pad10)
- U1 pad 7: Net-(J1-Pad7) -> /GND
- U2 pad 10: (no net) -> Net-(U2-Pad10)
- U2 pad 11: (no net) -> Net-(U2-Pad11)
- U2 pad 12: (no net) -> Net-(U2-Pad12)
- U2 pad 13: (no net) -> Net-(U2-Pad13)
- U2 pad 14: (no net) -> Net-(U2-Pad14)
- U2 pad 3: (no net) -> /GND
- U2 pad 4: (no net) -> /GND
- U2 pad 5: (no net) -> /GND
- U2 pad 6: (no net) -> /GND
- U2 pad 7: (no net) -> /GND
Routing:
- net Net-(J1-Pad7): track 28.6 -> 0.00 mm
- net /GND: track 65.1 -> 69.3 mm
- net /In_Engine_Crank_Mag: track 26.1 -> 26.8 mm

Commit message: PCBS
Other:
- board text added: "5V"
- board text added: "PWM"
Changed lines of the file:
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@@
   (general
     (thickness 1.6)
-    (drawings 31)
+    (drawings 37)
     (tracks 212)
     (zones 0)
@@
     (pad 1 np_thru_hole circle (at 0 0) (size 3.2 3.2) (drill 3.2) (layers *.Cu *.Mask))
   )
+  (gr_text PWM (at 185.547 80.137) (layer F.SilkS)
+    (effects (font (size 1 1) (thickness 0.15)))
+  )
+  (gr_text 5V (at 188.849 80.137) (layer F.SilkS)
+    (effects (font (size 1 1) (thickness 0.15)))
+  )
+  (gr_text GND (at 191.897 80.137) (layer F.SilkS)
+    (effects (font (size 1 1) (thickness 0.15)))
+  )
+  (gr_text GND (at 178.943 80.137) (layer F.SilkS)
+    (effects (font (size 1 1) (thickness 0.15)))
+  )
+  (gr_text 5V (at 175.895 80.137) (layer F.SilkS)
+    (effects (font (size 1 1) (thickness 0.15)))
+  )
+  (gr_text PWM (at 172.593 80.137) (layer F.SilkS)
+    (effects (font (size 1 1) (thickness 0.15)))
+  )
   (gr_text "Hook Ovrde" (at 179.578 60.833 90) (layer F.SilkS)

Commit message: PCBs
Parts:
- removed J6: Landing Gear Handle, PT_Library_v001:Molex_1x02_P2.54mm_Vertical
- removed R1, R2: 560, PT_Library_v001:R_Axial_DIN0207_L6.3mm_D2.5mm_P7.62mm_Horizontal
- removed U2: ULN2003A, Package_DIP:DIP-16_W7.62mm
- added D1: APU LED, PT_Library_v001:Molex_1x02_P2.54mm_Vertical, F.Cu at (187.1, 62.9)
- added D2: LANDING GEAR LED, PT_Library_v001:Molex_1x02_P2.54mm_Vertical, F.Cu at (198.5, 62.9)
- J4: value APU LED -> LED IN; footprint PT_Library_v001:Molex_1x02_P2.54mm_Vertical -> PT_Library_v001:Molex_1x04_P2.54mm_Vertical
- moved J5 16.6 mm to (157.6, 47.4)
- moved J10 15.6 mm to (170.1, 64.5)
- moved J7 15.6 mm to (156.5, 64.5)
- moved J4 14.3 mm to (193.5, 51.4)
- moved U1 13.9 mm to (138.0, 45.8)
- moved J9 11.4 mm to (185.3, 40.4)
- moved J3 7.55 mm to (169.5, 40.4)
Connections:
- net Net-(J11-Pad1) renamed /SERVO_PWM
- net Net-(J11-Pad2) renamed /SERVO_5V
- net Net-(J11-Pad3) renamed /SERVO_GND
- J1 pad 7: Net-(J1-Pad7) -> (no net)
- J1 pad 8: /In_Landing_Gear_LED -> (no net)
- J1 pad 9: /In_APU_Led -> (no net)
- J4 pad 1: Net-(J4-Pad1) -> /LEDCOL1
- J4 pad 2: /Out_APU_LED -> (no net)
- U1 pad 10: Net-(U1-Pad10) -> (no net)
Routing:
- net /Out_APU_LED: track 64.8 -> 0.00 mm
- net /Out_Landing_Gear_LED: track 54.1 -> 0.00 mm
- net /+12V: track 130.5 -> 88.9 mm
- net /In_APU_Led: track 27.0 -> 0.00 mm
- net /In_Landing_Gear_LED: track 23.4 -> 0.00 mm
- net /LEDCOL1: track 0.00 -> 23.2 mm
- net /GND: track 69.3 -> 52.0 mm
- net /LEDROW1: track 0.00 -> 16.9 mm
- net /LEDROW2: track 0.00 -> 12.5 mm
- net /In_Landing_Gear_Sol: track 18.2 -> 8.34 mm
- net Net-(J4-Pad1): track 9.51 -> 0.00 mm
- net /In_Launch_Bar_Mag: track 21.1 -> 12.1 mm
- net /Out_Fuel_Dump_Mag: track 20.9 -> 29.3 mm
- net Net-(J3-Pad3): track 24.4 -> 17.6 mm
- net Net-(J3-Pad2): track 24.6 -> 17.9 mm
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Other:
- board text removed: "+"
- board text removed: "-"

Commit message: PCBs
Parts:
- removed D1: APU LED, PT_Library_v001:Molex_1x02_P2.54mm_Vertical
- removed D2: LANDING GEAR LED, PT_Library_v001:Molex_1x02_P2.54mm_Vertical
- removed the J4 at (193.5, 51.4)
- added J2: LED IN, PT_Library_v001:Molex_1x03_P2.54mm_Vertical, F.Cu at (184.2, 52.3)
- added J5: APU LED, PT_Library_v001:Molex_1x02_P2.54mm_Vertical, F.Cu at (195.8, 52.2)
- added J6: LANDING GEAR LED, PT_Library_v001:Molex_1x02_P2.54mm_Vertical, F.Cu at (196.0, 63.0)
- renumbered J9 to J10, J10 to J11, J11 to J12, J12 to J13, J2 to J3, J3 to J4, J5 to J7, J7 to J8, J8 to J9
Routing:
- net /LEDROW1: track 16.9 -> 12.8 mm
- net /Out_Fuel_Dump_Mag: track 29.3 -> 33.2 mm
- net /Out_Launch_Bar_Mag: track 24.1 -> 27.8 mm
- net /Out_APU_Mag: track 34.5 -> 31.0 mm
- net /LEDROW2: track 12.5 -> 15.2 mm
- net /LEDCOL1: track 23.2 -> 21.0 mm
- net /+12V: track 88.9 -> 87.5 mm
- net /Out_Engine_Crank_Mag: track 34.8 -> 36.0 mm
- net /GND: track 52.0 -> 51.1 mm
- net /In_Engine_Crank_Mag: track 26.9 -> 26.3 mm
Other:
- board text added: "v002"
- board text removed: "v001"

Commit message: PCBS
Parts:
- J1: value Central Output -> CENTRAL OUTPUT; footprint PT_Library_v001:Molex_1x10_P2.54mm_Vertical -> PT_Library_v001:Molex_1x08_P2.54mm_Vertical
Connections:
- J1 pad 8: (no net) -> /GND
Routing:
- net /Out_Hook_Bypass_Mag: track 24.4 -> 32.8 mm
- net /GND: track 51.1 -> 46.6 mm
- net /+12V: track 87.5 -> 83.2 mm
- net /Out_APU_Mag: track 31.0 -> 34.6 mm
- net /Out_Launch_Bar_Mag: track 27.8 -> 26.4 mm
- net /Out_Engine_Crank_Mag: track 36.0 -> 34.8 mm
Other:
- board text removed: "SPR"

Commit message: PCBS
Parts:
- added J14: 5V APU, PT_Library_v001:Molex_1x04_P2.54mm_Vertical, F.Cu at (169.4, 46.1)
- added J3: 5V Landing Gear Sol, PT_Library_v001:Molex_1x02_P2.54mm_Vertical, F.Cu at (169.7, 58.0)
- added J5: 5V Fuel Dump, PT_Library_v001:Molex_1x02_P2.54mm_Vertical, F.Cu at (169.7, 64.8)
- added J6: 5V Select Jet, PT_Library_v001:Molex_1x04_P2.54mm_Vertical, F.Cu at (169.5, 34.3)
- added U2: 5V ULN2003A, Package_DIP:DIP-16_W7.62mm, F.Cu at (154.9, 50.5)
- J10: renamed from J8; value Select Jet -> 12V Select Jet
- J11: renamed from J9; value Fuel Dump -> 12V Fuel Dump
- J12: renamed from J10; value Brake Pressure Out -> Brake Pressure
- J13: renamed from J11; value APU -> 12V APU
- J15: renamed from J12; value Trim Servo In -> Trim Servo
- J17: renamed from J13; value Trim Servo Out -> Trim Servo
- J2: renamed from J3; value Power In -> 12V Power In; footprint PT_Library_v001:Molex_1x02_P2.54mm_Vertical -> Connector_BarrelJack:BarrelJack_Horizontal
- J7: renamed from J4; value Brake Pressure In -> Brake Pressure
- J9: renamed from J7; value Landing Gear Sol -> 12V Landing Gear Sol
- U1: value ULN2003A -> 12V ULN2003A
- moved J11 41.1 mm to (150.2, 34.8), turned to 270 degrees
- moved J1 38.6 mm to (134.7, 76.1)
- moved J13 31.2 mm to (139.1, 60.7), turned to 270 degrees
- moved J10 23.3 mm to (138.9, 49.1), turned to 270 degrees
- moved J2 18.2 mm to (141.0, 41.5), turned to 270 degrees
- moved J7 16.7 mm to (185.3, 34.8)
- moved J16 16.1 mm to (199.8, 48.3)
- moved J17 15.5 mm to (186.1, 65.8)
- moved U1 13.7 mm to (124.3, 46.7)
- moved J9 9.50 mm to (150.1, 41.5), turned to 270 degrees
- moved J4 7.62 mm to (201.9, 56.8)
- moved J8 6.37 mm to (201.8, 65.5)
- moved J12 2.04 mm to (185.4, 42.4)
- renumbered J2 to J16, J5 to J4, J6 to J8
Connections:
- net /Out_APU_Mag renamed /12V_APU_Mag
- net /Out_Engine_Crank_Mag renamed /12V_Engine_Crank_Mag
- net /Out_Fuel_Dump_Mag renamed /12V_Fuel_Dump_Mag
- net /Out_Hook_Bypass_Mag renamed /12V_Hook_Bypass_Mag
- net /Out_Landing_Gear_Sol renamed /12V_Landing_Gear_Sol
- net /Out_Launch_Bar_Mag renamed /12V_Launch_Bar_Mag
- J15 pad 3: /SERVO_GND -> /GND
- J17 pad 3: /SERVO_GND -> /GND
Routing:
- net /GND: track 46.6 -> 124.9 mm
- net /In_Landing_Gear_Sol: track 8.36 -> 67.2 mm
- net /SERVO_5V: track 14.8 -> 71.8 mm
- net /In_Launch_Bar_Mag: track 12.2 -> 63.8 mm
- net /In_Hook_Bypass_Mag: track 15.5 -> 59.0 mm
- net /In_Fuel_Dump_Mag: track 19.8 -> 55.4 mm
- net /In_APU_Mag: track 23.4 -> 51.8 mm
- net /12V_APU_Mag: track 34.6 -> 10.0 mm
- net /12V_Engine_Crank_Mag: track 34.8 -> 12.1 mm
- net /In_Engine_Crank_Mag: track 26.3 -> 48.2 mm
- net /12V_Hook_Bypass_Mag: track 32.8 -> 12.6 mm
- net /5V_Launch_Bar_Mag: track 0.00 -> 19.4 mm
- net /12V_Launch_Bar_Mag: track 26.4 -> 7.98 mm
- net /5V_Hook_Bypass_Mag: track 0.00 -> 16.9 mm
- net /5V_APU_Mag: track 0.00 -> 15.2 mm
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Other:
- net class GND AND POWER added: clearance 0.2, trace_width 0.45, via_dia 0.8, via_drill 0.4
- board text added: "12V"

Commit message: pcbs and front test
Connections:
- J3 pad 1: /+12V -> /SERVO_5V
Routing:
- net /+12V: track 85.6 -> 58.0 mm
- net /In_Launch_Bar_Mag: track 63.8 -> 66.0 mm
- net /SERVO_5V: track 71.8 -> 73.3 mm
- net /In_Landing_Gear_Sol: track 67.2 -> 66.2 mm
Other:
- board text added: "5V supplied via Servo"
- board text added: "v003"
- board text removed: "v002"
