File: PCBs/Pi GPS Serial/Pi GPS Serial.sch (KiCad schematic (older format))
At the start: 10 parts, among them J1 RS232 OUT, J2 5V In, J3 40HAT, U1 MAX232

Commit message: GPS
Other:
- note added: "Add I2C connector with same pinout as Arduino\nAdd general data connector for OLED\nAdd connector for stick shaker"
Changed lines of the file:
@@
 Wire Wire Line
 	11150 7400 11800 7400
+Text Notes 6950 3600 0    50   ~ 0
+Add I2C connector with same pinout as Arduino\nAdd general data connector for OLED\nAdd connector for stick shaker
 $EndSCHEMATC
