File: PCBs/Pi GPS Serial/Pi GPS Serial.kicad_sch (KiCad schematic)
At the start: 13 parts, among them J1 RS232 OUT, J2 5V In, J3 40HAT, J4 SPI, J5 I2C, J6 Stick Shaker, U1 MAX232

Commit message: Doc
Other:
- moved on the sheet: C1, C2, H1, H2, H3, H4, J1, J2, J3, J4, J5, J6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

Commit message: large update
Parts:
- added C3, C4: 0.1uF, Capacitor_THT:C_Disc_D4.3mm_W1.9mm_P5.00mm, symbol Device:C
Connections:
- net GND: now also C3.2, C4.2
- net at U1.2 (VS+): now also C4.1
- net at U1.6 (VS-): now also C3.1
- no-connect marks 27 -> 25
Changed lines of the file:
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@@
     (rev "A")
   )
-  (no_connect (at 167.005 48.895))
-  (no_connect (at 167.005 41.275))
   (no_connect (at 126.365 69.215))
   (no_connect (at 126.365 59.055))
@@
     (stroke (width 0) (type default) (color 0 0 0 0))
   )
+  (wire (pts (xy 188.595 33.655) (xy 183.515 33.655))
+    (stroke (width 0) (type default) (color 0 0 0 0))
+  )
+  (wire (pts (xy 167.005 48.895) (xy 170.18 48.895))
+    (stroke (width 0) (type default) (color 0 0 0 0))
+  )
   (wire (pts (xy 48.895 41.91) (xy 18.415 41.91))
     (stroke (width 0) (type default) (color 0 0 0 0))
@@
     (stroke (width 0) (type default) (color 0 0 0 0))
   )
+  (wire (pts (xy 167.005 38.1) (xy 167.005 41.275))
+    (stroke (width 0) (type default) (color 0 0 0 0))
+  )
   (wire (pts (xy 48.895 62.23) (xy 18.415 62.23))
     (stroke (width 0) (type default) (color 0 0 0 0))
@@
     (stroke (width 0) (type default) (color 0 0 0 0))
   )
+  (wire (pts (xy 183.515 33.655) (xy 183.515 38.1))
+    (stroke (width 0) (type default) (color 0 0 0 0))
+  )
+  (wire (pts (xy 170.18 43.18) (xy 179.07 43.18))
+    (stroke (width 0) (type default) (color 0 0 0 0))
+  )
   (wire (pts (xy 126.365 28.575) (xy 116.205 28.575))
     (stroke (width 0) (type default) (color 0 0 0 0))
   )
+  (wire (pts (xy 170.18 48.895) (xy 170.18 43.18))
+    (stroke (width 0) (type default) (color 0 0 0 0))
+  )
   (wire (pts (xy 167.005 53.975) (xy 183.515 53.975))
     (stroke (width 0) (type default) (color 0 0 0 0))
   )
   (wire (pts (xy 48.895 31.75) (xy 18.415 31.75))
+    (stroke (width 0) (type default) (color 0 0 0 0))
+  )
+  (wire (pts (xy 183.515 38.1) (xy 167.005 38.1))
     (stroke (width 0) (type default) (color 0 0 0 0))
   )
@@
     (pin "3")
   )
+  (symbol (lib_id "power:GND") (at 188.595 41.275 0) (unit 1)
+    (in_bom yes) (on_board yes)
+    (property "Reference" "#PWR05" (id 0) (at 188.595 47.625 0)
+      (effects (font (size 1.27 1.27)) hide)
+    )
+    (property "Value" "GND" (id 1) (at 188.722 45.6692 0))
+    (property "Footprint" "" (id 2) (at 188.595 41.275 0)
+      (effects (font (size 1.27 1.27)) hide)
+    )
+    (property "Datasheet" "" (id 3) (at 188.595 41.275 0)
+      (effects (font (size 1.27 1.27)) hide)
+    )
+    (pin "1")
+  )
+  (symbol (lib_id "Device:C") (at 188.595 37.465 0) (unit 1)
+    (in_bom yes) (on_board yes)
+    (property "Reference" "C4" (id 0) (at 191.516 36.2966 0)
+      (effects (font (size 1.27 1.27)) (justify left))
+    )
+    (property "Value" "0.1uF" (id 1) (at 191.516 38.608 0)
+      (effects (font (size 1.27 1.27)) (justify left))
+    )
+    (property "Footprint" "Capacitor_THT:C_Disc_D4.3mm_W1.9mm_P5.00mm" (id 2) (at 189.5602 41.275 0)
+      (effects (font (size 1.27 1.27)) hide)
+    )
+    (property "Datasheet" "~" (id 3) (at 188.595 37.465 0)
+      (effects (font (size 1.27 1.27)) hide)
+    )
+    (pin "1")
+    (pin "2")
+  )
   (symbol (lib_id "Connector:Conn_01x04_Female") (at 120.015 91.44 0) (unit 1)
     (in_bom yes) (on_board yes) (fields_autoplaced)
@@
     (pin "6")
   )
+  (symbol (lib_id "power:GND") (at 179.07 50.8 0) (unit 1)
+    (in_bom yes) (on_board yes)
+    (property "Reference" "#PWR04" (id 0) (at 179.07 57.15 0)
+      (effects (font (size 1.27 1.27)) hide)
+    )
+    (property "Value" "GND" (id 1) (at 179.197 55.1942 0))
+    (property "Footprint" "" (id 2) (at 179.07 50.8 0)
+      (effects (font (size 1.27 1.27)) hide)
+    )
+    (property "Datasheet" "" (id 3) (at 179.07 50.8 0)
+      (effects (font (size 1.27 1.27)) hide)
+    )
+    (pin "1")
+  )
+  (symbol (lib_id "Device:C") (at 179.07 46.99 0) (unit 1)
+    (in_bom yes) (on_board yes)
+    (property "Reference" "C3" (id 0) (at 181.991 45.8216 0)
+      (effects (font (size 1.27 1.27)) (justify left))
+    )
+    (property "Value" "0.1uF" (id 1) (at 181.991 48.133 0)
+      (effects (font (size 1.27 1.27)) (justify left))
+    )
+    (property "Footprint" "Capacitor_THT:C_Disc_D4.3mm_W1.9mm_P5.00mm" (id 2) (at 180.0352 50.8 0)
+      (effects (font (size 1.27 1.27)) hide)
+    )
+    (property "Datasheet" "~" (id 3) (at 179.07 46.99 0)
+      (effects (font (size 1.27 1.27)) hide)
+    )
+    (pin "1")
+    (pin "2")
+  )
   (sheet_instances
     (path "/" (page "1"))
@@
       (reference "#PWR03") (unit 1) (value "GND") (footprint "")
     )
+    (path "/7d293cae-cbe1-4a5e-a7fa-41cce3d33b53"
+      (reference "#PWR04") (unit 1) (value "GND") (footprint "")
+    )
+    (path "/143ad586-7f36-4cf9-bd03-3cc28fcfe7e9"
+      (reference "#PWR05") (unit 1) (value "GND") (footprint "")
+    )
     (path "/00000000-0000-0000-0000-00006284bd5e"
       (reference "C1") (unit 1) (value "0.1uF") (footprint "Capacitor_THT:C_Disc_D4.3mm_W1.9mm_P5.00mm")
@@
       (reference "C2") (unit 1) (value "0.1uF") (footprint "Capacitor_THT:C_Disc_D4.3mm_W1.9mm_P5.00mm")
     )
+    (path "/80a9a6ef-e99b-43f0-8470-b41370404370"
+      (reference "C3") (unit 1) (value "0.1uF") (footprint "Capacitor_THT:C_Disc_D4.3mm_W1.9mm_P5.00mm")
+    )
+    (path "/25c0cbb9-13ac-407b-a364-b917d0e78dc7"
+      (reference "C4") (unit 1) (value "0.1uF") (footprint "Capacitor_THT:C_Disc_D4.3mm_W1.9mm_P5.00mm")
+    )
     (path "/00000000-0000-0000-0000-00005834bc4a"
