File: PCBs/OH - Hornet Forward Upper Output Shield/Hornet Forward Output Upper Shield.sch (KiCad schematic (older format))
At the start: 48 parts, among them J1 LOWER 12V IN, J10 FLOOD, J11 5V IN, J12 RIGHT FORM, J13 PORT SIDE, J14 LEFT FORM, J15 RELAY OUT, J18 NEXTION ANA, J19 STARBOARD SIDE, J2 UPPER 12V IN, J3 MAP, J4 LOWER 12V OUT, J5 LOWER 5V IN, J6 UPPER 5V OUT, J7 NEXTION, J8 7219 OUT, J9 BACKLIGHT, P1 Power, P2 Analog, P3 Analog, P4 Digital, P5 PWM, P6 PWM, P7 Communication, Q1 IRF1405PBF, Q2 IRF1405PBF, Q3 IRF1405PBF, Q4 IRF1405PBF, Q5 IRF1405PBF, Q6 IRF1405PBF

Commit message: Upper Output PCB and Compass start
Parts:
- added J16: Compass, PT_Library_v001:Molex_1x08_P2.54mm_Vertical, symbol Connector:Conn_01x08_Female
Connections:
- net GNDD: now also J16.7 (Pin_7)
- net UPPER_OUTPUT_5V: now also J16.6 (Pin_6)
- net D11 renamed Compass_Stepper_B
- net Compass_Stepper_B: now also J16.2 (Pin_2)
- net D12 renamed Compass_Stepper_A
- net Compass_Stepper_A: now also J16.1 (Pin_1)
- net D2 renamed Compass_Stepper_D
- net Compass_Stepper_D: now also J16.4 (Pin_4)
- net D3 renamed Compass_Stepper_C
- net Compass_Stepper_C: now also J16.3 (Pin_3)
- net D9 renamed Compass_Zero_Sensor
- net Compass_Zero_Sensor: now also J16.5 (Pin_5)
- no-connect marks 59 -> 55
Changed lines of the file:
@@
 	5400 3950 5250 3950
 NoConn ~ 8250 5400
-NoConn ~ 10600 1950
-NoConn ~ 10600 1650
-NoConn ~ 10600 1750
 NoConn ~ 8900 2450
 NoConn ~ 8900 2550
@@
 	1    0    0    -1
 $EndComp
-NoConn ~ 10400 2850
-NoConn ~ 10400 2950
 $Comp
 L power:GND #PWR0108
@@
 RELAY_4
 NoConn ~ 6050 6950
+$Comp
+L Connector:Conn_01x08_Female J16
+U 1 1 62BA5FC7
+P 6450 2700
+F 0 "J16" H 6478 2676 50  0000 L CNN
+F 1 "Compass" H 6478 2585 50  0000 L CNN
+F 2 "PT_Library_v001:Molex_1x08_P2.54mm_Vertical" H 6450 2700 50  0001 C CNN
+F 3 "~" H 6450 2700 50  0001 C CNN
+	1    6450 2700
+	1    0    0    -1
+$EndComp
+Text Label 6250 2400 2    50   ~ 0
+Compass_Stepper_A
+Text Label 6250 2500 2    50   ~ 0
+Compass_Stepper_B
+Text Label 6250 2600 2    50   ~ 0
+Compass_Stepper_C
+Text Label 6250 2700 2    50   ~ 0
+Compass_Stepper_D
+NoConn ~ 6250 3100
+Text Label 6250 2800 2    50   ~ 0
+Compass_Zero_Sensor
+Text Label 6250 2900 2    50   ~ 0
+UPPER_OUTPUT_5V
+$Comp
+L power:GNDD #PWR07
+U 1 1 62BB8EAE
+P 5950 3000
+F 0 "#PWR07" H 5950 2750 50  0001 C CNN
+F 1 "GNDD" H 5954 2845 50  0000 C CNN
+F 2 "" H 5950 3000 50  0001 C CNN
+F 3 "" H 5950 3000 50  0001 C CNN
+	1    5950 3000
+	1    0    0    -1
+$EndComp
+Wire Wire Line
+	6250 3000 5950 3000
+Text Label 10600 1650 0    50   ~ 0
+Compass_Stepper_A
+Text Label 10600 1750 0    50   ~ 0
+Compass_Stepper_B
+Text Label 10400 2850 0    50   ~ 0
+Compass_Stepper_C
+Text Label 10400 2950 0    50   ~ 0
+Compass_Stepper_D
+Text Label 10600 1950 0    50   ~ 0
+Compass_Zero_Sensor
 $EndSCHEMATC
