File: PCBs/OH - Power_Distro_PCB_V2/Power Distro PCB V2.kicad_pcb (KiCad board)
At the start: 2 copper layers, 95 x 95 mm, 34 parts, among them J1 Conn_01x04_Female, J10 Conn_01x04_Female, J11 Conn_01x04_Female, J12 Conn_01x02_Female, J13 Conn_01x02_Female, J14 Conn_01x02_Female, J15 Conn_01x02_Female, J16 Conn_01x02_Female, J17 Conn_01x02_Female, J18 Conn_01x02_Female, J19 Conn_01x02_Female, J2 Conn_01x04_Female, J20 Conn_01x02_Female, J22 Conn_01x02_Female, J23 Conn_01x02_Female, J24 Conn_01x02_Female, J25 Conn_01x02_Female, J26 Conn_01x08_Female, J27 Conn_01x24_Female, J28 Conn_01x02_Female, J29 Conn_01x02_Female, J3 Conn_01x04_Female, J30 Conn_01x02_Female, J31 Conn_01x02_Female, J32 Conn_01x02_Female, J35 Conn_01x04_Female, J4 Conn_01x04_Female, J5 Conn_01x04_Female, J6 Conn_01x04_Female, J7 Conn_01x08_Female, J8 Conn_01x04_Female, J9 Conn_01x04_Female

Commit message: s
Routing:
- net /LEDGND: track 416.9 -> 0.00 mm
- net /LED5V1: track 269.1 -> 0.00 mm
- net /12VSOCKETS+: track 105.5 -> 0.00 mm
- net /LEDDATA7: track 43.9 -> 0.00 mm
- net /FAN+: track 34.3 -> 0.00 mm
- net /LEDDATA1: track 31.4 -> 0.00 mm
- net /PWRGOOD: track 29.0 -> 0.00 mm
- net /LEDDATA6: track 27.6 -> 0.00 mm
- net /LEDDATA2: track 19.5 -> 0.00 mm
- net /PSUSW: track 18.1 -> 0.00 mm
- net /LEDDATA5: track 17.7 -> 0.00 mm
- net /FAN1Control: track 15.8 -> 0.00 mm
- net /FAN1Tach: track 15.8 -> 0.00 mm
- net /LEDDATA3: track 14.7 -> 0.00 mm
- net /FAN4Control: track 13.8 -> 0.00 mm
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Other:
- net class LED POWER: trace_width 4 -> 3
- net class LED POWER -: trace_width 2.5 -> 3

Commit message: Power
Routing:
- net /LEDGND: track 0.00 -> 417.6 mm
- net /LED5V1: track 0.00 -> 255.7 mm
- net /12VSOCKETS+: track 0.00 -> 114.0 mm
- net /LEDDATA7: track 0.00 -> 44.0 mm
- net /FAN+: track 0.00 -> 34.3 mm
- net /LEDDATA1: track 0.00 -> 31.5 mm
- net /LEDDATA6: track 0.00 -> 28.8 mm
- net /PWRGOOD: track 0.00 -> 23.2 mm
- net /LEDDATA2: track 0.00 -> 19.6 mm
- net /PSUSW: track 0.00 -> 18.2 mm
- net /LEDDATA5: track 0.00 -> 17.7 mm
- net /FAN1Control: track 0.00 -> 15.8 mm
- net /FAN1Tach: track 0.00 -> 15.8 mm
- net /LEDDATA3: track 0.00 -> 14.7 mm
- net /FAN4Control: track 0.00 -> 13.8 mm
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Other:
- net class 5V SOCKETS: trace_width 3 -> 2
- net class LED POWER: trace_width 3 -> 2
- net class LED POWER -: trace_width 3 -> 2

Commit message: power
Parts:
- removed J26: Conn_01x08_Female, Connector_PinHeader_2.54mm:PinHeader_2x04_P2.54mm_Vertical
- J10, J11, J8, J9: value Conn_01x04_Female -> Conn_01x02_Female; footprint Connector:FanPinHeader_1x04_P2.54mm_Vertical -> Connector_Molex:Molex_KK-254_AE-6410-02A_1x02_P2.54mm_Vertical
- moved J8 35.1 mm to (60.8, 90.0), turned to 180 degrees
- moved J11 33.0 mm to (27.1, 92.1)
- moved J10 26.5 mm to (27.1, 85.8)
- moved J9 21.0 mm to (54.3, 90.0), turned to 180 degrees
- moved J12 0.96 mm to (67.4, 90.0)
- moved J13 0.62 mm to (73.9, 90.0)
- moved J14 0.29 mm to (80.4, 90.0)
Connections:
- J10 pad 1: /LEDGND -> /12VSOCKETS+
- J10 pad 2: /FAN+ -> /LEDGND
- J11 pad 1: /LEDGND -> /12VSOCKETS+
- J11 pad 2: /FAN+ -> /LEDGND
- J27 pad 1: (no net) -> Net-(J27-Pad1)
- J27 pad 12: (no net) -> Net-(J27-Pad12)
- J27 pad 13: (no net) -> Net-(J27-Pad13)
- J27 pad 14: (no net) -> Net-(J27-Pad14)
- J27 pad 2: (no net) -> Net-(J27-Pad2)
- J27 pad 20: (no net) -> Net-(J27-Pad20)
- J27 pad 9: (no net) -> Net-(J27-Pad9)
- J8 pad 1: /LEDGND -> /LED5V1
- J8 pad 2: /FAN+ -> /LEDGND
- J9 pad 1: /LEDGND -> /LED5V1
- J9 pad 2: /FAN+ -> /LEDGND
Routing:
- net /FAN+: track 34.3 -> 0.00 mm
- net /LED5V1: track 255.7 -> 275.9 mm
- net /12VSOCKETS+: track 114.0 -> 131.4 mm
- net /FAN1Control: track 15.8 -> 0.00 mm
- net /FAN1Tach: track 15.8 -> 0.00 mm
- net /FAN4Control: track 13.8 -> 0.00 mm
- net /FAN4Tach: track 13.8 -> 0.00 mm
- net /FAN2Tach: track 10.5 -> 0.00 mm
- net /FAN2Control: track 10.3 -> 0.00 mm
- net /FAN3Tach: track 8.83 -> 0.00 mm
- net /FAN3Control: track 8.54 -> 0.00 mm
- net /LEDGND: track 417.6 -> 425.4 mm
Other:
- board text removed: "FAN 1"
- board text removed: "FAN 2"
- board text removed: "FAN 3"
- board text removed: "FAN 4"
- board text removed: "NOTE: ALL FAN PORTS SUPPLY 12V"
- board text removed: "PWM CONTROL"
- board text removed: "TACHOMETER"
