File: PCBs/SARI_LEDS/SARI_LEDS.kicad_sch (KiCad schematic)
At the start: 4 parts, among them J1 BL OUT, J2 BL OUT

Commit message: PCBS
Parts:
- added H1, H2: MountingHole, MountingHole:MountingHole_3.5mm, symbol Mechanical:MountingHole
Changed lines of the file:
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@@
     (pin "4")
+  )
+  (symbol (lib_id "Mechanical:MountingHole") (at 134.62 112.395 0) (unit 1)
+    (in_bom yes) (on_board yes) (fields_autoplaced)
+    (property "Reference" "H1" (id 0) (at 137.16 111.5603 0)
+      (effects (font (size 1.27 1.27)) (justify left))
+    )
+    (property "Value" "MountingHole" (id 1) (at 137.16 114.0972 0)
+      (effects (font (size 1.27 1.27)) (justify left))
+    )
+    (property "Footprint" "MountingHole:MountingHole_3.5mm" (id 2) (at 134.62 112.395 0)
+      (effects (font (size 1.27 1.27)) hide)
+    )
+    (property "Datasheet" "~" (id 3) (at 134.62 112.395 0)
+      (effects (font (size 1.27 1.27)) hide)
+    )
+  )
+  (symbol (lib_id "Mechanical:MountingHole") (at 134.62 118.745 0) (unit 1)
+    (in_bom yes) (on_board yes) (fields_autoplaced)
+    (property "Reference" "H2" (id 0) (at 137.16 117.9103 0)
+      (effects (font (size 1.27 1.27)) (justify left))
+    )
+    (property "Value" "MountingHole" (id 1) (at 137.16 120.4472 0)
+      (effects (font (size 1.27 1.27)) (justify left))
+    )
+    (property "Footprint" "MountingHole:MountingHole_3.5mm" (id 2) (at 134.62 118.745 0)
+      (effects (font (size 1.27 1.27)) hide)
+    )
+    (property "Datasheet" "~" (id 3) (at 134.62 118.745 0)
+      (effects (font (size 1.27 1.27)) hide)
+    )
   )
   (sheet_instances
@@
       (reference "D2") (unit 1) (value "NeoPixel_THT") (footprint "LED_THT:LED_D5.0mm-4_RGB")
     )
+    (path "/db255932-1161-4ee7-91ce-ce1b0fe44fc0"
+      (reference "H1") (unit 1) (value "MountingHole") (footprint "MountingHole:MountingHole_3.5mm")
+    )
+    (path "/ddaf4972-cfbf-47bc-aae1-eb85987956c3"
+      (reference "H2") (unit 1) (value "MountingHole") (footprint "MountingHole:MountingHole_3.5mm")
+    )
     (path "/add7b91f-b3b9-45f6-ac45-8de434c8eab3"
