File: PCBs/F16 Input Shield with Ethernet/F16 Input Shield with Ethernet.kicad_pcb (KiCad board)
At the start: 2 copper layers, 121.8 x 53.3 mm, 48 parts, among them J1 5V to Max7219, J10 DIGITAL B, J11 ANALOG A, J2 7219 OUT, J3 Address Select 0, J4 Address Select 1, J5 ANALOG B, J6 ENCODERS, J7 MATRIX INPUT, J8 DIGITAL A, J9 DIGITAL C, P1 PWM, P2 PWM, P3 Communication, P4 Digital, P5 Power, P6 Analog, P7 Analog, U1 USR-ES1

Commit message: PCBS
Parts:
- added J7: Reset, Connector_PinHeader_2.54mm:PinHeader_1x02_P2.54mm_Vertical, F.Cu at (118.1, 116.8)
- added R1: 10K, PT_Library_v001:PT_R_Axial_DIN0204_L3.6mm_D1.6mm_P2.54mm_Vertical, F.Cu at (110.5, 115.6)
- C1: renamed from C5; value 0.1uF -> 0.1
- C10: value 0.1uF -> 0.1
- C11: renamed from C13; value 0.1uF -> 0.1
- C12: renamed from C8; value 0.1uF -> 0.1
- C13: renamed from C11; value 0.1uF -> 0.1
- C14: renamed from C12; value 0.1uF -> 0.1
- C2: renamed from C4; value 0.1uF -> 0.1
- C3: renamed from C1; value 0.1uF -> 0.1
- C4: renamed from C3; value 0.1uF -> 0.1
- C5: renamed from C2; value 0.1uF -> 0.1
- C6: renamed from C14; value 0.1uF -> 0.1
- C7: renamed from C6; value 0.1uF -> 0.1
- C8: renamed from C9; value 0.1uF -> 0.1
- C9: renamed from C7; value 0.1uF -> 0.1
- J8: renamed from J3; value Address Select 0 -> Addr Sel 0; footprint PT_Library_v001:Molex_1x02_P2.54mm_Vertical -> Connector_PinHeader_2.54mm:PinHeader_1x02_P2.54mm_Vertical
- J9: renamed from J4; value Address Select 1 -> Addr Sel 1; footprint PT_Library_v001:Molex_1x02_P2.54mm_Vertical -> Connector_PinHeader_2.54mm:PinHeader_1x02_P2.54mm_Vertical
- P1: footprint Connector_PinHeader_2.54mm:PinHeader_1x08_P2.54mm_Vertical -> Socket_Arduino_Mega:Socket_Strip_Arduino_1x08
- moved R2 82.6 mm to (138.4, 101.6), turned to 90 degrees
- moved R13 78.8 mm to (141.0, 101.6), turned to 90 degrees
- moved R12 75.2 mm to (143.5, 101.6), turned to 90 degrees
- moved R11 71.7 mm to (146.1, 101.6), turned to 90 degrees
- moved R10 68.4 mm to (148.6, 101.6), turned to 90 degrees
- moved R9 65.3 mm to (151.1, 101.6), turned to 90 degrees
- moved R8 62.4 mm to (153.7, 101.6), turned to 90 degrees
- moved J10 62.1 mm to (147.3, 91.4), turned to 90 degrees
- moved R7 59.8 mm to (156.2, 101.6), turned to 90 degrees
- moved R6 57.4 mm to (158.8, 101.6), turned to 90 degrees
- moved R5 55.4 mm to (161.3, 101.6), turned to 90 degrees
- moved R14 53.7 mm to (163.8, 101.6), turned to 90 degrees
- moved J1 41.8 mm to (105.4, 73.7)
- moved J6 37.2 mm to (130.8, 107.3), turned to 0 degrees
- moved J2 26.0 mm to (105.4, 83.2)
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- renumbered J9 to J1, J7 to J10, J6 to J11, J5 to J12, J8 to J2, J1 to J3, J2 to J4, J10 to J5, J11 to J6, P5 to P2, P2 to P3, P6 to P4, P3 to P5, P7 to P6, P4 to P7, R11 to R10, R4 to R11, R5 to R12, R6 to R13, R9 to R14, R3 to R2, R2 to R3, R1 to R4, R13 to R5, R12 to R6, R8 to R7, R10 to R8, R7 to R9
Connections:
- C10 pad 2: GND -> GNDD
- C11 pad 2: GND -> GNDD
- C12 pad 2: GND -> GNDD
- C14 pad 2: GND -> GNDD
- C6 pad 2: GND -> GNDD
- C7 pad 2: GND -> GNDD
- C8 pad 2: GND -> GNDD
- C9 pad 2: GND -> GNDD
- J1 pad 1: +5VL -> +5V
- J10 pad 1: (no net) -> unconnected-(J1-Pad1)
- J10 pad 29: (no net) -> unconnected-(J1-Pad29)
- J10 pad 30: (no net) -> unconnected-(J1-Pad30)
- J10 pad 31: (no net) -> unconnected-(J1-Pad31)
- J10 pad 32: (no net) -> unconnected-(J1-Pad32)
- J10 pad 33: (no net) -> unconnected-(J1-Pad33)
- J10 pad 34: (no net) -> unconnected-(J1-Pad34)
- J11 pad 1: GND -> GNDD
- J11 pad 10: (no net) -> unconnected-(J5-Pad10)
- J12 pad 2: GND -> GNDD
- J2 pad 1: +5VL -> +5V
- J3 pad 1: +5VL -> +5V
- J4 pad 6: (no net) -> unconnected-(J3-Pad6)
- J5 pad 1: +5VL -> +5V
- J6 pad 1: +5VL -> +5V
- P1 pad 1: (no net) -> unconnected-(P5-Pad1)
- P1 pad 6: (no net) -> /SS
- P2 pad 1: (no net) -> unconnected-(P1-Pad1)
- P2 pad 2: (no net) -> /IOREF
- P2 pad 3: (no net) -> /Reset
- P2 pad 4: (no net) -> +3V3
- P2 pad 5: +5VL -> +5V
- P2 pad 8: (no net) -> /Vin
- P3 pad 4: (no net) -> unconnected-(P6-Pad4)
- P7 pad 1: GND -> GNDD
- P7 pad 2: GND -> GNDD
- P7 pad 3: (no net) -> /52
- P7 pad 4: (no net) -> /53
- P7 pad 5: (no net) -> /50
- P7 pad 6: (no net) -> /51
- P7 pad 8: (no net) -> /49
Routing:
- net GNDD: track 0.00 -> 271.3 mm
- net +5V: track 0.00 -> 195.7 mm
- net /50: track 0.00 -> 100.1 mm
- net /51: track 0.00 -> 91.2 mm
- net /49: track 0.00 -> 89.0 mm
- net /52: track 0.00 -> 83.5 mm
- net /39: track 0.00 -> 74.0 mm, vias 0 -> 1
- net /38: track 0.00 -> 67.9 mm
- net /41: track 0.00 -> 65.8 mm, vias 0 -> 1
- net /D0: track 0.00 -> 65.4 mm
- net /40: track 0.00 -> 65.0 mm
- net /42: track 0.00 -> 63.1 mm
- net /D9: track 0.00 -> 62.7 mm
- net /23: track 0.00 -> 59.9 mm
- net /D1: track 0.00 -> 59.5 mm
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Other:
- board size 121.8 x 53.3 mm -> 104.1 x 53.3 mm
- board text added: "RESET"

Commit message: PCBS
Parts:
- renumbered C13 to C1, C11 to C10, C4 to C11, C8 to C12, C12 to C13, C9 to C14, C14 to C2, C5 to C3, C7 to C4, C3 to C5, C1 to C7, C10 to C8, C2 to C9, D2 to D1, D1 to D2, J10 to J1, J2 to J10, J5 to J11, J1 to J12, J3 to J2, J4 to J3, J12 to J4, J11 to J5, P2 to P1, P4 to P2, P6 to P3, P7 to P4, P1 to P5, P3 to P6, P5 to P7, R6 to R10, R5 to R11, R14 to R12, R4 to R13, R3 to R14, R13 to R3, R12 to R4, R11 to R5, R10 to R6, R9 to R7, R7 to R9
Connections:
- U1 pad B5: /49 -> /53
Routing:
- net /53: track 0.00 -> 91.9 mm
- net /49: track 89.0 -> 0.00 mm
- net /41: track 65.8 -> 93.1 mm
- net /50: track 100.1 -> 85.3 mm
- net GNDD: track 271.3 -> 261.3 mm, vias 0 -> 1
- net /48: track 47.9 -> 57.0 mm
- net /35: track 42.2 -> 49.6 mm, vias 0 -> 1
- net /39: track 74.0 -> 68.6 mm, vias 1 -> 0
- net /40: track 65.0 -> 68.3 mm
- net /33: track 44.4 -> 41.6 mm
- net +5V: track 195.7 -> 193.5 mm
- net /51: track 91.2 -> 93.4 mm
- net /43: track 56.9 -> 55.4 mm
- net /45: track 51.4 -> 52.9 mm
- net /42: track 63.1 -> 64.6 mm
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Other:
- board size 104.1 x 53.3 mm -> 99.8 x 53.3 mm

Commit message: PCB
Connections:
- P1 pad 4: +3V3 -> +3.3V
Routing:
- net /39: track 68.6 -> 104.0 mm
- net /41: track 93.1 -> 61.2 mm, vias 1 -> 0
- net +3.3V: track 28.2 -> 57.9 mm
- net GNDD: track 261.3 -> 273.5 mm, vias 1 -> 0
- net /35: track 49.6 -> 40.1 mm, vias 1 -> 0
- net /48: track 57.0 -> 48.4 mm
- net +5V: track 193.5 -> 188.4 mm
- net /40: track 68.3 -> 65.4 mm
- net /29: track 50.6 -> 47.7 mm
- net /42: track 64.6 -> 61.8 mm
- net /45: track 52.9 -> 53.8 mm
- net /53: track 91.9 -> 91.1 mm
- net /D0: track 65.4 -> 64.7 mm
- net /34: track 37.4 -> 36.7 mm
- net /27: track 52.3 -> 51.7 mm
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