File: A10/A10 PCBs/GAUGE_Analog Instruments/GAUGE_Analog Instruments.kicad_sch (KiCad schematic)
At the start: 11 parts, among them J1 Conn_01x02_Female, J2 STEPPER, J3 Conn_01x03_Female, J4 ZERO, M1 VID29-02

Commit message: A10 AND HORNET
Parts:
- removed J1: Conn_01x02_Female, Connector_Molex:Molex_KK-254_AE-6410-02A_1x02_P2.54mm_Vertical, symbol Connector:Conn_01x02_Female
- removed J3: Conn_01x03_Female, Connector_Molex:Molex_KK-254_AE-6410-03A_1x03_P2.54mm_Vertical, symbol Connector:Conn_01x03_Female
- added J4: ZERO_AND_BACKLIGHT, Connector_Molex:Molex_PicoBlade_53047-0510_1x05_P1.25mm_Vertical, symbol Connector:Conn_01x05_Female
- J1: renamed from J2; footprint Connector_PinHeader_2.54mm:PinHeader_2x02_P2.54mm_Vertical -> Connector_Molex:Molex_PicoBlade_53047-0410_1x04_P1.25mm_Vertical
- renumbered J4 to J3
Connections:
- net 5V: now also J4.1 (Pin_1)
- net GND: now also J4.2 (Pin_2)
- net ZERO_DETECT: now also J4.3 (Pin_3)
- net BACKLIGHT_+12V: now reaches R1.1
- net BACKLIGHT_+12V: now also J4.4 (Pin_4)
- net BACKLIGHT_GND: now reaches D2.1 (K)
- net BACKLIGHT_GND: now also J4.5 (Pin_5)
Other:
- moved on the sheet: R1
Changed lines of the file:
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@@
     (rev "2")
-  )
-  (junction (at 105.664 77.47) (diameter 0) (color 0 0 0 0)
   )
   (wire (pts (xy 182.88 31.75) (xy 182.88 29.21))
     (stroke (width 0) (type default) (color 0 0 0 0))
   )
-  (wire (pts (xy 127.762 71.12) (xy 127.762 77.47))
-    (stroke (width 0) (type default) (color 0 0 0 0))
-  )
-  (wire (pts (xy 105.664 77.47) (xy 105.41 77.47))
-    (stroke (width 0) (type default) (color 0 0 0 0))
-  )
-  (wire (pts (xy 127.762 66.802) (xy 105.41 66.802))
-    (stroke (width 0) (type default) (color 0 0 0 0))
-  )
-  (wire (pts (xy 127.762 68.58) (xy 127.762 66.802))
-    (stroke (width 0) (type default) (color 0 0 0 0))
-  )
-  (wire (pts (xy 105.41 77.47) (xy 105.41 74.422))
-    (stroke (width 0) (type default) (color 0 0 0 0))
-  )
   (wire (pts (xy 180.34 31.75) (xy 182.88 31.75))
     (stroke (width 0) (type default) (color 0 0 0 0))
   )
-  (wire (pts (xy 145.796 26.67) (xy 148.082 26.67))
-    (stroke (width 0) (type default) (color 0 0 0 0))
-  )
-  (wire (pts (xy 105.918 77.47) (xy 105.664 77.47))
-    (stroke (width 0) (type default) (color 0 0 0 0))
-  )
   (wire (pts (xy 182.88 36.83) (xy 180.34 36.83))
     (stroke (width 0) (type default) (color 0 0 0 0))
   )
-  (wire (pts (xy 127.762 77.47) (xy 120.904 77.47))
-    (stroke (width 0) (type default) (color 0 0 0 0))
-  )
   (text "1) XXXX" (at 12.7 20.32 0)
     (effects (font (size 1.27 1.27)) (justify left bottom))
@@
     (effects (font (size 2.54 2.54)) (justify left bottom))
   )
-  (label "GND" (at 148.082 29.21 180)
+  (label "BACKLIGHT_GND" (at 209.804 41.402 180)
+    (effects (font (size 1.27 1.27)) (justify right bottom))
+  )
+  (label "GND" (at 209.804 33.782 180)
     (effects (font (size 1.27 1.27)) (justify right bottom))
   )
@@
     (effects (font (size 1.27 1.27)) (justify left bottom))
   )
+  (label "BACKLIGHT_+12V" (at 98.044 77.47 180)
+    (effects (font (size 1.27 1.27)) (justify right bottom))
+  )
   (label "COIL2" (at 144.78 43.18 180)
     (effects (font (size 1.27 1.27)) (justify right bottom))
   )
-  (label "5V" (at 145.796 26.67 0)
-    (effects (font (size 1.27 1.27)) (justify left bottom))
+  (label "5V" (at 209.804 31.242 180)
+    (effects (font (size 1.27 1.27)) (justify right bottom))
   )
   (label "5V" (at 182.88 29.21 0)
     (effects (font (size 1.27 1.27)) (justify left bottom))
   )
+  (label "BACKLIGHT_+12V" (at 209.804 38.862 180)
+    (effects (font (size 1.27 1.27)) (justify right bottom))
+  )
   (label "COIL3" (at 144.78 57.15 180)
     (effects (font (size 1.27 1.27)) (justify right bottom))
   )
-  (label "ZERO_DETECT" (at 148.082 31.75 180)
+  (label "ZERO_DETECT" (at 209.804 36.322 180)
     (effects (font (size 1.27 1.27)) (justify right bottom))
   )
@@
     (effects (font (size 1.27 1.27)) (justify right bottom))
   )
+  (label "BACKLIGHT_GND" (at 120.904 77.47 0)
+    (effects (font (size 1.27 1.27)) (justify left bottom))
+  )
   (label "COIL4" (at 157.48 40.64 0)
     (effects (font (size 1.27 1.27)) (justify left bottom))
@@
   (symbol (lib_id "power:GND") (at 176.53 68.58 270) (unit 1)
     (in_bom yes) (on_board yes)
-    (property "Reference" "#PWR04" (id 0) (at 170.18 68.58 0)
+    (property "Reference" "#PWR02" (id 0) (at 170.18 68.58 0)
       (effects (font (size 1.27 1.27)) hide)
     )
@@
   (symbol (lib_id "Connector:Conn_01x03_Male") (at 175.26 34.29 0) (unit 1)
     (in_bom yes) (on_board yes)
-    (property "Reference" "J4" (id 0) (at 172.72 33.02 0))
+    (property "Reference" "J3" (id 0) (at 172.72 33.02 0))
     (property "Value" "ZERO" (id 1) (at 171.45 35.56 0))
     (property "Footprint" "Connector_PinHeader_2.54mm:PinHeader_1x03_P2.54mm_Vertical" (id 2) (at 175.26 34.29 0)
@@
   (symbol (lib_id "power:+5V") (at 176.53 66.04 90) (unit 1)
     (in_bom yes) (on_board yes)
-    (property "Reference" "#PWR03" (id 0) (at 180.34 66.04 0)
+    (property "Reference" "#PWR01" (id 0) (at 180.34 66.04 0)
       (effects (font (size 1.27 1.27)) hide)
     )
@@
   (symbol (lib_id "Connector_Generic:Conn_02x02_Odd_Even") (at 149.86 40.64 0) (unit 1)
     (in_bom yes) (on_board yes)
-    (property "Reference" "J2" (id 0) (at 151.13 35.56 0))
+    (property "Reference" "J1" (id 0) (at 151.13 35.56 0))
     (property "Value" "STEPPER" (id 1) (at 151.13 38.1 0))
-    (property "Footprint" "Connector_PinHeader_2.54mm:PinHeader_2x02_P2.54mm_Vertical" (id 2) (at 149.86 40.64 0)
+    (property "Footprint" "Connector_Molex:Molex_PicoBlade_53047-0410_1x04_P1.25mm_Vertical" (id 2) (at 149.86 40.64 0)
       (effects (font (size 1.27 1.27)) hide)
     )
@@
     (pin "4")
   )
-  (symbol (lib_id "Connector:Conn_01x03_Female") (at 153.162 29.21 0) (unit 1)
+  (symbol (lib_id "Connector:Conn_01x05_Female") (at 214.884 36.322 0) (unit 1)
     (in_bom yes) (on_board yes) (fields_autoplaced)
-    (property "Reference" "J3" (id 0) (at 153.8732 28.3753 0)
-      (effects (font (size 1.27 1.27)) (justify left))
-    )
-    (property "Value" "Conn_01x03_Female" (id 1) (at 153.8732 30.9122 0)
-      (effects (font (size 1.27 1.27)) (justify left))
-    )
-    (property "Footprint" "Connector_Molex:Molex_KK-254_AE-6410-03A_1x03_P2.54mm_Vertical" (id 2) (at 153.162 29.21 0)
-      (effects (font (size 1.27 1.27)) hide)
-    )
-    (property "Datasheet" "~" (id 3) (at 153.162 29.21 0)
+    (property "Reference" "J4" (id 0) (at 215.5952 35.4873 0)
+      (effects (font (size 1.27 1.27)) (justify left))
+    )
+    (property "Value" "ZERO_AND_BACKLIGHT" (id 1) (at 215.5952 38.0242 0)
+      (effects (font (size 1.27 1.27)) (justify left))
+    )
+    (property "Footprint" "Connector_Molex:Molex_PicoBlade_53047-0510_1x05_P1.25mm_Vertical" (id 2) (at 214.884 36.322 0)
+      (effects (font (size 1.27 1.27)) hide)
+    )
+    (property "Datasheet" "~" (id 3) (at 214.884 36.322 0)
       (effects (font (size 1.27 1.27)) hide)
     )
@@
     (pin "2")
     (pin "3")
-  )
-  (symbol (lib_id "Device:R") (at 105.41 70.612 0) (unit 1)
+    (pin "4")
+    (pin "5")
+  )
+  (symbol (lib_id "Device:R") (at 101.854 77.47 90) (unit 1)
     (in_bom yes) (on_board yes) (fields_autoplaced)
-    (property "Reference" "R1" (id 0) (at 107.188 69.7773 0)
-      (effects (font (size 1.27 1.27)) (justify left))
-    )
-    (property "Value" "R" (id 1) (at 107.188 72.3142 0)
-      (effects (font (size 1.27 1.27)) (justify left))
-    )
-    (property "Footprint" "Resistor_THT:R_Axial_DIN0204_L3.6mm_D1.6mm_P1.90mm_Vertical" (id 2) (at 103.632 70.612 90)
-      (effects (font (size 1.27 1.27)) hide)
-    )
-    (property "Datasheet" "~" (id 3) (at 105.41 70.612 0)
+    (property "Reference" "R1" (id 0) (at 101.854 72.7542 90))
+    (property "Value" "R" (id 1) (at 101.854 75.2911 90))
+    (property "Footprint" "Resistor_THT:R_Axial_DIN0204_L3.6mm_D1.6mm_P1.90mm_Vertical" (id 2) (at 101.854 79.248 90)
+      (effects (font (size 1.27 1.27)) hide)
+    )
+    (property "Datasheet" "~" (id 3) (at 101.854 77.47 0)
       (effects (font (size 1.27 1.27)) hide)
     )
@@
     (pin "2")
   )
-  (symbol (lib_id "Connector:Conn_01x02_Female") (at 132.842 68.58 0) (unit 1)
-    (in_bom yes) (on_board yes) (fields_autoplaced)
-    (property "Reference" "J1" (id 0) (at 133.5532 69.0153 0)
-      (effects (font (size 1.27 1.27)) (justify left))
-    )
-    (property "Value" "Conn_01x02_Female" (id 1) (at 133.5532 71.5522 0)
-      (effects (font (size 1.27 1.27)) (justify left))
-    )
-    (property "Footprint" "Connector_Molex:Molex_KK-254_AE-6410-02A_1x02_P2.54mm_Vertical" (id 2) (at 132.842 68.58 0)
-      (effects (font (size 1.27 1.27)) hide)
-    )
-    (property "Datasheet" "~" (id 3) (at 132.842 68.58 0)
-      (effects (font (size 1.27 1.27)) hide)
-    )
-    (pin "1")
-    (pin "2")
-  )
   (sheet_instances
     (path "/" (page "1"))
@@
     )
     (path "/00000000-0000-0000-0000-00006137e4cf"
-      (reference "#PWR03") (unit 1) (value "+5V") (footprint "")
+      (reference "#PWR01") (unit 1) (value "+5V") (footprint "")
     )
     (path "/00000000-0000-0000-0000-00006134005a"
-      (reference "#PWR04") (unit 1) (value "GND") (footprint "")
+      (reference "#PWR02") (unit 1) (value "GND") (footprint "")
     )
     (path "/a56238bb-cf17-4e99-bcb1-68f472cf0a01"
@@
       (reference "H3") (unit 1) (value "MountingHole") (footprint "MountingHole:MountingHole_2.5mm")
     )
-    (path "/c0356fd2-ac1a-40ac-a9a6-3aeb1bcb0000"
-      (reference "J1") (unit 1) (value "Conn_01x02_Female") (footprint "Connector_Molex:Molex_KK-254_AE-6410-02A_1x02_P2.54mm_Vertical")
-    )
     (path "/00000000-0000-0000-0000-000062ec0411"
-      (reference "J2") (unit 1) (value "STEPPER") (footprint "Connector_PinHeader_2.54mm:PinHeader_2x02_P2.54mm_Vertical")
-    )
-    (path "/28fb6b2d-1ab2-4bbf-91f8-12b95c433815"
-      (reference "J3") (unit 1) (value "Conn_01x03_Female") (footprint "Connector_Molex:Molex_KK-254_AE-6410-03A_1x03_P2.54mm_Vertical")
+      (reference "J1") (unit 1) (value "STEPPER") (footprint "Connector_Molex:Molex_PicoBlade_53047-0410_1x04_P1.25mm_Vertical")
     )
     (path "/00000000-0000-0000-0000-00006137a947"
-      (reference "J4") (unit 1) (value "ZERO") (footprint "Connector_PinHeader_2.54mm:PinHeader_1x03_P2.54mm_Vertical")
+      (reference "J3") (unit 1) (value "ZERO") (footprint "Connector_PinHeader_2.54mm:PinHeader_1x03_P2.54mm_Vertical")
+    )
+    (path "/1feeb685-c8e4-41ec-8cc2-7c73ca665321"
+      (reference "J4") (unit 1) (value "ZERO_AND_BACKLIGHT") (footprint "Connector_Molex:Molex_PicoBlade_53047-0510_1x05_P1.25mm_Vertical")
     )
     (path "/00000000-0000-0000-0000-000061379ede"

Commit message: A10
Parts:
- renumbered J3 to J2, J4 to J3
Changed lines of the file:
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@@
   (symbol (lib_id "Connector:Conn_01x03_Male") (at 175.26 34.29 0) (unit 1)
     (in_bom yes) (on_board yes)
-    (property "Reference" "J3" (id 0) (at 172.72 33.02 0))
+    (property "Reference" "J2" (id 0) (at 172.72 33.02 0))
     (property "Value" "ZERO" (id 1) (at 171.45 35.56 0))
     (property "Footprint" "Connector_PinHeader_2.54mm:PinHeader_1x03_P2.54mm_Vertical" (id 2) (at 175.26 34.29 0)
@@
   (symbol (lib_id "Connector:Conn_01x05_Female") (at 214.884 36.322 0) (unit 1)
     (in_bom yes) (on_board yes) (fields_autoplaced)
-    (property "Reference" "J4" (id 0) (at 215.5952 35.4873 0)
+    (property "Reference" "J3" (id 0) (at 215.5952 35.4873 0)
       (effects (font (size 1.27 1.27)) (justify left))
     )
@@
     )
     (path "/00000000-0000-0000-0000-00006137a947"
-      (reference "J3") (unit 1) (value "ZERO") (footprint "Connector_PinHeader_2.54mm:PinHeader_1x03_P2.54mm_Vertical")
+      (reference "J2") (unit 1) (value "ZERO") (footprint "Connector_PinHeader_2.54mm:PinHeader_1x03_P2.54mm_Vertical")
     )
     (path "/1feeb685-c8e4-41ec-8cc2-7c73ca665321"
-      (reference "J4") (unit 1) (value "ZERO_AND_BACKLIGHT") (footprint "Connector_Molex:Molex_PicoBlade_53047-0510_1x05_P1.25mm_Vertical")
+      (reference "J3") (unit 1) (value "ZERO_AND_BACKLIGHT") (footprint "Connector_Molex:Molex_PicoBlade_53047-0510_1x05_P1.25mm_Vertical")
     )
     (path "/00000000-0000-0000-0000-000061379ede"
