File: A10/A10 PCBs/Caution Panel/Caution Panel.kicad_sch (KiCad schematic)
At the start: 100 parts, among them J1 CAUTION_UPPER_SEG, J2 CAUTION_UPPER_DIGIT, J3 CAUTION_LOWER_SEG, J4 CAUTION_LOW_DIGITS

Commit message: A10
Other:
- note added: "Note - SEG_DP is Col 0 - not 8"
Changed lines of the file:
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@@
     (effects (font (size 1.27 1.27)) (justify right bottom))
+  )
+  (text "Note - SEG_DP is Col 0 - not 8" (at 149.606 151.638 0)
+    (effects (font (size 1.27 1.27)) (justify left bottom))
   )
   (text "AIL DISENG" (at 47.752 53.086 180)
