File: A10/A10 PCBs/Right Console Overview/ELECT POWER.kicad_sch (KiCad schematic)
At the start: 13 parts

Commit message: Right Console
Parts:
- J?: value Conn_01x06_Female -> ELEC POWER
Changed lines of the file:
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@@
       (effects (font (size 1.27 1.27)) (justify left))
     )
-    (property "Value" "Conn_01x06_Female" (id 1) (at 215.8492 68.7582 0)
+    (property "Value" "ELEC POWER" (id 1) (at 215.8492 68.7582 0)
       (effects (font (size 1.27 1.27)) (justify left))
     )

Commit message: A10
Other:
- note added: "A_10C:defineToggleSwitch("EPP_APU_GEN_PWR", 1, 3001, 241, "Electrical Power Panel", "APU GEN PWR") A_10C:defineSpringloaded_3PosTumb("EPP_INVERTER", 1, 3055, 3002, 242, "Electrical Power Panel", "Inverter TEST - OFF - STBY") A_10C:defineToggleSwitch("EPP_AC_GEN_PWR_L", 1, 3004, 244, "Electrical Power Panel", "AC GEN PWR Left") A_10C:defineToggleSwitch("EPP_AC_GEN_PWR_R", 1, 3005, 245, "Electrical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"
Changed lines of the file:
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@@
     (stroke (width 0) (type default) (color 0 0 0 0))
+  )
+  (text "A_10C:defineToggleSwitch(\"EPP_APU_GEN_PWR\", 1, 3001, 241, \"Electrical Power Panel\", \"APU GEN PWR\")\nA_10C:defineSpringloaded_3PosTumb(\"EPP_INVERTER\", 1, 3055, 3002, 242, \"Electrical Power Panel\", \"Inverter TEST - OFF - STBY\")\nA_10C:defineToggleSwitch(\"EPP_AC_GEN_PWR_L\", 1, 3004, 244, \"Electrical Power Panel\", \"AC GEN PWR Left\")\nA_10C:defineToggleSwitch(\"EPP_AC_GEN_PWR_R\", 1, 3005, 245, \"Electrical Power Panel\", \"AC GEN PWR Right\")\nA_10C:defineToggleSwitch(\"EPP_BATTERY_PWR\", 1, 3006, 246, \"Electrical Power Panel\", \"Battery Power\")\nA_10C:defineToggleSwitch(\"EPP_EMER_FLOOD\", 49, 3007, 243, \"Electrical Power Panel\", \"Emergency Flood Light\")\n"
+    (at 31.242 164.338 0)
+    (effects (font (size 1.27 1.27)) (justify left bottom))
   )
   (label "ROW6" (at 183.134 50.8 0)

Commit message: A10
Parts:
- gave numbers to parts that had none: 13
Connections:
- net COL2 renamed COL8
- net COL3 renamed COL9
- net ROW5 renamed ROW0
- net ROW6 renamed ROW1
- net ROW7 renamed ROW2
- net ROW8 renamed ROW3
Other:
- moved on the sheet: D25, D28, D30, SW23, SW26, SW28
