File: A10/A10 PCBs/Right Console Overview/ENVIRONMENT.kicad_sch (KiCad schematic)
At the start: 9 parts

Commit message: A10
Parts:
- removed J?: SWITCH_INPUT, symbol Connector:Conn_01x06_Female
- removed RV?: ENG INST, symbol Device:R_Potentiometer_US
- removed RV?: FORMATION, symbol Device:R_Potentiometer_US
- added D? (x5): D, PT_Library_v001:D_Signal_P7.62mm_Horizontal, symbol Device:D
- added D?: LED, Connector_Molex:Molex_KK-254_AE-6410-02A_1x02_P2.54mm_Vertical, symbol Device:LED
- added J?: Conn_01x08_Female, symbol Connector:Conn_01x08_Female
- added J?: Conn_01x02_Female, symbol Connector:Conn_01x02_Female
- added R?: 500, symbol Device:R_US
- added SW?: BLEED AIR, symbol Switch:SW_SPST
- added SW?: NORM / RAM, symbol Switch:SW_SPST
- added SW?: MAIN AIR, symbol Switch:SW_SPST
- added SW?: NVG, symbol Switch:SW_SPST
- added SW?: POTIT HEAT, symbol Switch:SW_SPST
- SW?: value POSITION -> EMEGY NORM TEST
- SW?: value NOSE ILLUM -> 100% OXY
Connections:
- net ROW12 is gone; now on net ROW0: SW?.1
- net ROW0: now also SW?.2 (B), J?.3 (Pin_3); no longer SW?.2
- net COL0 renamed COL2
- net COL2: now also D?.2 (A), D?.2 (A), J?.1 (Pin_1)
- net COL1 renamed COL3
- net COL3: now also D?.2 (A), D?.2 (A), D?.2 (A), J?.2 (Pin_2)
- net ROW13 renamed ROW1
- net ROW1: now also J?.4 (Pin_4), SW?.2 (B); no longer SW?.2 (B)
- new net: D?.1 (K), SW?.1 (A) (x5)
- new net: J?.2 (Pin_2), R?.1
- new net: D?.2 (A), R?.2
- new net: D?.1 (K), J?.1 (Pin_1)
- new net ROW2: J?.5 (Pin_5), SW?.2, SW?.2 (B)
- new net ROW3: J?.6 (Pin_6), SW?.2 (B), SW?.2 (B)
- new net ROW4: J?.7 (Pin_7), SW?.2 (B)
- no-connect marks 0 -> 1
Other:
- moved on the sheet: D?, SW?

Commit message: Right Console
Parts:
- J?: value Conn_01x08_Female -> ENVIRONMENT
Changed lines of the file:
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@@
       (effects (font (size 1.27 1.27)) (justify left))
     )
-    (property "Value" "Conn_01x08_Female" (id 1) (at 207.2132 98.4762 0)
+    (property "Value" "ENVIRONMENT" (id 1) (at 207.2132 98.4762 0)
       (effects (font (size 1.27 1.27)) (justify left))
     )

Commit message: A10
Other:
- note added: "A_10C:defineFloat("OXY_VOLUME", 274, { 0, 1 }, "Environment Control Panel", "Oxygen Volume (0 to 5 liters)") A_10C:defineFloat("CABIN_PRESS_ALT", 281, { 0, 1 }, "Environment Control Panel", "Cabin Pressure Altitude") A_10C:definePushButton("ENVCP_OXY_TEST", 41, 3001, 275, "Environment Control Panel", "Oxygen Indicator Test") A_10C:defineToggleSwitch("ENVCP_WINDSHIELD_DEFOG", 41, 3002, 276, "Envir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"
- note added: "A_10C:defineSpringloaded_3PosTumb("OXY_EMERGENCY", 40, 3004, 3003, 601, "Oxygen Regulator Panel", "Oxygen Flow: Emergency / Normal / Test") A_10C:defineToggleSwitch("OXY_DILUTER", 40, 3002, 602, "Oxygen Regulator Panel", "Oxygen Normal/100%") A_10C:defineToggleSwitch("OXY_SUPPLY", 40, 3001, 603, "Oxygen Regulator Panel", "Oxygen Supply On/Off") A_10C:defineFloat("OXY_PRESS", 604, { 0, 1 }, "Oxyge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"
Changed lines of the file:
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@@
     (stroke (width 0) (type default) (color 0 0 0 0))
+  )
+  (text "A_10C:defineFloat(\"OXY_VOLUME\", 274, { 0, 1 }, \"Environment Control Panel\", \"Oxygen Volume (0 to 5 liters)\")\nA_10C:defineFloat(\"CABIN_PRESS_ALT\", 281, { 0, 1 }, \"Environment Control Panel\", \"Cabin Pressure Altitude\")\nA_10C:definePushButton(\"ENVCP_OXY_TEST\", 41, 3001, 275, \"Environment Control Panel\", \"Oxygen Indicator Test\")\nA_10C:defineToggleSwitch(\"ENVCP_WINDSHIELD_DEFOG\", 41, 3002, 276, \"Environment Control Panel\", \"Windshield Defog/Deice\")\nA_10C:definePotentiometer(\"ENVCP_CANOPY_DEFOG\", 41, 3003, 277, { 0, 1 }, \"Environment Control Panel\", \"Canopy Defog\")\nA_10C:define3PosTumb(\"ENVCP_WRRW\", 41, 3004, 278, \"Environment Control Panel\", \"Windshield Rain Removal/Wash\")\nA_10C:defineToggleSwitch(\"ENVCP_PITOT_HEAT\", 41, 3005, 279, \"Environment Control Panel\", \"Pitot Heat\")\nA_10C:defineToggleSwitch(\"ENVCP_BLEED_AIR\", 41, 3006, 280, \"Environment Control Panel\", \"Bleed Air\")\nA_10C:define3PosTumb(\"ENVCP_TEMP_PRESS\", 41, 3007, 282, \"Environment Control Panel\", \"Temperature/Pressure Control\")\nA_10C:reserveIntValue(7)\nA_10C:defineToggleSwitch(\"ENVCP_AIR_SUPPLY\", 41, 3008, 283, \"Environment Control Panel\", \"Main Air Supply\")\nA_10C:definePotentiometer(\"ENVCP_FLOW_LEVEL\", 41, 3009, 284, { 0, 1 }, \"Environment Control Panel\", \"Flow Level\")\nA_10C:definePotentiometer(\"ENVCP_TEMP_LEVEL\", 41, 3013, 286, { 0, 1 }, \"Environment Control Panel\", \"Temp Level Control\")\nA_10C:defineTumb(\"ENVCP_AC_OPER\", 41, 3010, 285, 0.1, { 0, 0.3 }, nil, false, \"Environment Control Panel\", \"Air Conditioner MAN/AUTO/COLD/HOT\")"
+    (at 20.828 185.674 0)
+    (effects (font (size 1.27 1.27)) (justify left bottom))
+  )
+  (text "A_10C:defineSpringloaded_3PosTumb(\"OXY_EMERGENCY\", 40, 3004, 3003, 601, \"Oxygen Regulator Panel\", \"Oxygen Flow: Emergency / Normal / Test\")\nA_10C:defineToggleSwitch(\"OXY_DILUTER\", 40, 3002, 602, \"Oxygen Regulator Panel\", \"Oxygen Normal/100%\")\nA_10C:defineToggleSwitch(\"OXY_SUPPLY\", 40, 3001, 603, \"Oxygen Regulator Panel\", \"Oxygen Supply On/Off\")\nA_10C:defineFloat(\"OXY_PRESS\", 604, { 0, 1 }, \"Oxygen Regulator Panel\", \"Oxygen Pressure Indicator\")\nA_10C:defineIndicatorLight(\"OXY_FLOW\", 600, \"Oxygen Regulator Panel\", \"Flow Indicator (on/off) (white)\")"
+    (at 21.336 148.844 0)
+    (effects (font (size 1.27 1.27)) (justify left bottom))
   )
   (label "ROW0" (at 138.938 68.072 0)

Commit message: A10
Parts:
- gave numbers to parts that had none: 20
