File: A10/A10 PCBs/Right Console Overview/WARNING DISPLAY.kicad_sch (KiCad schematic)
At the start: 96 parts

Commit message: A10
Other:
- note added: "-- Caution Lights A_10C:defineIndicatorLight("CL_A1", 480, "Caution Lights Panel", "ENG START CYCLE Light (green)") A_10C:defineIndicatorLight("CL_A2", 481, "Caution Lights Panel", "L-HYD PRESS Light (green)") A_10C:defineIndicatorLight("CL_A3", 482, "Caution Lights Panel", "R-HYD PRESS Light (green)") A_10C:defineIndicatorLight("CL_A4", 483, "Caution Lights Panel", "GUN UNSAFE Light (green)") A_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"
- moved on the sheet: D?

Commit message: A10
Parts:
- gave numbers to parts that had none: 96
