File: A10/A10 PCBs/Left Console Overview/AUDIO_KEYPAD.kicad_sch (KiCad schematic)
At the start: 0 parts

Commit message: A10
Parts:
- added D? (x7): D, Diode_THT:D_A-405_P7.62mm_Horizontal, symbol Device:D
- added J?: AUDIO_KEYPAD, symbol Connector:Conn_01x08_Female
- added SW? (x12): LOAD, Connector_Molex:Molex_KK-254_AE-6410-02A_1x02_P2.54mm_Vertical, symbol Switch:SW_Push
- added SW?: ARM, Connector_Molex:Molex_KK-254_AE-6410-02A_1x02_P2.54mm_Vertical, symbol Switch:SW_Push
- added SW?: VHF, Connector_Molex:Molex_KK-254_AE-6410-02A_1x02_P2.54mm_Vertical, symbol Switch:SW_Push
- added SW?: INTERCOMM, Connector_Molex:Molex_KK-254_AE-6410-02A_1x02_P2.54mm_Vertical, symbol Switch:SW_Push
- added SW?: ESC, Connector_Molex:Molex_KK-254_AE-6410-02A_1x02_P2.54mm_Vertical, symbol Switch:SW_Push
Connections:
- new net: D?.1 (K), SW?.1, SW?.1, SW?.1, SW?.1 (x3)
- new net: D?.1 (K), SW?.1 (x4)
- new net COL0: J?.1 (Pin_1)
- new net COL1: J?.2 (Pin_2)
- new net COL2: J?.3 (Pin_3)
- new net COL3: J?.4 (Pin_4)
- new net ROW0: J?.5 (Pin_5)
- new net ROW1: J?.6 (Pin_6), SW?.2, SW?.2, SW?.2, SW?.2
- new net ROW2: J?.7 (Pin_7)
- new net ROW3: J?.8 (Pin_8)

Commit message: A10
Changed lines of the file:
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@@
   )
   (symbol (lib_id "Connector:Conn_01x08_Female") (at 167.386 67.31 0) (unit 1)
-    (in_bom yes) (on_board yes) (fields_autoplaced)
+    (in_bom yes) (on_board yes)
     (property "Reference" "J?" (id 0) (at 168.0972 67.7453 0)
       (effects (font (size 1.27 1.27)) (justify left))
     )
-    (property "Value" "AUDIO_KEYPAD" (id 1) (at 168.0972 70.2822 0)
+    (property "Value" "AUDIO_KEYPAD" (id 1) (at 157.48 55.372 0)
       (effects (font (size 1.27 1.27)) (justify left))
     )

Commit message: A10 and F16
Parts:
- gave numbers to parts that had none: 24
Changed lines of the file:
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@@
   (symbol (lib_id "Switch:SW_Push") (at 65.786 101.092 0) (unit 1)
     (in_bom yes) (on_board yes) (fields_autoplaced)
-    (property "Reference" "SW?" (id 0) (at 65.786 94.4712 0))
+    (property "Reference" "SW53" (id 0) (at 65.786 94.4712 0))
     (property "Value" "LOAD" (id 1) (at 65.786 97.0081 0))
     (property "Footprint" "Connector_Molex:Molex_KK-254_AE-6410-02A_1x02_P2.54mm_Vertical" (id 2) (at 65.786 96.012 0)
@@
   (symbol (lib_id "Switch:SW_Push") (at 81.788 65.532 0) (unit 1)
     (in_bom yes) (on_board yes) (fields_autoplaced)
-    (property "Reference" "SW?" (id 0) (at 81.788 58.9112 0))
+    (property "Reference" "SW54" (id 0) (at 81.788 58.9112 0))
     (property "Value" "LOAD" (id 1) (at 81.788 61.4481 0))
     (property "Footprint" "Connector_Molex:Molex_KK-254_AE-6410-02A_1x02_P2.54mm_Vertical" (id 2) (at 81.788 60.452 0)
@@
   (symbol (lib_id "Switch:SW_Push") (at 101.092 101.092 0) (unit 1)
     (in_bom yes) (on_board yes) (fields_autoplaced)
-    (property "Reference" "SW?" (id 0) (at 101.092 94.4712 0))
+    (property "Reference" "SW61" (id 0) (at 101.092 94.4712 0))
     (property "Value" "LOAD" (id 1) (at 101.092 97.0081 0))
     (property "Footprint" "Connector_Molex:Molex_KK-254_AE-6410-02A_1x02_P2.54mm_Vertical" (id 2) (at 101.092 96.012 0)
@@
   (symbol (lib_id "Device:D") (at 93.218 135.128 0) (mirror y) (unit 1)
     (in_bom yes) (on_board yes)
-    (property "Reference" "D?" (id 0) (at 93.218 129.6416 0))
+    (property "Reference" "D55" (id 0) (at 93.218 129.6416 0))
     (property "Value" "D" (id 1) (at 93.218 131.953 0))
     (property "Footprint" "Diode_THT:D_A-405_P7.62mm_Horizontal" (id 2) (at 93.218 135.128 0)
@@
   (symbol (lib_id "Switch:SW_Push") (at 65.786 65.532 0) (unit 1)
     (in_bom yes) (on_board yes) (fields_autoplaced)
-    (property "Reference" "SW?" (id 0) (at 65.786 58.9112 0))
+    (property "Reference" "SW50" (id 0) (at 65.786 58.9112 0))
     (property "Value" "LOAD" (id 1) (at 65.786 61.4481 0))
     (property "Footprint" "Connector_Molex:Molex_KK-254_AE-6410-02A_1x02_P2.54mm_Vertical" (id 2) (at 65.786 60.452 0)
@@
   (symbol (lib_id "Switch:SW_Push") (at 81.788 75.438 0) (unit 1)
     (in_bom yes) (on_board yes) (fields_autoplaced)
-    (property "Reference" "SW?" (id 0) (at 81.788 68.8172 0))
+    (property "Reference" "SW55" (id 0) (at 81.788 68.8172 0))
     (property "Value" "LOAD" (id 1) (at 81.788 71.3541 0))
     (property "Footprint" "Connector_Molex:Molex_KK-254_AE-6410-02A_1x02_P2.54mm_Vertical" (id 2) (at 81.788 70.358 0)
@@
   (symbol (lib_id "Switch:SW_Push") (at 102.108 135.128 0) (unit 1)
     (in_bom yes) (on_board yes) (fields_autoplaced)
-    (property "Reference" "SW?" (id 0) (at 102.108 128.5072 0))
+    (property "Reference" "SW65" (id 0) (at 102.108 128.5072 0))
     (property "Value" "ARM" (id 1) (at 102.108 131.0441 0))
     (property "Footprint" "Connector_Molex:Molex_KK-254_AE-6410-02A_1x02_P2.54mm_Vertical" (id 2) (at 102.108 130.048 0)
@@
   (symbol (lib_id "Device:D") (at 92.964 145.796 0) (mirror y) (unit 1)
     (in_bom yes) (on_board yes)
-    (property "Reference" "D?" (id 0) (at 92.964 140.3096 0))
+    (property "Reference" "D53" (id 0) (at 92.964 140.3096 0))
     (property "Value" "D" (id 1) (at 92.964 142.621 0))
     (property "Footprint" "Diode_THT:D_A-405_P7.62mm_Horizontal" (id 2) (at 92.964 145.796 0)
@@
   (symbol (lib_id "Switch:SW_Push") (at 101.854 156.464 0) (unit 1)
     (in_bom yes) (on_board yes) (fields_autoplaced)
-    (property "Reference" "SW?" (id 0) (at 101.854 149.8432 0))
+    (property "Reference" "SW64" (id 0) (at 101.854 149.8432 0))
     (property "Value" "VHF" (id 1) (at 101.854 152.3801 0))
     (property "Footprint" "Connector_Molex:Molex_KK-254_AE-6410-02A_1x02_P2.54mm_Vertical" (id 2) (at 101.854 151.384 0)
@@
   (symbol (lib_id "Switch:SW_Push") (at 81.788 86.106 0) (unit 1)
     (in_bom yes) (on_board yes) (fields_autoplaced)
-    (property "Reference" "SW?" (id 0) (at 81.788 79.4852 0))
+    (property "Reference" "SW56" (id 0) (at 81.788 79.4852 0))
     (property "Value" "LOAD" (id 1) (at 81.788 82.0221 0))
     (property "Footprint" "Connector_Molex:Molex_KK-254_AE-6410-02A_1x02_P2.54mm_Vertical" (id 2) (at 81.788 81.026 0)
@@
   (symbol (lib_id "Switch:SW_Push") (at 101.854 145.796 0) (unit 1)
     (in_bom yes) (on_board yes) (fields_autoplaced)
-    (property "Reference" "SW?" (id 0) (at 101.854 139.1752 0))
+    (property "Reference" "SW63" (id 0) (at 101.854 139.1752 0))
     (property "Value" "INTERCOMM" (id 1) (at 101.854 141.7121 0))
     (property "Footprint" "Connector_Molex:Molex_KK-254_AE-6410-02A_1x02_P2.54mm_Vertical" (id 2) (at 101.854 140.716 0)
@@
   (symbol (lib_id "Device:D") (at 92.71 125.222 0) (mirror y) (unit 1)
     (in_bom yes) (on_board yes)
-    (property "Reference" "D?" (id 0) (at 92.71 119.7356 0))
+    (property "Reference" "D52" (id 0) (at 92.71 119.7356 0))
     (property "Value" "D" (id 1) (at 92.71 122.047 0))
     (property "Footprint" "Diode_THT:D_A-405_P7.62mm_Horizontal" (id 2) (at 92.71 125.222 0)
@@
   (symbol (lib_id "Connector:Conn_01x08_Female") (at 167.386 67.31 0) (unit 1)
     (in_bom yes) (on_board yes)
-    (property "Reference" "J?" (id 0) (at 168.0972 67.7453 0)
+    (property "Reference" "J36" (id 0) (at 168.0972 67.7453 0)
       (effects (font (size 1.27 1.27)) (justify left))
     )
@@
   (symbol (lib_id "Device:D") (at 92.964 156.464 0) (mirror y) (unit 1)
     (in_bom yes) (on_board yes)
-    (property "Reference" "D?" (id 0) (at 92.964 150.9776 0))
+    (property "Reference" "D54" (id 0) (at 92.964 150.9776 0))
     (property "Value" "D" (id 1) (at 92.964 153.289 0))
     (property "Footprint" "Diode_THT:D_A-405_P7.62mm_Horizontal" (id 2) (at 92.964 156.464 0)
@@
   (symbol (lib_id "Device:D") (at 88.138 112.776 0) (mirror y) (unit 1)
     (in_bom yes) (on_board yes)
-    (property "Reference" "D?" (id 0) (at 88.138 107.2896 0))
+    (property "Reference" "D51" (id 0) (at 88.138 107.2896 0))
     (property "Value" "D" (id 1) (at 88.138 109.601 0))
     (property "Footprint" "Diode_THT:D_A-405_P7.62mm_Horizontal" (id 2) (at 88.138 112.776 0)
@@
   (symbol (lib_id "Switch:SW_Push") (at 81.788 101.092 0) (unit 1)
     (in_bom yes) (on_board yes) (fields_autoplaced)
-    (property "Reference" "SW?" (id 0) (at 81.788 94.4712 0))
+    (property "Reference" "SW57" (id 0) (at 81.788 94.4712 0))
     (property "Value" "LOAD" (id 1) (at 81.788 97.0081 0))
     (property "Footprint" "Connector_Molex:Molex_KK-254_AE-6410-02A_1x02_P2.54mm_Vertical" (id 2) (at 81.788 96.012 0)
@@
   (symbol (lib_id "Switch:SW_Push") (at 101.092 86.106 0) (unit 1)
     (in_bom yes) (on_board yes) (fields_autoplaced)
-    (property "Reference" "SW?" (id 0) (at 101.092 79.4852 0))
+    (property "Reference" "SW60" (id 0) (at 101.092 79.4852 0))
     (property "Value" "LOAD" (id 1) (at 101.092 82.0221 0))
     (property "Footprint" "Connector_Molex:Molex_KK-254_AE-6410-02A_1x02_P2.54mm_Vertical" (id 2) (at 101.092 81.026 0)
@@
   (symbol (lib_id "Switch:SW_Push") (at 65.786 86.106 0) (unit 1)
     (in_bom yes) (on_board yes) (fields_autoplaced)
-    (property "Reference" "SW?" (id 0) (at 65.786 79.4852 0))
+    (property "Reference" "SW52" (id 0) (at 65.786 79.4852 0))
     (property "Value" "LOAD" (id 1) (at 65.786 82.0221 0))
     (property "Footprint" "Connector_Molex:Molex_KK-254_AE-6410-02A_1x02_P2.54mm_Vertical" (id 2) (at 65.786 81.026 0)
@@
   (symbol (lib_id "Switch:SW_Push") (at 101.092 65.532 0) (unit 1)
     (in_bom yes) (on_board yes) (fields_autoplaced)
-    (property "Reference" "SW?" (id 0) (at 101.092 58.9112 0))
+    (property "Reference" "SW58" (id 0) (at 101.092 58.9112 0))
     (property "Value" "LOAD" (id 1) (at 101.092 61.4481 0))
     (property "Footprint" "Connector_Molex:Molex_KK-254_AE-6410-02A_1x02_P2.54mm_Vertical" (id 2) (at 101.092 60.452 0)
@@
   (symbol (lib_id "Device:D") (at 72.39 112.776 0) (mirror y) (unit 1)
     (in_bom yes) (on_board yes)
-    (property "Reference" "D?" (id 0) (at 72.39 107.2896 0))
+    (property "Reference" "D50" (id 0) (at 72.39 107.2896 0))
     (property "Value" "D" (id 1) (at 72.39 109.601 0))
     (property "Footprint" "Diode_THT:D_A-405_P7.62mm_Horizontal" (id 2) (at 72.39 112.776 0)
@@
   (symbol (lib_id "Device:D") (at 56.642 112.776 0) (mirror y) (unit 1)
     (in_bom yes) (on_board yes)
-    (property "Reference" "D?" (id 0) (at 56.642 107.2896 0))
+    (property "Reference" "D49" (id 0) (at 56.642 107.2896 0))
     (property "Value" "D" (id 1) (at 56.642 109.601 0))
     (property "Footprint" "Diode_THT:D_A-405_P7.62mm_Horizontal" (id 2) (at 56.642 112.776 0)
@@
   (symbol (lib_id "Switch:SW_Push") (at 101.6 125.222 0) (unit 1)
     (in_bom yes) (on_board yes) (fields_autoplaced)
-    (property "Reference" "SW?" (id 0) (at 101.6 118.6012 0))
+    (property "Reference" "SW62" (id 0) (at 101.6 118.6012 0))
     (property "Value" "ESC" (id 1) (at 101.6 121.1381 0))
     (property "Footprint" "Connector_Molex:Molex_KK-254_AE-6410-02A_1x02_P2.54mm_Vertical" (id 2) (at 101.6 120.142 0)
@@
   (symbol (lib_id "Switch:SW_Push") (at 65.786 75.438 0) (unit 1)
     (in_bom yes) (on_board yes) (fields_autoplaced)
-    (property "Reference" "SW?" (id 0) (at 65.786 68.8172 0))
+    (property "Reference" "SW51" (id 0) (at 65.786 68.8172 0))
     (property "Value" "LOAD" (id 1) (at 65.786 71.3541 0))
     (property "Footprint" "Connector_Molex:Molex_KK-254_AE-6410-02A_1x02_P2.54mm_Vertical" (id 2) (at 65.786 70.358 0)
@@
   (symbol (lib_id "Switch:SW_Push") (at 101.092 75.438 0) (unit 1)
     (in_bom yes) (on_board yes) (fields_autoplaced)
-    (property "Reference" "SW?" (id 0) (at 101.092 68.8172 0))
+    (property "Reference" "SW59" (id 0) (at 101.092 68.8172 0))
     (property "Value" "LOAD" (id 1) (at 101.092 71.3541 0))
     (property "Footprint" "Connector_Molex:Molex_KK-254_AE-6410-02A_1x02_P2.54mm_Vertical" (id 2) (at 101.092 70.358 0)
