File: A10/A10 PCBs/Left Console Overview/FUEL.kicad_sch (KiCad schematic)
At the start: 30 parts

Commit message: A10
Parts:
- added J?: Conn_01x10_Female, symbol Connector:Conn_01x10_Female
- added J?: Conn_01x08_Female, symbol Connector:Conn_01x08_Female
Connections:
- net ROW7 is gone; now on net ROW6: SW?.2 (B)
- net COL6: now also D?.2 (A), D?.2 (A), J?.7 (Pin_7), J?.7 (Pin_7); no longer D?.2 (A)
- net ROW6: now reaches SW?.2 (B)
- net ROW6: now also SW?.2, SW?.2, SW?.2, SW?.2, SW?.3, J?.10 (Pin_10)
- net ROW5: now reaches SW?.2 (B)
- net ROW5: now also SW?.1, SW?.2 (B), SW?.2 (B), SW?.2 (B), SW?.2 (B), SW?.2 (B), SW?.2 (B), J?.9 (Pin_9)
- net COL2: now reaches D?.2 (A)
- net COL2: now also D?.2 (A), J?.3 (Pin_3), J?.3 (Pin_3)
- net COL4: now reaches D?.2 (A)
- net COL4: now also D?.2 (A), J?.5 (Pin_5), J?.5 (Pin_5)
- net COL3: now reaches D?.2 (A)
- net COL3: now also D?.2 (A), J?.4 (Pin_4), J?.4 (Pin_4)
- net COL1: now reaches D?.2 (A)
- net COL1: now also D?.2 (A), J?.2 (Pin_2), J?.2 (Pin_2)
- net COL5: now reaches D?.2 (A)
- net COL5: now also J?.6 (Pin_6), J?.6 (Pin_6)
- net COL0: now reaches D?.2 (A)
- net COL0: now also D?.2 (A), J?.1 (Pin_1), J?.1 (Pin_1)
- net COL7: now reaches D?.2 (A)
- net COL7: now also J?.8 (Pin_8), J?.8 (Pin_8)
Changed lines of the file:
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@@
     (stroke (width 0) (type default) (color 0 0 0 0))
   )
+  (label "COL7" (at 232.918 62.738 180)
+    (effects (font (size 1.27 1.27)) (justify right bottom))
+  )
+  (label "COL6" (at 230.632 85.344 180)
+    (effects (font (size 1.27 1.27)) (justify right bottom))
+  )
+  (label "COL0" (at 39.116 63.754 180)
+    (effects (font (size 1.27 1.27)) (justify right bottom))
+  )
+  (label "COL1" (at 232.918 47.498 180)
+    (effects (font (size 1.27 1.27)) (justify right bottom))
+  )
+  (label "COL2" (at 115.316 107.188 180)
+    (effects (font (size 1.27 1.27)) (justify right bottom))
+  )
   (label "ANALOG_5V" (at 121.158 60.452 180)
     (effects (font (size 1.27 1.27)) (justify right bottom))
   )
+  (label "COL3" (at 115.57 124.206 180)
+    (effects (font (size 1.27 1.27)) (justify right bottom))
+  )
   (label "RCVR_BRIGHT" (at 124.968 64.262 0)
     (effects (font (size 1.27 1.27)) (justify left bottom))
   )
+  (label "COL7" (at 134.112 85.344 180)
+    (effects (font (size 1.27 1.27)) (justify right bottom))
+  )
+  (label "ROW5" (at 151.13 82.804 0)
+    (effects (font (size 1.27 1.27)) (justify left bottom))
+  )
   (label "ANALOG_GND" (at 121.158 68.072 0)
     (effects (font (size 1.27 1.27)) (justify left bottom))
   )
+  (label "ROW5" (at 93.98 107.95 0)
+    (effects (font (size 1.27 1.27)) (justify left bottom))
+  )
+  (label "ROW5" (at 94.996 79.756 0)
+    (effects (font (size 1.27 1.27)) (justify left bottom))
+  )
+  (label "COL6" (at 232.918 60.198 180)
+    (effects (font (size 1.27 1.27)) (justify right bottom))
+  )
+  (label "COL1" (at 38.862 79.756 180)
+    (effects (font (size 1.27 1.27)) (justify right bottom))
+  )
+  (label "ROW6" (at 93.726 122.936 0)
+    (effects (font (size 1.27 1.27)) (justify left bottom))
+  )
+  (label "ROW5" (at 55.372 122.936 0)
+    (effects (font (size 1.27 1.27)) (justify left bottom))
+  )
   (label "RCVR_BRIGHT" (at 152.4 66.548 180)
     (effects (font (size 1.27 1.27)) (justify right bottom))
   )
+  (label "COL1" (at 230.632 72.644 180)
+    (effects (font (size 1.27 1.27)) (justify right bottom))
+  )
   (label "ANALOG_5V" (at 152.4 64.008 180)
     (effects (font (size 1.27 1.27)) (justify right bottom))
   )
-  (label "ROW7" (at 133.096 51.054 0)
+  (label "ROW5" (at 56.896 63.754 0)
+    (effects (font (size 1.27 1.27)) (justify left bottom))
+  )
+  (label "ROW5" (at 95.25 64.77 0)
+    (effects (font (size 1.27 1.27)) (justify left bottom))
+  )
+  (label "ROW5" (at 56.642 79.756 0)
+    (effects (font (size 1.27 1.27)) (justify left bottom))
+  )
+  (label "COL2" (at 77.47 64.77 180)
+    (effects (font (size 1.27 1.27)) (justify right bottom))
+  )
+  (label "COL3" (at 232.918 52.578 180)
+    (effects (font (size 1.27 1.27)) (justify right bottom))
+  )
+  (label "COL1" (at 115.316 51.054 180)
+    (effects (font (size 1.27 1.27)) (justify right bottom))
+  )
+  (label "ROW6" (at 165.1 108.204 0)
+    (effects (font (size 1.27 1.27)) (justify left bottom))
+  )
+  (label "COL7" (at 230.632 87.884 180)
+    (effects (font (size 1.27 1.27)) (justify right bottom))
+  )
+  (label "COL2" (at 230.632 75.184 180)
+    (effects (font (size 1.27 1.27)) (justify right bottom))
+  )
+  (label "COL5" (at 230.632 82.804 180)
+    (effects (font (size 1.27 1.27)) (justify right bottom))
+  )
+  (label "COL0" (at 230.632 70.104 180)
+    (effects (font (size 1.27 1.27)) (justify right bottom))
+  )
+  (label "COL0" (at 75.946 122.936 180)
+    (effects (font (size 1.27 1.27)) (justify right bottom))
+  )
+  (label "COL3" (at 230.632 77.724 180)
+    (effects (font (size 1.27 1.27)) (justify right bottom))
+  )
+  (label "COL2" (at 232.918 50.038 180)
+    (effects (font (size 1.27 1.27)) (justify right bottom))
+  )
+  (label "ROW6" (at 165.354 124.206 0)
+    (effects (font (size 1.27 1.27)) (justify left bottom))
+  )
+  (label "COL5" (at 76.2 107.95 180)
+    (effects (font (size 1.27 1.27)) (justify right bottom))
+  )
+  (label "COL3" (at 77.216 79.756 180)
+    (effects (font (size 1.27 1.27)) (justify right bottom))
+  )
+  (label "COL0" (at 232.918 44.958 180)
+    (effects (font (size 1.27 1.27)) (justify right bottom))
+  )
+  (label "COL6" (at 37.592 122.936 180)
+    (effects (font (size 1.27 1.27)) (justify right bottom))
+  )
+  (label "COL6" (at 147.574 124.206 180)
+    (effects (font (size 1.27 1.27)) (justify right bottom))
+  )
+  (label "ROW6" (at 133.35 124.206 0)
     (effects (font (size 1.27 1.27)) (justify left bottom))
   )
@@
     (effects (font (size 1.27 1.27)) (justify right bottom))
   )
-  (label "COL6" (at 115.316 51.054 180)
+  (label "ROW6" (at 133.096 107.188 0)
+    (effects (font (size 1.27 1.27)) (justify left bottom))
+  )
+  (label "ROW6" (at 133.096 51.054 0)
+    (effects (font (size 1.27 1.27)) (justify left bottom))
+  )
+  (label "COL5" (at 232.918 57.658 180)
+    (effects (font (size 1.27 1.27)) (justify right bottom))
+  )
+  (label "COL4" (at 232.918 55.118 180)
+    (effects (font (size 1.27 1.27)) (justify right bottom))
+  )
+  (label "ROW5" (at 55.626 106.934 0)
+    (effects (font (size 1.27 1.27)) (justify left bottom))
+  )
+  (label "ROW6" (at 230.632 92.964 180)
+    (effects (font (size 1.27 1.27)) (justify right bottom))
+  )
+  (label "ROW6" (at 151.13 87.884 0)
+    (effects (font (size 1.27 1.27)) (justify left bottom))
+  )
+  (label "COL4" (at 230.632 80.264 180)
+    (effects (font (size 1.27 1.27)) (justify right bottom))
+  )
+  (label "COL4" (at 147.32 108.204 180)
+    (effects (font (size 1.27 1.27)) (justify right bottom))
+  )
+  (label "ROW5" (at 230.632 90.424 180)
+    (effects (font (size 1.27 1.27)) (justify right bottom))
+  )
+  (label "COL4" (at 37.846 106.934 180)
     (effects (font (size 1.27 1.27)) (justify right bottom))
   )
@@
     (pin "2")
   )
+  (symbol (lib_id "Connector:Conn_01x10_Female") (at 235.712 80.264 0) (unit 1)
+    (in_bom yes) (on_board yes) (fields_autoplaced)
+    (property "Reference" "J?" (id 0) (at 236.4232 80.6993 0)
+      (effects (font (size 1.27 1.27)) (justify left))
+    )
+    (property "Value" "Conn_01x10_Female" (id 1) (at 236.4232 83.2362 0)
+      (effects (font (size 1.27 1.27)) (justify left))
+    )
+    (property "Footprint" "" (id 2) (at 235.712 80.264 0)
+      (effects (font (size 1.27 1.27)) hide)
+    )
+    (property "Datasheet" "~" (id 3) (at 235.712 80.264 0)
+      (effects (font (size 1.27 1.27)) hide)
+    )
+    (pin "1")
+    (pin "10")
+    (pin "2")
+    (pin "3")
+    (pin "4")
+    (pin "5")
+    (pin "6")
+    (pin "7")
+    (pin "8")
+    (pin "9")
+  )
   (symbol (lib_id "Device:D") (at 81.026 79.756 0) (mirror y) (unit 1)
     (in_bom yes) (on_board yes)
@@
     (pin "2")
   )
+  (symbol (lib_id "Connector:Conn_01x08_Female") (at 237.998 52.578 0) (unit 1)
+    (in_bom yes) (on_board yes) (fields_autoplaced)
+    (property "Reference" "J?" (id 0) (at 238.7092 53.0133 0)
+      (effects (font (size 1.27 1.27)) (justify left))
+    )
+    (property "Value" "Conn_01x08_Female" (id 1) (at 238.7092 55.5502 0)
+      (effects (font (size 1.27 1.27)) (justify left))
+    )
+    (property "Footprint" "" (id 2) (at 237.998 52.578 0)
+      (effects (font (size 1.27 1.27)) hide)
+    )
+    (property "Datasheet" "~" (id 3) (at 237.998 52.578 0)
+      (effects (font (size 1.27 1.27)) hide)
+    )
+    (pin "1")
+    (pin "2")
+    (pin "3")
+    (pin "4")
+    (pin "5")
+    (pin "6")
+    (pin "7")
+    (pin "8")
+  )
   (symbol (lib_id "Device:D") (at 81.28 64.77 0) (mirror y) (unit 1)

Commit message: A10
Parts:
- removed J?: Conn_01x08_Female, symbol Connector:Conn_01x08_Female
- J?: value Conn_01x10_Female -> FUEL
Other:
- moved on the sheet: J?
Changed lines of the file:
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@@
     (stroke (width 0) (type default) (color 0 0 0 0))
   )
-  (label "COL7" (at 232.918 62.738 180)
-    (effects (font (size 1.27 1.27)) (justify right bottom))
-  )
   (label "COL6" (at 230.632 85.344 180)
     (effects (font (size 1.27 1.27)) (justify right bottom))
@@
     (effects (font (size 1.27 1.27)) (justify right bottom))
   )
-  (label "COL1" (at 232.918 47.498 180)
-    (effects (font (size 1.27 1.27)) (justify right bottom))
-  )
   (label "COL2" (at 115.316 107.188 180)
     (effects (font (size 1.27 1.27)) (justify right bottom))
@@
     (effects (font (size 1.27 1.27)) (justify left bottom))
   )
-  (label "COL6" (at 232.918 60.198 180)
-    (effects (font (size 1.27 1.27)) (justify right bottom))
-  )
   (label "COL1" (at 38.862 79.756 180)
     (effects (font (size 1.27 1.27)) (justify right bottom))
@@
     (effects (font (size 1.27 1.27)) (justify left bottom))
   )
-  (label "RCVR_BRIGHT" (at 152.4 66.548 180)
+  (label "RCVR_BRIGHT" (at 235.712 56.896 180)
     (effects (font (size 1.27 1.27)) (justify right bottom))
   )
@@
     (effects (font (size 1.27 1.27)) (justify right bottom))
   )
-  (label "ANALOG_5V" (at 152.4 64.008 180)
+  (label "ANALOG_5V" (at 235.712 54.356 180)
     (effects (font (size 1.27 1.27)) (justify right bottom))
   )
@@
     (effects (font (size 1.27 1.27)) (justify right bottom))
   )
-  (label "COL3" (at 232.918 52.578 180)
-    (effects (font (size 1.27 1.27)) (justify right bottom))
-  )
   (label "COL1" (at 115.316 51.054 180)
     (effects (font (size 1.27 1.27)) (justify right bottom))
@@
     (effects (font (size 1.27 1.27)) (justify right bottom))
   )
-  (label "COL2" (at 232.918 50.038 180)
-    (effects (font (size 1.27 1.27)) (justify right bottom))
-  )
   (label "ROW6" (at 165.354 124.206 0)
     (effects (font (size 1.27 1.27)) (justify left bottom))
@@
     (effects (font (size 1.27 1.27)) (justify right bottom))
   )
-  (label "COL0" (at 232.918 44.958 180)
-    (effects (font (size 1.27 1.27)) (justify right bottom))
-  )
   (label "COL6" (at 37.592 122.936 180)
     (effects (font (size 1.27 1.27)) (justify right bottom))
@@
     (effects (font (size 1.27 1.27)) (justify left bottom))
   )
-  (label "ANALOG_GND" (at 152.4 69.088 180)
+  (label "ANALOG_GND" (at 235.712 59.436 180)
     (effects (font (size 1.27 1.27)) (justify right bottom))
   )
@@
   (label "ROW6" (at 133.096 51.054 0)
     (effects (font (size 1.27 1.27)) (justify left bottom))
-  )
-  (label "COL5" (at 232.918 57.658 180)
-    (effects (font (size 1.27 1.27)) (justify right bottom))
-  )
-  (label "COL4" (at 232.918 55.118 180)
-    (effects (font (size 1.27 1.27)) (justify right bottom))
   )
   (label "ROW5" (at 55.626 106.934 0)
@@
       (effects (font (size 1.27 1.27)) (justify left))
     )
-    (property "Value" "Conn_01x10_Female" (id 1) (at 236.4232 83.2362 0)
+    (property "Value" "FUEL" (id 1) (at 236.4232 83.2362 0)
       (effects (font (size 1.27 1.27)) (justify left))
     )
@@
     (pin "2")
   )
-  (symbol (lib_id "Connector:Conn_01x03_Female") (at 157.48 66.548 0) (unit 1)
-    (in_bom yes) (on_board yes) (fields_autoplaced)
-    (property "Reference" "J?" (id 0) (at 158.1912 65.7133 0)
+  (symbol (lib_id "Connector:Conn_01x03_Female") (at 240.792 56.896 0) (unit 1)
+    (in_bom yes) (on_board yes) (fields_autoplaced)
+    (property "Reference" "J?" (id 0) (at 241.5032 56.0613 0)
       (effects (font (size 1.27 1.27)) (justify left))
     )
-    (property "Value" "FUEL ANALOG" (id 1) (at 158.1912 68.2502 0)
+    (property "Value" "FUEL ANALOG" (id 1) (at 241.5032 58.5982 0)
       (effects (font (size 1.27 1.27)) (justify left))
     )
-    (property "Footprint" "" (id 2) (at 157.48 66.548 0)
-      (effects (font (size 1.27 1.27)) hide)
-    )
-    (property "Datasheet" "~" (id 3) (at 157.48 66.548 0)
+    (property "Footprint" "" (id 2) (at 240.792 56.896 0)
+      (effects (font (size 1.27 1.27)) hide)
+    )
+    (property "Datasheet" "~" (id 3) (at 240.792 56.896 0)
       (effects (font (size 1.27 1.27)) hide)
     )
@@
     (pin "2")
   )
-  (symbol (lib_id "Connector:Conn_01x08_Female") (at 237.998 52.578 0) (unit 1)
-    (in_bom yes) (on_board yes) (fields_autoplaced)
-    (property "Reference" "J?" (id 0) (at 238.7092 53.0133 0)
-      (effects (font (size 1.27 1.27)) (justify left))
-    )
-    (property "Value" "Conn_01x08_Female" (id 1) (at 238.7092 55.5502 0)
-      (effects (font (size 1.27 1.27)) (justify left))
-    )
-    (property "Footprint" "" (id 2) (at 237.998 52.578 0)
-      (effects (font (size 1.27 1.27)) hide)
-    )
-    (property "Datasheet" "~" (id 3) (at 237.998 52.578 0)
-      (effects (font (size 1.27 1.27)) hide)
-    )
-    (pin "1")
-    (pin "2")
-    (pin "3")
-    (pin "4")
-    (pin "5")
-    (pin "6")
-    (pin "7")
-    (pin "8")
-  )
   (symbol (lib_id "Device:D") (at 81.28 64.77 0) (mirror y) (unit 1)

Commit message: A10 and F16
Parts:
- gave numbers to parts that had none: 31
