File: A10/A10 PCBs/Left Console Overview/UHF.kicad_sch (KiCad schematic)
At the start: 18 parts

Commit message: A10
Parts:
- added J?: UHF, symbol Connector:Conn_01x06_Female
Connections:
- net COL1 is gone; now on net COL9: D?.2 (A)
- net ROW0: now also J?.3 (Pin_3)
- net ROW1: now also J?.4 (Pin_4); no longer SW?.2
- net ROW2: now also J?.5 (Pin_5)
- net ROW3: now also SW?.2, J?.6 (Pin_6)
- net COL9: now reaches D?.2 (A)
- net COL9: now also J?.2 (Pin_2)
- net COL0 renamed COL8
- net COL8: now also J?.1 (Pin_1)
Changed lines of the file:
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@@
     (effects (font (size 1.27 1.27)) (justify right bottom))
   )
-  (label "ROW1" (at 160.528 97.79 0)
+  (label "UHF_ENC_3_A" (at 54.356 58.166 180)
+    (effects (font (size 1.27 1.27)) (justify right bottom))
+  )
+  (label "UHF_PRESET_B" (at 54.102 103.632 180)
+    (effects (font (size 1.27 1.27)) (justify right bottom))
+  )
+  (label "UHF_ENC_5_B" (at 104.14 57.912 180)
+    (effects (font (size 1.27 1.27)) (justify right bottom))
+  )
+  (label "ROW1" (at 226.314 51.054 180)
+    (effects (font (size 1.27 1.27)) (justify right bottom))
+  )
+  (label "ROW3" (at 160.528 97.79 0)
     (effects (font (size 1.27 1.27)) (justify left bottom))
   )
-  (label "UHF_ENC_3_A" (at 54.356 58.166 180)
-    (effects (font (size 1.27 1.27)) (justify right bottom))
-  )
-  (label "UHF_PRESET_B" (at 54.102 103.632 180)
-    (effects (font (size 1.27 1.27)) (justify right bottom))
-  )
-  (label "UHF_ENC_5_B" (at 104.14 57.912 180)
-    (effects (font (size 1.27 1.27)) (justify right bottom))
-  )
   (label "ROW2" (at 152.4 84.074 180)
     (effects (font (size 1.27 1.27)) (justify right bottom))
@@
     (effects (font (size 1.27 1.27)) (justify right bottom))
   )
+  (label "COL9" (at 226.314 45.974 180)
+    (effects (font (size 1.27 1.27)) (justify right bottom))
+  )
   (label "UHF_PRESET_B" (at 104.14 62.992 180)
     (effects (font (size 1.27 1.27)) (justify right bottom))
@@
     (effects (font (size 1.27 1.27)) (justify right bottom))
   )
-  (label "COL1" (at 139.7 76.454 180)
+  (label "ROW3" (at 226.314 56.134 180)
+    (effects (font (size 1.27 1.27)) (justify right bottom))
+  )
+  (label "COL9" (at 139.7 76.454 180)
     (effects (font (size 1.27 1.27)) (justify right bottom))
   )
@@
     (effects (font (size 1.27 1.27)) (justify right bottom))
   )
+  (label "COL9" (at 142.748 97.79 180)
+    (effects (font (size 1.27 1.27)) (justify right bottom))
+  )
   (label "UHF_ENC_2_A" (at 53.848 45.72 180)
     (effects (font (size 1.27 1.27)) (justify right bottom))
   )
   (label "UHF_ENC_5_A" (at 54.356 84.582 180)
+    (effects (font (size 1.27 1.27)) (justify right bottom))
+  )
+  (label "ROW2" (at 226.314 53.594 180)
     (effects (font (size 1.27 1.27)) (justify right bottom))
   )
@@
     (effects (font (size 1.27 1.27)) (justify right bottom))
   )
+  (label "COL8" (at 226.314 43.434 180)
+    (effects (font (size 1.27 1.27)) (justify right bottom))
+  )
   (label "UHF_ENC_2_A" (at 104.14 34.036 180)
     (effects (font (size 1.27 1.27)) (justify right bottom))
@@
     (effects (font (size 1.27 1.27)) (justify right bottom))
   )
+  (label "ROW0" (at 226.314 48.514 180)
+    (effects (font (size 1.27 1.27)) (justify right bottom))
+  )
   (label "UHF_ENC_1_A" (at 54.102 31.75 180)
     (effects (font (size 1.27 1.27)) (justify right bottom))
   )
-  (label "COL0" (at 139.7 54.61 180)
+  (label "COL8" (at 139.7 54.61 180)
     (effects (font (size 1.27 1.27)) (justify right bottom))
   )
@@
     (pin "2")
   )
+  (symbol (lib_id "Connector:Conn_01x06_Female") (at 231.394 48.514 0) (unit 1)
+    (in_bom yes) (on_board yes) (fields_autoplaced)
+    (property "Reference" "J?" (id 0) (at 232.1052 48.9493 0)
+      (effects (font (size 1.27 1.27)) (justify left))
+    )
+    (property "Value" "UHF" (id 1) (at 232.1052 51.4862 0)
+      (effects (font (size 1.27 1.27)) (justify left))
+    )
+    (property "Footprint" "" (id 2) (at 231.394 48.514 0)
+      (effects (font (size 1.27 1.27)) hide)
+    )
+    (property "Datasheet" "~" (id 3) (at 231.394 48.514 0)
+      (effects (font (size 1.27 1.27)) hide)
+    )
+    (pin "1")
+    (pin "2")
+    (pin "3")
+    (pin "4")
+    (pin "5")
+    (pin "6")
+  )
   (symbol (lib_id "Device:R_Potentiometer_US") (at 142.24 127.254 0) (unit 1)

Commit message: A10
Parts:
- J?: value Conn_01x08_Female -> UHF_ENC_2
- J?: value Conn_01x08_Female -> UHF_ENC_1
Changed lines of the file:
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@@
       (effects (font (size 1.27 1.27)) (justify left))
     )
-    (property "Value" "Conn_01x08_Female" (id 1) (at 109.9312 58.3442 0)
+    (property "Value" "UHF_ENC_2" (id 1) (at 109.9312 58.3442 0)
       (effects (font (size 1.27 1.27)) (justify left))
     )
@@
       (effects (font (size 1.27 1.27)) (justify left))
     )
-    (property "Value" "Conn_01x08_Female" (id 1) (at 109.9312 37.0082 0)
+    (property "Value" "UHF_ENC_1" (id 1) (at 109.9312 37.0082 0)
       (effects (font (size 1.27 1.27)) (justify left))
     )

Commit message: A10 and F16
Parts:
- gave numbers to parts that had none: 19
Changed lines of the file:
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@@
   (symbol (lib_id "Connector:Conn_01x04_Female") (at 157.48 78.994 0) (unit 1)
     (in_bom yes) (on_board yes) (fields_autoplaced)
-    (property "Reference" "J?" (id 0) (at 158.1912 79.4293 0)
+    (property "Reference" "J16" (id 0) (at 158.1912 79.4293 0)
       (effects (font (size 1.27 1.27)) (justify left))
     )
@@
   (symbol (lib_id "power:GND") (at 40.386 34.29 0) (unit 1)
     (in_bom yes) (on_board yes) (fields_autoplaced)
-    (property "Reference" "#PWR?" (id 0) (at 40.386 40.64 0)
+    (property "Reference" "#PWR04" (id 0) (at 40.386 40.64 0)
       (effects (font (size 1.27 1.27)) hide)
     )
@@
   (symbol (lib_id "power:GND") (at 40.64 74.676 0) (unit 1)
     (in_bom yes) (on_board yes) (fields_autoplaced)
-    (property "Reference" "#PWR?" (id 0) (at 40.64 81.026 0)
+    (property "Reference" "#PWR07" (id 0) (at 40.64 81.026 0)
       (effects (font (size 1.27 1.27)) hide)
     )
@@
   (symbol (lib_id "Connector:Conn_01x03_Female") (at 178.054 128.27 0) (unit 1)
     (in_bom yes) (on_board yes) (fields_autoplaced)
-    (property "Reference" "J?" (id 0) (at 178.7652 127.4353 0)
+    (property "Reference" "J17" (id 0) (at 178.7652 127.4353 0)
       (effects (font (size 1.27 1.27)) (justify left))
     )
@@
   (symbol (lib_id "Device:D") (at 143.51 76.454 0) (mirror y) (unit 1)
     (in_bom yes) (on_board yes)
-    (property "Reference" "D?" (id 0) (at 143.51 70.9676 0))
+    (property "Reference" "D36" (id 0) (at 143.51 70.9676 0))
     (property "Value" "D" (id 1) (at 143.51 73.279 0))
     (property "Footprint" "Diode_THT:D_A-405_P7.62mm_Horizontal" (id 2) (at 143.51 76.454 0)
@@
   (symbol (lib_id "Device:RotaryEncoder") (at 61.976 87.122 0) (unit 1)
     (in_bom yes) (on_board yes) (fields_autoplaced)
-    (property "Reference" "SW?" (id 0) (at 67.818 86.2873 0)
+    (property "Reference" "SW32" (id 0) (at 67.818 86.2873 0)
       (effects (font (size 1.27 1.27)) (justify left))
     )
@@
   (symbol (lib_id "Device:RotaryEncoder") (at 61.722 34.29 0) (unit 1)
     (in_bom yes) (on_board yes) (fields_autoplaced)
-    (property "Reference" "SW?" (id 0) (at 67.564 33.4553 0)
+    (property "Reference" "SW28" (id 0) (at 67.564 33.4553 0)
       (effects (font (size 1.27 1.27)) (justify left))
     )
@@
   (symbol (lib_id "power:GND") (at 40.386 48.26 0) (unit 1)
     (in_bom yes) (on_board yes) (fields_autoplaced)
-    (property "Reference" "#PWR?" (id 0) (at 40.386 54.61 0)
+    (property "Reference" "#PWR05" (id 0) (at 40.386 54.61 0)
       (effects (font (size 1.27 1.27)) hide)
     )
@@
   (symbol (lib_id "Device:RotaryEncoder") (at 61.468 48.26 0) (unit 1)
     (in_bom yes) (on_board yes) (fields_autoplaced)
-    (property "Reference" "SW?" (id 0) (at 67.31 47.4253 0)
+    (property "Reference" "SW27" (id 0) (at 67.31 47.4253 0)
       (effects (font (size 1.27 1.27)) (justify left))
     )
@@
   (symbol (lib_id "Device:D") (at 143.51 54.61 0) (mirror y) (unit 1)
     (in_bom yes) (on_board yes)
-    (property "Reference" "D?" (id 0) (at 143.51 49.1236 0))
+    (property "Reference" "D35" (id 0) (at 143.51 49.1236 0))
     (property "Value" "D" (id 1) (at 143.51 51.435 0))
     (property "Footprint" "Diode_THT:D_A-405_P7.62mm_Horizontal" (id 2) (at 143.51 54.61 0)
@@
   (symbol (lib_id "Connector:Conn_01x08_Female") (at 109.22 55.372 0) (unit 1)
     (in_bom yes) (on_board yes) (fields_autoplaced)
-    (property "Reference" "J?" (id 0) (at 109.9312 55.8073 0)
+    (property "Reference" "J14" (id 0) (at 109.9312 55.8073 0)
       (effects (font (size 1.27 1.27)) (justify left))
     )
@@
   (symbol (lib_id "power:GND") (at 40.64 87.122 0) (unit 1)
     (in_bom yes) (on_board yes) (fields_autoplaced)
-    (property "Reference" "#PWR?" (id 0) (at 40.64 93.472 0)
+    (property "Reference" "#PWR08" (id 0) (at 40.64 93.472 0)
       (effects (font (size 1.27 1.27)) hide)
     )
@@
   (symbol (lib_id "power:GND") (at 40.64 101.092 0) (unit 1)
     (in_bom yes) (on_board yes) (fields_autoplaced)
-    (property "Reference" "#PWR?" (id 0) (at 40.64 107.442 0)
+    (property "Reference" "#PWR09" (id 0) (at 40.64 107.442 0)
       (effects (font (size 1.27 1.27)) hide)
     )
@@
   (symbol (lib_id "Switch:SW_Push") (at 155.448 97.79 0) (unit 1)
     (in_bom yes) (on_board yes) (fields_autoplaced)
-    (property "Reference" "SW?" (id 0) (at 155.448 91.1692 0))
+    (property "Reference" "SW33" (id 0) (at 155.448 91.1692 0))
     (property "Value" "LOAD" (id 1) (at 155.448 93.7061 0))
     (property "Footprint" "Connector_Molex:Molex_KK-254_AE-6410-02A_1x02_P2.54mm_Vertical" (id 2) (at 155.448 92.71 0)
@@
   (symbol (lib_id "Connector:Conn_01x06_Female") (at 231.394 48.514 0) (unit 1)
     (in_bom yes) (on_board yes) (fields_autoplaced)
-    (property "Reference" "J?" (id 0) (at 232.1052 48.9493 0)
+    (property "Reference" "J18" (id 0) (at 232.1052 48.9493 0)
       (effects (font (size 1.27 1.27)) (justify left))
     )
@@
   (symbol (lib_id "Device:R_Potentiometer_US") (at 142.24 127.254 0) (unit 1)
     (in_bom yes) (on_board yes) (fields_autoplaced)
-    (property "Reference" "RV?" (id 0) (at 140.5891 126.4193 0)
+    (property "Reference" "RV4" (id 0) (at 140.5891 126.4193 0)
       (effects (font (size 1.27 1.27)) (justify right))
     )
@@
   (symbol (lib_id "Connector:Conn_01x04_Female") (at 53.848 130.302 0) (mirror y) (unit 1)
     (in_bom yes) (on_board yes)
-    (property "Reference" "J?" (id 0) (at 54.483 123.605 0))
+    (property "Reference" "J11" (id 0) (at 54.483 123.605 0))
     (property "Value" "UHF_DISP" (id 1) (at 48.514 133.096 0))
     (property "Footprint" "" (id 2) (at 53.848 130.302 0)
@@
   (symbol (lib_id "Device:RotaryEncoder") (at 61.722 74.676 0) (unit 1)
     (in_bom yes) (on_board yes) (fields_autoplaced)
-    (property "Reference" "SW?" (id 0) (at 67.564 73.8413 0)
+    (property "Reference" "SW29" (id 0) (at 67.564 73.8413 0)
       (effects (font (size 1.27 1.27)) (justify left))
     )
@@
   (symbol (lib_id "Device:D") (at 146.558 97.79 0) (mirror y) (unit 1)
     (in_bom yes) (on_board yes)
-    (property "Reference" "D?" (id 0) (at 146.558 92.3036 0))
+    (property "Reference" "D37" (id 0) (at 146.558 92.3036 0))
     (property "Value" "D" (id 1) (at 146.558 94.615 0))
     (property "Footprint" "Diode_THT:D_A-405_P7.62mm_Horizontal" (id 2) (at 146.558 97.79 0)
@@
   (symbol (lib_id "Connector:Conn_01x08_Female") (at 109.22 34.036 0) (unit 1)
     (in_bom yes) (on_board yes) (fields_autoplaced)
-    (property "Reference" "J?" (id 0) (at 109.9312 34.4713 0)
+    (property "Reference" "J13" (id 0) (at 109.9312 34.4713 0)
       (effects (font (size 1.27 1.27)) (justify left))
     )
@@
   (symbol (lib_id "power:GND") (at 40.64 60.706 0) (unit 1)
     (in_bom yes) (on_board yes) (fields_autoplaced)
-    (property "Reference" "#PWR?" (id 0) (at 40.64 67.056 0)
+    (property "Reference" "#PWR06" (id 0) (at 40.64 67.056 0)
       (effects (font (size 1.27 1.27)) hide)
     )
@@
   (symbol (lib_id "Connector:Conn_01x06_Female") (at 157.48 59.69 0) (unit 1)
     (in_bom yes) (on_board yes)
-    (property "Reference" "J?" (id 0) (at 158.1912 60.1253 0)
+    (property "Reference" "J15" (id 0) (at 158.1912 60.1253 0)
       (effects (font (size 1.27 1.27)) (justify left))
     )
@@
   (symbol (lib_id "Device:RotaryEncoder") (at 61.976 60.706 0) (unit 1)
     (in_bom yes) (on_board yes) (fields_autoplaced)
-    (property "Reference" "SW?" (id 0) (at 67.818 59.8713 0)
+    (property "Reference" "SW31" (id 0) (at 67.818 59.8713 0)
       (effects (font (size 1.27 1.27)) (justify left))
     )
@@
   (symbol (lib_id "power:GND") (at 88.9 47.752 0) (unit 1)
     (in_bom yes) (on_board yes) (fields_autoplaced)
-    (property "Reference" "#PWR?" (id 0) (at 88.9 54.102 0)
+    (property "Reference" "#PWR011" (id 0) (at 88.9 54.102 0)
       (effects (font (size 1.27 1.27)) hide)
     )
@@
   (symbol (lib_id "Device:RotaryEncoder") (at 61.722 101.092 0) (unit 1)
     (in_bom yes) (on_board yes) (fields_autoplaced)
-    (property "Reference" "SW?" (id 0) (at 67.564 100.2573 0)
+    (property "Reference" "SW30" (id 0) (at 67.564 100.2573 0)
       (effects (font (size 1.27 1.27)) (justify left))
     )
@@
   (symbol (lib_id "power:GND") (at 88.9 26.416 0) (unit 1)
     (in_bom yes) (on_board yes) (fields_autoplaced)
-    (property "Reference" "#PWR?" (id 0) (at 88.9 32.766 0)
+    (property "Reference" "#PWR010" (id 0) (at 88.9 32.766 0)
       (effects (font (size 1.27 1.27)) hide)
     )
@@
   (symbol (lib_id "Connector:Conn_01x04_Female") (at 64.008 130.302 0) (unit 1)
     (in_bom yes) (on_board yes) (fields_autoplaced)
-    (property "Reference" "J?" (id 0) (at 64.7192 130.7373 0)
-      (effects (font (size 1.27 1.27)) (justify left))
-    )
+    (property "Reference" "J12" (id 0) (at 64.7192 130.7373 0)
+      (effects (font (size 1.27 1.27)) (justify left))
+    )
