File: A10/A10 PCBs/Left Console Overview/VHF_FM.kicad_sch (KiCad schematic)
At the start: 0 parts

Commit message: A10
Parts:
- added D? (x4): D, Diode_THT:D_A-405_P7.62mm_Horizontal, symbol Device:D
- added J?: UVHF_FM_MAIN, Connector_Molex:Molex_KK-254_AE-6410-06A_1x06_P2.54mm_Vertical, symbol Connector:Conn_01x06_Female
- added J?: VHF_FM_ANALOG, symbol Connector:Conn_01x03_Female
- added J? (x2): VHF_FM, symbol Connector:Conn_01x04_Female
- added J?: VHF_FM_1, symbol Connector:Conn_01x08_Female
- added J?: VHF_FM_OFF_TR_DF, symbol Connector:Conn_01x04_Female
- added J?: VHF_AM, symbol Connector:Conn_01x08_Female
- added RV?: VHF_FM_VOL, symbol Device:R_Potentiometer_US
- added SW?: TONE, Connector_Molex:Molex_KK-254_AE-6410-02A_1x02_P2.54mm_Vertical, symbol Switch:SW_Push
- added SW?: ENCODER_3, Connector_Molex:Molex_KK-254_AE-6410-03A_1x03_P2.54mm_Vertical, symbol Device:RotaryEncoder
- added SW?: ENCODER_1, Connector_Molex:Molex_KK-254_AE-6410-03A_1x03_P2.54mm_Vertical, symbol Device:RotaryEncoder
- added SW?: ENCODER_2, Connector_Molex:Molex_KK-254_AE-6410-03A_1x03_P2.54mm_Vertical, symbol Device:RotaryEncoder
- added SW?: ENCODER_4, Connector_Molex:Molex_KK-254_AE-6410-03A_1x03_P2.54mm_Vertical, symbol Device:RotaryEncoder
- added SW?: PRESET, Connector_Molex:Molex_KK-254_AE-6410-03A_1x03_P2.54mm_Vertical, symbol Device:RotaryEncoder
- added SW?: LOAD, Connector_Molex:Molex_KK-254_AE-6410-02A_1x02_P2.54mm_Vertical, symbol Switch:SW_Push
- added VHF_FM_2: UHF_MAIN, Connector_Molex:Molex_KK-254_AE-6410-06A_1x06_P2.54mm_Vertical, symbol Connector:Conn_01x06_Female
Connections:
- new net: D?.1 (K), J?.1 (Pin_1) (x2)
- new net: D?.1 (K), SW?.1 (x2)
- new net: J?.1 (Pin_1), J?.1 (Pin_1)
- new net: J?.2 (Pin_2), J?.2 (Pin_2)
- new net: J?.3 (Pin_3), J?.3 (Pin_3)
- new net: J?.4 (Pin_4), J?.4 (Pin_4)
- new net ANALOG_5V: J?.1 (Pin_1), RV?.1
- new net ANALOG_GND: J?.3 (Pin_3), RV?.3
- new net COL6: D?.2 (A), D?.2 (A), J?.1 (Pin_1)
- new net COL7: D?.2 (A), D?.2 (A), J?.2 (Pin_2)
- new net GND: J?.1 (Pin_1), SW?.C, SW?.C, SW?.C, SW?.C, SW?.C, VHF_FM_2.1 (Pin_1)
- new net ROW0: J?.2 (Pin_2), J?.2 (Pin_2), J?.3 (Pin_3)
- new net ROW1: J?.3 (Pin_3), J?.3 (Pin_3), J?.4 (Pin_4)
- new net ROW2: J?.4 (Pin_4), J?.4 (Pin_4), J?.5 (Pin_5)
- new net ROW3: J?.5 (Pin_5), J?.6 (Pin_6), SW?.2
- new net ROW4: J?.7 (Pin_7), SW?.2
- new net VHF_FM_VOL: J?.2 (Pin_2), RV?.2
- new net VHF__FM_ENC_1_A: J?.2 (Pin_2), SW?.A
- new net VHF__FM_ENC_1_B: J?.3 (Pin_3), SW?.B
- new net VHF__FM_ENC_2_A: J?.4 (Pin_4), SW?.A
- new net VHF__FM_ENC_2_B: J?.5 (Pin_5), SW?.B
- new net VHF__FM_ENC_3_A: J?.6 (Pin_6), SW?.A
- new net VHF__FM_ENC_3_B: J?.7 (Pin_7), SW?.B
- new net VHF__FM_ENC_4_A: SW?.A, VHF_FM_2.2 (Pin_2)
- new net VHF__FM_ENC_4_B: SW?.B, VHF_FM_2.3 (Pin_3)
- new net VHF__FM_PRESET_A: SW?.A, VHF_FM_2.4 (Pin_4)
- new net VHF__FM_PRESET_B: SW?.B, VHF_FM_2.5 (Pin_5)
- no-connect marks 0 -> 4

Commit message: A10
Parts:
- J?: value VHF_AM -> VHF_FM
Changed lines of the file:
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@@
   )
   (symbol (lib_id "Connector:Conn_01x03_Female") (at 202.438 143.002 0) (unit 1)
-    (in_bom yes) (on_board yes) (fields_autoplaced)
+    (in_bom yes) (on_board yes)
     (property "Reference" "J?" (id 0) (at 203.1492 142.1673 0)
       (effects (font (size 1.27 1.27)) (justify left))
     )
-    (property "Value" "VHF_FM_ANALOG" (id 1) (at 203.1492 144.7042 0)
+    (property "Value" "VHF_FM_ANALOG" (id 1) (at 187.706 136.398 0)
       (effects (font (size 1.27 1.27)) (justify left))
     )
@@
       (effects (font (size 1.27 1.27)) (justify left))
     )
-    (property "Value" "VHF_AM" (id 1) (at 248.8692 74.0922 0)
-      (effects (font (size 1.27 1.27)) (justify left))
-    )
+    (property "Value" "VHF_FM" (id 1) (at 248.8692 74.0922 0)
+      (effects (font (size 1.27 1.27)) (justify left))
+    )

Commit message: A10 and F16
Parts:
- gave numbers to parts that had none: 19
- renumbered VHF_FM_2 to VHF_FM_1
Changed lines of the file:
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@@
   (symbol (lib_id "Connector:Conn_01x06_Female") (at 181.864 74.422 0) (unit 1)
     (in_bom yes) (on_board yes)
-    (property "Reference" "J?" (id 0) (at 182.5752 74.8573 0)
+    (property "Reference" "J22" (id 0) (at 182.5752 74.8573 0)
       (effects (font (size 1.27 1.27)) (justify left))
     )
@@
   (symbol (lib_id "Device:R_Potentiometer_US") (at 166.624 141.986 0) (unit 1)
     (in_bom yes) (on_board yes) (fields_autoplaced)
-    (property "Reference" "RV?" (id 0) (at 164.973 141.1513 0)
+    (property "Reference" "RV5" (id 0) (at 164.973 141.1513 0)
       (effects (font (size 1.27 1.27)) (justify right))
     )
@@
   (symbol (lib_id "power:GND") (at 51.308 49.022 0) (unit 1)
     (in_bom yes) (on_board yes) (fields_autoplaced)
-    (property "Reference" "#PWR?" (id 0) (at 51.308 55.372 0)
+    (property "Reference" "#PWR013" (id 0) (at 51.308 55.372 0)
       (effects (font (size 1.27 1.27)) hide)
     )
@@
   (symbol (lib_id "power:GND") (at 50.8 104.14 0) (unit 1)
     (in_bom yes) (on_board yes) (fields_autoplaced)
-    (property "Reference" "#PWR?" (id 0) (at 50.8 110.49 0)
+    (property "Reference" "#PWR012" (id 0) (at 50.8 110.49 0)
       (effects (font (size 1.27 1.27)) hide)
     )
@@
   (symbol (lib_id "Switch:SW_Push") (at 180.34 122.428 0) (unit 1)
     (in_bom yes) (on_board yes) (fields_autoplaced)
-    (property "Reference" "SW?" (id 0) (at 180.34 115.8072 0))
+    (property "Reference" "SW40" (id 0) (at 180.34 115.8072 0))
     (property "Value" "TONE" (id 1) (at 180.34 118.3441 0))
     (property "Footprint" "Connector_Molex:Molex_KK-254_AE-6410-02A_1x02_P2.54mm_Vertical" (id 2) (at 180.34 117.348 0)
@@
   (symbol (lib_id "power:GND") (at 108.712 67.056 0) (unit 1)
     (in_bom yes) (on_board yes) (fields_autoplaced)
-    (property "Reference" "#PWR?" (id 0) (at 108.712 73.406 0)
+    (property "Reference" "#PWR018" (id 0) (at 108.712 73.406 0)
       (effects (font (size 1.27 1.27)) hide)
     )
@@
   (symbol (lib_id "Device:RotaryEncoder") (at 86.36 75.438 0) (unit 1)
     (in_bom yes) (on_board yes) (fields_autoplaced)
-    (property "Reference" "SW?" (id 0) (at 92.202 74.6033 0)
+    (property "Reference" "SW38" (id 0) (at 92.202 74.6033 0)
       (effects (font (size 1.27 1.27)) (justify left))
     )
@@
   (symbol (lib_id "Device:D") (at 167.894 69.342 0) (mirror y) (unit 1)
     (in_bom yes) (on_board yes)
-    (property "Reference" "D?" (id 0) (at 167.894 63.8556 0))
+    (property "Reference" "D38" (id 0) (at 167.894 63.8556 0))
     (property "Value" "D" (id 1) (at 167.894 66.167 0))
     (property "Footprint" "Diode_THT:D_A-405_P7.62mm_Horizontal" (id 2) (at 167.894 69.342 0)
@@
   (symbol (lib_id "Connector:Conn_01x03_Female") (at 202.438 143.002 0) (unit 1)
     (in_bom yes) (on_board yes)
-    (property "Reference" "J?" (id 0) (at 203.1492 142.1673 0)
+    (property "Reference" "J24" (id 0) (at 203.1492 142.1673 0)
       (effects (font (size 1.27 1.27)) (justify left))
     )
@@
   (symbol (lib_id "Connector:Conn_01x04_Female") (at 78.232 145.034 0) (mirror y) (unit 1)
     (in_bom yes) (on_board yes)
-    (property "Reference" "J?" (id 0) (at 78.867 138.337 0))
+    (property "Reference" "J19" (id 0) (at 78.867 138.337 0))
     (property "Value" "VHF_FM" (id 1) (at 72.898 147.828 0))
     (property "Footprint" "" (id 2) (at 78.232 145.034 0)
@@
   (symbol (lib_id "Connector:Conn_01x08_Female") (at 133.604 48.768 0) (unit 1)
     (in_bom yes) (on_board yes) (fields_autoplaced)
-    (property "Reference" "J?" (id 0) (at 134.3152 49.2033 0)
+    (property "Reference" "J21" (id 0) (at 134.3152 49.2033 0)
       (effects (font (size 1.27 1.27)) (justify left))
     )
@@
   (symbol (lib_id "power:GND") (at 51.308 89.408 0) (unit 1)
     (in_bom yes) (on_board yes) (fields_autoplaced)
-    (property "Reference" "#PWR?" (id 0) (at 51.308 95.758 0)
+    (property "Reference" "#PWR016" (id 0) (at 51.308 95.758 0)
       (effects (font (size 1.27 1.27)) hide)
     )
@@
   (symbol (lib_id "Device:RotaryEncoder") (at 86.106 49.022 0) (unit 1)
     (in_bom yes) (on_board yes) (fields_autoplaced)
-    (property "Reference" "SW?" (id 0) (at 91.948 48.1873 0)
+    (property "Reference" "SW36" (id 0) (at 91.948 48.1873 0)
       (effects (font (size 1.27 1.27)) (justify left))
     )
@@
   (symbol (lib_id "power:GND") (at 108.712 41.148 0) (unit 1)
     (in_bom yes) (on_board yes) (fields_autoplaced)
-    (property "Reference" "#PWR?" (id 0) (at 108.712 47.498 0)
+    (property "Reference" "#PWR017" (id 0) (at 108.712 47.498 0)
       (effects (font (size 1.27 1.27)) hide)
     )
@@
   (symbol (lib_id "Device:D") (at 170.942 112.522 0) (mirror y) (unit 1)
     (in_bom yes) (on_board yes)
-    (property "Reference" "D?" (id 0) (at 170.942 107.0356 0))
+    (property "Reference" "D40" (id 0) (at 170.942 107.0356 0))
     (property "Value" "D" (id 1) (at 170.942 109.347 0))
     (property "Footprint" "Diode_THT:D_A-405_P7.62mm_Horizontal" (id 2) (at 170.942 112.522 0)
@@
   (symbol (lib_id "Device:D") (at 171.45 122.428 0) (mirror y) (unit 1)
     (in_bom yes) (on_board yes)
-    (property "Reference" "D?" (id 0) (at 171.45 116.9416 0))
+    (property "Reference" "D41" (id 0) (at 171.45 116.9416 0))
     (property "Value" "D" (id 1) (at 171.45 119.253 0))
     (property "Footprint" "Diode_THT:D_A-405_P7.62mm_Horizontal" (id 2) (at 171.45 122.428 0)
@@
   (symbol (lib_id "Connector:Conn_01x04_Female") (at 181.864 93.726 0) (unit 1)
     (in_bom yes) (on_board yes) (fields_autoplaced)
-    (property "Reference" "J?" (id 0) (at 182.5752 94.1613 0)
+    (property "Reference" "J23" (id 0) (at 182.5752 94.1613 0)
       (effects (font (size 1.27 1.27)) (justify left))
     )
@@
   (symbol (lib_id "Device:RotaryEncoder") (at 85.852 62.992 0) (unit 1)
     (in_bom yes) (on_board yes) (fields_autoplaced)
-    (property "Reference" "SW?" (id 0) (at 91.694 62.1573 0)
+    (property "Reference" "SW35" (id 0) (at 91.694 62.1573 0)
       (effects (font (size 1.27 1.27)) (justify left))
     )
@@
   (symbol (lib_id "Device:RotaryEncoder") (at 86.106 89.408 0) (unit 1)
     (in_bom yes) (on_board yes) (fields_autoplaced)
-    (property "Reference" "SW?" (id 0) (at 91.948 88.5733 0)
+    (property "Reference" "SW37" (id 0) (at 91.948 88.5733 0)
       (effects (font (size 1.27 1.27)) (justify left))
     )
@@
   (symbol (lib_id "Connector:Conn_01x06_Female") (at 133.604 72.136 0) (unit 1)
     (in_bom yes) (on_board yes)
-    (property "Reference" "VHF_FM_2" (id 0) (at 134.3152 72.5713 0)
+    (property "Reference" "VHF_FM_1" (id 0) (at 134.3152 72.5713 0)
       (effects (font (size 1.27 1.27)) (justify left))
     )
@@
   (symbol (lib_id "power:GND") (at 51.308 62.992 0) (unit 1)
     (in_bom yes) (on_board yes) (fields_autoplaced)
-    (property "Reference" "#PWR?" (id 0) (at 51.308 69.342 0)
+    (property "Reference" "#PWR014" (id 0) (at 51.308 69.342 0)
       (effects (font (size 1.27 1.27)) hide)
     )
@@
   (symbol (lib_id "Device:RotaryEncoder") (at 85.598 104.14 0) (unit 1)
     (in_bom yes) (on_board yes) (fields_autoplaced)
-    (property "Reference" "SW?" (id 0) (at 91.44 103.3053 0)
+    (property "Reference" "SW34" (id 0) (at 91.44 103.3053 0)
       (effects (font (size 1.27 1.27)) (justify left))
     )
@@
   (symbol (lib_id "Switch:SW_Push") (at 179.832 112.522 0) (unit 1)
     (in_bom yes) (on_board yes) (fields_autoplaced)
-    (property "Reference" "SW?" (id 0) (at 179.832 105.9012 0))
+    (property "Reference" "SW39" (id 0) (at 179.832 105.9012 0))
     (property "Value" "LOAD" (id 1) (at 179.832 108.4381 0))
     (property "Footprint" "Connector_Molex:Molex_KK-254_AE-6410-02A_1x02_P2.54mm_Vertical" (id 2) (at 179.832 107.442 0)
@@
   (symbol (lib_id "Connector:Conn_01x04_Female") (at 88.392 145.034 0) (unit 1)
     (in_bom yes) (on_board yes) (fields_autoplaced)
-    (property "Reference" "J?" (id 0) (at 89.1032 145.4693 0)
+    (property "Reference" "J20" (id 0) (at 89.1032 145.4693 0)
       (effects (font (size 1.27 1.27)) (justify left))
     )
@@
   (symbol (lib_id "power:GND") (at 51.308 75.438 0) (unit 1)
     (in_bom yes) (on_board yes) (fields_autoplaced)
-    (property "Reference" "#PWR?" (id 0) (at 51.308 81.788 0)
+    (property "Reference" "#PWR015" (id 0) (at 51.308 81.788 0)
       (effects (font (size 1.27 1.27)) hide)
     )
@@
   (symbol (lib_id "Connector:Conn_01x08_Female") (at 248.158 71.12 0) (unit 1)
     (in_bom yes) (on_board yes) (fields_autoplaced)
-    (property "Reference" "J?" (id 0) (at 248.8692 71.5553 0)
+    (property "Reference" "J25" (id 0) (at 248.8692 71.5553 0)
       (effects (font (size 1.27 1.27)) (justify left))
     )
@@
   (symbol (lib_id "Device:D") (at 167.894 91.186 0) (mirror y) (unit 1)
     (in_bom yes) (on_board yes)
-    (property "Reference" "D?" (id 0) (at 167.894 85.6996 0))
+    (property "Reference" "D39" (id 0) (at 167.894 85.6996 0))
     (property "Value" "D" (id 1) (at 167.894 88.011 0))
     (property "Footprint" "Diode_THT:D_A-405_P7.62mm_Horizontal" (id 2) (at 167.894 91.186 0)

Commit message: A10
Parts:
- removed J19, J20: VHF_FM, symbol Connector:Conn_01x04_Female
- removed SW34: PRESET, Connector_Molex:Molex_KK-254_AE-6410-03A_1x03_P2.54mm_Vertical, symbol Device:RotaryEncoder
- removed SW35: ENCODER_2, Connector_Molex:Molex_KK-254_AE-6410-03A_1x03_P2.54mm_Vertical, symbol Device:RotaryEncoder
- removed SW36: ENCODER_1, Connector_Molex:Molex_KK-254_AE-6410-03A_1x03_P2.54mm_Vertical, symbol Device:RotaryEncoder
- removed SW37: ENCODER_4, Connector_Molex:Molex_KK-254_AE-6410-03A_1x03_P2.54mm_Vertical, symbol Device:RotaryEncoder
- removed SW38: ENCODER_3, Connector_Molex:Molex_KK-254_AE-6410-03A_1x03_P2.54mm_Vertical, symbol Device:RotaryEncoder
- added J3, J6: OLED, Connector_Molex:Molex_KK-254_AE-6410-04A_1x04_P2.54mm_Vertical, symbol Connector:Conn_01x04_Socket
- added J4, J5: BKLGHT, Connector_Molex:Molex_KK-254_AE-6410-02A_1x02_P2.54mm_Vertical, symbol Connector:Conn_01x02_Socket
- added SW8: ENCODER_4, Connector_Molex:Molex_KK-254_AE-6410-03A_1x03_P2.54mm_Vertical, symbol Device:RotaryEncoder
- added SW8: PRESET, Connector_Molex:Molex_KK-254_AE-6410-03A_1x03_P2.54mm_Vertical, symbol Device:RotaryEncoder
- added SW8: ENCODER_1, Connector_Molex:Molex_KK-254_AE-6410-03A_1x03_P2.54mm_Vertical, symbol Device:RotaryEncoder
- added SW8: ENCODER_3, Connector_Molex:Molex_KK-254_AE-6410-03A_1x03_P2.54mm_Vertical, symbol Device:RotaryEncoder
- added SW8: ENCODER_2, Connector_Molex:Molex_KK-254_AE-6410-03A_1x03_P2.54mm_Vertical, symbol Device:RotaryEncoder
Connections:
- net GND: now also SW8.2, SW8.2, SW8.2, SW8.2, SW8.2
- net VHF__FM_ENC_1_A: now also SW8.1
- net VHF__FM_ENC_1_B: now also SW8.3
- net VHF__FM_ENC_2_A: now also SW8.1
- net VHF__FM_ENC_2_B: now also SW8.3
- net VHF__FM_ENC_3_A: now also SW8.1
- net VHF__FM_ENC_3_B: now also SW8.3
- net VHF__FM_ENC_4_A: now also SW8.1
- net VHF__FM_ENC_4_B: now also SW8.3
- net VHF__FM_PRESET_A: now also SW8.1
- net VHF__FM_PRESET_B: now also SW8.3
- new net: J3.1 (Pin_1), J6.1 (Pin_1)
- new net: J3.2 (Pin_2), J6.2 (Pin_2)
- new net: J3.3 (Pin_3), J6.3 (Pin_3)
- new net: J3.4 (Pin_4), J6.4 (Pin_4)
- new net: J4.1 (Pin_1), J5.1 (Pin_1)
- new net: J4.2 (Pin_2), J5.2 (Pin_2)
