File: A10/A10 PCBs/Forward Console Overview/Forward Console Overview.kicad_pcb (KiCad board)
At the start: 2 copper layers, 18 parts, among them J1 Conn_01x03_Female, J10 I2C Out, J11 INPUT COLS, J2 Conn_01x03_Female, J3 Conn_01x03_Female, J4 Conn_01x03_Female, J5 Conn_01x02_Female, J6 Conn_01x02_Female, J7 TACAN ROTARY SWITCH, J8 Conn_01x08_Female, J9 I2C In, SW1 Right Encoder, SW2 SW_Rotary2x6, SW3 Test, SW4 Encoder_Push

Commit message: a10
Parts:
- added D10: LED, Connector_Molex:Molex_KK-254_AE-6410-02A_1x02_P2.54mm_Vertical, F.Cu at (144.2, 86.8)
- added D100: LED, LED_THT:LED_D3.0mm_FlatTop, F.Cu at (42.5, 113.4)
- added D101: LED, LED_THT:LED_D3.0mm_FlatTop, F.Cu at (42.5, 118.9)
- added D102: LED, LED_THT:LED_D3.0mm_FlatTop, F.Cu at (42.5, 124.5)
- added D103: LED, LED_THT:LED_D3.0mm_FlatTop, F.Cu at (42.5, 130.0)
- added D104: LED, LED_THT:LED_D3.0mm_FlatTop, F.Cu at (42.5, 135.6)
- added D105: LED, LED_THT:LED_D3.0mm_FlatTop, F.Cu at (48.4, 107.8)
- added D106: LED, LED_THT:LED_D3.0mm_FlatTop, F.Cu at (48.4, 113.4)
- added D107: LED, LED_THT:LED_D3.0mm_FlatTop, F.Cu at (48.4, 118.9)
- added D108: LED, LED_THT:LED_D3.0mm_FlatTop, F.Cu at (48.4, 124.5)
- added D109: LED, LED_THT:LED_D3.0mm_FlatTop, F.Cu at (48.4, 130.0)
- added D11: D, Diode_THT:D_A-405_P7.62mm_Horizontal, F.Cu at (99.6, 84.9)
- added D110: LED, LED_THT:LED_D3.0mm_FlatTop, F.Cu at (48.4, 135.6)
- added D12: D, Diode_THT:D_A-405_P7.62mm_Horizontal, F.Cu at (99.6, 89.2)
- added D13: D, Diode_THT:D_A-405_P7.62mm_Horizontal, F.Cu at (99.6, 93.4)
- added D14: D, Diode_THT:D_A-405_P7.62mm_Horizontal, F.Cu at (99.6, 97.7)
- added D15: D, Diode_THT:D_A-405_P7.62mm_Horizontal, F.Cu at (99.6, 101.9)
- added D16: D, Diode_THT:D_A-405_P7.62mm_Horizontal, F.Cu at (99.6, 106.2)
- added D17: D, Diode_THT:D_A-405_P7.62mm_Horizontal, F.Cu at (99.6, 110.4)
- added D18: D, Diode_THT:D_A-405_P7.62mm_Horizontal, F.Cu at (99.6, 114.7)
- added D19: D, Diode_THT:D_A-405_P7.62mm_Horizontal, F.Cu at (99.6, 118.9)
- added D20: D, Diode_THT:D_A-405_P7.62mm_Horizontal, F.Cu at (99.6, 123.2)
- added D21: D, Diode_THT:D_A-405_P7.62mm_Horizontal, F.Cu at (99.6, 31.9)
- added D22: D, Diode_THT:D_A-405_P7.62mm_Horizontal, F.Cu at (99.6, 36.2)
- added D23: D, Diode_THT:D_A-405_P7.62mm_Horizontal, F.Cu at (99.6, 40.4)
- added D24: PRI, Connector_Molex:Molex_KK-254_AE-6410-02A_1x02_P2.54mm_Vertical, F.Cu at (111.2, 33.8)
- added D25: HARS, Connector_Molex:Molex_KK-254_AE-6410-02A_1x02_P2.54mm_Vertical, F.Cu at (118.3, 33.8)
- added D26: STR PT, Connector_Molex:Molex_KK-254_AE-6410-02A_1x02_P2.54mm_Vertical, F.Cu at (125.4, 33.8)
- added D27: VHF, Connector_Molex:Molex_KK-254_AE-6410-02A_1x02_P2.54mm_Vertical, F.Cu at (132.6, 33.8)
- added D28: D, Diode_THT:D_A-405_P7.62mm_Horizontal, F.Cu at (99.6, 44.7)
- added D29: D, Diode_THT:D_A-405_P7.62mm_Horizontal, F.Cu at (99.6, 48.9)
- added D30: D, Diode_THT:D_A-405_P7.62mm_Horizontal, F.Cu at (99.6, 53.2)
- added D31: D, Diode_THT:D_A-405_P7.62mm_Horizontal, F.Cu at (99.6, 57.4)
- added D32: SEP, Connector_Molex:Molex_KK-254_AE-6410-02A_1x02_P2.54mm_Vertical, F.Cu at (139.7, 33.8)
- added D33: MISSLE LAUNCH, Connector_Molex:Molex_KK-254_AE-6410-02A_1x02_P2.54mm_Vertical, F.Cu at (111.2, 41.6)
- added D34: ANCHR, Connector_Molex:Molex_KK-254_AE-6410-02A_1x02_P2.54mm_Vertical, F.Cu at (118.3, 41.6)
- added D35: D, Diode_THT:D_A-405_P7.62mm_Horizontal, F.Cu at (99.6, 61.7)
- added D36: SPARE, Connector_Molex:Molex_KK-254_AE-6410-02A_1x02_P2.54mm_Vertical, F.Cu at (125.4, 41.6)
- added D37: D, Diode_THT:D_A-405_P7.62mm_Horizontal, F.Cu at (99.6, 65.9)
- added D38: D, Diode_THT:D_A-405_P7.62mm_Horizontal, F.Cu at (99.6, 70.2)
- added D39: EGI, Connector_Molex:Molex_KK-254_AE-6410-02A_1x02_P2.54mm_Vertical, F.Cu at (132.6, 41.6)
- added D4: D, Diode_THT:D_A-405_P7.62mm_Horizontal, F.Cu at (133.9, 92.8)
- added D40: TCN, Connector_Molex:Molex_KK-254_AE-6410-02A_1x02_P2.54mm_Vertical, F.Cu at (139.7, 41.6)
- added D41: UHF, Connector_Molex:Molex_KK-254_AE-6410-02A_1x02_P2.54mm_Vertical, F.Cu at (111.2, 49.5)
- added D42: D, Diode_THT:D_A-405_P7.62mm_Horizontal, F.Cu at (99.6, 74.4)
- added D43: D, Diode_THT:D_A-405_P7.62mm_Horizontal, F.Cu at (99.6, 78.7)
- added D44: TISL, Connector_Molex:Molex_KK-254_AE-6410-02A_1x02_P2.54mm_Vertical, F.Cu at (118.3, 49.5)
- added D45: ILS, Connector_Molex:Molex_KK-254_AE-6410-02A_1x02_P2.54mm_Vertical, F.Cu at (125.4, 49.5)
- added D46: D, Diode_THT:D_A-405_P7.62mm_Horizontal, F.Cu at (36.6, 71.2)
- added D47: D, Diode_THT:D_A-405_P7.62mm_Horizontal, F.Cu at (36.6, 75.4)
- added D48: D, Diode_THT:D_A-405_P7.62mm_Horizontal, F.Cu at (36.6, 79.7)
- added D49: D, Diode_THT:D_A-405_P7.62mm_Horizontal, F.Cu at (36.6, 83.9)
- added D5: D, Diode_THT:D_A-405_P7.62mm_Horizontal, F.Cu at (133.9, 97.0)
- added D50: D, Diode_THT:D_A-405_P7.62mm_Horizontal, F.Cu at (36.6, 88.2)
- added D51: D, Diode_THT:D_A-405_P7.62mm_Horizontal, F.Cu at (36.6, 92.4)
- added D52: D, Diode_THT:D_A-405_P7.62mm_Horizontal, F.Cu at (36.6, 96.7)
- added D53: D, Diode_THT:D_A-405_P7.62mm_Horizontal, F.Cu at (36.6, 100.9)
- added D54: D, Diode_THT:D_A-405_P7.62mm_Horizontal, F.Cu at (47.6, 71.2)
- added D55: D, Diode_THT:D_A-405_P7.62mm_Horizontal, F.Cu at (47.6, 75.4)
- added D56: D, Diode_THT:D_A-405_P7.62mm_Horizontal, F.Cu at (47.6, 79.7)
- added D57: D, Diode_THT:D_A-405_P7.62mm_Horizontal, F.Cu at (47.6, 83.9)
- added D58: D, Diode_THT:D_A-405_P7.62mm_Horizontal, F.Cu at (47.6, 88.2)
- added D59: D, Diode_THT:D_A-405_P7.62mm_Horizontal, F.Cu at (47.6, 92.4)
- added D6: D, Diode_THT:D_A-405_P7.62mm_Horizontal, F.Cu at (133.9, 101.3)
- added D60: D, Diode_THT:D_A-405_P7.62mm_Horizontal, F.Cu at (47.6, 96.7)
- added D61: D, Diode_THT:D_A-405_P7.62mm_Horizontal, F.Cu at (47.6, 100.9)
- added D62: D, Diode_THT:D_A-405_P7.62mm_Horizontal, F.Cu at (58.6, 71.2)
- added D63: D, Diode_THT:D_A-405_P7.62mm_Horizontal, F.Cu at (58.6, 75.4)
- added D64: D, Diode_THT:D_A-405_P7.62mm_Horizontal, F.Cu at (58.6, 79.7)
- added D65: MASTER CAUTION, Connector_Molex:Molex_KK-254_AE-6410-02A_1x02_P2.54mm_Vertical, F.Cu at (37.2, 33.8)
- added D66: D, Diode_THT:D_A-405_P7.62mm_Horizontal, F.Cu at (58.6, 83.9)
- added D67: D, Diode_THT:D_A-405_P7.62mm_Horizontal, F.Cu at (58.6, 88.2)
- added D68: D, Diode_THT:D_A-405_P7.62mm_Horizontal, F.Cu at (58.6, 92.4)
- added D69: D, Diode_THT:D_A-405_P7.62mm_Horizontal, F.Cu at (58.6, 96.7)
- added D7: LED, Connector_Molex:Molex_KK-254_AE-6410-02A_1x02_P2.54mm_Vertical, F.Cu at (122.8, 86.8)
- added D70: D, Diode_THT:D_A-405_P7.62mm_Horizontal, F.Cu at (58.6, 100.9)
- added D71: D, Diode_THT:D_A-405_P7.62mm_Horizontal, F.Cu at (69.5, 71.2)
- added D72: D, Diode_THT:D_A-405_P7.62mm_Horizontal, F.Cu at (69.5, 75.4)
- added D73: D, Diode_THT:D_A-405_P7.62mm_Horizontal, F.Cu at (69.5, 79.7)
- added D74: D, Diode_THT:D_A-405_P7.62mm_Horizontal, F.Cu at (69.5, 83.9)
- added D75: D, Diode_THT:D_A-405_P7.62mm_Horizontal, F.Cu at (69.5, 88.2)
- added D76: D, Diode_THT:D_A-405_P7.62mm_Horizontal, F.Cu at (69.5, 92.4)
- added D77: D, Diode_THT:D_A-405_P7.62mm_Horizontal, F.Cu at (69.5, 96.7)
- added D78: GUN READY A, Connector_Molex:Molex_KK-254_AE-6410-02A_1x02_P2.54mm_Vertical, F.Cu at (63.1, 109.0)
- added D79: GUN READY B, Connector_Molex:Molex_KK-254_AE-6410-02A_1x02_P2.54mm_Vertical, F.Cu at (70.2, 109.0)
- added D8: LED, Connector_Molex:Molex_KK-254_AE-6410-02A_1x02_P2.54mm_Vertical, F.Cu at (130.0, 86.8)
- added D80: D, Diode_THT:D_A-405_P7.62mm_Horizontal, F.Cu at (83.8, 107.2)
- added D81: STEERING A, Connector_Molex:Molex_KK-254_AE-6410-02A_1x02_P2.54mm_Vertical, F.Cu at (77.3, 109.0)
- added D82: STEERING B, Connector_Molex:Molex_KK-254_AE-6410-02A_1x02_P2.54mm_Vertical, F.Cu at (63.1, 116.8)
- added D83: D, Diode_THT:D_A-405_P7.62mm_Horizontal, F.Cu at (83.8, 111.4)
- added D84: D, Diode_THT:D_A-405_P7.62mm_Horizontal, F.Cu at (83.8, 115.7)
- added D85: D, Diode_THT:D_A-405_P7.62mm_Horizontal, F.Cu at (83.8, 119.9)
- added D86: MKR BEACON A, Connector_Molex:Molex_KK-254_AE-6410-02A_1x02_P2.54mm_Vertical, F.Cu at (70.2, 116.8)
- added D87: MKR BEACON B, Connector_Molex:Molex_KK-254_AE-6410-02A_1x02_P2.54mm_Vertical, F.Cu at (77.3, 116.8)
- added D88: D, Diode_THT:D_A-405_P7.62mm_Horizontal, F.Cu at (83.8, 124.2)
- added D89: CANOPY UNLOCKED A, Connector_Molex:Molex_KK-254_AE-6410-02A_1x02_P2.54mm_Vertical, F.Cu at (63.1, 124.7)
- added D9: LED, Connector_Molex:Molex_KK-254_AE-6410-02A_1x02_P2.54mm_Vertical, F.Cu at (137.1, 86.8)
- added D90: CANOPY UNLOCKED B, Connector_Molex:Molex_KK-254_AE-6410-02A_1x02_P2.54mm_Vertical, F.Cu at (70.2, 124.7)
- added D91: D, Diode_THT:D_A-405_P7.62mm_Horizontal, F.Cu at (122.2, 128.4)
- added D92: D, Diode_THT:D_A-405_P7.62mm_Horizontal, F.Cu at (122.2, 132.6)
- added D93: LED, LED_THT:LED_D3.0mm_FlatTop, F.Cu at (36.6, 107.8)
- added D94: LED, LED_THT:LED_D3.0mm_FlatTop, F.Cu at (36.6, 113.4)
- added D95: LED, LED_THT:LED_D3.0mm_FlatTop, F.Cu at (36.6, 118.9)
- added D96: LED, LED_THT:LED_D3.0mm_FlatTop, F.Cu at (36.6, 124.5)
- added D97: LED, LED_THT:LED_D3.0mm_FlatTop, F.Cu at (36.6, 130.0)
- added D98: LED, LED_THT:LED_D3.0mm_FlatTop, F.Cu at (36.6, 135.6)
- added D99: LED, LED_THT:LED_D3.0mm_FlatTop, F.Cu at (42.5, 107.8)
- added K1: ANIT-SKID, Relay_THT:Relay_1P1T_NO_10x24x18.8mm_Panasonic_ADW11xxxxW_THT, F.Cu at (122.7, 93.1)
- added R1: R_US, Resistor_THT:R_Axial_DIN0207_L6.3mm_D2.5mm_P2.54mm_Vertical, F.Cu at (54.7, 107.1)
- added R2: R_US, Resistor_THT:R_Axial_DIN0207_L6.3mm_D2.5mm_P2.54mm_Vertical, F.Cu at (54.7, 111.1)
- added R3: R_US, Resistor_THT:R_Axial_DIN0207_L6.3mm_D2.5mm_P2.54mm_Vertical, F.Cu at (54.7, 115.2)
- added R4: R_US, Resistor_THT:R_Axial_DIN0207_L6.3mm_D2.5mm_P2.54mm_Vertical, F.Cu at (54.7, 119.2)
- added R5: R_US, Resistor_THT:R_Axial_DIN0207_L6.3mm_D2.5mm_P2.54mm_Vertical, F.Cu at (54.7, 123.3)
- added R6: R_US, Resistor_THT:R_Axial_DIN0207_L6.3mm_D2.5mm_P2.54mm_Vertical, F.Cu at (54.7, 127.3)
- added SW13: IFCC, Connector_Molex:Molex_KK-254_AE-6410-03A_1x03_P2.54mm_Vertical, F.Cu at (111.2, 118.2)
- added SW15: PRI, Connector_Molex:Molex_KK-254_AE-6410-02A_1x02_P2.54mm_Vertical, F.Cu at (132.6, 49.5)
- added SW16: HARS, Connector_Molex:Molex_KK-254_AE-6410-02A_1x02_P2.54mm_Vertical, F.Cu at (139.7, 49.5)
- added SW17: STR PT, Connector_Molex:Molex_KK-254_AE-6410-02A_1x02_P2.54mm_Vertical, F.Cu at (111.2, 57.3)
- added SW18: SEP, Connector_Molex:Molex_KK-254_AE-6410-02A_1x02_P2.54mm_Vertical, F.Cu at (118.3, 57.3)
- added SW19: PTR, Connector_Molex:Molex_KK-254_AE-6410-02A_1x02_P2.54mm_Vertical, F.Cu at (125.4, 57.3)
- added SW20: MISSLE LAUNCH, Connector_Molex:Molex_KK-254_AE-6410-02A_1x02_P2.54mm_Vertical, F.Cu at (132.6, 57.3)
- added SW21: ANCHR, Connector_Molex:Molex_KK-254_AE-6410-02A_1x02_P2.54mm_Vertical, F.Cu at (139.7, 57.3)
- added SW22: SPARE, Connector_Molex:Molex_KK-254_AE-6410-02A_1x02_P2.54mm_Vertical, F.Cu at (111.2, 65.2)
- added SW23: EGI, Connector_Molex:Molex_KK-254_AE-6410-02A_1x02_P2.54mm_Vertical, F.Cu at (118.3, 65.2)
- added SW24: TCN, Connector_Molex:Molex_KK-254_AE-6410-02A_1x02_P2.54mm_Vertical, F.Cu at (125.4, 65.2)
- added SW25: TISL, Connector_Molex:Molex_KK-254_AE-6410-02A_1x02_P2.54mm_Vertical, F.Cu at (132.6, 65.2)
- added SW26: ILS, Connector_Molex:Molex_KK-254_AE-6410-02A_1x02_P2.54mm_Vertical, F.Cu at (139.7, 65.2)
- added SW27: STEER +, Button_Switch_THT:SW_PUSH-12mm, F.Cu at (81.1, 73.3)
- added SW28: STEER -, Connector_Molex:Molex_KK-254_AE-6410-02A_1x02_P2.54mm_Vertical, F.Cu at (44.4, 33.8)
- added SW29: 1, Connector_Molex:Molex_KK-254_AE-6410-02A_1x02_P2.54mm_Vertical, F.Cu at (51.5, 33.8)
- added SW30: 4, Connector_Molex:Molex_KK-254_AE-6410-02A_1x02_P2.54mm_Vertical, F.Cu at (58.6, 33.8)
- added SW31: 7, Connector_Molex:Molex_KK-254_AE-6410-02A_1x02_P2.54mm_Vertical, F.Cu at (65.8, 33.8)
- added SW32: FUNC, Connector_Molex:Molex_KK-254_AE-6410-02A_1x02_P2.54mm_Vertical, F.Cu at (72.9, 33.8)
- added SW33: LTR, Connector_Molex:Molex_KK-254_AE-6410-02A_1x02_P2.54mm_Vertical, F.Cu at (80.0, 33.8)
- added SW34: CLR, Connector_Molex:Molex_KK-254_AE-6410-02A_1x02_P2.54mm_Vertical, F.Cu at (37.2, 41.6)
- added SW35: 2, Connector_Molex:Molex_KK-254_AE-6410-02A_1x02_P2.54mm_Vertical, F.Cu at (44.4, 41.6)
- added SW36: 5, Connector_Molex:Molex_KK-254_AE-6410-02A_1x02_P2.54mm_Vertical, F.Cu at (51.5, 41.6)
- added SW37: 8, Connector_Molex:Molex_KK-254_AE-6410-02A_1x02_P2.54mm_Vertical, F.Cu at (58.6, 41.6)
- added SW38: ENT, Connector_Molex:Molex_KK-254_AE-6410-02A_1x02_P2.54mm_Vertical, F.Cu at (65.8, 41.6)
- added SW39: MK, Connector_Molex:Molex_KK-254_AE-6410-02A_1x02_P2.54mm_Vertical, F.Cu at (72.9, 41.6)
- added SW40: 3, Connector_Molex:Molex_KK-254_AE-6410-02A_1x02_P2.54mm_Vertical, F.Cu at (80.0, 41.6)
- added SW41: 6, Connector_Molex:Molex_KK-254_AE-6410-02A_1x02_P2.54mm_Vertical, F.Cu at (37.2, 49.5)
- added SW42: 9, Connector_Molex:Molex_KK-254_AE-6410-02A_1x02_P2.54mm_Vertical, F.Cu at (44.4, 49.5)
- added SW43: INTEN LEFT, Connector_Molex:Molex_KK-254_AE-6410-02A_1x02_P2.54mm_Vertical, F.Cu at (51.5, 49.5)
- added SW44: MASTER CAUTION, Connector_Molex:Molex_KK-254_AE-6410-02A_1x02_P2.54mm_Vertical, F.Cu at (58.6, 49.5)
- added SW45: INTEN LEFT, Connector_Molex:Molex_KK-254_AE-6410-02A_1x02_P2.54mm_Vertical, F.Cu at (65.8, 49.5)
- added SW46: POS, Connector_Molex:Molex_KK-254_AE-6410-02A_1x02_P2.54mm_Vertical, F.Cu at (72.9, 49.5)
- added SW47: 0, Connector_Molex:Molex_KK-254_AE-6410-02A_1x02_P2.54mm_Vertical, F.Cu at (80.0, 49.5)
- added SW48: SPC, Connector_Molex:Molex_KK-254_AE-6410-02A_1x02_P2.54mm_Vertical, F.Cu at (37.2, 57.3)
- added SW49: INTEN RIGHT, Connector_Molex:Molex_KK-254_AE-6410-02A_1x02_P2.54mm_Vertical, F.Cu at (44.4, 57.3)
- added SW5: MASTER ARM, Connector_Molex:Molex_KK-254_AE-6410-03A_1x03_P2.54mm_Vertical, F.Cu at (111.2, 86.8)
- added SW50: INTEN LEFT, Connector_Molex:Molex_KK-254_AE-6410-02A_1x02_P2.54mm_Vertical, F.Cu at (51.5, 57.3)
- added SW51: DATA UP, Connector_Molex:Molex_KK-254_AE-6410-02A_1x02_P2.54mm_Vertical, F.Cu at (58.6, 57.3)
- added SW52: DATA DOWN, Connector_Molex:Molex_KK-254_AE-6410-02A_1x02_P2.54mm_Vertical, F.Cu at (65.8, 57.3)
- added SW53: INTEN RIGHT, Connector_Molex:Molex_KK-254_AE-6410-02A_1x02_P2.54mm_Vertical, F.Cu at (72.9, 57.3)
- added SW54: SEL UP, Connector_Molex:Molex_KK-254_AE-6410-02A_1x02_P2.54mm_Vertical, F.Cu at (80.0, 57.3)
- added SW55: SEL DOWN, Connector_Molex:Molex_KK-254_AE-6410-02A_1x02_P2.54mm_Vertical, F.Cu at (37.2, 65.2)
- added SW56: DEPR UP, Connector_Molex:Molex_KK-254_AE-6410-02A_1x02_P2.54mm_Vertical, F.Cu at (44.4, 65.2)
- added SW57: DEPR DOWN, Connector_Molex:Molex_KK-254_AE-6410-02A_1x02_P2.54mm_Vertical, F.Cu at (51.5, 65.2)
- added SW58: EXT STORES JET, Connector_Molex:Molex_KK-254_AE-6410-02A_1x02_P2.54mm_Vertical, F.Cu at (77.3, 124.7)
- added SW59: ANCHR, Connector_Molex:Molex_KK-254_AE-6410-02A_1x02_P2.54mm_Vertical, F.Cu at (63.1, 132.6)
- added SW6: LASER, Connector_Molex:Molex_KK-254_AE-6410-03A_1x03_P2.54mm_Vertical, F.Cu at (111.2, 94.6)
- added SW60: ANCHR, Connector_Molex:Molex_KK-254_AE-6410-02A_1x02_P2.54mm_Vertical, F.Cu at (70.2, 132.6)
- added SW61: ANCHR, Connector_Molex:Molex_KK-254_AE-6410-02A_1x02_P2.54mm_Vertical, F.Cu at (77.3, 132.6)
- added SW62: FIRE EXT DISC, Connector_Molex:Molex_KK-254_AE-6410-03A_1x03_P2.54mm_Vertical, F.Cu at (84.5, 130.2)
- added SW63: JAMMER, Connector_Molex:Molex_KK-254_AE-6410-02A_1x02_P2.54mm_Vertical, F.Cu at (122.8, 122.3)
- added SW64: MWS, Connector_Molex:Molex_KK-254_AE-6410-02A_1x02_P2.54mm_Vertical, F.Cu at (130.0, 122.3)
- added SW7: ALT SCE, Connector_Molex:Molex_KK-254_AE-6410-03A_1x03_P2.54mm_Vertical, F.Cu at (111.2, 102.5)
- added SW9: GUM / PAC, Connector_Molex:Molex_KK-254_AE-6410-03A_1x03_P2.54mm_Vertical, F.Cu at (111.2, 110.3)
- J10: value I2C Out -> BKLGHT; footprint Connector_Molex:Molex_KK-254_AE-6410-04A_1x04_P2.54mm_Vertical -> Connector_Molex:Molex_KK-254_AE-6410-02A_1x02_P2.54mm_Vertical
- J11: value INPUT COLS -> BKLGHT; footprint Connector_Molex:Molex_KK-254_AE-6410-08A_1x08_P2.54mm_Vertical -> Connector_Molex:Molex_KK-254_AE-6410-02A_1x02_P2.54mm_Vertical
- J5: value Conn_01x02_Female -> Conn_01x02_Socket
- J6: value Conn_01x02_Female -> UFC COLS; footprint Connector_Molex:Molex_KK-254_AE-6410-02A_1x02_P2.54mm_Vertical -> Connector_Molex:Molex_KK-254_AE-6410-06A_1x06_P2.54mm_Vertical
- J7: value TACAN ROTARY SWITCH -> UFC ROWS
- SW1: value Right Encoder -> FLAPS
- SW2: value SW_Rotary2x6 -> LANDING LIGHTS; footprint Connector_Molex:Molex_KK-254_AE-6410-06A_1x06_P2.54mm_Vertical -> Connector_Molex:Molex_KK-254_AE-6410-03A_1x03_P2.54mm_Vertical
- SW3: value Test -> BRAKE; footprint Connector_Molex:Molex_KK-254_AE-6410-02A_1x02_P2.54mm_Vertical -> Connector_Molex:Molex_KK-254_AE-6410-03A_1x03_P2.54mm_Vertical
Connections:
- D1 pad 1: Net-(D1-Pad1) -> Net-(D1-K)
- D1 pad 2: /TACAN/COL2 -> /LANDING GEAR/COL0
- D2 pad 1: Net-(D2-Pad1) -> Net-(D2-K)
- D2 pad 2: unconnected-(D2-Pad2) -> /LANDING GEAR/COL0
- D3 pad 1: Net-(D3-Pad1) -> /LANDING GEAR/COIL_28V
- D3 pad 2: /TACAN/COL1 -> /LANDING GEAR/COIL_ANTI_SKID
- J10 pad 1: Net-(J10-Pad1) -> /UFC/UFC_BACKLIGHTING/BACKLIGHT_+12V
- J10 pad 2: Net-(J10-Pad2) -> /UFC/UFC_BACKLIGHTING/BACKLIGHT_GND
- J11 pad 1: /TACAN/COL1 -> /UFC/UFC_BACKLIGHTING/BACKLIGHT_+12V
- J11 pad 2: /TACAN/COL2 -> /UFC/UFC_BACKLIGHTING/BACKLIGHT_GND
- J5 pad 1: unconnected-(J5-Pad1) -> /UFC/CAUTION_LED+
- J5 pad 2: unconnected-(J5-Pad2) -> /UFC/CAUTION_LED-
- J6 pad 1: unconnected-(J6-Pad1) -> /UFC/COL0
- J6 pad 2: unconnected-(J6-Pad2) -> /UFC/COL1
- J7 pad 1: Net-(D3-Pad1) -> /UFC/ROW0
- J7 pad 2: /TACAN/ROW1 -> /UFC/ROW1
- J7 pad 3: /TACAN/ROW2 -> /UFC/ROW2
- J7 pad 4: /TACAN/ROW3 -> /UFC/ROW3
- J7 pad 5: /TACAN/ROW4 -> /UFC/ROW4
- J7 pad 6: /TACAN/ROW5 -> /UFC/ROW5
- SW1 pad 1: (no net) -> /LANDING GEAR/ROW10
- SW1 pad 2: (no net) -> Net-(D1-K)
- SW1 pad 3: (no net) -> /LANDING GEAR/ROW11
- SW2 pad 1: unconnected-(SW2-Pad1) -> /LANDING GEAR/ROW12
- SW2 pad 2: unconnected-(SW2-Pad2) -> Net-(D2-K)
- SW2 pad 3: unconnected-(SW2-Pad3) -> /LANDING GEAR/ROW13
- SW3 pad 1: Net-(D1-Pad1) -> /LANDING GEAR/ROW10
- SW3 pad 2: /TACAN/ROW1 -> Net-(D4-K)
