File: A10/A10 PCBs/Forward Console Overview/UFC.kicad_sch (KiCad schematic)
At the start: 63 parts

Commit message: A10
Parts:
- removed D? (x6): D, Diode_THT:D_A-405_P7.62mm_Horizontal, symbol Device:D
- removed SW?: 0, Connector_Molex:Molex_KK-254_AE-6410-02A_1x02_P2.54mm_Vertical, symbol Switch:SW_Push
- removed SW?: 9, Connector_Molex:Molex_KK-254_AE-6410-02A_1x02_P2.54mm_Vertical, symbol Switch:SW_Push
- removed SW?: SPC, Connector_Molex:Molex_KK-254_AE-6410-02A_1x02_P2.54mm_Vertical, symbol Switch:SW_Push
- removed SW?: 3, Connector_Molex:Molex_KK-254_AE-6410-02A_1x02_P2.54mm_Vertical, symbol Switch:SW_Push
- removed SW?: POS, Connector_Molex:Molex_KK-254_AE-6410-02A_1x02_P2.54mm_Vertical, symbol Switch:SW_Push
- removed SW?: 6, Connector_Molex:Molex_KK-254_AE-6410-02A_1x02_P2.54mm_Vertical, symbol Switch:SW_Push
- added D? (x6): D, Diode_THT:D_A-405_P7.62mm_Horizontal, symbol Device:D
- added SW?: 6, Connector_Molex:Molex_KK-254_AE-6410-02A_1x02_P2.54mm_Vertical, symbol Switch:SW_Push
- added SW?: POS, Connector_Molex:Molex_KK-254_AE-6410-02A_1x02_P2.54mm_Vertical, symbol Switch:SW_Push
- added SW?: 9, Connector_Molex:Molex_KK-254_AE-6410-02A_1x02_P2.54mm_Vertical, symbol Switch:SW_Push
- added SW?: SPC, Connector_Molex:Molex_KK-254_AE-6410-02A_1x02_P2.54mm_Vertical, symbol Switch:SW_Push
- added SW?: 0, Connector_Molex:Molex_KK-254_AE-6410-02A_1x02_P2.54mm_Vertical, symbol Switch:SW_Push
- added SW?: 3, Connector_Molex:Molex_KK-254_AE-6410-02A_1x02_P2.54mm_Vertical, symbol Switch:SW_Push
Connections:
- net COL1: now reaches D?.2 (A)
- net COL1: now also D?.2 (A)
- net COL0: now reaches D?.2 (A)
- net COL0: now also D?.2 (A)
- net ROW5: now reaches SW?.2
- net ROW5: now also SW?.2
- net ROW0: now reaches SW?.2
- net ROW0: now also SW?.2
- net ROW4: now reaches SW?.2
- net ROW4: now also SW?.2
- net ROW1: now reaches SW?.2
- net ROW1: now also SW?.2
- net ROW2: now reaches SW?.2
- net ROW2: now also SW?.2
- net COL2: now reaches D?.2 (A)
- net COL2: now also D?.2 (A)
- net ROW3: now reaches SW?.2
- net ROW3: now also SW?.2
- new net: D?.1 (K), SW?.1 (x6)
- new net COL3: D?.2 (A)
- new net COL4: D?.2 (A)
- new net COL5: D?.2 (A)
- new net COL6: D?.2 (A)
- new net COL7: D?.2 (A), D?.2 (A)
Other:
- moved on the sheet: D?, SW?

Commit message: A10
Parts:
- added J?: UFC ROWS, symbol Connector:Conn_01x06_Female
- added J?: UFC COLS, symbol Connector:Conn_01x06_Female
Connections:
- net COL6 is gone; now on net COL1: D?.2 (A)
- net COL7 is gone; now on net COL1: D?.2 (A), D?.2 (A)
- net COL0: now also D?.2 (A), D?.2 (A), D?.2 (A), D?.2 (A), J?.1 (Pin_1)
- net COL1: now also D?.2 (A), D?.2 (A), D?.2 (A), J?.2 (Pin_2); no longer D?.2 (A), D?.2 (A)
- net COL2: now also D?.2 (A), D?.2 (A), D?.2 (A), D?.2 (A), D?.2 (A), D?.2 (A), J?.3 (Pin_3); no longer D?.2 (A), D?.2 (A)
- net COL3: now also D?.2 (A), D?.2 (A), D?.2 (A), D?.2 (A), D?.2 (A), D?.2 (A), J?.4 (Pin_4); no longer D?.2 (A)
- net COL4: now also D?.2 (A), D?.2 (A), D?.2 (A), D?.2 (A), D?.2 (A), D?.2 (A), J?.5 (Pin_5); no longer D?.2 (A)
- net COL5: now also D?.2 (A), J?.6 (Pin_6); no longer D?.2 (A)
- net ROW0: now also SW?.2, SW?.2, SW?.2, SW?.2, J?.1 (Pin_1)
- net ROW1: now also SW?.2, SW?.2, SW?.2, J?.2 (Pin_2)
- net ROW2: now also SW?.2, SW?.2, SW?.2, J?.3 (Pin_3)
- net ROW3: now also SW?.2, SW?.2, SW?.2, J?.4 (Pin_4)
- net ROW4: now also SW?.2, SW?.2, SW?.2, J?.5 (Pin_5)
- net ROW5: now also SW?.2, SW?.2, SW?.2, J?.6 (Pin_6)
- net at D?.1 (K): no longer SW?.1 (x2)
Other:
- moved on the sheet: D?, SW?

Commit message: a10
Parts:
- added J5: Conn_01x02_Socket, Connector_Molex:Molex_KK-254_AE-6410-02A_1x02_P2.54mm_Vertical, symbol Connector:Conn_01x02_Socket
- J6, J7: renamed from J?; footprint (none) -> Connector_Molex:Molex_KK-254_AE-6410-06A_1x06_P2.54mm_Vertical
- SW27, SW28, SW29, SW30, SW31, SW32, SW33, SW34, SW35, SW36, SW37, SW38, SW39, SW40, SW41, SW42, SW43, SW45, SW46, SW47, SW48, SW49, SW50, SW51, SW52, SW53, SW54, SW55, SW56, SW57: renamed from SW?; footprint Connector_Molex:Molex_KK-254_AE-6410-02A_1x02_P2.54mm_Vertical -> Button_Switch_THT:SW_PUSH-12mm
- gave numbers to parts that had none: 33
Connections:
- net CAUTION_LED-: now reaches D65.1 (K)
- net CAUTION_LED-: now also J5.2 (Pin_2)
- net CAUTION_LED+: now reaches D65.2 (A)
- net CAUTION_LED+: now also J5.1 (Pin_1)
Other:
- added sheet UFC_BACKLIGHTING (UFC_BACKLIGHTING.kicad_sch)
