File: A10/A10 PCBs/Forward Console Overview/NMSP CMSP.kicad_sch (KiCad schematic)
At the start: 37 parts

Commit message: A10
Parts:
- added J?: NMSP CMSP, symbol Connector:Conn_01x08_Female
Connections:
- net ROW6: now reaches SW?.2
- net ROW6: now also SW?.2, J?.3 (Pin_3)
- net COL5: now reaches D?.2 (A)
- net COL5: now also D?.2 (A), D?.2 (A), D?.2 (A), D?.2 (A), D?.2 (A), J?.2 (Pin_2)
- net COL4: now reaches D?.2 (A)
- net COL4: now also D?.2 (A), D?.2 (A), D?.2 (A), D?.2 (A), D?.2 (A), J?.1 (Pin_1)
- net ROW9: now reaches SW?.2
- net ROW9: now also SW?.2, J?.6 (Pin_6)
- net ROW10: now reaches SW?.2
- net ROW10: now also SW?.2, J?.7 (Pin_7)
- net ROW7: now reaches SW?.2
- net ROW7: now also SW?.2, J?.4 (Pin_4)
- net ROW8: now reaches SW?.2
- net ROW8: now also SW?.2 (B), J?.5 (Pin_5)
- net ROW11: now reaches SW?.2
- net ROW11: now also SW?.2, J?.8 (Pin_8)
Changed lines of the file:
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@@
 (kicad_sch (version 20211123) (generator eeschema)
   (paper "A4")
+  (label "ROW10" (at 136.652 97.536 0)
+    (effects (font (size 1.27 1.27)) (justify left bottom))
+  )
+  (label "COL5" (at 77.978 122.174 180)
+    (effects (font (size 1.27 1.27)) (justify right bottom))
+  )
+  (label "ROW8" (at 218.44 74.676 180)
+    (effects (font (size 1.27 1.27)) (justify right bottom))
+  )
+  (label "ROW8" (at 94.996 93.726 0)
+    (effects (font (size 1.27 1.27)) (justify left bottom))
+  )
+  (label "ROW6" (at 218.44 69.596 180)
+    (effects (font (size 1.27 1.27)) (justify right bottom))
+  )
+  (label "ROW7" (at 218.44 72.136 180)
+    (effects (font (size 1.27 1.27)) (justify right bottom))
+  )
+  (label "ROW10" (at 136.906 122.174 0)
+    (effects (font (size 1.27 1.27)) (justify left bottom))
+  )
+  (label "ROW11" (at 173.99 122.174 0)
+    (effects (font (size 1.27 1.27)) (justify left bottom))
+  )
+  (label "ROW9" (at 52.832 122.174 0)
+    (effects (font (size 1.27 1.27)) (justify left bottom))
+  )
+  (label "COL5" (at 76.454 48.26 180)
+    (effects (font (size 1.27 1.27)) (justify right bottom))
+  )
+  (label "COL5" (at 218.44 67.056 180)
+    (effects (font (size 1.27 1.27)) (justify right bottom))
+  )
+  (label "ROW6" (at 52.324 48.26 0)
+    (effects (font (size 1.27 1.27)) (justify left bottom))
+  )
+  (label "COL4" (at 218.44 64.516 180)
+    (effects (font (size 1.27 1.27)) (justify right bottom))
+  )
+  (label "ROW10" (at 218.44 79.756 180)
+    (effects (font (size 1.27 1.27)) (justify right bottom))
+  )
+  (label "COL5" (at 119.126 122.174 180)
+    (effects (font (size 1.27 1.27)) (justify right bottom))
+  )
+  (label "ROW6" (at 94.234 48.26 0)
+    (effects (font (size 1.27 1.27)) (justify left bottom))
+  )
+  (label "ROW7" (at 131.318 48.26 0)
+    (effects (font (size 1.27 1.27)) (justify left bottom))
+  )
+  (label "COL5" (at 156.21 122.174 180)
+    (effects (font (size 1.27 1.27)) (justify right bottom))
+  )
+  (label "COL4" (at 118.872 97.536 180)
+    (effects (font (size 1.27 1.27)) (justify right bottom))
+  )
+  (label "ROW7" (at 95.504 70.104 0)
+    (effects (font (size 1.27 1.27)) (justify left bottom))
+  )
+  (label "ROW11" (at 173.736 97.536 0)
+    (effects (font (size 1.27 1.27)) (justify left bottom))
+  )
+  (label "COL4" (at 155.956 97.536 180)
+    (effects (font (size 1.27 1.27)) (justify right bottom))
+  )
+  (label "COL4" (at 34.798 97.536 180)
+    (effects (font (size 1.27 1.27)) (justify right bottom))
+  )
+  (label "ROW11" (at 218.44 82.296 180)
+    (effects (font (size 1.27 1.27)) (justify right bottom))
+  )
+  (label "COL5" (at 77.724 70.104 180)
+    (effects (font (size 1.27 1.27)) (justify right bottom))
+  )
+  (label "COL4" (at 34.544 48.26 180)
+    (effects (font (size 1.27 1.27)) (justify right bottom))
+  )
+  (label "COL4" (at 113.538 48.26 180)
+    (effects (font (size 1.27 1.27)) (justify right bottom))
+  )
+  (label "COL5" (at 77.216 93.726 180)
+    (effects (font (size 1.27 1.27)) (justify right bottom))
+  )
+  (label "COL4" (at 35.052 122.174 180)
+    (effects (font (size 1.27 1.27)) (justify right bottom))
+  )
+  (label "ROW9" (at 218.44 77.216 180)
+    (effects (font (size 1.27 1.27)) (justify right bottom))
+  )
+  (label "ROW8" (at 52.578 97.536 0)
+    (effects (font (size 1.27 1.27)) (justify left bottom))
+  )
+  (label "ROW9" (at 95.758 122.174 0)
+    (effects (font (size 1.27 1.27)) (justify left bottom))
+  )
   (symbol (lib_id "Switch:SW_Push") (at 89.154 48.26 0) (unit 1)
     (in_bom yes) (on_board yes) (fields_autoplaced)
@@
     (pin "2")
   )
+  (symbol (lib_id "Connector:Conn_01x08_Female") (at 223.52 72.136 0) (unit 1)
+    (in_bom yes) (on_board yes) (fields_autoplaced)
+    (property "Reference" "J?" (id 0) (at 224.2312 72.5713 0)
+      (effects (font (size 1.27 1.27)) (justify left))
+    )
+    (property "Value" "NMSP CMSP" (id 1) (at 224.2312 75.1082 0)
+      (effects (font (size 1.27 1.27)) (justify left))
+    )
+    (property "Footprint" "" (id 2) (at 223.52 72.136 0)
+      (effects (font (size 1.27 1.27)) hide)
+    )
+    (property "Datasheet" "~" (id 3) (at 223.52 72.136 0)
+      (effects (font (size 1.27 1.27)) hide)
+    )
+    (pin "1")
+    (pin "2")
+    (pin "3")
+    (pin "4")
+    (pin "5")
+    (pin "6")
+    (pin "7")
+    (pin "8")
+  )
   (symbol (lib_id "Device:LED") (at 165.1 86.106 180) (unit 1)

Commit message: a10
Parts:
- D29: renamed from D?; footprint PT_Library_v001:D_Signal_P7.62mm_Horizontal -> Diode_THT:D_A-405_P7.62mm_Horizontal
- SW15, SW16, SW17, SW18, SW20, SW21, SW22, SW23, SW24, SW25, SW26: renamed from SW?; footprint Connector_Molex:Molex_KK-254_AE-6410-02A_1x02_P2.54mm_Vertical -> Button_Switch_THT:SW_PUSH-12mm
- SW19: renamed from SW?; footprint (none) -> Button_Switch_THT:SW_PUSH-12mm
- gave numbers to parts that had none: 25

Commit message: A10
Parts:
- removed D24: PRI, Connector_Molex:Molex_KK-254_AE-6410-02A_1x02_P2.54mm_Vertical, symbol Device:LED
- removed D25: HARS, Connector_Molex:Molex_KK-254_AE-6410-02A_1x02_P2.54mm_Vertical, symbol Device:LED
- removed D26: STR PT, Connector_Molex:Molex_KK-254_AE-6410-02A_1x02_P2.54mm_Vertical, symbol Device:LED
- removed D32: SEP, Connector_Molex:Molex_KK-254_AE-6410-02A_1x02_P2.54mm_Vertical, symbol Device:LED
- removed D33: MISSLE LAUNCH, Connector_Molex:Molex_KK-254_AE-6410-02A_1x02_P2.54mm_Vertical, symbol Device:LED
- removed D34: ANCHR, Connector_Molex:Molex_KK-254_AE-6410-02A_1x02_P2.54mm_Vertical, symbol Device:LED
- removed D36: SPARE, Connector_Molex:Molex_KK-254_AE-6410-02A_1x02_P2.54mm_Vertical, symbol Device:LED
- removed D39: EGI, Connector_Molex:Molex_KK-254_AE-6410-02A_1x02_P2.54mm_Vertical, symbol Device:LED
- removed D40: TCN, Connector_Molex:Molex_KK-254_AE-6410-02A_1x02_P2.54mm_Vertical, symbol Device:LED
- removed D44: TISL, Connector_Molex:Molex_KK-254_AE-6410-02A_1x02_P2.54mm_Vertical, symbol Device:LED
- removed D45: ILS, Connector_Molex:Molex_KK-254_AE-6410-02A_1x02_P2.54mm_Vertical, symbol Device:LED
- added J16: BULB_B, symbol Connector:Conn_01x06_Socket
- added J17: NMSP LED, symbol Connector:Conn_01x03_Socket
- added J2: BULB_A, symbol Connector:Conn_01x06_Socket
- added J49, J50: BKLIGHT, Connector_Molex:Molex_KK-254_AE-6410-02A_1x02_P2.54mm_Vertical, symbol Connector:Conn_01x02_Socket
- added LA4: MISSLE LAUNCH, Connector_Molex:Molex_KK-254_AE-6410-02A_1x02_P2.54mm_Vertical, symbol Device:Lamp
- added LA4: HARS, Connector_Molex:Molex_KK-254_AE-6410-02A_1x02_P2.54mm_Vertical, symbol Device:Lamp
- added LA4: EGI, Connector_Molex:Molex_KK-254_AE-6410-02A_1x02_P2.54mm_Vertical, symbol Device:Lamp
- added LA4: ANCHR, Connector_Molex:Molex_KK-254_AE-6410-02A_1x02_P2.54mm_Vertical, symbol Device:Lamp
- added LA4: PRI, Connector_Molex:Molex_KK-254_AE-6410-02A_1x02_P2.54mm_Vertical, symbol Device:Lamp
- added LA4: STR PT, Connector_Molex:Molex_KK-254_AE-6410-02A_1x02_P2.54mm_Vertical, symbol Device:Lamp
- added LA4: TISL, Connector_Molex:Molex_KK-254_AE-6410-02A_1x02_P2.54mm_Vertical, symbol Device:Lamp
- added LA4: SEP, Connector_Molex:Molex_KK-254_AE-6410-02A_1x02_P2.54mm_Vertical, symbol Device:Lamp
- added LA4: TCN, Connector_Molex:Molex_KK-254_AE-6410-02A_1x02_P2.54mm_Vertical, symbol Device:Lamp
- added LA4: ILS, Connector_Molex:Molex_KK-254_AE-6410-02A_1x02_P2.54mm_Vertical, symbol Device:Lamp
Connections:
- net at D41.1 (K): now also J17.1 (Pin_1)
- net at D41.2 (A): now also D27.2 (A), J17.2 (Pin_2)
- net at D27.1 (K): now also J17.3 (Pin_3)
- new net: J49.1 (Pin_1), J50.1 (Pin_1)
- new net: J49.2 (Pin_2), J50.2 (Pin_2)
- new net +12V: J16.1 (Pin_1), J2.1 (Pin_1), LA4.2 (+), LA4.2 (+), LA4.2 (+), LA4.2 (+), LA4.2 (+), LA4.2 (+), LA4.2 (+), LA4.2 (+), LA4.2 (+), LA4.2 (+)
- new net ANCHR: J16.4 (Pin_4), LA4.1 (-)
- new net EGI: J2.6 (Pin_6), LA4.1 (-)
- new net HARS: J2.5 (Pin_5), LA4.1 (-)
- new net ILS: J16.6 (Pin_6), LA4.1 (-)
- new net MISSLE LAUNCH: J2.4 (Pin_4), LA4.1 (-)
- new net PRI: J2.2 (Pin_2), LA4.1 (-)
- new net SEP: J2.3 (Pin_3), LA4.1 (-)
- new net STR PT: J16.3 (Pin_3), LA4.1 (-)
- new net TCN: J16.5 (Pin_5), LA4.1 (-)
- new net TISL: J16.2 (Pin_2), LA4.1 (-)
Other:
- moved on the sheet: D27
