File: A10/A10 PCBs/Forward Console Inidividual PCBS/UFC/BACKLIGHTING.kicad_sch (KiCad schematic)
At the start: 26 parts, among them J1 BKLGHT, J2 BKLGHT

Commit message: A10
Parts:
- removed D10, D11, D12, D13, D14, D15, D16, D17, D18, D19, D20, D3, D4, D5, D6, D7, D8, D9: LED, LED_THT:LED_D3.0mm_FlatTop, symbol Device:LED
- removed J1, J2: BKLGHT, Connector_Molex:Molex_KK-254_AE-6410-02A_1x02_P2.54mm_Vertical, symbol Connector:Conn_01x02_Socket
- removed R1, R2, R3, R4, R5, R6: R_US, Resistor_THT:R_Axial_DIN0207_L6.3mm_D2.5mm_P2.54mm_Vertical, symbol Device:R_US

Commit message: A10
Parts:
- added D10, D11, D12, D13, D14 (x3), D15, D16, D17, D18, D19, D20 (x3), D3, D4, D5, D6, D7, D8 (x3), D9: LED, LED_THT:LED_D3.0mm_FlatTop, symbol Device:LED
- added J2: BKLGHT, Connector_Molex:Molex_KK-254_AE-6410-02A_1x02_P2.54mm_Vertical, symbol Connector:Conn_01x02_Socket
- added R1, R2, R3, R4, R5, R6 (x3): R_US, Resistor_THT:R_Axial_DIN0207_L6.3mm_D2.5mm_P2.54mm_Vertical, symbol Device:R_US
Connections:
- new net: D12.1 (K), D18.2 (A)
- new net: D12.2 (A), D6.1 (K)
- new net: D14.1 (K), D20.2 (A) (x3)
- new net: D14.2 (A), D8.1 (K) (x3)
- new net: D8.2 (A), R6.2 (x3)
- new net: D15.2 (A), D9.1 (K)
- new net: D11.1 (K), D17.2 (A)
- new net: D11.2 (A), D5.1 (K)
- new net: D13.2 (A), D7.1 (K)
- new net: D7.2 (A), R5.2
- new net: D5.2 (A), R3.2
- new net: D10.2 (A), D4.1 (K)
- new net: D4.2 (A), R2.2
- new net: D3.1 (K), D9.2 (A)
- new net: D6.2 (A), R4.2
- new net: D3.2 (A), R1.2
- new net: D10.1 (K), D16.2 (A)
- new net: D13.1 (K), D19.2 (A)
- new net BACKLIGHT_+12V: J2.1 (Pin_1), R1.1, R2.1, R3.1, R4.1, R5.1, R6.1, R6.1, R6.1
- new net BACKLIGHT_GND: D15.1 (K), D16.1 (K), D17.1 (K), D18.1 (K), D19.1 (K), D20.1 (K), D20.1 (K), D20.1 (K), J2.2 (Pin_2)
