File: A10/A10 PCBs/Forward Console Inidividual PCBS/UFC/UFC.kicad_pcb (KiCad board)
At the start: 2 copper layers, 226.4 x 76.2 mm, 92 parts, among them J1 Conn_01x02_Socket, J2 UFC COLS, J3 UFC ROWS, J4 BKLGHT, J5 BKLGHT, SW1 STEER +, SW10 5, SW11 8, SW12 ENT, SW13 MK, SW14 3, SW15 6, SW16 9, SW17 INTEN LEFT, SW18 MASTER CAUTION, SW19 INTEN LEFT, SW2 STEER -, SW20 POS, SW21 0, SW22 SPC, SW23 INTEN RIGHT, SW24 INTEN LEFT, SW25 DATA UP, SW26 DATA DOWN, SW27 INTEN RIGHT, SW28 SEL UP, SW29 SEL DOWN, SW3 1, SW30 DEPR UP, SW31 DEPR DOWN, SW4 4, SW5 7, SW6 FUNC, SW7 LTR, SW8 CLR, SW9 2

Commit message: A10
Parts:
- removed D33, D34, D35, D36, D37, D38, D39, D40, D41, D42, D43, D44, D45, D46, D47, D48, D49, D50: LED, LED_THT:LED_D3.0mm_FlatTop
- removed J4, J5: BKLGHT, Connector_Molex:Molex_KK-254_AE-6410-02A_1x02_P2.54mm_Vertical
- removed R1, R2, R3, R4, R5, R6: R_US, Resistor_THT:R_Axial_DIN0207_L6.3mm_D2.5mm_P2.54mm_Vertical
- added D51: D, Diode_THT:D_A-405_P7.62mm_Horizontal, B.Cu at (186.8, 83.3)
- added SW32: TBA3, Button_Switch_THT:SW_PUSH-12mm, F.Cu at (169.0, 82.8)
- D1, D10, D11, D12, D13, D14, D15, D16, D17, D18, D19, D2, D21, D22, D23, D24, D25, D26, D27, D28, D29, D3, D30, D31, D32, D4, D5, D6, D7, D8, D9, J2, J3, SW18: moved to B.Cu
- D20: value MASTER CAUTION -> MASTER CAUTION LED; moved to B.Cu
- J1: value Conn_01x02_Socket -> CAUTION LED; moved to B.Cu
- SW17: value INTEN LEFT -> TBA1
- SW23: value INTEN RIGHT -> TBA2
- SW24: value INTEN LEFT -> TBA3
- moved J1 219.2 mm to (246.3, 91.2), turned to 180 degrees
- moved SW5 184.6 mm to (63.2, 89.1), turned to 90 degrees
- moved SW27 181.0 mm to (213.6, 94.2), turned to 90 degrees
- moved SW2 172.2 mm to (41.8, 75.3)
- moved SW31 168.8 mm to (239.3, 80.6), turned to 180 degrees
- moved SW11 168.7 mm to (78.6, 89.1), turned to 90 degrees
- moved SW19 165.9 mm to (198.2, 94.2), turned to 90 degrees
- moved SW4 165.5 mm to (63.2, 71.3), turned to 90 degrees
- moved D20 165.2 mm to (209.2, 45.7), turned to 180 degrees
- moved SW30 164.6 mm to (239.3, 67.9), turned to 180 degrees
- moved J2 161.1 mm to (239.1, 91.1), turned to 180 degrees
- moved SW8 159.5 mm to (126.9, 89.1), turned to 90 degrees
- moved SW28 157.7 mm to (223.2, 59.9), turned to 180 degrees
- moved SW1 155.3 mm to (41.8, 60.0)
- moved SW16 153.5 mm to (93.9, 89.1), turned to 90 degrees
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Connections:
- D13 pad 1: unconnected-(D13-K-Pad1) -> Net-(D13-K)
- D26 pad 1: unconnected-(D26-K-Pad1) -> Net-(D26-K)
- SW13 pad 1: unconnected-(SW13-Pad1) -> Net-(D13-K)
- SW25 pad 1: unconnected-(SW25-Pad1) -> Net-(D26-K)
Routing:
- net /ROW2: track 0.00 -> 299.8 mm
- net /ROW0: track 0.00 -> 298.5 mm
- net /ROW5: track 0.00 -> 253.7 mm
- net /ROW1: track 0.00 -> 250.3 mm
- net /ROW3: track 0.00 -> 248.9 mm
- net /COL2: track 0.00 -> 241.5 mm
- net /COL0: track 0.00 -> 240.8 mm
- net /ROW4: track 0.00 -> 213.2 mm, vias 0 -> 1
- net /COL1: track 0.00 -> 210.8 mm
- net /COL3: track 0.00 -> 150.1 mm
- net /COL4: track 0.00 -> 102.7 mm
- net /CAUTION_LED+: track 0.00 -> 76.8 mm
- net /CAUTION_LED-: track 0.00 -> 69.1 mm
- net /COL5: track 0.00 -> 64.4 mm
- net Net-(D26-K): track 0.00 -> 34.4 mm
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Other:
- board size 226.4 x 76.2 mm -> 226.1 x 75.5 mm

Commit message: A10
Parts:
- added D33: LED, LED_THT:LED_D3.0mm_FlatTop, F.Cu at (65.6, 93.5)
- added D34: LED, LED_THT:LED_D3.0mm_FlatTop, F.Cu at (81.1, 93.3)
- added D35: LED, LED_THT:LED_D3.0mm_FlatTop, F.Cu at (96.4, 93.4)
- added D36: LED, LED_THT:LED_D3.0mm_FlatTop, F.Cu at (111.2, 93.4)
- added D37: LED, LED_THT:LED_D3.0mm_FlatTop, F.Cu at (129.6, 93.4)
- added D38: LED, LED_THT:LED_D3.0mm_FlatTop, F.Cu at (147.4, 93.4)
- added D39: LED, LED_THT:LED_D3.0mm_FlatTop, F.Cu at (65.7, 75.2)
- added D40: LED, LED_THT:LED_D3.0mm_FlatTop, F.Cu at (81.1, 75.2)
- added D41: LED, LED_THT:LED_D3.0mm_FlatTop, F.Cu at (96.4, 75.2)
- added D42: LED, LED_THT:LED_D3.0mm_FlatTop, F.Cu at (111.0, 75.2)
- added D43: LED, LED_THT:LED_D3.0mm_FlatTop, F.Cu at (129.3, 75.2)
- added D44: LED, LED_THT:LED_D3.0mm_FlatTop, F.Cu at (147.3, 75.2)
- added D45: LED, LED_THT:LED_D3.0mm_FlatTop, F.Cu at (65.9, 57.2)
- added D46: LED, LED_THT:LED_D3.0mm_FlatTop, F.Cu at (81.1, 57.4)
- added D47: LED, LED_THT:LED_D3.0mm_FlatTop, F.Cu at (96.4, 57.4)
- added D48: LED, LED_THT:LED_D3.0mm_FlatTop, F.Cu at (111.4, 57.2)
- added D49: LED, LED_THT:LED_D3.0mm_FlatTop, F.Cu at (129.4, 57.4)
- added D50: LED, LED_THT:LED_D3.0mm_FlatTop, F.Cu at (147.3, 57.3)
- added D52: LED, LED_THT:LED_D3.0mm_FlatTop, F.Cu at (190.5, 63.9)
- added D53: LED, LED_THT:LED_D3.0mm_FlatTop, F.Cu at (207.5, 98.9)
- added D54: LED, LED_THT:LED_D3.0mm_FlatTop, F.Cu at (240.5, 72.3)
- added D55: LED, LED_THT:LED_D3.0mm_FlatTop, F.Cu at (47.0, 54.0)
- added D56: LED, LED_THT:LED_D3.0mm_FlatTop, F.Cu at (36.8, 70.1)
- added D57: LED, LED_THT:LED_D3.0mm_FlatTop, F.Cu at (46.9, 87.3)
- added J5: BKLGHT, Connector_Molex:Molex_KK-254_AE-6410-02A_1x02_P2.54mm_Vertical, B.Cu at (180.4, 96.1)
- added R1: R_US, Resistor_THT:R_Axial_DIN0207_L6.3mm_D2.5mm_P2.54mm_Vertical, B.Cu at (74.8, 92.8)
- added R2: R_US, Resistor_THT:R_Axial_DIN0207_L6.3mm_D2.5mm_P2.54mm_Vertical, B.Cu at (90.2, 92.7)
- added R3: R_US, Resistor_THT:R_Axial_DIN0207_L6.3mm_D2.5mm_P2.54mm_Vertical, B.Cu at (104.0, 92.6)
- added R4: R_US, Resistor_THT:R_Axial_DIN0207_L6.3mm_D2.5mm_P2.54mm_Vertical, B.Cu at (121.2, 92.5)
- added R5: R_US, Resistor_THT:R_Axial_DIN0207_L6.3mm_D2.5mm_P2.54mm_Vertical, B.Cu at (136.7, 92.4)
- added R6: R_US, Resistor_THT:R_Axial_DIN0207_L6.3mm_D2.5mm_P2.54mm_Vertical, B.Cu at (142.0, 92.5)
- added R7: R_US, Resistor_THT:R_Axial_DIN0207_L6.3mm_D2.5mm_P2.54mm_Vertical, B.Cu at (191.2, 90.4)
- added R8: R_US, Resistor_THT:R_Axial_DIN0207_L6.3mm_D2.5mm_P2.54mm_Vertical, B.Cu at (56.7, 88.0)
- D1, D10, D11, D12, D13, D14, D15, D16, D17, D18, D19, D2, D21, D22, D23, D24, D25, D26, D27, D28, D29, D3, D30, D31, D32, D4, D5, D51, D6, D7, D8, D9: footprint Diode_THT:D_A-405_P7.62mm_Horizontal -> Diode_THT:D_A-405_P2.54mm_Vertical_AnodeUp
- moved D18 17.6 mm to (234.6, 48.9)
- moved D31 13.8 mm to (238.2, 49.0)
- moved D26 10.8 mm to (231.1, 49.0)
- moved D32 1.04 mm to (244.0, 75.6)
- renumbered SW16 to locked
Routing:
- net /BACKLIGHTING/BACKLIGHT_GND: track 0.00 -> 283.8 mm
- net /BACKLIGHTING/BACKLIGHT_+12V: track 0.00 -> 147.2 mm
- net Net-(D53-K): track 0.00 -> 56.5 mm
- net Net-(D52-K): track 0.00 -> 54.6 mm
- net Net-(D55-A): track 0.00 -> 36.0 mm
- net Net-(D52-A): track 0.00 -> 31.0 mm
- net Net-(D43-K): track 0.00 -> 25.3 mm
- net Net-(D38-K): track 0.00 -> 25.2 mm
- net Net-(D35-K): track 0.00 -> 25.1 mm
- net Net-(D44-K): track 0.00 -> 24.8 mm
- net Net-(D39-K): track 0.00 -> 24.6 mm
- net Net-(D42-K): track 0.00 -> 24.5 mm
- net Net-(D37-K): track 0.00 -> 22.9 mm
- net Net-(D56-K): track 0.00 -> 22.4 mm
- net Net-(D33-K): track 0.00 -> 22.2 mm
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Other:
- board text added: "UFC 1.0"

Commit message: a10
Parts:
- removed D20: MASTER CAUTION LED, Connector_Molex:Molex_KK-254_AE-6410-02A_1x02_P2.54mm_Vertical
- added LA1: MASTER CAUTION LAMP, Connector_Molex:Molex_KK-254_AE-6410-02A_1x02_P2.54mm_Vertical, B.Cu at (214.6, 44.5)
- J1: value CAUTION LED -> CAUTION LAMP
Connections:
- J1 pad 1: /CAUTION_LED+ -> /CAUTION_LAMP+
- J1 pad 2: /CAUTION_LED- -> /CAUTION_LAMP-
Routing:
- net /CAUTION_LED+: track 77.4 -> 0.00 mm
- net /CAUTION_LED-: track 72.6 -> 0.00 mm
- net /CAUTION_LAMP+: track 0.00 -> 71.9 mm
- net /CAUTION_LAMP-: track 0.00 -> 66.8 mm
- net /ROW4: track 213.3 -> 252.3 mm, vias 0 -> 1
- net /ROW2: track 284.9 -> 311.8 mm, vias 0 -> 1
- net Net-(D39-K): track 24.6 -> 50.8 mm
- net /COL3: track 137.0 -> 162.6 mm
- net /ROW3: track 256.1 -> 232.1 mm
- net /ROW1: track 258.0 -> 277.0 mm, vias 0 -> 1
- net /COL4: track 96.9 -> 115.4 mm
- net Net-(D23-K): track 26.4 -> 44.3 mm
- net /COL2: track 253.9 -> 240.2 mm
- net /ROW5: track 247.7 -> 257.4 mm, vias 0 -> 1
- net Net-(D33-K): track 22.2 -> 31.1 mm
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