File: A10/A10 PCBs/Front Console 12 Stepper/Datasheets.kicad_sch (KiCad schematic)
At the start: 0 parts

Commit message: A10 12 Stepper
Other:
- title: (none) -> FRONT CONSOLE STEPPER
Changed lines of the file:
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@@
 (kicad_sch (version 20230121) (generator eeschema)
   (paper "A4")
+  (title_block
+    (title "FRONT CONSOLE STEPPER")
+    (date "2024-01-26")
+    (rev "1.2")
+  )
   (image (at 96.012 143.51)
     (data
