File: A10/A10 PCBs/Front Console Output/Front Console Output.kicad_pcb (KiCad board)
At the start: 2 copper layers, 154.7 x 53.3 mm, 49 parts, among them J1 TO LCD, J10 B/L ALT SOURCE, J11 BL OUT, J12 BL IN, J13 TO SARI PCB, J14 ROLL STEPPER, J15 VERT STEPPER, J2 STANDBY ALT, J3 VVI, J4 5V IN, J5 AIRSPEED, J6 RWR BRT, J7 STEPPER IN 12-20VDC, J8 WTR STEPPER, J9 HOZ STEPPER, P1 Power, P2 Analog, P3 Analog, P4 Digital, P5 PWM, P6 PWM, P7 Communication, Q1 IRF540N, SW1 MICRO STEP, U1 USR-ES1

Commit message: A10
Other:
- board text added: "12 Engine Steppers Airspeed (Zero Sense) Altitude (Zero Sense) VSI (Zero Sense) Compass (could be relocated to Right Console) G Meter (Could be relocated to Left Console) Clock (could be located to left console) Need to also consider SARI Holding current per coil is 14mA, which gives 28mA per stepper Mega absolute max is 40mA per pin, with a total max of 200mA Could do up to 6 steppers, which wou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"
Changed lines of the file:
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@@
     (effects (font (size 1 1) (thickness 0.15)))
+  )
+  (gr_text "12 Engine Steppers\nAirspeed (Zero Sense)\nAltitude (Zero Sense)\nVSI (Zero Sense)\nCompass (could be relocated to Right Console)\nG Meter (Could be relocated to Left Console)\nClock (could be located to left console)\n\nNeed to also consider SARI\n\nHolding current per coil is 14mA, which gives 28mA per stepper\nMega absolute max is 40mA per pin, with a total max of 200mA\nCould do up to 6 steppers, which would consume 24 pins.\n\n\n54 Digital IO Pins(of which 15 provide PWM output)\nLess two for Leds, two for UART, 5 for ethernet shield\nLeaves 47 pins\n\nAt a minimum 3 pins per stepper are needed when using driver\n1: Direction\n2: Step\n3: Sleep\n\n15 Servos gives 45 pins - not including zero position sense, \nAnalog inputs can be used as digital inputs.\n\n\n" (at 39.2 155.64) (layer "Dwgs.User")
+    (effects (font (size 1 1) (thickness 0.15)) (justify left bottom))
   )
   (group "" (id 3fd75294-da22-4e57-8fcc-45f0c43895d4)

Commit message: A10
Parts:
- removed C-H1, C-R1, C-V1: 100uF, Capacitor_THT:C_Radial_D8.0mm_H7.0mm_P3.50mm
- removed the C-W1 at (39.6, 96.9)
- removed the C-W1 at (208.6, 90.5)
- removed C1: 0.1uF, Capacitor_THT:C_Disc_D6.0mm_W2.5mm_P5.00mm
- removed D3: LED, LED_THT:LED_D3.0mm
- removed H1: H1, MountingHole:MountingHole_2.5mm
- removed H2: H2, MountingHole:MountingHole_2.5mm
- removed J4: 5V IN, Connector_BarrelJack:BarrelJack_Horizontal
- removed the J8 at (47.5, 105.5)
- removed Q1: IRF540N, Package_TO_SOT_THT:TO-220-3_Vertical
- removed R10, R7, R8, R9: 10K, Resistor_THT:R_Axial_DIN0204_L3.6mm_D1.6mm_P2.54mm_Vertical
- removed SW1: MICRO STEP, Button_Switch_THT:SW_DIP_SPSTx08_Slide_9.78x22.5mm_W7.62mm_P2.54mm
- added C-W1: 100uF, Capacitor_THT:C_Radial_D8.0mm_H7.0mm_P3.50mm, F.Cu at (214.3, 70.9)
- added C-W2: 100uF, Capacitor_THT:C_Radial_D8.0mm_H7.0mm_P3.50mm, F.Cu at (165.8, 146.8)
- added C-W3: 100uF, Capacitor_THT:C_Radial_D8.0mm_H7.0mm_P3.50mm, F.Cu at (147.7, 100.6)
- added C-W4: 100uF, Capacitor_THT:C_Radial_D8.0mm_H7.0mm_P3.50mm, F.Cu at (181.7, 146.9)
- added C-W5: 100uF, Capacitor_THT:C_Radial_D8.0mm_H7.0mm_P3.50mm, F.Cu at (214.7, 94.2)
- added C-W6: 100uF, Capacitor_THT:C_Radial_D8.0mm_H7.0mm_P3.50mm, F.Cu at (198.6, 146.8)
- added C-W7: 100uF, Capacitor_THT:C_Radial_D8.0mm_H7.0mm_P3.50mm, F.Cu at (214.9, 146.7)
- added J16: 7_MS2, Connector_PinHeader_2.54mm:PinHeader_1x02_P2.54mm_Vertical, F.Cu at (218.5, 60.4)
- added J17: STEPPER_8, Connector_Molex:Molex_KK-254_AE-6410-04A_1x04_P2.54mm_Vertical, F.Cu at (197.7, 59.5)
- added J18: 8_MS1, Connector_PinHeader_2.54mm:PinHeader_1x02_P2.54mm_Vertical, F.Cu at (214.0, 83.8)
- added J19: STEPPER_8, Module:Pololu_Breakout-16_15.2x20.3mm, F.Cu at (209.9, 81.4)
- added J20: 8_MS2, Connector_PinHeader_2.54mm:PinHeader_1x02_P2.54mm_Vertical, F.Cu at (218.7, 83.8)
- added J21: 10_MS1, Connector_PinHeader_2.54mm:PinHeader_1x02_P2.54mm_Vertical, F.Cu at (165.0, 136.5)
- added J22: STEPPER_10, Module:Pololu_Breakout-16_15.2x20.3mm, F.Cu at (160.9, 134.2)
- added J23: 10_MS2, Connector_PinHeader_2.54mm:PinHeader_1x02_P2.54mm_Vertical, F.Cu at (169.7, 136.5)
- added J24: STEPPER_10, Connector_Molex:Molex_KK-254_AE-6410-04A_1x04_P2.54mm_Vertical, F.Cu at (163.3, 126.2)
- added J25: STEPPER_11, Connector_Molex:Molex_KK-254_AE-6410-04A_1x04_P2.54mm_Vertical, F.Cu at (179.3, 126.3)
- added J26: STEPPER_12, Connector_Molex:Molex_KK-254_AE-6410-04A_1x04_P2.54mm_Vertical, F.Cu at (196.4, 126.2)
- added J27: STEPPER_13, Connector_Molex:Molex_KK-254_AE-6410-04A_1x04_P2.54mm_Vertical, F.Cu at (213.6, 127.6)
- added J28: 11_MS1, Connector_PinHeader_2.54mm:PinHeader_1x02_P2.54mm_Vertical, F.Cu at (181.4, 136.4)
- added J29: STEPPER_11, Module:Pololu_Breakout-16_15.2x20.3mm, F.Cu at (177.2, 134.0)
- added J30: 11_MS2, Connector_PinHeader_2.54mm:PinHeader_1x02_P2.54mm_Vertical, F.Cu at (186.0, 136.4)
- added J31: 12_MS1, Connector_PinHeader_2.54mm:PinHeader_1x02_P2.54mm_Vertical, F.Cu at (197.9, 136.1)
- added J32: STEPPER_12, Module:Pololu_Breakout-16_15.2x20.3mm, F.Cu at (193.9, 134.0)
- added J33: 12_MS2, Connector_PinHeader_2.54mm:PinHeader_1x02_P2.54mm_Vertical, F.Cu at (202.5, 136.1)
- added J34: 13_MS1, Connector_PinHeader_2.54mm:PinHeader_1x02_P2.54mm_Vertical, F.Cu at (214.6, 135.8)
- added J35: STEPPER_13, Module:Pololu_Breakout-16_15.2x20.3mm, F.Cu at (210.3, 134.0)
- added J36: 13_MS2, Connector_PinHeader_2.54mm:PinHeader_1x02_P2.54mm_Vertical, F.Cu at (219.5, 135.8)
- added R12: 10K, Resistor_THT:R_Axial_DIN0204_L3.6mm_D1.6mm_P2.54mm_Vertical, F.Cu at (185.1, 88.1)
- added R13: 10K, Resistor_THT:R_Axial_DIN0204_L3.6mm_D1.6mm_P2.54mm_Vertical, F.Cu at (185.1, 91.3)
- added R14: 10K, Resistor_THT:R_Axial_DIN0204_L3.6mm_D1.6mm_P2.54mm_Vertical, F.Cu at (185.1, 94.4)
- added R15: 10K, Resistor_THT:R_Axial_DIN0204_L3.6mm_D1.6mm_P2.54mm_Vertical, F.Cu at (185.1, 97.6)
- J1: value TO LCD -> STEPPER_9; footprint Connector_USB:USB_A_Molex_67643_Horizontal -> Connector_Molex:Molex_KK-254_AE-6410-04A_1x04_P2.54mm_Vertical
- J10: value B/L ALT SOURCE -> STEPPER_5; footprint Connector_PinHeader_2.54mm:PinHeader_1x02_P2.54mm_Vertical -> Connector_Molex:Molex_KK-254_AE-6410-04A_1x04_P2.54mm_Vertical
- J11: value BL OUT -> STEPPER_6; footprint Connector_Molex:Molex_Mini-Fit_Jr_5566-04A_2x02_P4.20mm_Vertical -> Connector_Molex:Molex_KK-254_AE-6410-04A_1x04_P2.54mm_Vertical
- J12: value BL IN -> 9_MS2; footprint Connector_Molex:Molex_Mini-Fit_Jr_5566-04A_2x02_P4.20mm_Vertical -> Connector_PinHeader_2.54mm:PinHeader_1x02_P2.54mm_Vertical
- J13: value TO SARI PCB -> STEPPER_7; footprint Connector_IDC:IDC-Header_2x20_P2.54mm_Vertical -> Connector_Molex:Molex_KK-254_AE-6410-04A_1x04_P2.54mm_Vertical
- J14: value ROLL STEPPER -> 7_MS1; footprint Module:Pololu_Breakout-16_15.2x20.3mm -> Connector_PinHeader_2.54mm:PinHeader_1x02_P2.54mm_Vertical
- J15: value VERT STEPPER -> STEPPER_7
- J2: value STANDBY ALT -> STEPPER_1; footprint Connector_IDC:IDC-Header_2x07_P2.54mm_Vertical -> Connector_Molex:Molex_KK-254_AE-6410-04A_1x04_P2.54mm_Vertical
- J3: value VVI -> STEPPER_2; footprint Connector_JST:JST_XH_B10B-XH-A_1x10_P2.50mm_Vertical -> Connector_Molex:Molex_KK-254_AE-6410-04A_1x04_P2.54mm_Vertical
- J5: value AIRSPEED -> STEPPER_3; footprint Connector_JST:JST_XH_B10B-XH-A_1x10_P2.50mm_Vertical -> Connector_Molex:Molex_KK-254_AE-6410-04A_1x04_P2.54mm_Vertical
- J6: value RWR BRT -> STEPPER_4; footprint Connector_JST:JST_XH_B3B-XH-A_1x03_P2.50mm_Vertical -> Connector_Molex:Molex_KK-254_AE-6410-04A_1x04_P2.54mm_Vertical
- J8: value WTR STEPPER -> 9_MS1; footprint Module:Pololu_Breakout-16_15.2x20.3mm -> Connector_PinHeader_2.54mm:PinHeader_1x02_P2.54mm_Vertical
- J9: value HOZ STEPPER -> STEPPER_9
- R3: value 500 -> 10K
- R5: value 220 -> 10K
- moved J11 119.9 mm to (151.9, 65.4), turned to 0 degrees
- moved J10 116.2 mm to (151.9, 58.4), turned to 0 degrees
- moved J2 98.6 mm to (128.2, 58.4), turned to 0 degrees
- moved R5 93.8 mm to (185.1, 81.8)
- moved R6 90.3 mm to (185.1, 85.0), turned to 0 degrees
- moved J15 68.7 mm to (209.8, 58.1), turned to 0 degrees
- moved J1 61.8 mm to (188.9, 112.1), turned to 90 degrees
- moved J5 60.5 mm to (140.0, 58.5)
- moved J3 54.0 mm to (128.2, 65.4)
- moved J12 52.3 mm to (218.5, 108.4), turned to 0 degrees
- moved J14 52.3 mm to (213.9, 60.4), turned to 0 degrees
- moved J6 45.9 mm to (140.0, 65.4), turned to 0 degrees
- moved R3 41.3 mm to (185.1, 78.7), turned to 0 degrees
- moved J13 28.2 mm to (185.2, 59.4), turned to 0 degrees
- moved J9 24.0 mm to (209.8, 106.2), turned to 0 degrees
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Connections:
- J1 pad 1: /LOWER_OUTPUT_5V -> /STEPPER_9_D
- J1 pad 2: unconnected-(J1-Pad2) -> /STEPPER_9_C
- J1 pad 3: unconnected-(J1-Pad3) -> /STEPPER_9_B
- J1 pad 4: GNDD -> /STEPPER_9_A
- J10 pad 1: /LED_DATA_IN -> /STEPPER_5_D
- J10 pad 2: /ALT_B/L -> /STEPPER_5_C
- J11 pad 1: /LED+5V -> /STEPPER_6_D
- J11 pad 2: /LED+5V -> /STEPPER_6_C
- J11 pad 3: GNDD -> /STEPPER_6_B
- J11 pad 4: /LED_DATA_OUT -> /STEPPER_6_A
- J12 pad 1: /LED+5V -> +5VL
- J12 pad 2: /LED+5V -> /9_MS2
- J13 pad 1: /ROLL_1B -> /STEPPER_7_D
- J13 pad 2: /WL_1A -> /STEPPER_7_C
- J13 pad 3: /ROLL_1A -> /STEPPER_7_B
- J13 pad 4: /WL_1B -> /STEPPER_7_A
- J14 pad 1: /ROLL_EN -> +5VL
- J14 pad 2: /ROLL_MS1 -> /7_MS1
- J15 pad 1: /VER_EN -> /7_EN
- J15 pad 10: /LOWER_OUTPUT_5V -> +5VL
- J15 pad 11: /VER_2B -> /STEPPER_7_A
- J15 pad 12: /VER_2A -> /STEPPER_7_B
- J15 pad 13: /VER_1A -> /STEPPER_7_C
- J15 pad 14: /VER_1B -> /STEPPER_7_D
- J15 pad 16: /HOZ_STEP_V+ -> /ROLL_STEP_V+
- J15 pad 2: /VER_MS1 -> /7_MS1
- J15 pad 3: /VER_MS2 -> /7_MS2
- J15 pad 7: /VER_STEP -> /7_STEP
- J15 pad 8: /VER_DIR -> /7_DIR
- J2 pad 1: /LED_DATA_LOOP_1 -> /STEPPER_1_D
- J2 pad 2: /SCL -> /STEPPER_1_C
- J2 pad 3: /ALT_COIL_C -> /STEPPER_1_B
- J2 pad 4: /SDA -> /STEPPER_1_A
- J3 pad 1: /LED_DATA_LOOP_1 -> /STEPPER_2_D
- J3 pad 2: /LED_DATA_LOOP_2 -> /STEPPER_2_C
- J3 pad 3: /VVI_ZERO_DET -> /STEPPER_2_B
- J3 pad 4: /VVI_COIL_A -> /STEPPER_2_A
- J5 pad 1: /LED_DATA_LOOP_2 -> /STEPPER_3_D
- J5 pad 2: /LED_DATA_LOOP_3 -> /STEPPER_3_C
- J5 pad 3: /AIR_ZERO_DET -> /STEPPER_3_B
- J5 pad 4: /AIR_COIL_A -> /STEPPER_3_A
- J6 pad 1: /LOWER_OUTPUT_5V -> /STEPPER_4_D
- J6 pad 2: /RWR_BRT_ANA -> /STEPPER_4_C
- J6 pad 3: GNDD -> /STEPPER_4_B
- J7 pad 1: /HOZ_STEP_V+ -> /ROLL_STEP_V+
- J8 pad 1: /WL_EN -> +5VL
- J8 pad 2: /WL_MS1 -> /9_MS1
- J9 pad 1: /HOZ_EN -> /9_EN
- J9 pad 10: /LOWER_OUTPUT_5V -> +5VL
- J9 pad 11: /HOZ_2B -> /STEPPER_9_A
- J9 pad 12: /HOZ_2A -> /STEPPER_9_B
- J9 pad 13: /HOZ_1A -> /STEPPER_9_C
- J9 pad 14: /HOZ_1B -> /STEPPER_9_D
- J9 pad 16: /HOZ_STEP_V+ -> /ROLL_STEP_V+
- J9 pad 2: /HOZ_MS1 -> /9_MS1
- J9 pad 3: /HOZ_MS2 -> /9_MS2
- J9 pad 7: /HOZ_STEP -> /9_STEP
- J9 pad 8: /HOZ_DIR -> /9_DIR
- P2 pad 1: /RWR_BRT_ANA -> unconnected-(P2-Pin_1-Pad1)
- P3 pad 5: /TEST_PUSH -> unconnected-(P3-Pin_5-Pad5)
- P3 pad 6: /ENCODER_PUSH -> unconnected-(P3-Pin_6-Pad6)
- P3 pad 7: /AIR_ZERO_DET -> unconnected-(P3-Pin_7-Pad7)
- P3 pad 8: /VVI_ZERO_DET -> unconnected-(P3-Pin_8-Pad8)
- P4 pad 10: /ROLL_STEP -> unconnected-(P4-Pin_10-Pad10)
- P4 pad 11: /ALT_COIL_B -> /9_EN
- P4 pad 12: /ROLL_DIR -> /13_DIR
- P4 pad 13: /ALT_COIL_A -> /8_DIR
- P4 pad 14: /HOZ_EN -> /13_STEP
- P4 pad 15: /ALT_COIL_D -> /8_STEP
- P4 pad 16: /HOZ_STEP -> /13_EN
- P4 pad 17: /ALT_COIL_C -> /8_EN
- P4 pad 18: /HOZ_DIR -> /12_DIR
- P4 pad 19: /VVI_COIL_D -> /7_DIR
- P4 pad 20: /VER_EN -> /12_STEP
- P4 pad 21: /VVI_COIL_C -> /7_STEP
- P4 pad 22: /VER_STEP -> /12_EN
- P4 pad 23: /VVI_COIL_B -> /7_EN
- P4 pad 24: /VER_DIR -> /11_DIR
- P4 pad 25: /VVI_COIL_A -> /STEPPER_6_D
- P4 pad 26: /WL_DIR -> /11_STEP
- P4 pad 27: /ENCODER_A -> /STEPPER_6_C
- P4 pad 28: /WL_STEP -> /11_EN
- P4 pad 29: /ENCODER_B -> /STEPPER_6_B
- P4 pad 30: /WL_EN -> /10_DIR
- P4 pad 31: /HOZ_ZERO_IR -> /STEPPER_6_A
- P4 pad 32: /VER_ZERO_IR -> /10_STEP
- P4 pad 33: /ROLL_ZERO_IR -> /STEPPER_5_D
- P4 pad 34: /WL_ZERO_IR -> /10_EN
- P4 pad 7: /ALT_ENC_A -> /9_DIR
- P4 pad 8: /ROLL_EN -> unconnected-(P4-Pin_8-Pad8)
- P4 pad 9: /ALT_ENC_B -> /9_STEP
- P5 pad 3: unconnected-(P5-Pad3) -> /STEPPER_1_A
- P5 pad 4: unconnected-(P5-Pad4) -> /STEPPER_1_B
- P5 pad 5: unconnected-(P5-Pad5) -> /STEPPER_1_C
- P6 pad 1: /SERVO_PITCH -> /STEPPER_1_D
- P6 pad 2: unconnected-(P6-Pad2) -> /STEPPER_2_A
- P6 pad 3: /FLAG_PIN -> /STEPPER_2_B
- P6 pad 4: unconnected-(P6-Pad4) -> /STEPPER_2_C
- P6 pad 5: unconnected-(P6-Pad5) -> /STEPPER_2_D
- P6 pad 6: /ALT_B/L_UPPER -> /STEPPER_3_A
- P6 pad 7: /ALT_B/L -> /STEPPER_3_B
- P6 pad 8: unconnected-(P6-Pad8) -> /STEPPER_3_C
- P7 pad 1: /AIR_COIL_A -> /STEPPER_3_D
- P7 pad 2: /AIR_COIL_B -> /STEPPER_4_A
- P7 pad 3: /AIR_COIL_C -> /STEPPER_4_B
- P7 pad 4: /AIR_COIL_D -> /STEPPER_4_C
- P7 pad 5: /ALT_ZERO_DET -> /STEPPER_4_D
- P7 pad 6: unconnected-(P7-Pad6) -> /STEPPER_5_A
- P7 pad 7: /SDA -> /STEPPER_5_B
- P7 pad 8: /SCL -> /STEPPER_5_C
- R3 pad 1: /LOWER_OUTPUT_5V -> +5VL
- R3 pad 2: Net-(D3-Pad2) -> /7_EN
- R4 pad 1: /HOZ_STEP_V+ -> /ROLL_STEP_V+
- R5 pad 1: /FLAG_PIN -> +5VL
- R5 pad 2: Net-(Q1-Pad1) -> /8_EN
- R6 pad 1: Net-(Q1-Pad1) -> +5VL
- R6 pad 2: GNDD -> /9_EN
Routing:
- net GNDD: track 0.00 -> 420.0 mm, vias 0 -> 1
- net +5VL: track 0.00 -> 349.0 mm, vias 0 -> 1
- net /ROLL_STEP_V+: track 0.00 -> 294.6 mm, vias 0 -> 1
- net /10_STEP: track 0.00 -> 102.7 mm, vias 0 -> 1
- net /10_DIR: track 0.00 -> 102.3 mm, vias 0 -> 3
- net /10_EN: track 0.00 -> 97.5 mm
- net /11_DIR: track 0.00 -> 87.3 mm
- net MOSI: track 0.00 -> 83.6 mm
- net SS: track 0.00 -> 81.4 mm
- net SCLK: track 0.00 -> 81.0 mm, vias 0 -> 1
- net /11_STEP: track 0.00 -> 78.2 mm
- net Net-(U1-INT): track 0.00 -> 70.6 mm
- net ES1_RST: track 0.00 -> 65.8 mm
- net /12_DIR: track 0.00 -> 64.8 mm
- net /11_EN: track 0.00 -> 64.3 mm
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Other:
- board size 154.7 x 53.3 mm -> 99.8 x 99.5 mm
- board text removed: "### ENSURE CURRENT LIMITS ARE SET FOR STEPPERS ###"
- board text removed: "(MS3) NOT USED"
- board text removed: "1/2"
- board text removed: "1/4"
- board text removed: "1/8"
- board text removed: "2"
- board text removed: "500R"
- board text removed: "5V"
- board text removed: "5V IN"
- board text removed: "5V LCD OUT"
- board text removed: "5V OK"
- board text removed: "ADD DIODE AT SOLENOID"
- board text removed: "B/L LED"
- board text removed: "B/L LOOP"
- board text removed: "BRT"
- board text removed: "DIODE"
- board text removed: "EN"
- board text removed: "FLAG SWITCH"
- board text removed: "FULL"
- board text removed: "GND"
- board text removed: "HOZ"
- board text removed: "HOZ STEPPER"
- board text removed: "IMPORTANT ADD 1N5408 DIODE AT SOLENOID"
- board text removed: "LCD PWR OUT"
- board text removed: "N/C"
- board text removed: "OFF"
- board text removed: "ON"
- board text removed: "RJ45 PORT"
- board text removed: "ROLL"
- board text removed: "ROLL STEPPER"
- board text removed: "SIG"
- board text removed: "STANDBY/SARI INST ETHER SHIELD OZ HORNET"
- board text removed: "STEP A"
- board text removed: "STEP B"
- board text removed: "STEP C"
- board text removed: "STEP D"
- board text removed: "TOP VIEW"
- board text removed: "USE A4988 STEPPER DRIVER"
- board text removed: "USR-ES1 ETHERNET MODULE"
- board text removed: "V002"
- board text removed: "VERT"
- board text removed: "VERT STEPPER"
- board text removed: "WTR"
- board text removed: "WTR STEPPER"
- board text removed: "ZERO"

Commit message: A10
Parts:
- added J37: ZERO DETECT_2, Connector_Molex:Molex_KK-254_AE-6410-03A_1x03_P2.54mm_Vertical, F.Cu at (161.3, 92.7)
- added J38: ZERO DETECT_3, Connector_Molex:Molex_KK-254_AE-6410-03A_1x03_P2.54mm_Vertical, F.Cu at (161.3, 102.2)
- added J39: ZERO DETECT_4, Connector_Molex:Molex_KK-254_AE-6410-03A_1x03_P2.54mm_Vertical, F.Cu at (161.3, 111.8)
- added J4: ZERO DETECT_1, Connector_Molex:Molex_KK-254_AE-6410-03A_1x03_P2.54mm_Vertical, F.Cu at (161.3, 83.2)
- added J41: PWM, Connector_PinSocket_2.54mm:PinSocket_1x08_P2.54mm_Vertical, F.Cu at (149.2, 76.2)
- added J42: Communication, Connector_PinSocket_2.54mm:PinSocket_1x08_P2.54mm_Vertical, F.Cu at (172.1, 76.2)
- added J43: Analog, Connector_PinSocket_2.54mm:PinSocket_1x08_P2.54mm_Vertical, F.Cu at (154.3, 123.2)
- added J44: Analog, Connector_PinSocket_2.54mm:PinSocket_1x08_P2.54mm_Vertical, F.Cu at (177.2, 123.2)
- added J45: Power, Connector_PinSocket_2.54mm:PinSocket_1x08_P2.54mm_Vertical, F.Cu at (131.4, 123.2)
- added P8: PWM, Socket_Arduino_Mega:Socket_Strip_Arduino_1x08, F.Cu at (127.0, 76.2)
- moved R11 19.9 mm to (136.7, 98.0)
- moved R2 19.9 mm to (136.7, 93.0)
- moved R1 19.9 mm to (136.7, 89.3)
- moved D1 18.7 mm to (130.2, 92.1)
- moved D2 18.7 mm to (130.2, 97.6)
- moved J24 9.38 mm to (154.3, 128.9)
- moved R12 8.08 mm to (177.2, 89.5)
- moved R13 8.08 mm to (177.2, 92.6)
- moved R14 8.08 mm to (177.2, 95.8)
- moved R15 8.08 mm to (177.2, 98.9)
- moved R3 8.08 mm to (177.2, 80.0)
- moved R5 8.08 mm to (177.2, 83.2)
- moved R6 8.08 mm to (177.2, 86.3)
- moved J7 3.07 mm to (136.0, 107.2)
- moved J25 2.86 mm to (180.3, 128.9)
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Connections:
- net /GREEN_LED renamed /*9
- net /RED_LED renamed /*8
- net /STEPPER_1_A renamed /*13
- net /STEPPER_1_B renamed /*12
- net /STEPPER_1_C renamed /*11
- net /STEPPER_1_D renamed /*7
- net /STEPPER_2_A renamed /*6
- net /STEPPER_2_B renamed /*5
- net /STEPPER_2_C renamed /*4
- net /STEPPER_2_D renamed /*3
- net /STEPPER_3_A renamed /*2
- net /STEPPER_3_C renamed /RX0/0
- net /STEPPER_4_A renamed /RX3/15
- net /STEPPER_4_C renamed /RX2/17
- net /STEPPER_5_A renamed /RX1/19
- net /STEPPER_5_B renamed /SDA/20
- net /STEPPER_5_C renamed /SCL/21
- net GNDD renamed GND
- P1 pad 8: /Vin -> VCC
- P2 pad 1: unconnected-(P2-Pin_1-Pad1) -> /A0
- P2 pad 2: unconnected-(P2-Pin_2-Pad2) -> /A1
- P2 pad 3: unconnected-(P2-Pin_3-Pad3) -> /A2
- P2 pad 4: unconnected-(P2-Pin_4-Pad4) -> /A3
- P2 pad 5: unconnected-(P2-Pin_5-Pad5) -> /A4
- P2 pad 6: unconnected-(P2-Pin_6-Pad6) -> /A5
- P2 pad 7: unconnected-(P2-Pin_7-Pad7) -> /A6
- P2 pad 8: unconnected-(P2-Pin_8-Pad8) -> /A7
- P3 pad 1: unconnected-(P3-Pin_1-Pad1) -> /A8
- P3 pad 2: unconnected-(P3-Pin_2-Pad2) -> /A9
- P3 pad 3: unconnected-(P3-Pin_3-Pad3) -> /A10
- P3 pad 4: unconnected-(P3-Pin_4-Pad4) -> /A11
- P3 pad 5: unconnected-(P3-Pin_5-Pad5) -> /A12
- P3 pad 6: unconnected-(P3-Pin_6-Pad6) -> /A13
- P3 pad 7: unconnected-(P3-Pin_7-Pad7) -> /A14
- P3 pad 8: unconnected-(P3-Pin_8-Pad8) -> /A15
- P5 pad 1: unconnected-(P5-Pin_1-Pad1) -> /AREF
Routing:
- net /A0: track 0.00 -> 44.8 mm
- net /A1: track 0.00 -> 34.2 mm
- net GND: track 420.0 -> 452.2 mm, vias 1 -> 0
- net /10_STEP: track 102.7 -> 126.7 mm, vias 1 -> 0
- net /A2: track 0.00 -> 23.6 mm
- net +5VL: track 349.0 -> 370.1 mm, vias 1 -> 0
- net Net-(U1-INT): track 70.6 -> 51.9 mm
- net /ROLL_STEP_V+: track 294.6 -> 276.2 mm, vias 1 -> 0
- net +3V3: track 50.9 -> 33.3 mm
- net /STEPPER_3_B: track 28.6 -> 44.4 mm
- net /*8: track 11.1 -> 25.6 mm
- net /10_EN: track 97.5 -> 83.8 mm, vias 0 -> 1
- net /A3: track 0.00 -> 13.0 mm
- net /STEPPER_7_B: track 50.9 -> 38.1 mm
- net /*3: track 34.9 -> 46.8 mm
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Other:
- board text added: "STEPPER V1.0"

Commit message: A10
Parts:
- removed J12: 9_MS2, Connector_PinHeader_2.54mm:PinHeader_1x02_P2.54mm_Vertical
- removed J14: 7_MS1, Connector_PinHeader_2.54mm:PinHeader_1x02_P2.54mm_Vertical
- removed J15: STEPPER_7, Module:Pololu_Breakout-16_15.2x20.3mm
- removed J16: 7_MS2, Connector_PinHeader_2.54mm:PinHeader_1x02_P2.54mm_Vertical
- removed J18: 8_MS1, Connector_PinHeader_2.54mm:PinHeader_1x02_P2.54mm_Vertical
- removed J19: STEPPER_8, Module:Pololu_Breakout-16_15.2x20.3mm
- removed J21: 10_MS1, Connector_PinHeader_2.54mm:PinHeader_1x02_P2.54mm_Vertical
- removed J22: STEPPER_10, Module:Pololu_Breakout-16_15.2x20.3mm
- removed J23: 10_MS2, Connector_PinHeader_2.54mm:PinHeader_1x02_P2.54mm_Vertical
- removed J28: 11_MS1, Connector_PinHeader_2.54mm:PinHeader_1x02_P2.54mm_Vertical
- removed J29: STEPPER_11, Module:Pololu_Breakout-16_15.2x20.3mm
- removed J30: 11_MS2, Connector_PinHeader_2.54mm:PinHeader_1x02_P2.54mm_Vertical
- removed J31: 12_MS1, Connector_PinHeader_2.54mm:PinHeader_1x02_P2.54mm_Vertical
- removed J32: STEPPER_12, Module:Pololu_Breakout-16_15.2x20.3mm
- removed J33: 12_MS2, Connector_PinHeader_2.54mm:PinHeader_1x02_P2.54mm_Vertical
- removed J34: 13_MS1, Connector_PinHeader_2.54mm:PinHeader_1x02_P2.54mm_Vertical
- removed J35: STEPPER_13, Module:Pololu_Breakout-16_15.2x20.3mm
- removed J36: 13_MS2, Connector_PinHeader_2.54mm:PinHeader_1x02_P2.54mm_Vertical
- removed J37: ZERO DETECT_2, Connector_Molex:Molex_KK-254_AE-6410-03A_1x03_P2.54mm_Vertical
- removed J38: ZERO DETECT_3, Connector_Molex:Molex_KK-254_AE-6410-03A_1x03_P2.54mm_Vertical
- removed J39: ZERO DETECT_4, Connector_Molex:Molex_KK-254_AE-6410-03A_1x03_P2.54mm_Vertical
- removed J4: ZERO DETECT_1, Connector_Molex:Molex_KK-254_AE-6410-03A_1x03_P2.54mm_Vertical
- removed J8: 9_MS1, Connector_PinHeader_2.54mm:PinHeader_1x02_P2.54mm_Vertical
- removed J9: STEPPER_9, Module:Pololu_Breakout-16_15.2x20.3mm
- removed R12, R13, R14, R15, R3, R5, R6: 10K, Resistor_THT:R_Axial_DIN0204_L3.6mm_D1.6mm_P2.54mm_Vertical
Connections:
- net /ROLL_STEP_V+ renamed /STEP_V+
- J10 pad 1: /STEPPER_5_D -> /SCL/21
- J10 pad 2: /SCL/21 -> /SDA/20
- J10 pad 3: /SDA/20 -> /RX1/19
- J10 pad 4: /RX1/19 -> /STEPPER_5_A
- J2 pad 1: /*7 -> /*9
- J3 pad 1: /*3 -> /*4
- J3 pad 2: /*4 -> /*5
- J3 pad 3: /*5 -> /*6
- J3 pad 4: /*6 -> /*7
- J41 pad 7: /STEPPER_3_B -> /STEPPER_3_C
- J42 pad 1: /STEPPER_3_D -> /STEPPER_4_A
- J42 pad 3: /STEPPER_4_B -> /STEPPER_4_C
- J42 pad 5: /STEPPER_4_D -> /STEPPER_5_A
- J5 pad 1: /STEPPER_3_D -> /RX0/0
- J5 pad 2: /RX0/0 -> /STEPPER_3_C
- J5 pad 3: /STEPPER_3_B -> /*2
- J5 pad 4: /*2 -> /*3
- J6 pad 1: /STEPPER_4_D -> /RX2/17
- J6 pad 2: /RX2/17 -> /STEPPER_4_C
- J6 pad 3: /STEPPER_4_B -> /RX3/15
- J6 pad 4: /RX3/15 -> /STEPPER_4_A
- P4 pad 10: unconnected-(P4-Pin_10-Pad10) -> /STEPPER_11_A
- P4 pad 11: /9_EN -> /STEPPER_8_D
- P4 pad 12: /13_DIR -> /STEPPER_11_D
- P4 pad 13: /8_DIR -> /STEPPER_8_C
- P4 pad 14: /13_STEP -> /STEPPER_11_C
- P4 pad 15: /8_STEP -> /STEPPER_8_B
- P4 pad 16: /13_EN -> /STEPPER_11_B
- P4 pad 17: /8_EN -> /STEPPER_8_A
- P4 pad 18: /12_DIR -> /STEPPER_11_A
- P4 pad 19: /7_DIR -> /STEPPER_7_D
- P4 pad 20: /12_STEP -> /STEPPER_10_D
- P4 pad 21: /7_STEP -> /STEPPER_7_C
- P4 pad 22: /12_EN -> /STEPPER_10_C
- P4 pad 23: /7_EN -> /STEPPER_7_B
- P4 pad 24: /11_DIR -> /STEPPER_10_B
- P4 pad 25: /STEPPER_6_D -> /STEPPER_7_A
- P4 pad 26: /11_STEP -> /STEPPER_10_A
- P4 pad 27: /STEPPER_6_C -> /STEPPER_6_D
- P4 pad 28: /11_EN -> /STEPPER_9_D
- P4 pad 29: /STEPPER_6_B -> /STEPPER_6_C
- P4 pad 30: /10_DIR -> /STEPPER_9_C
- P4 pad 31: /STEPPER_6_A -> /STEPPER_6_B
- P4 pad 32: /10_STEP -> /STEPPER_9_B
- P4 pad 33: /STEPPER_5_D -> /STEPPER_6_A
- P4 pad 34: /10_EN -> /STEPPER_9_A
- P4 pad 7: /9_DIR -> /STEPPER_11_D
- P4 pad 8: unconnected-(P4-Pin_8-Pad8) -> /STEPPER_11_B
- P4 pad 9: /9_STEP -> /STEPPER_11_C
- P6 pad 7: /STEPPER_3_B -> /STEPPER_3_C
- P7 pad 1: /STEPPER_3_D -> /STEPPER_4_A
- P7 pad 3: /STEPPER_4_B -> /STEPPER_4_C
- P7 pad 5: /STEPPER_4_D -> /STEPPER_5_A
- R1 pad 1: /*9 -> /GREEN_LED
Routing:
- net GND: track 452.2 -> 0.00 mm
- net +5VL: track 370.1 -> 0.00 mm
- net /STEP_V+: track 276.2 -> 0.00 mm
- net /10_STEP: track 126.7 -> 0.00 mm
- net /10_DIR: track 99.6 -> 0.00 mm
- net MOSI: track 88.6 -> 0.00 mm
- net /11_DIR: track 88.2 -> 0.00 mm
- net /10_EN: track 83.8 -> 0.00 mm, vias 1 -> 0
- net SS: track 83.5 -> 0.00 mm
- net /11_STEP: track 80.2 -> 0.00 mm, vias 1 -> 0
- net SCLK: track 77.0 -> 0.00 mm
- net /11_EN: track 67.9 -> 0.00 mm
- net ES1_RST: track 66.7 -> 0.00 mm
- net /12_DIR: track 66.2 -> 0.00 mm
- net /12_STEP: track 65.8 -> 0.00 mm
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Other:
- board text added: "STEPPER V1.1"
- board text removed: "STEPPER V1.0"
