File: A10/A10 PCBs/Left Console Individual PCBs/UHF-ROTARIES/UHF-ROTARIES.kicad_sch (KiCad schematic)
At the start: 25 parts, among them J1 VHF_AM, J10 VHF_AM_OFF-TR-DF, J3 OLED, J4 BKLGHT, J9 VHF_AM_MAIN, SW1 SECOND CHANNEL, SW2 THIRD CHANNEL, SW3 FORTH CHANNEL, SW4 PRESET, SW5 FIRST CHANNEL, SW6 LOAD, SW7 TONE, SW8 PRESET, SW9 THIRD CHANNEL

Commit message: A10
Parts:
- added D11, D12, D13: D, Diode_THT:D_A-405_P7.62mm_Horizontal, symbol Device:D
- added SW10: TEST DISPLAY, Connector_Molex:Molex_KK-254_AE-6410-02A_1x02_P2.54mm_Vertical, symbol Switch:SW_Push
- added SW11: TONE, Connector_Molex:Molex_KK-254_AE-6410-02A_1x02_P2.54mm_Vertical, symbol Switch:SW_Push
- added SW12: LOAD, Connector_Molex:Molex_KK-254_AE-6410-02A_1x02_P2.54mm_Vertical, symbol Switch:SW_Push
- J1: value VHF_AM -> UHF
- SW6: value LOAD -> TEST DISPLAY
- SW7: value TONE -> STATUS
Connections:
- net VHF__AM_PRESET_A is gone; now on net UHF_PRESET_A: SW8.1
- net VHF__AM_PRESET_B is gone; now on net UHF_PRESET_B: SW8.3
- net COL1: now also D11.2 (A), D12.2 (A), D13.2 (A); no longer D3.2 (A)
- net COL8: now also D3.2 (A)
- net ROW14: now also SW10.2
- net ROW15: now also SW11.2, SW12.2
- net VHF_AM_OLED_SC renamed UHF_OLED_SC
- net VHF_AM_OLED_SD renamed UHF_OLED_SD
- net VHF_AM_PRESET_A renamed UHF_PRESET_A
- net VHF_AM_PRESET_B renamed UHF_PRESET_B
- net VHF_AM_VOL renamed UHF_VOL
- new net: D11.1 (K), SW10.1
- new net: D12.1 (K), SW11.1
- new net: D13.1 (K), SW12.1
Other:
- note added: "ADF"
- note added: "BOTH"
- note added: "GRD"
- note added: "MAIN"
- note added: "MAN"
- note added: "OFF"
- note added: "PRESET"
- moved on the sheet: J3, RV1

Commit message: A10 VHF and UHF
Parts:
- removed SW10: TEST DISPLAY, Connector_Molex:Molex_KK-254_AE-6410-02A_1x02_P2.54mm_Vertical, symbol Switch:SW_Push
- removed SW11: TONE, Connector_Molex:Molex_KK-254_AE-6410-02A_1x02_P2.54mm_Vertical, symbol Switch:SW_Push
- added SW10: T-TONE, symbol Switch:SW_SP3T
- added SW13: SQELCH, symbol Switch:SW_SPST
- J10: value VHF_AM_OFF-TR-DF -> UHF_OFF-TR-DF
- J9: value VHF_AM_MAIN -> UHF_MAIN
- RV1: value VHF_AM_VOL -> UHF_VOL
Connections:
- net COL0 is gone; now on net COL7: J1.1 (Pin_1)
- net COL11 is gone; now on net COL10: D9.2 (A)
- net COL3 is gone; now on net COL10: J1.4 (Pin_4)
- net ANALOG_5V: now also J1.22 (Pin_22); no longer J1.21 (Pin_21)
- net ANALOG_GND: now also J1.24 (Pin_24); no longer J1.23 (Pin_23)
- net COL7: now also D1.2 (A)
- net COL8: now also D11.2 (A), D2.2 (A), D4.2 (A), J1.2 (Pin_2)
- net COL9: now also D12.2 (A), D13.2 (A), J1.3 (Pin_3)
- net ROW0: no longer SW4.1, SW4.7
- net ROW1: no longer SW4.2, SW4.8
- net ROW10: now also J9.5 (Pin_5), SW4.1, SW4.7, SW10.1; no longer J9.2 (Pin_2)
- net ROW11: now also SW4.2, SW4.8, SW10.4; no longer J9.3 (Pin_3)
- net ROW12: now also SW12.2, SW4.3, SW4.9; no longer J9.4 (Pin_4)
- net ROW13: now also SW4.10, SW4.4, SW6.2; no longer J9.5 (Pin_5)
- net ROW14: now also SW4.11, SW4.5, SW7.2; no longer SW6.2
- net ROW15: now also SW4.12, SW4.6, SW13.2 (B); no longer SW12.2, SW7.2
- net ROW2: no longer SW4.3, SW4.9
- net ROW3: no longer SW4.10, SW4.4
- net ROW4: no longer SW4.11, SW4.5
- net ROW5: no longer SW4.12, SW4.6
- net ROW7: now also J9.2 (Pin_2)
- net ROW8: now also J9.3 (Pin_3)
- net ROW9: now also J9.4 (Pin_4)
- net UHF_VOL: now also J1.23 (Pin_23); no longer J1.22 (Pin_22)
- net at D11.1 (K): now also SW13.1 (A)
- net at D12.1 (K): now also SW10.3
- removed net COL1: D1.2 (A), D11.2 (A), D12.2 (A), D13.2 (A), D4.2 (A), J1.2 (Pin_2)
- removed net COL2: D2.2 (A), J1.3 (Pin_3)
- no-connect marks 17 -> 26
Other:
- note added: "MON-OFF-MON"
- moved on the sheet: D1, D11, D12, D13, D2, D3, D4, J1, J10, J3, J4, J9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

Commit message: A10 PCBS
Parts:
- J1: footprint Connector_IDC:IDC-Header_2x17_P2.54mm_Latch_Vertical -> Connector_IDC:IDC-Header_2x17_P2.54mm_Vertical
Changed lines of the file:
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@@
 			)
 		)
-		(property "Footprint" "Connector_IDC:IDC-Header_2x17_P2.54mm_Latch_Vertical"
+		(property "Footprint" "Connector_IDC:IDC-Header_2x17_P2.54mm_Vertical"
 			(at 265.684 117.602 0)
 			(effects

Commit message: A10 PCBS
Parts:
- added J2: BKLGHT, Connector_Molex:Molex_KK-254_AE-6410-02A_1x02_P2.54mm_Vertical, symbol Connector:Conn_01x02_Socket
- J10: footprint Connector_Molex:Molex_KK-254_AE-6410-04A_1x04_P2.54mm_Vertical -> Footprint Library:ALPHA 12 POS; symbol Connector:Conn_01x04_Female -> Switch:SW_Rotary_1x12
- J9: footprint Connector_Molex:Molex_KK-254_AE-6410-06A_1x06_P2.54mm_Vertical -> Footprint Library:ALPHA 12 POS; symbol Connector:Conn_01x06_Female -> Switch:SW_Rotary_1x12
- SW10: footprint (none) -> Connector_Molex:Molex_KK-254_AE-6410-02A_1x02_P2.54mm_Vertical; symbol Switch:SW_SP3T -> Switch:SW_SPDT
- SW13: footprint (none) -> Connector_Molex:Molex_KK-254_AE-6410-02A_1x02_P2.54mm_Vertical
- SW3: value FORTH CHANNEL -> FIFTH CHANNEL
- SW9: value THIRD CHANNEL -> FORTH CHANNEL
Connections:
- net +12V: now also J2.1 (Pin_1)
- net BACKLIGHT_-V: now also J2.2 (Pin_2)
- net ROW10: now also J10.1, J9.4; no longer J10.2 (Pin_2), J9.5 (Pin_5)
- net ROW11: now also J10.2, SW10.3 (C); no longer J10.3 (Pin_3), SW10.4
- net ROW12: now also J10.3; no longer J10.4 (Pin_4)
- net ROW7: now also J9.1; no longer J9.2 (Pin_2)
- net ROW8: now also J9.2; no longer J9.3 (Pin_3)
- net ROW9: now also J9.3; no longer J9.4 (Pin_4)
- net at D1.1 (K): now also J9.A1; no longer J9.1 (Pin_1)
- net at SW10.2 (B): now also D12.1 (K)
- net at D2.1 (K): now also J10.A1; no longer J10.1 (Pin_1)
- no-connect marks 26 -> 42
Other:
- moved on the sheet: D1, D11, D12, D13, D2, D3, D4, J3, J4, RV1, SW12, SW13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

Commit message: A10
Parts:
- added J5: PRESET, Connector_JST:JST_XH_B4B-XH-A_1x04_P2.50mm_Vertical, symbol Connector:Conn_01x04_Socket
- J2, J4, SW12, SW13, SW6, SW7: footprint Connector_Molex:Molex_KK-254_AE-6410-02A_1x02_P2.54mm_Vertical -> Connector_JST:JST_XH_B2B-XH-A_1x02_P2.50mm_Vertical
- J3: value OLED -> CHANNEL; footprint Connector_Molex:Molex_KK-254_AE-6410-04A_1x04_P2.54mm_Vertical -> Connector_JST:JST_XH_B4B-XH-A_1x04_P2.50mm_Vertical
- RV1, SW8: footprint Connector_Molex:Molex_KK-254_AE-6410-03A_1x03_P2.54mm_Vertical -> Connector_JST:JST_XH_B3B-XH-A_1x03_P2.50mm_Vertical
- SW10: footprint Connector_Molex:Molex_KK-254_AE-6410-02A_1x02_P2.54mm_Vertical -> Connector_JST:JST_XH_B3B-XH-A_1x03_P2.50mm_Vertical
Connections:
- net +5V: now also J1.27 (Pin_27), J5.1 (Pin_1); no longer J1.29 (Pin_29)
- net ANALOG_5V: now also J1.21 (Pin_21); no longer J1.22 (Pin_22)
- net ANALOG_GND: now also J1.23 (Pin_23); no longer J1.24 (Pin_24)
- net GND: now also J1.25 (Pin_25), J1.28 (Pin_28), J5.2 (Pin_2); no longer J1.26 (Pin_26), J1.30 (Pin_30)
- net UHF_PRESET_A: now also J1.24 (Pin_24); no longer J1.25 (Pin_25)
- net UHF_PRESET_B: now also J1.26 (Pin_26); no longer J1.27 (Pin_27)
- net UHF_VOL: now also J1.22 (Pin_22); no longer J1.23 (Pin_23)
- net UHF_OLED_SC renamed UHF_CHANNEL_SC
- net UHF_OLED_SD renamed UHF_CHANNEL_SD
- new net UHF_PRESET_SC: J1.29 (Pin_29), J5.3 (Pin_3)
- new net UHF_PRESET_SD: J1.30 (Pin_30), J5.4 (Pin_4)
- no-connect marks 42 -> 40
