File: A10/A10 PCBs/Forward Console General Output/Forward Console General Output.kicad_pcb (KiCad board)
At the start: 2 copper layers, 99.7 x 98.4 mm, 79 parts, among them J1 BACKLIGHT, J10 PATCH, J11 PATCH, J12 BACKLIGHT, J13 BACKLIGHT, J14 BACKLIGHT, J15 PATCH, J16 PATCH, J17 BACKLIGHT, J18 BACKLIGHT, J19 BACKLIGHT, J2 BACKLIGHT, J20 5VIN, J21 LOX, J22 12VIN, J23 CABIN_PRES, J24 PWM, J25 PWM, J26 Communication, J27 OXY_REG, J28 RIGHT FUEL, J29 LEFT_FUEL, J3 BACKLIGHT, J30 RIGHT_HYD, J31 LEFT_HYD, J32 Analog, J33 Analog, J34 CABIN_PRES, J35 OXY_REG, J36 LOX, J37 RIGHT_HYD, J38 LEFT_FUEL, J39 RIGHT FUEL, J4 BACKLIGHT, J40 LEFT_HYD, J41 Power, J42 Power, J43 Analog, J44 Analog, J45 Digital, J46 PWM, J47 PWM, J48 Communication, J49 CAUTION_UPPER_DIGIT, J5 BACKLIGHT, J50 CAUTION_UPPER_SEG, J51 CAUTION_LOW_DIGITS, J52 CAUTION_LOWER_SEG, J53 OXY_LED, J54 TACAN_TEST, J55 FORWARD_SEGEMENTS, J56 FORWARD_DIGITS, J6 BACKLIGHT, J7 BACKLIGHT, J8 BACKLIGHT, J9 BACKLIGHT, Q1 IRF1405PBF, U1 USR-ES1, U2 MAX7219-A, U3 MAX7219-B, U4 TCA9548APWR

Commit message: A10
Parts:
- removed C3: 0.1uF, Capacitor_THT:C_Disc_D5.1mm_W3.2mm_P5.00mm
- removed C4: 100uF, Capacitor_THT:CP_Radial_D8.0mm_P5.00mm
- removed J21: LOX, Connector_Molex:Molex_KK-254_AE-6410-06A_1x06_P2.54mm_Vertical
- removed J36: LOX, Connector_Molex:Molex_KK-254_AE-6410-04A_1x04_P2.54mm_Vertical
- removed J55: FORWARD_SEGEMENTS, Connector_Molex:Molex_KK-254_AE-6410-08A_1x08_P2.54mm_Vertical
- removed J56: FORWARD_DIGITS, Connector_Molex:Molex_KK-254_AE-6410-04A_1x04_P2.54mm_Vertical
- removed R6, R7: 10K, Resistor_THT:R_Axial_DIN0204_L3.6mm_D1.6mm_P2.54mm_Vertical
- added U5: ULN2003A, Package_DIP:DIP-16_W7.62mm_LongPads, F.Cu at (82.9, 117.1)
- J49: value CAUTION_UPPER_DIGIT -> CAUTION LAMP; footprint Connector_Molex:Molex_KK-254_AE-6410-08A_1x08_P2.54mm_Vertical -> Connector_Molex:Molex_KK-254_AE-6410-02A_1x02_P2.54mm_Vertical
- J50: value CAUTION_UPPER_SEG -> 28V RELAY BOARD; footprint Connector_Molex:Molex_KK-254_AE-6410-08A_1x08_P2.54mm_Vertical -> Connector_Molex:Molex_KK-254_AE-6410-06A_1x06_P2.54mm_Vertical
- J51: value CAUTION_LOW_DIGITS -> BULB_A; footprint Connector_Molex:Molex_KK-254_AE-6410-04A_1x04_P2.54mm_Vertical -> Connector_Molex:Molex_KK-254_AE-6410-06A_1x06_P2.54mm_Vertical
- J52: value CAUTION_LOWER_SEG -> BULB_B; footprint Connector_Molex:Molex_KK-254_AE-6410-08A_1x08_P2.54mm_Vertical -> Connector_Molex:Molex_KK-254_AE-6410-06A_1x06_P2.54mm_Vertical
- J53: value OXY_LED -> ANTI-SKID-COIL
- J54: value TACAN_TEST -> SAS_COILS; footprint Connector_Molex:Molex_KK-254_AE-6410-02A_1x02_P2.54mm_Vertical -> Connector_Molex:Molex_KK-254_AE-6410-06A_1x06_P2.54mm_Vertical
- U2: value MAX7219-A -> ULN2003A; footprint Package_DIP:DIP-24_W7.62mm_Socket -> Package_DIP:DIP-16_W7.62mm_LongPads
- U3: value MAX7219-B -> ULN2003A; footprint Package_DIP:DIP-24_W7.62mm_Socket -> Package_DIP:DIP-16_W7.62mm_LongPads
- moved J54 119.1 mm to (71.6, 140.9)
- moved U3 117.0 mm to (71.3, 117.1)
- moved J50 91.6 mm to (230.8, 119.7)
- moved J52 91.5 mm to (230.8, 102.0)
- moved J51 90.0 mm to (230.8, 94.1)
- moved U2 67.9 mm to (72.1, 90.5)
- moved J49 53.2 mm to (91.1, 77.8)
- moved J53 42.7 mm to (230.8, 110.8)
- moved U4 13.6 mm to (249.9, 75.9)
- moved J16 4.65 mm to (171.8, 39.5)
- moved J11 4.02 mm to (171.8, 43.5)
- moved J10 1.02 mm to (204.1, 42.2)
- moved J15 1.02 mm to (204.1, 38.4)
Connections:
- net /A15 renamed O_ANTI_SKID
- J24 pad 1: /SCL/21 -> /SCL
- J24 pad 2: /SDA/20 -> /SDA
- J26 pad 1: CLK -> /TX3/14
- J26 pad 2: LOAD -> /RX3/15
- J26 pad 3: DIN -> /I2C_SEL_RESET
- J26 pad 4: /RX2/17 -> /I2C_SEL_A0
- J26 pad 5: /TX1/18 -> /I2C_SEL_A1
- J26 pad 6: /RX1/19 -> /I2C_SEL_A2
- J26 pad 7: /SDA/20 -> /SDA
- J26 pad 8: /SCL/21 -> /SCL
- J32 pad 5: /A4 -> O_CAUTION_LAMP-
- J32 pad 6: /A5 -> O_PRI_LAMP
- J32 pad 7: /A6 -> O_SEP_LAMP
- J32 pad 8: /A7 -> O_MISSILE_LAMP
- J33 pad 1: /A8 -> O_HARS_LAMP
- J33 pad 2: /A9 -> O_EGI_LAMP
- J33 pad 3: /A10 -> O_TISL_LAMP
- J33 pad 4: /A11 -> O_STR_PT_LAMP
- J33 pad 5: /A12 -> O_ANCHR_LAMP
- J33 pad 6: /A13 -> O_TCN_LAMP
- J33 pad 7: /A14 -> O_ILS_LAMP
- J43 pad 5: /A4 -> O_CAUTION_LAMP-
- J43 pad 6: /A5 -> O_PRI_LAMP
- J43 pad 7: /A6 -> O_SEP_LAMP
- J43 pad 8: /A7 -> O_MISSILE_LAMP
- J44 pad 1: /A8 -> O_HARS_LAMP
- J44 pad 2: /A9 -> O_EGI_LAMP
- J44 pad 3: /A10 -> O_TISL_LAMP
- J44 pad 4: /A11 -> O_STR_PT_LAMP
- J44 pad 5: /A12 -> O_ANCHR_LAMP
- J44 pad 6: /A13 -> O_TCN_LAMP
- J44 pad 7: /A14 -> O_ILS_LAMP
- J45 pad 12: /*45 -> O_COIL_L_YAW
- J45 pad 14: /43 -> O_COIL_R_YAW
- J45 pad 16: /41 -> O_COIL_L_PITCH
- J45 pad 18: /39 -> O_COIL_R_PITCH
- J46 pad 1: /SCL/21 -> /SCL
- J46 pad 2: /SDA/20 -> /SDA
- J48 pad 1: CLK -> /TX3/14
- J48 pad 2: LOAD -> /RX3/15
- J48 pad 3: DIN -> /I2C_SEL_RESET
- J48 pad 4: /RX2/17 -> /I2C_SEL_A0
- J48 pad 5: /TX1/18 -> /I2C_SEL_A1
- J48 pad 6: /RX1/19 -> /I2C_SEL_A2
- J48 pad 7: /SDA/20 -> /SDA
- J48 pad 8: /SCL/21 -> /SCL
- J49 pad 1: /MAX7219A/DIG_A0 -> +12V
- J49 pad 2: /MAX7219A/DIG_A1 -> /COIL AND LAMP DRIVERS/CAUTION_LAMP-
- J50 pad 1: /MAX7219A/SEG_A0 -> GND
- J50 pad 2: /MAX7219A/SEG_B0 -> /A0
- J50 pad 3: /MAX7219A/SEG_C0 -> /A1
- J50 pad 4: /MAX7219A/SEG_D0 -> /A2
- J50 pad 5: /MAX7219A/SEG_E0 -> /A3
- J50 pad 6: /MAX7219A/SEG_F0 -> +5VD
- J51 pad 1: /MAX7219A/DIG_B0 -> +12V
- J51 pad 2: /MAX7219A/DIG_B1 -> /COIL AND LAMP DRIVERS/PRI
- J51 pad 3: /MAX7219A/DIG_B2 -> /COIL AND LAMP DRIVERS/SEP
- J51 pad 4: /MAX7219A/DIG_B3 -> /COIL AND LAMP DRIVERS/MISSLE LAUNCH
- J52 pad 1: /MAX7219A/SEG_A1 -> +12V
- J52 pad 2: /MAX7219A/SEG_B1 -> /COIL AND LAMP DRIVERS/TISL
- J52 pad 3: /MAX7219A/SEG_C1 -> /COIL AND LAMP DRIVERS/STR PT
- J52 pad 4: /MAX7219A/SEG_D1 -> /COIL AND LAMP DRIVERS/ANCHR
- J52 pad 5: /MAX7219A/SEG_E1 -> /COIL AND LAMP DRIVERS/TCN
- J52 pad 6: /MAX7219A/SEG_F1 -> /COIL AND LAMP DRIVERS/ILS
- J53 pad 1: /MAX7219A/SEG_A1 -> +12V
- J53 pad 2: /MAX7219A/DIG_B4 -> /COIL AND LAMP DRIVERS/COIL_ANTI_SKID
- J54 pad 1: /MAX7219A/SEG_B1 -> +12V
- J54 pad 2: /MAX7219A/DIG_B4 -> /COIL AND LAMP DRIVERS/COIL_L_YAW
- U2 pad 1: DIN -> O_CAUTION_LAMP-
- U2 pad 10: /MAX7219A/DIG_A5 -> /COIL AND LAMP DRIVERS/TISL
- U2 pad 11: /MAX7219A/DIG_A1 -> /COIL AND LAMP DRIVERS/EGI
- U2 pad 12: LOAD -> /COIL AND LAMP DRIVERS/HARS
- U2 pad 13: CLK -> /COIL AND LAMP DRIVERS/MISSLE LAUNCH
- U2 pad 14: /MAX7219A/SEG_A0 -> /COIL AND LAMP DRIVERS/SEP
- U2 pad 15: /MAX7219A/SEG_F0 -> /COIL AND LAMP DRIVERS/PRI
- U2 pad 16: /MAX7219A/SEG_B0 -> /COIL AND LAMP DRIVERS/CAUTION_LAMP-
- U2 pad 2: /MAX7219A/DIG_A0 -> O_PRI_LAMP
- U2 pad 3: /MAX7219A/DIG_A4 -> O_SEP_LAMP
- U2 pad 4: GND -> O_MISSILE_LAMP
- U2 pad 5: /MAX7219A/DIG_A6 -> O_HARS_LAMP
- U2 pad 6: /MAX7219A/DIG_A2 -> O_EGI_LAMP
- U2 pad 7: /MAX7219A/DIG_A3 -> O_TISL_LAMP
- U2 pad 8: /MAX7219A/DIG_A7 -> GND
- U2 pad 9: GND -> +12V
- U3 pad 1: /MAX7219A/A-DOUT-B-DIN -> O_STR_PT_LAMP
- U3 pad 10: /MAX7219A/DIG_B5 -> unconnected-(U3-O7-Pad10)
- U3 pad 11: /MAX7219A/DIG_B1 -> unconnected-(U3-O6-Pad11)
- U3 pad 12: LOAD -> unconnected-(U3-O5-Pad12)
- U3 pad 13: CLK -> /COIL AND LAMP DRIVERS/ILS
- U3 pad 14: /MAX7219A/SEG_A1 -> /COIL AND LAMP DRIVERS/TCN
- U3 pad 15: /MAX7219A/SEG_F1 -> /COIL AND LAMP DRIVERS/ANCHR
- U3 pad 16: /MAX7219A/SEG_B1 -> /COIL AND LAMP DRIVERS/STR PT
- U3 pad 2: /MAX7219A/DIG_B0 -> O_ANCHR_LAMP
- U3 pad 3: /MAX7219A/DIG_B4 -> O_TCN_LAMP
- U3 pad 4: GND -> O_ILS_LAMP
- U3 pad 5: /MAX7219A/DIG_B6 -> GND
- U3 pad 6: /MAX7219A/DIG_B2 -> GND
- U3 pad 7: /MAX7219A/DIG_B3 -> GND
- U3 pad 8: /MAX7219A/DIG_B7 -> GND
- U3 pad 9: GND -> +12V
- U4 pad 1: unconnected-(U4-A0-Pad1) -> +3V3
- U4 pad 2: unconnected-(U4-A1-Pad2) -> GND
- U4 pad 3: unconnected-(U4-~{RESET}-Pad3) -> /SDA
- U4 pad 4: unconnected-(U4-SD0-Pad4) -> /SCL
- U4 pad 5: unconnected-(U4-SC0-Pad5) -> /I2C_SEL_RESET
- U4 pad 6: unconnected-(U4-SD1-Pad6) -> /I2C_SEL_A2
- U4 pad 7: unconnected-(U4-SC1-Pad7) -> /I2C_SEL_A1
- U4 pad 8: unconnected-(U4-SD2-Pad8) -> /I2C_SEL_A0
Routing:
- net GND: track 375.8 -> 0.00 mm, vias 1 -> 0
- net +12V: track 301.1 -> 0.00 mm, vias 1 -> 0
- net +5VD: track 299.7 -> 0.00 mm, vias 2 -> 0
- net /BACKLIGHT_-V: track 269.1 -> 0.00 mm
- net /*3: track 140.3 -> 0.00 mm
- net CLK: track 135.3 -> 0.00 mm, vias 2 -> 0
- net /MAX7219A/SEG_A1: track 130.2 -> 0.00 mm, vias 1 -> 0
- net /*4: track 114.7 -> 0.00 mm, vias 1 -> 0
- net +5V: track 113.1 -> 0.00 mm, vias 1 -> 0
- net /MAX7219A/SEG_B1: track 106.1 -> 0.00 mm, vias 1 -> 0
- net SCLK: track 99.1 -> 0.00 mm
- net MOSI: track 98.5 -> 0.00 mm, vias 1 -> 0
- net LOAD: track 83.8 -> 0.00 mm
- net SS: track 81.1 -> 0.00 mm
- net /SCL/21: track 78.5 -> 0.00 mm
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Other:
- board text removed: "DP G F E D C B A"

Commit message: a10
Parts:
- removed J1, J12, J13, J17, J18, J2, J4, J5, J7, J8: BACKLIGHT, Connector_Molex:Molex_KK-254_AE-6410-02A_1x02_P2.54mm_Vertical
- added J21: VHF_FM_OLED, Connector_Molex:Molex_KK-254_AE-6410-04A_1x04_P2.54mm_Vertical, F.Cu at (128.6, 67.0)
- added J36: VHF_AM_OLED, Connector_Molex:Molex_KK-254_AE-6410-04A_1x04_P2.54mm_Vertical, F.Cu at (128.6, 58.7)
- added J55: UHF_OLED, Connector_Molex:Molex_KK-254_AE-6410-04A_1x04_P2.54mm_Vertical, F.Cu at (140.0, 67.0)
- added J56: MWS_OLED, Connector_Molex:Molex_KK-254_AE-6410-04A_1x04_P2.54mm_Vertical, F.Cu at (140.0, 58.7)
- added J57: CMSP_OLED, Connector_Molex:Molex_KK-254_AE-6410-04A_1x04_P2.54mm_Vertical, F.Cu at (151.4, 67.0)
- added J58: ILS_OLED, Connector_Molex:Molex_KK-254_AE-6410-04A_1x04_P2.54mm_Vertical, F.Cu at (151.4, 58.7)
- added J59: TACAN_OLED, Connector_Molex:Molex_KK-254_AE-6410-04A_1x04_P2.54mm_Vertical, F.Cu at (181.9, 68.2)
- added J60: SPARE_OLED, Connector_Molex:Molex_KK-254_AE-6410-04A_1x04_P2.54mm_Vertical, F.Cu at (181.9, 58.7)
- moved U2 107.9 mm to (178.7, 106.3)
- moved U3 96.7 mm to (167.3, 106.3)
- moved J50 80.9 mm to (150.8, 107.6)
- moved J54 80.7 mm to (150.8, 125.4)
- moved J49 75.5 mm to (155.9, 116.5)
- moved U4 74.8 mm to (175.6, 84.8)
- moved J52 61.6 mm to (176.2, 130.5)
- moved J9 58.4 mm to (152.7, 75.9)
- moved U5 57.5 mm to (139.4, 106.3)
- moved Q1 55.5 mm to (132.4, 77.5)
- moved R2 49.4 mm to (146.4, 77.7), turned to 90 degrees
- moved J51 48.5 mm to (190.8, 121.6)
- moved J14 47.3 mm to (151.9, 84.9)
- moved J19 47.3 mm to (145.1, 84.9)
- moved J3 47.1 mm to (138.4, 84.9)
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Connections:
- U4 pad 10: unconnected-(U4-SC0-Pad10) -> /SC0
- U4 pad 11: unconnected-(U4-SD1-Pad11) -> /SD1
- U4 pad 12: unconnected-(U4-SC1-Pad12) -> /SC1
- U4 pad 13: unconnected-(U4-SD2-Pad13) -> /SD2
- U4 pad 14: unconnected-(U4-SC2-Pad14) -> /SC2
- U4 pad 15: unconnected-(U4-SD3-Pad15) -> /SD3
- U4 pad 16: unconnected-(U4-SC3-Pad16) -> /SC3
- U4 pad 17: unconnected-(U4-SD4-Pad17) -> /SD4
- U4 pad 18: unconnected-(U4-SC4-Pad18) -> /SC4
- U4 pad 19: unconnected-(U4-SD5-Pad19) -> /SD5
- U4 pad 20: unconnected-(U4-SC5-Pad20) -> /SC5
- U4 pad 21: unconnected-(U4-SD6-Pad21) -> /SD6
- U4 pad 22: unconnected-(U4-SC6-Pad22) -> /SC6
- U4 pad 23: unconnected-(U4-SD7-Pad23) -> /SD7
- U4 pad 24: unconnected-(U4-SC7-Pad24) -> /SC7
- U4 pad 9: unconnected-(U4-SD0-Pad9) -> /SD0
Routing:
- net GND: track 0.00 -> 474.1 mm
- net +12V: track 0.00 -> 260.0 mm
- net +5VD: track 0.00 -> 225.1 mm, vias 0 -> 2
- net /BACKLIGHT_-V: track 0.00 -> 190.5 mm
- net /*3: track 0.00 -> 151.7 mm
- net +5V: track 0.00 -> 150.3 mm
- net /SCL: track 0.00 -> 133.8 mm
- net /SDA: track 0.00 -> 130.3 mm
- net SCLK: track 0.00 -> 114.1 mm
- net O_COIL_R_PITCH: track 0.00 -> 100.1 mm, vias 0 -> 2
- net MOSI: track 0.00 -> 98.3 mm, vias 0 -> 2
- net MISO: track 0.00 -> 93.8 mm, vias 0 -> 1
- net O_COIL_L_YAW: track 0.00 -> 88.1 mm, vias 0 -> 1
- net SS: track 0.00 -> 85.6 mm
- net O_COIL_R_YAW: track 0.00 -> 85.1 mm, vias 0 -> 2
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Other:
- board text added: "A10 FRONT CONSOLE OUTPUT V1.0"
- board text removed: "A10 RIGHT CONSOLE OUTPUT V1.1"

Commit message: A10
Parts:
- removed J23: CABIN_PRES, Connector_Molex:Molex_KK-254_AE-6410-06A_1x06_P2.54mm_Vertical
- removed J27: OXY_REG, Connector_Molex:Molex_KK-254_AE-6410-06A_1x06_P2.54mm_Vertical
- removed J28: RIGHT FUEL, Connector_Molex:Molex_KK-254_AE-6410-06A_1x06_P2.54mm_Vertical
- removed J29: LEFT_FUEL, Connector_Molex:Molex_KK-254_AE-6410-06A_1x06_P2.54mm_Vertical
- removed J30: RIGHT_HYD, Connector_Molex:Molex_KK-254_AE-6410-06A_1x06_P2.54mm_Vertical
- removed J31: LEFT_HYD, Connector_Molex:Molex_KK-254_AE-6410-06A_1x06_P2.54mm_Vertical
- removed J34: CABIN_PRES, Connector_Molex:Molex_KK-254_AE-6410-04A_1x04_P2.54mm_Vertical
- removed J35: OXY_REG, Connector_Molex:Molex_KK-254_AE-6410-04A_1x04_P2.54mm_Vertical
- removed J37: RIGHT_HYD, Connector_Molex:Molex_KK-254_AE-6410-04A_1x04_P2.54mm_Vertical
- removed J38: LEFT_FUEL, Connector_Molex:Molex_KK-254_AE-6410-04A_1x04_P2.54mm_Vertical
- removed J39: RIGHT FUEL, Connector_Molex:Molex_KK-254_AE-6410-04A_1x04_P2.54mm_Vertical
- removed J40: LEFT_HYD, Connector_Molex:Molex_KK-254_AE-6410-04A_1x04_P2.54mm_Vertical
- removed J50: 28V RELAY BOARD, Connector_Molex:Molex_KK-254_AE-6410-06A_1x06_P2.54mm_Vertical
- removed J54: SAS_COILS, Connector_Molex:Molex_KK-254_AE-6410-06A_1x06_P2.54mm_Vertical
- added J61: APU_FIRE, Connector_Molex:Molex_KK-254_AE-6410-02A_1x02_P2.54mm_Vertical, F.Cu at (230.2, 81.2)
- added J62: RIGHT_FIRE, Connector_Molex:Molex_KK-254_AE-6410-02A_1x02_P2.54mm_Vertical, F.Cu at (237.3, 81.2)
- added J63: LEFT_FIRE, Connector_Molex:Molex_KK-254_AE-6410-02A_1x02_P2.54mm_Vertical, F.Cu at (244.4, 81.2)
- added J64: SARI-SERVO, Connector_Molex:Molex_KK-254_AE-6410-03A_1x03_P2.54mm_Vertical, F.Cu at (267.8, 91.1)
- added U7: VIRIABLE BUCK, VARIABLE_BUCK:VARIABLE_BUCK, F.Cu at (248.8, 67.9)
- J21: value VHF_FM_OLED -> CLOCK-OLED
- J36: value VHF_AM_OLED -> ALTIMETER-OLED
- J55: value UHF_OLED -> BARO-OLED
Connections:
- net /*11 renamed D11
- net /*2 renamed BACKLIGHT
- net /*3 renamed D3
- net /*4 renamed D4
- net /*5 renamed D5
- net /*6 renamed D6
- net /*7 renamed D7
- net /*8 renamed D8
- net /*9 renamed D9
- net /A3 renamed A3 D57
- net /BACKLIGHT_-V renamed BACKLIGHT_-V
- net /I2C_SEL_A0 renamed D17
- net /I2C_SEL_A1 renamed D18
- net /I2C_SEL_A2 renamed D19
- net /I2C_SEL_RESET renamed D16
- net /RX3/15 renamed D15
- net /SC0 renamed /OLED/SC0
- net /SC1 renamed /OLED/SC1
- net /SC2 renamed /OLED/SC2
- net /SC3 renamed /OLED/SC3
- net /SC4 renamed /OLED/SC4
- net /SC5 renamed /OLED/SC5
- net /SC6 renamed /OLED/SC6
- net /SC7 renamed /OLED/SC7
- net /SCL renamed D21 SCL
- net /SD0 renamed /OLED/SD0
- net /SD1 renamed /OLED/SD1
- net /SD2 renamed /OLED/SD2
- net /SD3 renamed /OLED/SD3
- net /SD4 renamed /OLED/SD4
- net /SD5 renamed /OLED/SD5
- net /SD6 renamed /OLED/SD6
- net /SD7 renamed /OLED/SD7
- net /SDA renamed D20 SDA
- net /TX3/14 renamed D14
- net O_ANCHR_LAMP renamed A12 D66
- net O_CAUTION_LAMP- renamed A4 D58
- net O_EGI_LAMP renamed A9 D63
- net O_HARS_LAMP renamed A8 D62
- net O_ILS_LAMP renamed A14 D68
- net O_MISSILE_LAMP renamed A7 D61
- net O_PRI_LAMP renamed A5 D59
- net O_SEP_LAMP renamed A6 D60
- net O_STR_PT_LAMP renamed A11 D65
- net O_TCN_LAMP renamed A13 D67
- net O_TISL_LAMP renamed A10 D64
- J32 pad 1: /A0 -> A0 D54
- J32 pad 2: /A1 -> A1 D55
- J32 pad 3: /A2 -> A2 D56
- J33 pad 8: O_ANTI_SKID -> A15 D69
- J43 pad 1: /A0 -> A0 D54
- J43 pad 2: /A1 -> A1 D55
- J43 pad 3: /A2 -> A2 D56
- J44 pad 8: O_ANTI_SKID -> A15 D69
- J45 pad 10: /47 -> D47
- J45 pad 11: /*44 -> D44
- J45 pad 12: O_COIL_L_YAW -> D45
- J45 pad 13: /42 -> D42
- J45 pad 14: O_COIL_R_YAW -> D43
- J45 pad 15: /40 -> D40
- J45 pad 16: O_COIL_L_PITCH -> D41
- J45 pad 17: /38 -> D38
- J45 pad 18: O_COIL_R_PITCH -> D39
- J45 pad 19: /36 -> D36
- J45 pad 20: /37 -> D37
- J45 pad 21: /34 -> D34
- J45 pad 22: /35 -> D35
- J45 pad 23: /32 -> D32
- J45 pad 24: /33 -> D33
- J45 pad 25: /30 -> D30
- J45 pad 26: /31 -> D31
- J45 pad 27: /28 -> D28
- J45 pad 28: /29 -> D29
- J45 pad 29: /26 -> D26
- J45 pad 30: /27 -> D27
- J45 pad 31: /24 -> D24
- J45 pad 32: /25 -> D25
- J45 pad 33: /22 -> D22
- J45 pad 34: /23 -> D23
- J45 pad 7: /48 -> D48
- J45 pad 8: /49 -> D49
- J45 pad 9: /*46 -> D46
- U3 pad 12: unconnected-(U3-O5-Pad12) -> /COIL AND LAMP DRIVERS/COIL_ANTI_SKID
- U3 pad 5: GND -> A15 D69
- U5 pad 1: O_ANTI_SKID -> A0 D54
- U5 pad 12: /COIL AND LAMP DRIVERS/COIL_R_PITCH -> unconnected-(U5-O5-Pad12)
- U5 pad 13: /COIL AND LAMP DRIVERS/COIL_L_PITCH -> unconnected-(U5-O4-Pad13)
- U5 pad 14: /COIL AND LAMP DRIVERS/COIL_R_YAW -> /COIL AND LAMP DRIVERS/B_RIGHT_FIRE
- U5 pad 15: /COIL AND LAMP DRIVERS/COIL_L_YAW -> /COIL AND LAMP DRIVERS/B_APU_FIRE
- U5 pad 16: /COIL AND LAMP DRIVERS/COIL_ANTI_SKID -> /COIL AND LAMP DRIVERS/B_LEFT_FIRE
- U5 pad 2: O_COIL_L_YAW -> A1 D55
- U5 pad 3: O_COIL_R_YAW -> A2 D56
- U5 pad 4: O_COIL_L_PITCH -> unconnected-(U5-I4-Pad4)
- U5 pad 5: O_COIL_R_PITCH -> unconnected-(U5-I5-Pad5)
- U5 pad 9: +12V -> +24V
Routing:
- net GND: track 474.1 -> 0.00 mm
- net +12V: track 260.0 -> 0.00 mm
- net +5VD: track 225.1 -> 0.00 mm, vias 2 -> 0
- net BACKLIGHT_-V: track 190.5 -> 0.00 mm
- net D3: track 151.7 -> 0.00 mm
- net +5V: track 150.3 -> 0.00 mm
- net D21 SCL: track 133.8 -> 0.00 mm
- net D20 SDA: track 130.3 -> 0.00 mm
- net SCLK: track 114.1 -> 0.00 mm
- net O_COIL_R_PITCH: track 100.1 -> 0.00 mm, vias 2 -> 0
- net MOSI: track 98.3 -> 0.00 mm, vias 2 -> 0
- net MISO: track 93.8 -> 0.00 mm, vias 1 -> 0
- net O_COIL_L_YAW: track 88.1 -> 0.00 mm, vias 1 -> 0
- net SS: track 85.6 -> 0.00 mm
- net O_COIL_R_YAW: track 85.1 -> 0.00 mm, vias 2 -> 0
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