File: A10/A10 PCBs/Right Console Output/Right Console Output.kicad_pcb (KiCad board)
At the start: 2 copper layers, 99.7 x 98.4 mm, 60 parts, among them J1 BACKLIGHT, J10 BACKLIGHT, J11 BACKLIGHT, J12 BACKLIGHT, J13 BACKLIGHT, J14 BACKLIGHT, J15 BACKLIGHT, J16 5VIN, J17 12VIN, J18 PWM, J19 PWM, J2 BACKLIGHT, J20 Communication, J21 Analog, J22 Analog, J23 Power, J24 Power, J25 Analog, J26 Analog, J27 Digital, J28 PWM, J29 PWM, J3 BACKLIGHT, J30 Communication, J31 CAUTION_UPPER_DIGIT, J32 CAUTION_UPPER_SEG, J33 CAUTION_LOW_DIGITS, J34 CAUTION_LOWER_SEG, J35 OXY_LED, J36 TACAN_TEST, J37 FORWARD_SEGEMENTS, J38 FORWARD_DIGITS, J4 BACKLIGHT, J5 BACKLIGHT, J6 BACKLIGHT, J7 BACKLIGHT, J8 BACKLIGHT, J9 BACKLIGHT, Q1 IRF1405PBF, U1 USR-ES1, U2 MAX7219-A, U3 MAX7219-B

Commit message: A10
Parts:
- added J23: Conn_01x04_Female, Connector_Molex:Molex_KK-254_AE-6410-04A_1x04_P2.54mm_Vertical, F.Cu at (202.6, 54.3)
- added J24: Conn_01x04_Female, Connector_Molex:Molex_KK-254_AE-6410-04A_1x04_P2.54mm_Vertical, F.Cu at (210.2, 54.3)
- renumbered J23 to J25, J24 to J26, J25 to J27, J26 to J28, J27 to J29, J28 to J30, J29 to J31, J30 to J32, J31 to J33, J32 to J34, J33 to J35, J34 to J36, J35 to J37, J36 to J38, J37 to J39, J38 to J40
Connections:
- net /BACKLIGHT renamed /*2

Commit message: A10 AND HORNET
Parts:
- added J16: STEPPER_F, Connector_Molex:Molex_KK-254_AE-6410-06A_1x06_P2.54mm_Vertical, F.Cu at (202.1, 126.4)
- added J23: STEPPER_E, Connector_Molex:Molex_KK-254_AE-6410-06A_1x06_P2.54mm_Vertical, F.Cu at (210.3, 126.4)
- added J24: STEPPER_D, Connector_Molex:Molex_KK-254_AE-6410-06A_1x06_P2.54mm_Vertical, F.Cu at (202.1, 109.9)
- added J25: STEPPER_C, Connector_Molex:Molex_KK-254_AE-6410-06A_1x06_P2.54mm_Vertical, F.Cu at (210.3, 109.9)
- added J26: STEPPER_B, Connector_Molex:Molex_KK-254_AE-6410-06A_1x06_P2.54mm_Vertical, F.Cu at (202.1, 93.1)
- added J27: STEPPER_A, Connector_Molex:Molex_KK-254_AE-6410-06A_1x06_P2.54mm_Vertical, F.Cu at (210.3, 93.1)
- added J30: STEPPER_E, Connector_Molex:Molex_KK-254_AE-6410-04A_1x04_P2.54mm_Vertical, F.Cu at (210.2, 76.6)
- added J31: STEPPER_F, Connector_Molex:Molex_KK-254_AE-6410-04A_1x04_P2.54mm_Vertical, F.Cu at (202.1, 76.6)
- added J33: STEPPER_C, Connector_Molex:Molex_KK-254_AE-6410-04A_1x04_P2.54mm_Vertical, F.Cu at (210.2, 65.2)
- added J34: STEPPER_D, Connector_Molex:Molex_KK-254_AE-6410-04A_1x04_P2.54mm_Vertical, F.Cu at (202.1, 65.2)
- J32: renamed from J23; value Conn_01x04_Female -> STEPPER_B
- J35: renamed from J24; value Conn_01x04_Female -> STEPPER_A
- moved J49 11.2 mm to (188.1, 116.3)
- moved J32 0.91 mm to (202.1, 53.5)
- moved J35 0.77 mm to (210.2, 53.5)
- renumbered J16 to J17, J17 to J19, J18 to J20, J19 to J21, J20 to J22, J21 to J28, J22 to J29, J25 to J36, J26 to J37, J27 to J38, J28 to J39, J29 to J40, J30 to J41, J31 to J42, J32 to J43, J33 to J44, J34 to J45, J35 to J46, J36 to J47, J37 to J48, J38 to J49, J39 to J50, J40 to J51
Connections:
- net Net-(J1-Pad2) renamed /BACKLIGHT_-V
- J32 pad 1: /29 -> /23
- J32 pad 2: /27 -> /25
- J32 pad 3: /25 -> /27
- J32 pad 4: /23 -> /29
- J40 pad 10: /47 -> /ZERO_B
- J40 pad 7: /48 -> /ZERO_C
- J40 pad 8: /49 -> /ZERO_D
- J40 pad 9: /*46 -> /ZERO_A
Routing:
- net GND: track 274.2 -> 0.00 mm
- net +12V: track 159.1 -> 0.00 mm, vias 1 -> 0
- net +5VD: track 150.6 -> 0.00 mm, vias 1 -> 0
- net /BACKLIGHT_-V: track 124.8 -> 0.00 mm
- net /MAX7219A/SEG_A1: track 105.5 -> 0.00 mm, vias 1 -> 0
- net +5V: track 99.3 -> 0.00 mm
- net /MAX7219A/SEG_B1: track 98.5 -> 0.00 mm
- net MOSI: track 96.7 -> 0.00 mm
- net CLK: track 88.2 -> 0.00 mm, vias 1 -> 0
- net LOAD: track 88.1 -> 0.00 mm
- net SS: track 84.6 -> 0.00 mm
- net SCLK: track 84.4 -> 0.00 mm
- net ES1_RST: track 78.1 -> 0.00 mm
- net /SCL/21: track 76.6 -> 0.00 mm
- net /MAX7219A/DIG_B4: track 74.7 -> 0.00 mm
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Other:
- board text added: "A10 RIGHT CONSOLE OUTPUT V1.0"
- board text removed: "A10 RIGHT CONSOLE OUTPUT VER 1.0"

Commit message: A10
Parts:
- added J10: PATCH, Connector_PinHeader_2.54mm:PinHeader_1x04_P2.54mm_Vertical, F.Cu at (203.1, 42.1)
- added J11: PATCH, Connector_PinHeader_2.54mm:PinHeader_1x08_P2.54mm_Vertical, F.Cu at (171.6, 39.5)
- added J15: PATCH, Connector_PinHeader_2.54mm:PinHeader_1x04_P2.54mm_Vertical, F.Cu at (203.1, 38.5)
- added J16: PATCH, Connector_PinHeader_2.54mm:PinHeader_1x08_P2.54mm_Vertical, F.Cu at (171.6, 44.1)
- added J23: CABIN_PRES, Connector_Molex:Molex_KK-254_AE-6410-06A_1x06_P2.54mm_Vertical, F.Cu at (155.1, 41.1)
- added J34: CABIN_PRES, Connector_Molex:Molex_KK-254_AE-6410-04A_1x04_P2.54mm_Vertical, F.Cu at (142.9, 41.1)
- J21: renamed from J16; value STEPPER_F -> LOX
- J27: renamed from J23; value STEPPER_E -> OXY_REG
- J28: renamed from J24; value STEPPER_D -> RIGHT FUEL
- J29: renamed from J25; value STEPPER_C -> LEFT_FUEL
- J30: renamed from J26; value STEPPER_B -> RIGHT_HYD
- J31: renamed from J27; value STEPPER_A -> LEFT_HYD
- J35: renamed from J30; value STEPPER_E -> OXY_REG
- J36: renamed from J31; value STEPPER_F -> LOX
- J37: renamed from J32; value STEPPER_B -> RIGHT_HYD
- J38: renamed from J33; value STEPPER_C -> LEFT_FUEL
- J39: renamed from J34; value STEPPER_D -> RIGHT FUEL
- J40: renamed from J35; value STEPPER_A -> LEFT_HYD
- moved R4 31.3 mm to (119.1, 45.6)
- moved R3 22.4 mm to (127.9, 42.8), turned to 90 degrees
- moved D1 2.97 mm to (122.6, 40.6)
- moved D2 2.27 mm to (117.0, 40.6)
- moved R7 1.02 mm to (166.9, 57.8)
- moved J31 0.25 mm to (210.2, 93.4)
- moved J30 0.25 mm to (202.1, 93.4)
- renumbered J10 to J12, J11 to J13, J12 to J14, J13 to J17, J14 to J18, J15 to J19, J17 to J20, J19 to J22, J20 to J24, J21 to J25, J22 to J26, J28 to J32, J29 to J33, J36 to J41, J37 to J42, J38 to J43, J39 to J44, J40 to J45, J41 to J46, J42 to J47, J43 to J48, J44 to J49, J45 to J50, J46 to J51, J47 to J52, J48 to J53, J49 to J54, J50 to J55, J51 to J56, MH3 to MH1
Connections:
- net /ZERO_A renamed /*46
- net /ZERO_B renamed /47
- net /ZERO_C renamed /48
- net /ZERO_D renamed /49
Routing:
- net GND: track 0.00 -> 372.2 mm
- net +12V: track 0.00 -> 329.0 mm, vias 0 -> 1
- net /BACKLIGHT_-V: track 0.00 -> 269.0 mm
- net +5VD: track 0.00 -> 260.4 mm, vias 0 -> 2
- net /*3: track 0.00 -> 118.6 mm, vias 0 -> 1
- net /*4: track 0.00 -> 110.6 mm, vias 0 -> 1
- net CLK: track 0.00 -> 104.4 mm, vias 0 -> 1
- net SCLK: track 0.00 -> 103.0 mm
- net +5V: track 0.00 -> 102.2 mm, vias 0 -> 1
- net /MAX7219A/SEG_B1: track 0.00 -> 99.8 mm, vias 0 -> 1
- net /MAX7219A/SEG_A1: track 0.00 -> 99.4 mm
- net MOSI: track 0.00 -> 94.2 mm
- net LOAD: track 0.00 -> 87.4 mm
- net SS: track 0.00 -> 84.7 mm
- net ES1_RST: track 0.00 -> 78.1 mm
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Other:
- board text added: "-12 BKLIGHT +12"
- board text added: "DP G F E D C B A"
- board text added: "ZERO GND +5V"

Commit message: A10 and F16
Other:
- board text added: "+"
- board text added: "A10 RIGHT CONSOLE OUTPUT V1.1"
- board text removed: "A10 RIGHT CONSOLE OUTPUT V1.0"
Changed lines of the file:
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@@
       (effects (font (size 1 1) (thickness 0.15)))
     )
-    (fp_text value "10K" (at 1.27 1.92) (layer "F.Fab")
+    (fp_text value "10K" (at 5.284 0) (layer "F.SilkS")
       (effects (font (size 1 1) (thickness 0.15)))
     )
@@
     (property "Sheetname" "MAX7219A")
     (attr through_hole)
-    (fp_text reference "U2" (at 3.81 -2.33) (layer "F.SilkS")
+    (fp_text reference "U2" (at 3.81 1.016) (layer "F.SilkS")
       (effects (font (size 1 1) (thickness 0.15)))
     )
@@
     (effects (font (size 1 1) (thickness 0.15)) (justify mirror))
   )
-  (gr_text "A10 RIGHT CONSOLE OUTPUT V1.0" (at 166.04 132.004) (layer "F.SilkS")
+  (gr_text "A10 RIGHT CONSOLE OUTPUT V1.1" (at 166.04 132.004) (layer "F.SilkS")
     (effects (font (size 2 2) (thickness 0.15)))
   )
+  (gr_text "+" (at 125.908 38.024) (layer "F.SilkS")
+    (effects (font (size 1 1) (thickness 0.15)))
+  )
+  (gr_text "+" (at 120.32 38.024) (layer "F.SilkS")
+    (effects (font (size 1 1) (thickness 0.15)))
+  )
   (segment (start 132.385 79.68) (end 131.1847 79.68) (width 0.4) (layer "F.Cu") (net 1))

Commit message: A10
Routing:
- net +5VD: track 260.4 -> 275.9 mm, vias 2 -> 1
- net +12V: track 329.0 -> 320.6 mm
- net /*3: track 118.6 -> 114.4 mm
- net /*4: track 110.6 -> 107.3 mm
- net Net-(Q1-Pad1): track 17.7 -> 14.6 mm
- net /BACKLIGHT_-V: track 269.0 -> 267.6 mm
- net /MAX7219A/SEG_E1: track 37.9 -> 36.9 mm
- net /MAX7219A/DIG_B2: track 25.9 -> 25.3 mm
- net MOSI: track 94.2 -> 93.7 mm

Commit message: a10 PC
Connections:
- R3 pad 1: /*5 -> /*13
- R4 pad 1: /*6 -> /*12
Routing:
- net /MAX7219A/DIG_A2: track 21.4 -> 71.6 mm, vias 1 -> 2
- net /MAX7219A/DIG_A4: track 30.3 -> 68.9 mm
- net /MAX7219A/DIG_A3: track 22.5 -> 57.8 mm, vias 0 -> 1
- net /30: track 19.8 -> 53.5 mm
- net /MAX7219A/DIG_A6: track 32.4 -> 65.2 mm, vias 0 -> 1
- net CLK: track 104.3 -> 135.3 mm, vias 1 -> 2
- net /MAX7219A/SEG_A1: track 99.4 -> 130.2 mm, vias 0 -> 1
- net /*5: track 44.8 -> 17.2 mm
- net /MAX7219A/SEG_G1: track 30.7 -> 57.1 mm, vias 0 -> 1
- net /*3: track 114.4 -> 140.3 mm, vias 1 -> 0
- net /MAX7219A/DIG_A5: track 26.6 -> 50.6 mm, vias 0 -> 1
- net +5VD: track 275.9 -> 299.7 mm, vias 1 -> 2
- net +12V: track 320.6 -> 301.1 mm
- net /*6: track 45.1 -> 26.2 mm
- net /MAX7219A/SEG_E1: track 36.9 -> 54.6 mm, vias 0 -> 1
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
Commit message: A10
Parts:
- removed J1, J17, J4: BACKLIGHT, Connector_Molex:Molex_KK-254_AE-6410-02A_1x02_P2.54mm_Vertical
- added J57: CMSP_OLED, Connector_Molex:Molex_KK-254_AE-6410-04A_1x04_P2.54mm_Vertical, F.Cu at (220.1, 41.5)
- added J58: FUEL_OLED, Connector_Molex:Molex_KK-254_AE-6410-04A_1x04_P2.54mm_Vertical, F.Cu at (219.9, 51.1)
- added J59: ILS_OLED, Connector_Molex:Molex_KK-254_AE-6410-04A_1x04_P2.54mm_Vertical, F.Cu at (219.9, 59.7)
- added J60: TACAN_OLED, Connector_Molex:Molex_KK-254_AE-6410-04A_1x04_P2.54mm_Vertical, F.Cu at (219.9, 68.3)
- added J61: SPARE_A_OLED, Connector_Molex:Molex_KK-254_AE-6410-04A_1x04_P2.54mm_Vertical, F.Cu at (219.9, 76.9)
- added J62: SPARE_B_OLED, Connector_Molex:Molex_KK-254_AE-6410-04A_1x04_P2.54mm_Vertical, F.Cu at (219.9, 85.4)
- added J63: SPARE_C_OLED, Connector_Molex:Molex_KK-254_AE-6410-04A_1x04_P2.54mm_Vertical, F.Cu at (219.9, 94.0)
- added Q2: IRF1405PBF, Package_TO_SOT_THT:TO-220-3_Vertical, F.Cu at (140.4, 108.5)
- added R8: 330, Resistor_THT:R_Axial_DIN0204_L3.6mm_D1.6mm_P2.54mm_Vertical, F.Cu at (150.1, 105.6)
- added R9: 10K, Resistor_THT:R_Axial_DIN0204_L3.6mm_D1.6mm_P2.54mm_Vertical, F.Cu at (149.8, 109.8)
- added U4: TCA9548APWR, Footprint Library:DIP-24_TCA9548A, F.Cu at (226.3, 118.7)
- J12, J7: value BACKLIGHT -> FLOODLIGHT
- moved J7 12.3 mm to (156.1, 107.8)
- moved J12 11.6 mm to (164.9, 107.9)
- moved J8 7.29 mm to (150.0, 116.2)
- moved J13 7.29 mm to (156.8, 116.2)
- moved J5 0.64 mm to (143.0, 116.2)
Connections:
- net /*11 renamed D11
- net /RX1/19 renamed D19
- net /RX2/17 renamed D17
- net /SCL/21 renamed D21 SCL
- net /SDA/20 renamed D20 SDA
- net /TX1/18 renamed D18
- J12 pad 2: /BACKLIGHT_-V -> /FLOODLIGHT_-V
- J27 pad 3: /*3 -> unconnected-(J27-Pin_3-Pad3)
- J7 pad 2: /BACKLIGHT_-V -> /FLOODLIGHT_-V
Routing:
- net GND: track 375.8 -> 0.00 mm, vias 1 -> 0
- net +12V: track 301.1 -> 0.00 mm, vias 1 -> 0
- net +5VD: track 299.7 -> 0.00 mm, vias 2 -> 0
- net /BACKLIGHT_-V: track 269.1 -> 0.00 mm
- net /*3: track 140.3 -> 0.00 mm
- net CLK: track 135.3 -> 0.00 mm, vias 2 -> 0
- net /MAX7219A/SEG_A1: track 130.2 -> 0.00 mm, vias 1 -> 0
- net /*4: track 114.7 -> 0.00 mm, vias 1 -> 0
- net +5V: track 113.1 -> 0.00 mm, vias 1 -> 0
- net /MAX7219A/SEG_B1: track 106.1 -> 0.00 mm, vias 1 -> 0
- net SCLK: track 99.1 -> 0.00 mm
- net MOSI: track 98.5 -> 0.00 mm, vias 1 -> 0
- net LOAD: track 83.8 -> 0.00 mm
- net SS: track 81.1 -> 0.00 mm
- net D21 SCL: track 78.5 -> 0.00 mm
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Other:
- board size 99.7 x 98.4 mm -> 123 x 98.4 mm

Commit message: a10
Parts:
- removed J10, J15: PATCH, Connector_PinHeader_2.54mm:PinHeader_1x04_P2.54mm_Vertical
- removed J11, J16: PATCH, Connector_PinHeader_2.54mm:PinHeader_1x08_P2.54mm_Vertical
- removed J21: LOX, Connector_Molex:Molex_KK-254_AE-6410-06A_1x06_P2.54mm_Vertical
- removed J23: CABIN_PRES, Connector_Molex:Molex_KK-254_AE-6410-06A_1x06_P2.54mm_Vertical
- removed J27: OXY_REG, Connector_Molex:Molex_KK-254_AE-6410-06A_1x06_P2.54mm_Vertical
- removed J28: RIGHT FUEL, Connector_Molex:Molex_KK-254_AE-6410-06A_1x06_P2.54mm_Vertical
- removed J29: LEFT_FUEL, Connector_Molex:Molex_KK-254_AE-6410-06A_1x06_P2.54mm_Vertical
- removed J30: RIGHT_HYD, Connector_Molex:Molex_KK-254_AE-6410-06A_1x06_P2.54mm_Vertical
- removed J31: LEFT_HYD, Connector_Molex:Molex_KK-254_AE-6410-06A_1x06_P2.54mm_Vertical
- removed J61: SPARE_A_OLED, Connector_Molex:Molex_KK-254_AE-6410-04A_1x04_P2.54mm_Vertical
- removed J62: SPARE_B_OLED, Connector_Molex:Molex_KK-254_AE-6410-04A_1x04_P2.54mm_Vertical
- removed J63: SPARE_C_OLED, Connector_Molex:Molex_KK-254_AE-6410-04A_1x04_P2.54mm_Vertical
- added J1: RIGHTSTROBE, Connector_Molex:Molex_KK-254_AE-6410-02A_1x02_P2.54mm_Vertical, F.Cu at (171.0, 116.0)
- added J4: RIGHTNAV, Connector_Molex:Molex_KK-254_AE-6410-02A_1x02_P2.54mm_Vertical, F.Cu at (162.0, 116.0)
- added Q3: IRF1405PBF, Package_TO_SOT_THT:TO-220-3_Vertical, F.Cu at (185.4, 117.9)
- added Q4: IRF1405PBF, Package_TO_SOT_THT:TO-220-3_Vertical, F.Cu at (185.4, 112.7)
- added R10: 330, Resistor_THT:R_Axial_DIN0204_L3.6mm_D1.6mm_P2.54mm_Vertical, F.Cu at (177.5, 118.5)
- added R11: 10K, Resistor_THT:R_Axial_DIN0204_L3.6mm_D1.6mm_P2.54mm_Vertical, F.Cu at (180.7, 118.5)
- added R12: 330, Resistor_THT:R_Axial_DIN0204_L3.6mm_D1.6mm_P2.54mm_Vertical, F.Cu at (177.5, 112.2)
- added R13: 10K, Resistor_THT:R_Axial_DIN0204_L3.6mm_D1.6mm_P2.54mm_Vertical, F.Cu at (180.7, 112.2)
- moved J40 56.8 mm to (154.9, 41.0), turned to 0 degrees
- moved J53 42.0 mm to (166.0, 73.5)
- moved J54 40.4 mm to (166.0, 82.5)
- moved J38 39.9 mm to (178.5, 41.0), turned to 0 degrees
- moved J37 37.4 mm to (166.9, 41.0), turned to 0 degrees
- moved J58 25.4 mm to (210.0, 74.5), turned to 90 degrees
- moved J59 25.4 mm to (211.1, 83.5), turned to 180 degrees
- moved J60 24.3 mm to (211.3, 91.0), turned to 180 degrees
- moved U4 23.5 mm to (203.9, 111.5), turned to -90 degrees
- moved Q1 13.8 mm to (185.5, 107.4)
- moved R2 11.7 mm to (173.0, 108.0), turned to 90 degrees
- moved J57 11.3 mm to (210.0, 46.5), turned to 90 degrees
- moved J36 11.1 mm to (202.5, 65.6)
- moved J39 11.1 mm to (202.5, 54.1)
- moved J35 7.91 mm to (202.4, 77.4)
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Routing:
- net GND: track 0.00 -> 361.2 mm
- net +3V3: track 0.00 -> 183.9 mm, vias 0 -> 2
- net +12V: track 0.00 -> 153.9 mm, vias 0 -> 1
- net +5VD: track 0.00 -> 142.1 mm
- net D21 SCL: track 0.00 -> 134.1 mm
- net D20 SDA: track 0.00 -> 127.8 mm, vias 0 -> 2
- net +5V: track 0.00 -> 101.6 mm
- net MOSI: track 0.00 -> 100.0 mm
- net CLK: track 0.00 -> 94.0 mm
- net /BACKLIGHT_-V: track 0.00 -> 92.7 mm
- net SCLK: track 0.00 -> 87.8 mm
- net /OLED/SC0: track 0.00 -> 85.5 mm
- net /OLED/SD0: track 0.00 -> 85.5 mm
- net /MAX7219A/SEG_A1: track 0.00 -> 85.1 mm
- net /*5: track 0.00 -> 84.7 mm
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Other:
- board size 123 x 98.4 mm -> 99.5 x 98.4 mm
- board text added: "A10 RIGHT CONSOLE OUTPUT V1.2"
- board text removed: "-12 BKLIGHT +12"
- board text removed: "A10 RIGHT CONSOLE OUTPUT V1.1"
- board text removed: "ZERO GND +5V"
