File: Jet Ranger/PCBs/Jet Ranger 13 Stepper/Jet Ranger 13 Stepper.kicad_pcb (KiCad board)
At the start: 2 copper layers, 100 x 99.1 mm, 49 parts, among them J1 Conn_01x03_Pin, J11 Conn_01x08, J12 Conn_01x08, J13 Conn_01x08, J14 Conn_01x08, J2 5V IN, J20 TURBINE_SPEED, J22 ROTOR_SPEED, J23 RADAR_ALT, J24 GAS_PRODUCER, J25 ENG_TORQUE, J26 AIRSPEED, J27 EGT, J29 Utility, J3 STEPPER IN 12-20VDC, J30 XMSN_OIL_TEMP, J34 Conn_01x08, J35 Conn_01x10, J36 Conn_01x02, J37 Conn_01x02, J38 Conn_01x02, J39 XMSN_OIL_PRESS, J4 FUEL_LEVEL, J40 ENG_OIL_PRES, J41 ENG_OIL_TEMP, J5 VVI, Q1 Q_NMOS_GSD, U3 USR-ES1

Commit message: Jet Ranger
Connections:
- net /STEPPER_FL_A renamed /STEPPER_FA_A
Other:
- board text added: "Jet Ranger 13 Stepper V ${REVISION} 20261012"
- board text removed: "Jet Ranger 13 Stepper V ${REVISION} 20260801"

Commit message: Jet Ranger
Parts:
- moved D1 2.50 mm to (110.5, 85.5)
- moved D2 2.50 mm to (110.5, 90.5)
- moved D3 2.50 mm to (110.5, 80.5)
- moved D4 2.50 mm to (125.0, 81.5)
- moved D5 2.50 mm to (125.3, 87.5)
- moved R2 2.50 mm to (115.2, 86.2)
- moved R3 2.50 mm to (115.2, 89.5)
- moved R4 2.50 mm to (115.2, 79.5)
- moved R5 2.50 mm to (115.2, 82.9)
- moved R6 2.50 mm to (122.5, 91.5)
Routing:
- net GND: track 307.4 -> 273.9 mm, vias 0 -> 1
- net /STEPPER_EGT_B: track 117.4 -> 138.3 mm, vias 1 -> 0
- net /STEPPER_RA_C: track 85.2 -> 66.1 mm, vias 1 -> 0
- net /STEPPER_EGT_C: track 122.0 -> 139.6 mm, vias 1 -> 0
- net /STEPPER_RA_D: track 88.3 -> 70.8 mm, vias 1 -> 2
- net /STEPPER_GP_A: track 75.0 -> 59.5 mm, vias 1 -> 0
- net +12V: track 249.2 -> 234.0 mm
- net /STEPPER_GP_B: track 81.6 -> 67.1 mm, vias 1 -> 0
- net /STEPPER_GP_D: track 94.7 -> 80.4 mm
- net /STEPPER_GP_C: track 81.0 -> 66.7 mm, vias 2 -> 0
- net /STEPPER_RA_A: track 75.5 -> 61.4 mm, vias 1 -> 0
- net /STEPPER_TS_D: track 61.5 -> 48.1 mm
- net /INT_5V: track 182.2 -> 195.0 mm
- net /STEPPER_RA_B: track 77.7 -> 65.6 mm, vias 2 -> 1
- net /STEPPER_SPD_D: track 34.2 -> 25.9 mm, vias 1 -> 0
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Other:
- board text added: "Jet Ranger 13 Stepper V ${REVISION} 20261016"
- board text removed: "Jet Ranger 13 Stepper V ${REVISION} 20261012"

Commit message: Jet Ranger MOSFET fix
Parts:
- Q1: value Q_NMOS_GSD -> IRF540N
Connections:
- Q1 pad 2: GND -> BACKLIGHT_-V
- Q1 pad 3: BACKLIGHT_-V -> GND
Routing:
- net /STEPPER_EGT_C: track 139.6 -> 112.5 mm
- net SS: track 52.0 -> 71.0 mm, vias 1 -> 0
- net /STEPPER_EGT_B: track 138.3 -> 129.7 mm
- net /INT_5V: track 195.0 -> 187.3 mm
- net /STEPPER_GP_D: track 80.4 -> 74.2 mm, vias 1 -> 0
- net /STEPPER_RA_D: track 70.8 -> 76.1 mm, vias 2 -> 1
- net /STEPPER_EGT_A: track 109.0 -> 103.7 mm, vias 0 -> 2
- net +12V: track 234.0 -> 239.1 mm
- net /STEPPER_ET_D: track 60.6 -> 57.7 mm
- net /+5v_IN: track 159.9 -> 157.7 mm
- net /STEPPER_EGT_D: track 129.2 -> 131.0 mm
- net /STEPPER_RS_B: track 62.5 -> 64.0 mm
- net Net-(D1-A): track 12.0 -> 11.0 mm
- net /STEPPER_GP_C: track 66.7 -> 67.5 mm
- net /STEPPER_SPD_C: track 29.8 -> 30.5 mm
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