File: Jet Ranger/PCBs/Jet Ranger Front Panel Servo/Jet Ranger Front Panel Servo.kicad_pcb (KiCad board)
At the start: 2 copper layers, 100 x 99.1 mm, 81 parts, among them J1 Conn_01x03_Pin, J10 BK_LIGHT, J11 Conn_01x08, J12 Conn_01x08, J13 Conn_01x08, J14 Conn_01x08, J15 BK_LIGHT, J16 BK_LIGHT, J17 BK_LIGHT, J18 BK_LIGHT, J19 BK_LIGHT, J2 5V IN, J20 AIRSPEED, J21 EGT, J22 TURBINE_SPEED, J23 RADAR_ALT, J24 ENG_TORQUE, J25 ROTOR_SPEED, J26 VVI, J27 ENG_OIL_TEMP, J28 FUEL_LEVEL, J29 Utility, J3 STEPPER IN 12-20VDC, J30 GAS_PRODUCER, J31 ENG_OIL_PRES, J32 XMSN_OIL_TEMP, J33 XMSN_OIL_PRESS, J34 Conn_01x08, J35 Conn_01x10, J36 Conn_01x02, J37 Conn_01x02, J38 Conn_01x02, J4 LHS_ANNUC, J42 PITCH, J43 ROLL, J44 ELEC_LOAD, J45 FUEL_LOAD, J5 RHS_ANNUC, J6 BK_LIGHT, J7 BK_LIGHT, J8 BK_LIGHT, J9 BK_LIGHT, Q1 Q_NMOS_GSD, SW1 TOT_CLEAR, SW2 FUEL_VALVE, SW3 WARNING_MUTE, U1 ULN2803A, U2 ULN2803A, U3 USR-ES1

Commit message: Servo PCB
Connections:
- J4 pad 1: /Fuel_Pump -> /AFT_Fuel_Filter
- J4 pad 13: /Low_Fuel -> /GroupB8
- J4 pad 14: /SC_Fail -> /GroupB9
- J4 pad 15: /GroupB8 -> /Low_Fuel
- J4 pad 16: /GroupB9 -> /SC_Fail
- J4 pad 3: /AFT_Fuel_Filter -> /Fuel_Pump
- J4 pad 5: /GroupB3 -> /Gen_Fail
- J4 pad 7: /Gen_Fail -> /GroupB3
Routing:
- net GND: track 0.00 -> 437.5 mm
- net /+12v-IN: track 0.00 -> 216.2 mm
- net /INT_5V: track 0.00 -> 207.5 mm
- net /+5v_SERVO: track 0.00 -> 153.0 mm
- net /+5v_IN: track 0.00 -> 142.7 mm, vias 0 -> 1
- net /BACKLIGHT_PANELS: track 0.00 -> 123.2 mm
- net /RESET_pin: track 0.00 -> 87.9 mm
- net ES1_RST: track 0.00 -> 80.4 mm, vias 0 -> 1
- net MOSI: track 0.00 -> 77.9 mm
- net MISO: track 0.00 -> 74.5 mm
- net SCLK: track 0.00 -> 72.2 mm
- net /RED_LED: track 0.00 -> 66.0 mm
- net /PWM_FUEL_LOAD: track 0.00 -> 64.9 mm
- net /PWM_ELEC_LOAD: track 0.00 -> 61.6 mm
- net /GREEN_LED: track 0.00 -> 58.5 mm
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Other:
- board text added: "Jet Ranger Servo V ${REVISION} 20261011"
- board text removed: "Jet Ranger Servo V ${REVISION} 20260111a"

Commit message: Jet Ranger MOSFET fix
Parts:
- removed Q1: Q_NMOS_GSD, Package_TO_SOT_THT:TO-220-3_Vertical
- added Q2: IRF540N, Package_TO_SOT_THT:TO-220-3_Vertical, F.Cu at (88.9, 56.5)
Routing:
- net /RESET_pin: track 87.9 -> 102.2 mm
- net /D_Low_Fuel: track 45.4 -> 38.8 mm, vias 0 -> 1
- net /+5v_SERVO: track 153.0 -> 146.8 mm
- net /+12v-IN: track 216.2 -> 221.9 mm
- net /+5v_IN: track 142.7 -> 147.7 mm
- net /D_SC_Fail: track 44.0 -> 39.9 mm, vias 0 -> 1
- net /PWM_XMSN_OIL_TEMP: track 51.0 -> 54.6 mm
- net /SW_TOT_CLEAR: track 21.4 -> 23.8 mm
- net /BACKLIGHT_PANELS: track 123.2 -> 125.1 mm
- net GND: track 437.5 -> 439.3 mm
- net /COL0: track 13.4 -> 15.0 mm
- net /D_Fuel_Pump: track 41.6 -> 43.1 mm
- net /D_T/R_Chip: track 41.5 -> 42.7 mm
- net /D_Engine_Chip: track 41.6 -> 42.6 mm
- net /COL9: track 21.9 -> 22.5 mm
Other:
- board text added: "Jet Ranger Servo V ${REVISION} ${ISSUE_DATE}"
- board text removed: "Jet Ranger Servo V ${REVISION} 20261011"
